File: Hardware/Satelite/PCB_A/Cargador de batería.sch (KiCad schematic (older format))
At the start: 0 parts

Commit message: Más modificaciones al esquema del PCB_A
Parts:
- added C1, C2: 1uF, symbol Device:C_Small
- added R4: 1k8, symbol Device:R
- added R5: 2k, symbol Device:R
- added R6: 100k, symbol Device:R
- added U2: BQ24091DGQT, SamacSys_Parts:SOP50P490X110-11N, symbol SamacSys_Parts:BQ24091DGQT
Connections:
- net labels added: CHG, CHG_DISABLE, GND, ISET, VBUS, VBat+
- wire segments 0 -> 24
Other:
- note added: "Corriente de carga a 300mA"
- note added: "Corriente de pre-carga 20% de carga"
- note added: "Corriente de terminación 10% de carga"
