File: Hardware/Satelite/PCB_A/Fuel Gauge.sch (KiCad schematic (older format))
At the start: 1 part

Commit message: Agregado fuel gauge a PCB_A
Parts:
- added C17: 0.47uF, symbol Device:C_Small
- added R15, R16, R17, R18: 10k, symbol Device:R
- added R?: 10m, symbol Device:R
- gave numbers to parts that had none: 1
Connections:
- net labels added: +3V3, GND, GPOUT, SCL, SDA, SYS, VBat+
- wire segments 0 -> 32
