File: Hardware/Satelite/PCB_A/PCB_A.sch (KiCad schematic (older format))
At the start: 0 parts

Commit message: Esquemas iniciales para PCB_A del satélite
Parts:
- added J? (x3): Conn_02x02_Counter_Clockwise, symbol Connector_Generic:Conn_02x02_Counter_Clockwise
- added J?: Servo Paracaídas, symbol Connector_Generic:Conn_01x03
- added J?: Servo Globo, symbol Connector_Generic:Conn_01x03
- added SW?: SW_SPDT, symbol Switch:SW_SPDT
- added U?: CONUFL001-SMD, symbol AXTEC_IC:CONUFL001-SMD
Connections:
- net labels added: +3V3, GND, GPS_TX, ISET, SCLK, SDI, SDO, VBAT, VBUS
- wire segments 0 -> 30

Commit message: Más modificaciones al esquema del PCB_A
Parts:
- added D1, D2, D3: LED, symbol Device:LED
- added J2: Batería LiPo, symbol Connector_Generic:Conn_01x02
- added J7: Conn_02x02_Counter_Clockwise, symbol Connector_Generic:Conn_02x02_Counter_Clockwise
- added MH1, MH2, MH3: MountingHole, symbol Mechanical:MountingHole
- added Q1: SSM3J338R,LF, SamacSys_Parts:SSM3J332RLFT, symbol SamacSys_Parts:SSM3J338R,LF
- added R1, R2, R3: 1k, symbol Device:R
- gave numbers to parts that had none: 7
Connections:
- net labels added: CHG, CHG_DISABLE, P1, P2, S_GLOBO, S_PARACAIDAS
- wire segments 30 -> 54

Commit message: Esquema inicial para fuel gauge en PCB_A y inicio de esquemas para PCB_B
Parts:
- added C?: 1uF, symbol Device:C_Small
Connections:
- net labels added: GPOUT, SCL, SDA, SYS
- wire segments 54 -> 64

Commit message: Agregado fuel gauge a PCB_A
Parts:
- added J?: Conn_02x02_Counter_Clockwise, symbol Connector_Generic:Conn_02x02_Counter_Clockwise
- gave numbers to parts that had none: 1
Connections:
- wire segments 64 -> 67
Changed lines of the file:
@@
 SCLK
 Wire Wire Line
-	8150 3250 8550 3250
+	8150 3250 8750 3250
 $Comp
 L Connector_Generic:Conn_02x02_Counter_Clockwise J6
@@
 Wire Wire Line
 	7250 3800 7650 3800
-Wire Wire Line
-	7250 3900 7650 3900
-Wire Wire Line
-	8150 3900 8750 3900
 Text Label 7300 3800 0    50   ~ 0
 GPS_TX
@@
 L power:+3V3 #PWR?
 U 1 1 5BA42A3A
-P 8750 3800
+P 7050 3750
 AR Path="/5BA17F9C/5BA42A3A" Ref="#PWR?"  Part="1"
 AR Path="/5BA42A3A" Ref="#PWR014"  Part="1"
-F 0 "#PWR014" H 8750 3650 50  0001 C CNN
-F 1 "+3V3" H 8765 3973 50  0000 C CNN
-F 2 "" H 8750 3800 50  0001 C CNN
-F 3 "" H 8750 3800 50  0001 C CNN
-	1    8750 3800
-	1    0    0    -1
-$EndComp
-Wire Wire Line
-	8750 3900 8750 3800
-$Comp
-L power:GND #PWR011
-U 1 1 5BA437E3
-P 7250 3900
-F 0 "#PWR011" H 7250 3650 50  0001 C CNN
-F 1 "GND" H 7255 3727 50  0000 C CNN
-F 2 "" H 7250 3900 50  0001 C CNN
-F 3 "" H 7250 3900 50  0001 C CNN
-	1    7250 3900
+F 0 "#PWR014" H 7050 3600 50  0001 C CNN
+F 1 "+3V3" H 7065 3923 50  0000 C CNN
+F 2 "" H 7050 3750 50  0001 C CNN
+F 3 "" H 7050 3750 50  0001 C CNN
+	1    7050 3750
 	1    0    0    -1
 $EndComp
@@
 Wire Wire Line
 	8150 4600 8550 4600
-$Comp
-L power:GND #PWR013
-U 1 1 5BADDBAE
-P 8750 3250
-F 0 "#PWR013" H 8750 3000 50  0001 C CNN
-F 1 "GND" H 8755 3077 50  0000 C CNN
-F 2 "" H 8750 3250 50  0001 C CNN
-F 3 "" H 8750 3250 50  0001 C CNN
-	1    8750 3250
-	1    0    0    -1
-$EndComp
 Wire Wire Line
 	8150 3150 8750 3150
-Wire Wire Line
-	8750 3150 8750 3250
 $Comp
 L Connector_Generic:Conn_01x02 J2
@@
 P1
 Wire Wire Line
-	8150 3800 8550 3800
+	8150 3800 8750 3800
 Text Label 8300 3800 0    50   ~ 0
 P2
@@
 AR Path="/5BA1A7F9/5BB16517" Ref="C?"  Part="1"
 AR Path="/5BA1A77A/5BB16517" Ref="C?"  Part="1"
-F 0 "C?" H 3850 2750 50  0000 L CNN
+AR Path="/5BB16517" Ref="C16"  Part="1"
+F 0 "C16" H 3850 2750 50  0000 L CNN
 F 1 "1uF" H 3800 2650 50  0000 L CNN
 F 2 "" H 3700 2750 50  0001 C CNN
@@
 	3700 2600 3700 2650
 $Comp
-L power:GND #PWR?
+L power:GND #PWR0101
 U 1 1 5BB18143
 P 3700 2900
-F 0 "#PWR?" H 3700 2650 50  0001 C CNN
+F 0 "#PWR0101" H 3700 2650 50  0001 C CNN
 F 1 "GND" H 3705 2727 50  0000 C CNN
 F 2 "" H 3700 2900 50  0001 C CNN
@@
 Text Label 3950 1700 0    50   ~ 0
 GPOUT
+$Comp
+L Connector_Generic:Conn_02x02_Counter_Clockwise J?
+U 1 1 5BB5DFD1
+P 7850 5200
+F 0 "J?" H 7900 5417 50  0000 C CNN
+F 1 "Conn_02x02_Counter_Clockwise" H 7900 5326 50  0000 C CNN
+F 2 "" H 7850 5200 50  0001 C CNN
+F 3 "~" H 7850 5200 50  0001 C CNN
+	1    7850 5200
+	1    0    0    -1
+$EndComp
+Wire Wire Line
+	6950 5200 7650 5200
+Wire Wire Line
+	8550 5200 8150 5200
+Wire Wire Line
+	8150 5300 8550 5300
+Text Label 8300 5200 0    50   ~ 0
+SDA
+Text Label 8300 5300 0    50   ~ 0
+SCL
+Text Label 7100 5200 0    50   ~ 0
+GPOUT
+Wire Wire Line
+	7250 5300 7650 5300
+$Comp
+L power:GND #PWR?
+U 1 1 5BB5F80C
+P 7250 5300
+F 0 "#PWR?" H 7250 5050 50  0001 C CNN
+F 1 "GND" H 7255 5127 50  0000 C CNN
+F 2 "" H 7250 5300 50  0001 C CNN
+F 3 "" H 7250 5300 50  0001 C CNN
+	1    7250 5300
+	1    0    0    -1
+$EndComp
+Text Label 8300 3150 0    50   ~ 0
+S_GLOBO
+Text Label 8300 3900 0    50   ~ 0
+S_PARACAIDAS
+Wire Wire Line
+	7050 3750 7050 3900
+Wire Wire Line
+	7050 3900 7650 3900
+Wire Wire Line
+	8150 3900 8750 3900
 $EndSCHEMATC

Commit message: Agregado sensor de corriente de batería
Connections:
- net labels added: OUT, VBat_I_SENSE, VIN
- wire segments 67 -> 70

Commit message: Completado esquema PCB_B. Mejoras en esquemas de PCB_A.
Parts:
- removed D2: LED, symbol Device:LED
- removed J4, J5, J6, J7, J?: Conn_02x02_Counter_Clockwise, symbol Connector_Generic:Conn_02x02_Counter_Clockwise
- removed R2: 1k, symbol Device:R
- added J? (x2): Conn_01x10, Connector_PinHeader_1.27mm:PinHeader_1x10_P1.27mm_Vertical, symbol Connector_Generic:Conn_01x10
Connections:
- net labels added: CS
- net labels removed: P2
- wire segments 70 -> 68

Commit message: Nuevos PCB_B y PCB_C
Connections:
- net labels added: +BATT
- net labels removed: CHG, CHG_DISABLE, GPOUT, ISET, OUT, SCL, SDA, SYS, VBAT, VBUS, VBat_I_SENSE, VIN
- wire segments 68 -> 50

Commit message: Agregados agujeros de montajes
Parts:
- removed MH1, MH2, MH3: MountingHole, symbol Mechanical:MountingHole
- added H? (x3): MountingHole_Pad, symbol Mechanical:MountingHole_Pad
Changed lines of the file:
@@
 	9300 2550 9900 2550
-$Comp
-L Mechanical:MountingHole MH1
-U 1 1 5BB03020
-P 9000 4300
-F 0 "MH1" H 9100 4346 50  0000 L CNN
-F 1 "MountingHole" H 9100 4255 50  0000 L CNN
-F 2 "" H 9000 4300 50  0001 C CNN
-F 3 "~" H 9000 4300 50  0001 C CNN
-	1    9000 4300
-	1    0    0    -1
-$EndComp
-$Comp
-L Mechanical:MountingHole MH2
-U 1 1 5BB03098
-P 9000 4600
-F 0 "MH2" H 9100 4646 50  0000 L CNN
-F 1 "MountingHole" H 9100 4555 50  0000 L CNN
-F 2 "" H 9000 4600 50  0001 C CNN
-F 3 "~" H 9000 4600 50  0001 C CNN
-	1    9000 4600
-	1    0    0    -1
-$EndComp
-$Comp
-L Mechanical:MountingHole MH3
-U 1 1 5BB03132
-P 9000 4900
-F 0 "MH3" H 9100 4946 50  0000 L CNN
-F 1 "MountingHole" H 9100 4855 50  0000 L CNN
-F 2 "" H 9000 4900 50  0001 C CNN
-F 3 "~" H 9000 4900 50  0001 C CNN
-	1    9000 4900
-	1    0    0    -1
-$EndComp
 $Comp
 L Device:C_Small C?
@@
 Text Label 7900 3450 0    50   ~ 0
 S_PARACAIDAS
+$Comp
+L Mechanical:MountingHole_Pad H?
+U 1 1 5C3B6679
+P 8850 4350
+F 0 "H?" H 8950 4401 50  0000 L CNN
+F 1 "MountingHole_Pad" H 8950 4309 50  0000 L CNN
+F 2 "" H 8850 4350 50  0001 C CNN
+F 3 "~" H 8850 4350 50  0001 C CNN
+	1    8850 4350
+	1    0    0    -1
+$EndComp
+$Comp
+L power:GND #PWR?
+U 1 1 5C3B6897
+P 8850 4450
+F 0 "#PWR?" H 8850 4200 50  0001 C CNN
+F 1 "GND" H 8855 4277 50  0000 C CNN
+F 2 "" H 8850 4450 50  0001 C CNN
+F 3 "" H 8850 4450 50  0001 C CNN
+	1    8850 4450
+	1    0    0    -1
+$EndComp
+$Comp
+L Mechanical:MountingHole_Pad H?
+U 1 1 5C3B68F0
+P 8850 4850
+F 0 "H?" H 8950 4901 50  0000 L CNN
+F 1 "MountingHole_Pad" H 8950 4809 50  0000 L CNN
+F 2 "" H 8850 4850 50  0001 C CNN
+F 3 "~" H 8850 4850 50  0001 C CNN
+	1    8850 4850
+	1    0    0    -1
+$EndComp
+$Comp
+L power:GND #PWR?
+U 1 1 5C3B68F7
+P 8850 4950
+F 0 "#PWR?" H 8850 4700 50  0001 C CNN
+F 1 "GND" H 8855 4777 50  0000 C CNN
+F 2 "" H 8850 4950 50  0001 C CNN
+F 3 "" H 8850 4950 50  0001 C CNN
+	1    8850 4950
+	1    0    0    -1
+$EndComp
+$Comp
+L Mechanical:MountingHole_Pad H?
+U 1 1 5C3B7311
+P 8850 5350
+F 0 "H?" H 8950 5401 50  0000 L CNN
+F 1 "MountingHole_Pad" H 8950 5309 50  0000 L CNN
+F 2 "" H 8850 5350 50  0001 C CNN
+F 3 "~" H 8850 5350 50  0001 C CNN
+	1    8850 5350
+	1    0    0    -1
+$EndComp
+$Comp
+L power:GND #PWR?
+U 1 1 5C3B7318
+P 8850 5450
+F 0 "#PWR?" H 8850 5200 50  0001 C CNN
+F 1 "GND" H 8855 5277 50  0000 C CNN
+F 2 "" H 8850 5450 50  0001 C CNN
+F 3 "" H 8850 5450 50  0001 C CNN
+	1    8850 5450
+	1    0    0    -1
+$EndComp
 $EndSCHEMATC
