File: Hardware/Satelite/PCB_A/PCB_A.sch (KiCad schematic (older format))
At the start: 16 parts, among them J1 Servo Globo, J2 Batería LiPo, J3 Servo Paracaídas, Q1 SSM3J338R,LF, SW1 SW_SPDT, U1 CONUFL001-SMD

Commit message: Footprints para PCB_A (WIP)
Parts:
- removed D3: LED, symbol Device:LED
- removed H? (x2): MountingHole_Pad, symbol Mechanical:MountingHole_Pad
- removed R3: 1k, symbol Device:R
- removed U1: CONUFL001-SMD, symbol AXTEC_IC:CONUFL001-SMD
- added D?: Verde, LED_SMD:LED_0603_1608Metric_Pad1.05x0.95mm_HandSolder, symbol Device:LED
- added H? (x2): MountingHole_Pad, MountingHole:MountingHole_3.2mm_M3_Pad, symbol Mechanical:MountingHole_Pad
- added J?: CONUFL001-SMD, CONUFL001-SMD, symbol SamacSys_Parts:CONUFL001-SMD
- added R?: 1k, Resistor_SMD:R_0603_1608Metric_Pad1.05x0.95mm_HandSolder, symbol Device:R
- C16: footprint (none) -> Capacitor_SMD:C_0603_1608Metric_Pad1.05x0.95mm_HandSolder; Dielectric (none) -> X7R; Manufacturer Part Number (none) -> EMK107B7104KAHT; Voltage (none) -> 10V
- D1: value LED -> Rojo; footprint (none) -> LED_SMD:LED_0603_1608Metric_Pad1.05x0.95mm_HandSolder; Manufacturer Part Number (none) -> 150060RS75000
- H?: footprint (none) -> MountingHole:MountingHole_3.2mm_M3_Pad
- J1, J3: footprint (none) -> Connector_PinHeader_2.54mm:PinHeader_1x03_P2.54mm_Vertical
- J2: value Batería LiPo -> Batería LiPo (Soldada); footprint (none) -> Connector_PinHeader_2.54mm:PinHeader_1x02_P2.54mm_Vertical
- R1: footprint (none) -> Resistor_SMD:R_0603_1608Metric_Pad1.05x0.95mm_HandSolder
Changed lines of the file:
@@
 F 0 "J3" H 6030 4692 50  0000 L CNN
 F 1 "Servo Paracaídas" H 6030 4601 50  0000 L CNN
-F 2 "" H 5950 4650 50  0001 C CNN
+F 2 "Connector_PinHeader_2.54mm:PinHeader_1x03_P2.54mm_Vertical" H 5950 4650 50  0001 C CNN
 F 3 "~" H 5950 4650 50  0001 C CNN
 	1    5950 4650
@@
 F 0 "J1" H 4580 4692 50  0000 L CNN
 F 1 "Servo Globo" H 4580 4601 50  0000 L CNN
-F 2 "" H 4500 4650 50  0001 C CNN
+F 2 "Connector_PinHeader_2.54mm:PinHeader_1x03_P2.54mm_Vertical" H 4500 4650 50  0001 C CNN
 F 3 "~" H 4500 4650 50  0001 C CNN
 	1    4500 4650
@@
 	7450 2450 7050 2450
 $Comp
-L AXTEC_IC:CONUFL001-SMD U1
-U 1 1 5BA4343B
-P 2500 3200
-F 0 "U1" H 2500 3465 50  0000 C CNN
-F 1 "CONUFL001-SMD" H 2500 3374 50  0000 C CNN
-F 2 "" H 2500 3400 50  0001 C CNN
-F 3 "https://componentsearchengine.com/Datasheets/1/CONUFL001-SMD.pdf" H 2500 3400 50  0001 C CNN
-F 4 "CONUFL001-SMD" H 2600 3450 50  0001 C CNN "Manufacturer Part Number"
-	1    2500 3200
-	-1   0    0    -1
-$EndComp
-Wire Wire Line
-	1350 3200 2100 3200
-$Comp
 L power:GND #PWR02
 U 1 1 5BA447BF
-P 3000 3450
-F 0 "#PWR02" H 3000 3200 50  0001 C CNN
-F 1 "GND" H 3005 3277 50  0000 C CNN
-F 2 "" H 3000 3450 50  0001 C CNN
-F 3 "" H 3000 3450 50  0001 C CNN
-	1    3000 3450
-	1    0    0    -1
-$EndComp
-Wire Wire Line
-	2900 3200 3000 3200
-Wire Wire Line
-	3000 3200 3000 3300
-Wire Wire Line
-	2900 3300 3000 3300
-Connection ~ 3000 3300
-Wire Wire Line
-	3000 3300 3000 3450
+P 3200 3450
+F 0 "#PWR02" H 3200 3200 50  0001 C CNN
+F 1 "GND" H 3205 3277 50  0000 C CNN
+F 2 "" H 3200 3450 50  0001 C CNN
+F 3 "" H 3200 3450 50  0001 C CNN
+	1    3200 3450
+	1    0    0    -1
+$EndComp
+Wire Wire Line
+	3100 3200 3200 3200
+Wire Wire Line
+	3200 3200 3200 3300
+Wire Wire Line
+	3100 3300 3200 3300
+Connection ~ 3200 3300
+Wire Wire Line
+	3200 3300 3200 3450
 $Sheet
 S 800  2600 550  700
@@
 P 2550 1400
 F 0 "J2" H 2629 1392 50  0000 L CNN
-F 1 "Batería LiPo" H 2629 1301 50  0000 L CNN
-F 2 "" H 2550 1400 50  0001 C CNN
+F 1 "Batería LiPo (Soldada)" H 2629 1301 50  0000 L CNN
+F 2 "Connector_PinHeader_2.54mm:PinHeader_1x02_P2.54mm_Vertical" H 2550 1400 50  0001 C CNN
 F 3 "~" H 2550 1400 50  0001 C CNN
 	1    2550 1400
@@
 Text Label 4400 5500 1    50   ~ 0
 S_GLOBO
-$Comp
-L Device:LED D3
-U 1 1 5BAF29A3
-P 7500 1650
-F 0 "D3" V 7445 1728 50  0000 L CNN
-F 1 "LED" V 7536 1728 50  0000 L CNN
-F 2 "" H 7500 1650 50  0001 C CNN
-F 3 "~" H 7500 1650 50  0001 C CNN
-	1    7500 1650
-	0    -1   -1   0
-$EndComp
-$Comp
-L Device:R R?
-U 1 1 5BAF2A92
-P 7500 1250
-AR Path="/5BA17F9C/5BAF2A92" Ref="R?"  Part="1"
-AR Path="/5BA1A7F9/5BAF2A92" Ref="R?"  Part="1"
-AR Path="/5BA1A77A/5BAF2A92" Ref="R?"  Part="1"
-AR Path="/5BAF2A92" Ref="R3"  Part="1"
-F 0 "R3" V 7600 1250 50  0000 L CNN
-F 1 "1k" V 7400 1250 50  0000 L CNN
-F 2 "" V 7430 1250 50  0001 C CNN
-F 3 "~" H 7500 1250 50  0001 C CNN
-	1    7500 1250
-	1    0    0    -1
-$EndComp
 Wire Wire Line
 	7500 1500 7500 1400
@@
 P 7050 1650
 F 0 "D1" V 6995 1728 50  0000 L CNN
-F 1 "LED" V 7086 1728 50  0000 L CNN
-F 2 "" H 7050 1650 50  0001 C CNN
+F 1 "Rojo" V 7086 1728 50  0000 L CNN
+F 2 "LED_SMD:LED_0603_1608Metric_Pad1.05x0.95mm_HandSolder" H 7050 1650 50  0001 C CNN
 F 3 "~" H 7050 1650 50  0001 C CNN
+F 4 "150060RS75000" V 7050 1650 50  0001 C CNN "Manufacturer Part Number"
 	1    7050 1650
 	0    -1   -1   0
@@
 F 0 "R1" V 7150 1250 50  0000 L CNN
 F 1 "1k" V 6950 1250 50  0000 L CNN
-F 2 "" V 6980 1250 50  0001 C CNN
+F 2 "Resistor_SMD:R_0603_1608Metric_Pad1.05x0.95mm_HandSolder" V 6980 1250 50  0001 C CNN
 F 3 "~" H 7050 1250 50  0001 C CNN
 	1    7050 1250
@@
 AR Path="/5BA1A77A/5BB16517" Ref="C?"  Part="1"
 AR Path="/5BB16517" Ref="C16"  Part="1"
-F 0 "C16" H 1500 1550 50  0000 L CNN
+F 0 "C16" H 1450 1550 50  0000 L CNN
 F 1 "1uF" H 1450 1450 50  0000 L CNN
-F 2 "" H 1350 1550 50  0001 C CNN
+F 2 "Capacitor_SMD:C_0603_1608Metric_Pad1.05x0.95mm_HandSolder" H 1350 1550 50  0001 C CNN
 F 3 "~" H 1350 1550 50  0001 C CNN
+F 4 "EMK107B7104KAHT" H 1350 1550 50  0001 C CNN "Manufacturer Part Number"
+F 5 "10V" H 1350 1550 50  0001 C CNN "Voltage"
+F 6 "X7R" H 1350 1550 50  0001 C CNN "Dielectric"
 	1    1350 1550
 	1    0    0    -1
@@
 F 0 "H?" H 8950 4401 50  0000 L CNN
 F 1 "MountingHole_Pad" H 8950 4309 50  0000 L CNN
-F 2 "" H 8850 4350 50  0001 C CNN
+F 2 "MountingHole:MountingHole_3.2mm_M3_Pad" H 8850 4350 50  0001 C CNN
 F 3 "~" H 8850 4350 50  0001 C CNN
 	1    8850 4350
@@
 $EndComp
 $Comp
-L Mechanical:MountingHole_Pad H?
-U 1 1 5C3B68F0
-P 8850 4850
-F 0 "H?" H 8950 4901 50  0000 L CNN
-F 1 "MountingHole_Pad" H 8950 4809 50  0000 L CNN
-F 2 "" H 8850 4850 50  0001 C CNN
-F 3 "~" H 8850 4850 50  0001 C CNN
-	1    8850 4850
-	1    0    0    -1
-$EndComp
-$Comp
 L power:GND #PWR?
 U 1 1 5C3B68F7
@@
 $EndComp
 $Comp
-L Mechanical:MountingHole_Pad H?
-U 1 1 5C3B7311
-P 8850 5350
-F 0 "H?" H 8950 5401 50  0000 L CNN
-F 1 "MountingHole_Pad" H 8950 5309 50  0000 L CNN
-F 2 "" H 8850 5350 50  0001 C CNN
-F 3 "~" H 8850 5350 50  0001 C CNN
-	1    8850 5350
-	1    0    0    -1
-$EndComp
-$Comp
 L power:GND #PWR?
 U 1 1 5C3B7318
@@
 	1    0    0    -1
 $EndComp
+$Comp
+L Device:R R?
+U 1 1 5C01D115
+P 7500 1250
+AR Path="/5BA17F9C/5C01D115" Ref="R?"  Part="1"
+AR Path="/5BA1A7F9/5C01D115" Ref="R?"  Part="1"
+AR Path="/5BA1A77A/5C01D115" Ref="R?"  Part="1"
+AR Path="/5C01D115" Ref="R?"  Part="1"
+F 0 "R?" V 7600 1250 50  0000 L CNN
+F 1 "1k" V 7400 1250 50  0000 L CNN
+F 2 "Resistor_SMD:R_0603_1608Metric_Pad1.05x0.95mm_HandSolder" V 7430 1250 50  0001 C CNN
+F 3 "~" H 7500 1250 50  0001 C CNN
+	1    7500 1250
+	1    0    0    -1
+$EndComp
+$Comp
+L Device:LED D?
+U 1 1 5C01D74F
+P 7500 1650
+F 0 "D?" V 7445 1728 50  0000 L CNN
+F 1 "Verde" V 7536 1728 50  0000 L CNN
+F 2 "LED_SMD:LED_0603_1608Metric_Pad1.05x0.95mm_HandSolder" H 7500 1650 50  0001 C CNN
+F 3 "~" H 7500 1650 50  0001 C CNN
+F 4 "150060RS75000" V 7500 1650 50  0001 C CNN "Manufacturer Part Number"
+	1    7500 1650
+	0    -1   -1   0
+$EndComp
+$Comp
+L Mechanical:MountingHole_Pad H?
+U 1 1 5C01DD03
+P 8850 4850
+F 0 "H?" H 8950 4901 50  0000 L CNN
+F 1 "MountingHole_Pad" H 8950 4809 50  0000 L CNN
+F 2 "MountingHole:MountingHole_3.2mm_M3_Pad" H 8850 4850 50  0001 C CNN
+F 3 "~" H 8850 4850 50  0001 C CNN
+	1    8850 4850
+	1    0    0    -1
+$EndComp
+$Comp
+L Mechanical:MountingHole_Pad H?
+U 1 1 5C01DD41
+P 8850 5350
+F 0 "H?" H 8950 5401 50  0000 L CNN
+F 1 "MountingHole_Pad" H 8950 5309 50  0000 L CNN
+F 2 "MountingHole:MountingHole_3.2mm_M3_Pad" H 8850 5350 50  0001 C CNN
+F 3 "~" H 8850 5350 50  0001 C CNN
+	1    8850 5350
+	1    0    0    -1
+$EndComp
+$Comp
+L SamacSys_Parts:CONUFL001-SMD J?
+U 1 1 5C01E8D4
+P 2650 3200
+F 0 "J?" H 2675 3466 50  0000 C CNN
+F 1 "CONUFL001-SMD" H 2675 3374 50  0000 C CNN
+F 2 "CONUFL001-SMD" H 2950 3300 50  0001 L CNN
+F 3 "https://componentsearchengine.com/Datasheets/1/CONUFL001-SMD.pdf" H 2950 3200 50  0001 L CNN
+F 4 "RF Connectors / Coaxial Connectors U.FL Straight Surface Mount Jack" H 2950 3100 50  0001 L CNN "Description"
+F 5 "Linx Technologies" H 2950 2900 50  0001 L CNN "Manufacturer_Name"
+F 6 "CONUFL001-SMD" H 2950 2800 50  0001 L CNN "Manufacturer_Part_Number"
+F 7 "CONUFL001-SMD" H 2950 2500 50  0001 L CNN "Arrow Part Number"
+	1    2650 3200
+	1    0    0    -1
+$EndComp
+Wire Wire Line
+	1350 3200 2250 3200
 $EndSCHEMATC

Commit message: PCB_A correciones, netlist y footprints
Parts:
- removed J?: CONUFL001-SMD, CONUFL001-SMD, symbol SamacSys_Parts:CONUFL001-SMD
- added J1: 5-1814832-1, SamacSys_Parts:5-1814832-1, symbol SamacSys_Parts:5-1814832-1
- SW1: footprint (none) -> Button_Switch_SMD:SW_SPDT_CK-JS102011SAQN
- gave numbers to parts that had none: 7
- renumbered C16 to C1, J1 to J3, J3 to J4
Connections:
- net labels added: +3V3_Internal
- net labels removed: +3V3
- wire segments 50 -> 56

Commit message: PCB_A agregado MH_CanSat y Conector PCB A-B por separados
Parts:
- removed H1, H2, H3: MountingHole_Pad, MountingHole:MountingHole_3.2mm_M3_Pad, symbol Mechanical:MountingHole_Pad
- removed J5, J6: Conn_01x10, Connector_PinHeader_1.27mm:PinHeader_1x10_P1.27mm_Vertical, symbol Connector_Generic:Conn_01x10
- added J4: Conector_PCB_A-B, AXTEC:Conector_PCB_A-B, symbol AXTEC_IC:Conector_PCB_A-B
- added MH1: MH_CanSat, AXTEC:MH_CanSat, symbol AXTEC_IC:MH_CanSat
- SW1: value SW_SPDT -> JS102011SAQN
- renumbered J2 to J1, J1 to J2, J4 to J5
Connections:
- wire segments 56 -> 61
Other:
- note added: "AGUJEROS DE MONTAJE\n\n\n\n"
- note added: "CC1101\n\n"
- note added: "Conector Bateria\n"
- note added: "Conector PCB A-B\n"
- note added: "GPS\n\n\n"
- note added: "SERVOS GLOBO Y PARACAIDA\n"

Commit message: PCB_A diseño WIP
Parts:
- removed J2: 5-1814832-1, SamacSys_Parts:5-1814832-1, symbol SamacSys_Parts:5-1814832-1
- added J2: CONUFL001-SMD, SamacSys_Parts:CONUFL001-SMD, symbol SamacSys_Parts:CONUFL001-SMD
Connections:
- wire segments 61 -> 57
Changed lines of the file:
@@
 L power:GND #PWR06
 U 1 1 5BCC3FF5
-P 2600 4200
-F 0 "#PWR06" H 2600 3950 50  0001 C CNN
-F 1 "GND" H 2605 4027 50  0000 C CNN
-F 2 "" H 2600 4200 50  0001 C CNN
-F 3 "" H 2600 4200 50  0001 C CNN
-	1    2600 4200
+P 3300 4050
+F 0 "#PWR06" H 3300 3800 50  0001 C CNN
+F 1 "GND" H 3305 3877 50  0000 C CNN
+F 2 "" H 3300 4050 50  0001 C CNN
+F 3 "" H 3300 4050 50  0001 C CNN
+	1    3300 4050
 	1    0    0    -1
 $EndComp
-$Comp
-L SamacSys_Parts:5-1814832-1 J2
-U 1 1 5BCC4004
-P 2600 3900
-F 0 "J2" H 2841 3876 50  0000 L CNN
-F 1 "5-1814832-1" H 2841 3784 50  0000 L CNN
-F 2 "SamacSys_Parts:5-1814832-1" H 3000 4000 50  0001 L CNN
-F 3 "http://www.te.com/commerce/DocumentDelivery/DDEController?Action=srchrtrv&DocNm=1814832&DocType=Customer+Drawing&DocLang=English" H 3000 3900 50  0001 L CNN
-F 4 "SUBMINIATURE COAX" H 3000 3800 50  0001 L CNN "Description"
-F 5 "TE Connectivity" H 3000 3600 50  0001 L CNN "Manufacturer_Name"
-F 6 "5-1814832-1" H 3000 3500 50  0001 L CNN "Manufacturer Part Number"
-F 7 "1355074" H 2800 3400 50  0001 L CNN "RS Part Number"
-F 8 "http://uk.rs-online.com/web/p/products/1355074" H 3000 3300 50  0001 L CNN "RS Price/Stock"
-F 9 "70084637" H 3000 3200 50  0001 L CNN "Allied_Number"
-F 10 "https://www.alliedelec.com/te-connectivity-5-1814832-1/70084637/" H 3000 3100 50  0001 L CNN "Allied Price/Stock"
-F 11 "5-1814832-1" H 3000 3000 50  0001 L CNN "Arrow Part Number"
-F 12 "https://www.arrow.com/en/products/5-1814832-1/te-connectivity" H 3000 2900 50  0001 L CNN "Arrow Price/Stock"
-	1    2600 3900
-	1    0    0    -1
-$EndComp
-Wire Wire Line
-	2500 4100 2500 4150
-Wire Wire Line
-	2500 4150 2600 4150
-Wire Wire Line
-	2800 4150 2800 4100
-Wire Wire Line
-	2700 4100 2700 4150
-Connection ~ 2700 4150
-Wire Wire Line
-	2700 4150 2800 4150
-Wire Wire Line
-	2600 4100 2600 4150
-Connection ~ 2600 4150
-Wire Wire Line
-	2600 4150 2700 4150
-Wire Wire Line
-	2600 4200 2600 4150
 Wire Wire Line
 	2400 3900 1600 3900
@@
 Text Notes 750  7250 0    157  ~ 0
 AGUJEROS DE MONTAJE\n\n\n\n
+$Comp
+L SamacSys_Parts:CONUFL001-SMD J2
+U 1 1 5BC6411A
+P 2800 3900
+F 0 "J2" H 2825 4165 50  0000 C CNN
+F 1 "CONUFL001-SMD" H 2825 4074 50  0000 C CNN
+F 2 "SamacSys_Parts:CONUFL001-SMD" H 3100 4000 50  0001 L CNN
+F 3 "https://componentsearchengine.com/Datasheets/1/CONUFL001-SMD.pdf" H 3100 3900 50  0001 L CNN
+F 4 "RF Connectors / Coaxial Connectors U.FL Straight Surface Mount Jack" H 3100 3800 50  0001 L CNN "Description"
+F 5 "Linx Technologies" H 3100 3600 50  0001 L CNN "Manufacturer_Name"
+F 6 "CONUFL001-SMD" H 3100 3500 50  0001 L CNN "Manufacturer_Part_Number"
+F 7 "CONUFL001-SMD" H 3100 3200 50  0001 L CNN "Arrow Part Number"
+	1    2800 3900
+	1    0    0    -1
+$EndComp
+Wire Wire Line
+	3250 3900 3300 3900
+Wire Wire Line
+	3300 3900 3300 4000
+Wire Wire Line
+	3250 4000 3300 4000
+Connection ~ 3300 4000
+Wire Wire Line
+	3300 4000 3300 4050
 $EndSCHEMATC

Commit message: PCB_A modificado coenctor PCB A-B
Changed lines of the file:
@@
 Wire Wire Line
 	8350 3250 8750 3250
-Text Label 9950 2550 0    50   ~ 0
+Text Label 9950 2650 0    50   ~ 0
 GPS_TX
 $Comp
@@
 Text Label 7350 1000 1    50   ~ 0
 P1
-Text Label 9950 2650 0    50   ~ 0
+Text Label 9950 2550 0    50   ~ 0
 P1
 $Comp
@@
 L AXTEC_IC:+3V3_Internal #PWR15
 U 1 1 5BCA5312
-P 10550 2750
-F 0 "#PWR15" H 10550 3150 50  0001 C CNN
-F 1 "+3V3_Internal" H 10535 2923 50  0000 C CNN
-F 2 "" H 10550 2750 50  0001 C CNN
-F 3 "" H 10550 2750 50  0001 C CNN
-	1    10550 2750
+P 10550 3050
+F 0 "#PWR15" H 10550 3450 50  0001 C CNN
+F 1 "+3V3_Internal" H 10535 3223 50  0000 C CNN
+F 2 "" H 10550 3050 50  0001 C CNN
+F 3 "" H 10550 3050 50  0001 C CNN
+	1    10550 3050
 	1    0    0    -1
 $EndComp
@@
 Wire Wire Line
 	2400 3900 1600 3900
-$Comp
-L AXTEC_IC:Conector_PCB_A-B J4
-U 1 1 5BC615BF
-P 9300 2850
-F 0 "J4" H 9300 3415 50  0000 C CNN
-F 1 "Conector_PCB_A-B" H 9300 3324 50  0000 C CNN
-F 2 "AXTEC:Conector_PCB_A-B" H 9050 3300 50  0001 C CNN
-F 3 "" H 9050 3300 50  0001 C CNN
-	1    9300 2850
-	1    0    0    -1
-$EndComp
-Wire Wire Line
-	9850 2750 10550 2750
+Wire Wire Line
+	9850 3050 10550 3050
+Wire Wire Line
+	9850 2650 10200 2650
 Wire Wire Line
 	9850 2550 10200 2550
-Wire Wire Line
-	9850 2650 10200 2650
 Text Notes 8100 850  0    157  ~ 0
 Conector PCB A-B\n
@@
 Wire Wire Line
 	3300 4000 3300 4050
+$Comp
+L AXTEC_IC:Conector_PCB_A-B J4
+U 1 1 5BC66E5E
+P 9300 2850
+F 0 "J4" H 9300 3415 50  0000 C CNN
+F 1 "Conector_PCB_A-B" H 9300 3324 50  0000 C CNN
+F 2 "AXTEC:Conector_PCB_A-B" H 9050 3300 50  0001 C CNN
+F 3 "" H 9050 3300 50  0001 C CNN
+	1    9300 2850
+	1    0    0    -1
+$EndComp
 $EndSCHEMATC

Commit message: Nueva modificacion en Coenctor PCB A-B
Changed lines of the file:
@@
 L power:GND #PWR010
 U 1 1 5BA1B3CD
-P 8100 2800
-F 0 "#PWR010" H 8100 2550 50  0001 C CNN
-F 1 "GND" H 8105 2627 50  0000 C CNN
-F 2 "" H 8100 2800 50  0001 C CNN
-F 3 "" H 8100 2800 50  0001 C CNN
-	1    8100 2800
-	1    0    0    -1
-$EndComp
-Wire Wire Line
-	8350 2950 8750 2950
-Wire Wire Line
-	8350 3050 8750 3050
-Text Label 8400 2950 0    50   ~ 0
+P 7850 2850
+F 0 "#PWR010" H 7850 2600 50  0001 C CNN
+F 1 "GND" H 7855 2677 50  0000 C CNN
+F 2 "" H 7850 2850 50  0001 C CNN
+F 3 "" H 7850 2850 50  0001 C CNN
+	1    7850 2850
+	1    0    0    -1
+$EndComp
+Text Label 8250 3150 0    50   ~ 0
 SDO
-Text Label 8400 3050 0    50   ~ 0
+Text Label 8250 3250 0    50   ~ 0
 SDI
-Text Label 8400 3250 0    50   ~ 0
+Text Label 8250 3450 0    50   ~ 0
 SCLK
-Wire Wire Line
-	8350 3250 8750 3250
-Text Label 9950 2650 0    50   ~ 0
+Text Label 10250 2650 0    50   ~ 0
 GPS_TX
 $Comp
@@
 F6 "CS" I R 1600 3350 50
 $EndSheet
-Wire Wire Line
-	8350 3150 8750 3150
 $Comp
 L Connector_Generic:Conn_01x02 J1
@@
 Text Label 7350 1000 1    50   ~ 0
 P1
-Text Label 9950 2550 0    50   ~ 0
+Text Label 10250 2550 0    50   ~ 0
 P1
 $Comp
@@
 	1350 1650 1350 1700
 Connection ~ 1350 1400
-Text Label 8400 3150 0    50   ~ 0
+Text Label 8250 3350 0    50   ~ 0
 CS
 Wire Wire Line
@@
 Text Label 2000 3350 0    50   ~ 0
 CS
-Wire Wire Line
-	8100 2750 8100 2800
-Wire Wire Line
-	8100 2750 8700 2750
 $Comp
 L power:+BATT #PWR01
@@
 Wire Wire Line
 	8700 2850 8700 2750
-Connection ~ 8700 2750
 Wire Wire Line
 	8700 2750 8750 2750
-Text Label 8200 3350 0    50   ~ 0
+Text Label 8250 2950 0    50   ~ 0
 S_GLOBO
-Wire Wire Line
-	8750 3350 8150 3350
-Wire Wire Line
-	8750 3450 8150 3450
-Text Label 8200 3450 0    50   ~ 0
+Text Label 8250 3050 0    50   ~ 0
 S_PARACAIDAS
 $Comp
@@
 Wire Wire Line
 	2400 3900 1600 3900
-Wire Wire Line
-	9850 3050 10550 3050
-Wire Wire Line
-	9850 2650 10200 2650
-Wire Wire Line
-	9850 2550 10200 2550
 Text Notes 8100 850  0    157  ~ 0
 Conector PCB A-B\n
@@
 	1    0    0    -1
 $EndComp
+Wire Wire Line
+	7850 2850 7850 2750
+Wire Wire Line
+	7850 2750 8700 2750
+Connection ~ 8700 2750
+Wire Wire Line
+	8250 2950 8750 2950
+Wire Wire Line
+	8250 3050 8750 3050
+Wire Wire Line
+	8250 3150 8750 3150
+Wire Wire Line
+	8250 3250 8750 3250
+Wire Wire Line
+	8250 3350 8750 3350
+Wire Wire Line
+	8750 3450 8250 3450
+Wire Wire Line
+	10150 2550 10550 2550
+Wire Wire Line
+	10150 2650 10550 2650
+Wire Wire Line
+	10150 3050 10550 3050
 $EndSCHEMATC
