File: Hardware/Satelite/PCB_A/PCB_A.sch (KiCad schematic (older format))
At the start: 13 parts, among them J1 Batería LiPo (Soldada), J2 CONUFL001-SMD, J3 Servo Globo, J4 Conector_PCB_A-B, J5 Servo Paracaídas, Q1 SSM3J338R,LF, SW1 JS102011SAQN

Commit message: PCB_A mas cambios
Parts:
- removed SW1: JS102011SAQN, Button_Switch_SMD:SW_SPDT_CK-JS102011SAQN, symbol Switch:SW_SPDT
- added S1: 500SSP1S1M6QEA, SamacSys_Parts:500SSP1S1M6QEA, symbol SamacSys_Parts:500SSP1S1M6QEA
Connections:
- wire segments 57 -> 63
Changed lines of the file:
@@
 GPS_TX
 $Comp
-L power:GND #PWR010
+L power:GND #PWR08
 U 1 1 5BA1B3CD
-P 7850 2850
-F 0 "#PWR010" H 7850 2600 50  0001 C CNN
-F 1 "GND" H 7855 2677 50  0000 C CNN
-F 2 "" H 7850 2850 50  0001 C CNN
-F 3 "" H 7850 2850 50  0001 C CNN
-	1    7850 2850
+P 7300 3300
+F 0 "#PWR08" H 7300 3050 50  0001 C CNN
+F 1 "GND" H 7305 3127 50  0000 C CNN
+F 2 "" H 7300 3300 50  0001 C CNN
+F 3 "" H 7300 3300 50  0001 C CNN
+	1    7300 3300
 	1    0    0    -1
 $EndComp
@@
 Text Label 10250 2650 0    50   ~ 0
 GPS_TX
-$Comp
-L Switch:SW_SPDT SW1
-U 1 1 5BA3F421
-P 7950 2450
-F 0 "SW1" H 7700 2550 50  0000 C CNN
-F 1 "JS102011SAQN" H 7700 2650 50  0000 C CNN
-F 2 "Button_Switch_SMD:SW_SPDT_CK-JS102011SAQN" H 7950 2450 50  0001 C CNN
-F 3 "" H 7950 2450 50  0001 C CNN
-	1    7950 2450
-	1    0    0    1
-$EndComp
-Wire Wire Line
-	7750 2450 7350 2450
 $Sheet
 S 1050 3300 550  700
@@
 F0 "CC1101" 50
 F1 "CC1101.sch" 50
-F2 "SDO" O R 1600 3450 50
-F3 "SDI" I R 1600 3550 50
-F4 "SCLK" O R 1600 3650 50
-F5 "ANT" B R 1600 3900 50
-F6 "CS" I R 1600 3350 50
+F2 "ANT" B R 1600 3900 50
+F3 "SCLK" I R 1600 3650 50
+F4 "SO" O R 1600 3450 50
+F5 "SI" I R 1600 3550 50
+F6 "CS" O R 1600 3350 50
 $EndSheet
 $Comp
@@
 $EndComp
 $Comp
-L power:GND #PWR011
+L power:GND #PWR012
 U 1 1 5BAE96AC
 P 8250 5250
-F 0 "#PWR011" H 8250 5000 50  0001 C CNN
+F 0 "#PWR012" H 8250 5000 50  0001 C CNN
 F 1 "GND" H 8255 5077 50  0000 C CNN
 F 2 "" H 8250 5250 50  0001 C CNN
@@
 $EndComp
 $Comp
-L power:GND #PWR013
+L power:GND #PWR014
 U 1 1 5BAE9E59
 P 9700 5250
-F 0 "#PWR013" H 9700 5000 50  0001 C CNN
+F 0 "#PWR014" H 9700 5000 50  0001 C CNN
 F 1 "GND" H 9705 5077 50  0000 C CNN
 F 2 "" H 9700 5250 50  0001 C CNN
@@
 	7800 1500 7800 1400
 $Comp
-L power:GND #PWR09
+L power:GND #PWR010
 U 1 1 5BAF7898
 P 7800 1800
-F 0 "#PWR09" H 7800 1550 50  0001 C CNN
+F 0 "#PWR010" H 7800 1550 50  0001 C CNN
 F 1 "GND" H 7805 1627 50  0000 C CNN
 F 2 "" H 7800 1800 50  0001 C CNN
@@
 	7350 1500 7350 1400
 $Comp
-L power:GND #PWR07
+L power:GND #PWR09
 U 1 1 5BAFD8D0
 P 7350 1800
-F 0 "#PWR07" H 7350 1550 50  0001 C CNN
+F 0 "#PWR09" H 7350 1550 50  0001 C CNN
 F 1 "GND" H 7355 1627 50  0000 C CNN
 F 2 "" H 7350 1800 50  0001 C CNN
@@
 	1000 1400 1350 1400
 $Comp
-L power:+BATT #PWR08
+L power:+BATT #PWR07
 U 1 1 5BC131BC
-P 7350 2450
-F 0 "#PWR08" H 7350 2300 50  0001 C CNN
-F 1 "+BATT" H 7364 2625 50  0000 C CNN
-F 2 "" H 7350 2450 50  0001 C CNN
-F 3 "" H 7350 2450 50  0001 C CNN
-	1    7350 2450
+P 7100 2300
+F 0 "#PWR07" H 7100 2150 50  0001 C CNN
+F 1 "+BATT" H 7114 2475 50  0000 C CNN
+F 2 "" H 7100 2300 50  0001 C CNN
+F 3 "" H 7100 2300 50  0001 C CNN
+	1    7100 2300
 	1    0    0    -1
 $EndComp
@@
 $EndComp
 $Comp
-L AXTEC_IC:+3V3_Internal #PWR12
+L AXTEC_IC:+3V3_Internal #PWR13
 U 1 1 5BCA17A3
 P 8600 5350
-F 0 "#PWR12" H 8600 5750 50  0001 C CNN
+F 0 "#PWR13" H 8600 5750 50  0001 C CNN
 F 1 "+3V3_Internal" H 8585 5523 50  0000 C CNN
 F 2 "" H 8600 5350 50  0001 C CNN
@@
 	8150 5550 8600 5550
 $Comp
-L AXTEC_IC:+3V3_Internal #PWR14
+L AXTEC_IC:+3V3_Internal #PWR15
 U 1 1 5BCA3BE2
 P 10050 5350
-F 0 "#PWR14" H 10050 5750 50  0001 C CNN
+F 0 "#PWR15" H 10050 5750 50  0001 C CNN
 F 1 "+3V3_Internal" H 10035 5523 50  0000 C CNN
 F 2 "" H 10050 5350 50  0001 C CNN
@@
 	9600 5550 10050 5550
 $Comp
-L AXTEC_IC:+3V3_Internal #PWR15
+L AXTEC_IC:+3V3_Internal #PWR16
 U 1 1 5BCA5312
 P 10550 3050
-F 0 "#PWR15" H 10550 3450 50  0001 C CNN
+F 0 "#PWR16" H 10550 3450 50  0001 C CNN
 F 1 "+3V3_Internal" H 10535 3223 50  0000 C CNN
 F 2 "" H 10550 3050 50  0001 C CNN
@@
 CC1101\n\n
 Wire Wire Line
-	8150 2550 8350 2550
-Wire Wire Line
-	8350 2550 8350 1000
+	8350 2550 8350 2350
 Wire Wire Line
 	8350 1000 7800 1000
 Wire Wire Line
 	7800 1000 7800 1100
-Connection ~ 8350 2550
 Wire Wire Line
 	8350 2550 8700 2550
@@
 $EndComp
 Wire Wire Line
-	7850 2850 7850 2750
-Wire Wire Line
-	7850 2750 8700 2750
+	8250 2950 8750 2950
+Wire Wire Line
+	8250 3050 8750 3050
+Wire Wire Line
+	8250 3150 8750 3150
+Wire Wire Line
+	8250 3250 8750 3250
+Wire Wire Line
+	8250 3350 8750 3350
+Wire Wire Line
+	8750 3450 8250 3450
+Wire Wire Line
+	10150 2550 10550 2550
+Wire Wire Line
+	10150 2650 10550 2650
+Wire Wire Line
+	10150 3050 10550 3050
+$Comp
+L SamacSys_Parts:500SSP1S1M6QEA S1
+U 1 1 5BC7E376
+P 7350 2450
+F 0 "S1" V 7704 2578 50  0000 L CNN
+F 1 "500SSP1S1M6QEA" V 7900 2600 50  0000 L CNN
+F 2 "SamacSys_Parts:500SSP1S1M6QEA" H 8000 2550 50  0001 L CNN
+F 3 "https://www.e-switch.com/system/asset/product_line/data_sheet/115/500.pdf" H 8000 2450 50  0001 L CNN
+F 4 "Slide Switches SPDT RA SLIDE PC MNT" H 8000 2350 50  0001 L CNN "Description"
+F 5 "6" H 8000 2250 50  0001 L CNN "Height"
+F 6 "E-Switch" H 8000 2150 50  0001 L CNN "Manufacturer_Name"
+F 7 "500SSP1S1M6QEA" H 8000 2050 50  0001 L CNN "Manufacturer_Part_Number"
+F 8 "" H 8000 1950 50  0001 L CNN "RS Part Number"
+F 9 "" H 8000 1850 50  0001 L CNN "RS Price/Stock"
+F 10 "500SSP1S1M6QEA" H 8000 1750 50  0001 L CNN "Arrow Part Number"
+F 11 "" H 8000 1650 50  0001 L CNN "Arrow Price/Stock"
+	1    7350 2450
+	0    1    1    0
+$EndComp
+Wire Wire Line
+	7250 3250 7300 3250
+Wire Wire Line
+	7300 3300 7300 3250
+Connection ~ 7300 3250
+Wire Wire Line
+	7300 3250 7350 3250
+$Comp
+L power:GND #PWR011
+U 1 1 5BC844C6
+P 8100 2750
+F 0 "#PWR011" H 8100 2500 50  0001 C CNN
+F 1 "GND" H 8105 2577 50  0000 C CNN
+F 2 "" H 8100 2750 50  0001 C CNN
+F 3 "" H 8100 2750 50  0001 C CNN
+	1    8100 2750
+	1    0    0    -1
+$EndComp
+Wire Wire Line
+	8100 2750 8700 2750
 Connection ~ 8700 2750
 Wire Wire Line
-	8250 2950 8750 2950
-Wire Wire Line
-	8250 3050 8750 3050
-Wire Wire Line
-	8250 3150 8750 3150
-Wire Wire Line
-	8250 3250 8750 3250
-Wire Wire Line
-	8250 3350 8750 3350
-Wire Wire Line
-	8750 3450 8250 3450
-Wire Wire Line
-	10150 2550 10550 2550
-Wire Wire Line
-	10150 2650 10550 2650
-Wire Wire Line
-	10150 3050 10550 3050
+	7100 2300 7100 2400
+Wire Wire Line
+	7100 2400 7150 2400
+Wire Wire Line
+	7150 2400 7150 2450
+Wire Wire Line
+	7250 2450 7250 2350
+Wire Wire Line
+	7250 2350 8350 2350
+Connection ~ 8350 2350
+Wire Wire Line
+	8350 2350 8350 1000
 $EndSCHEMATC

Commit message: Cambio en el simbolo de SW1 en PCB_A
Connections:
- wire segments 63 -> 61
Changed lines of the file:
@@
 L power:GND #PWR08
 U 1 1 5BA1B3CD
-P 7300 3300
-F 0 "#PWR08" H 7300 3050 50  0001 C CNN
-F 1 "GND" H 7305 3127 50  0000 C CNN
-F 2 "" H 7300 3300 50  0001 C CNN
-F 3 "" H 7300 3300 50  0001 C CNN
-	1    7300 3300
+P 7350 3150
+F 0 "#PWR08" H 7350 2900 50  0001 C CNN
+F 1 "GND" H 7355 2977 50  0000 C CNN
+F 2 "" H 7350 3150 50  0001 C CNN
+F 3 "" H 7350 3150 50  0001 C CNN
+	1    7350 3150
 	1    0    0    -1
 $EndComp
@@
 L power:+BATT #PWR07
 U 1 1 5BC131BC
-P 7100 2300
-F 0 "#PWR07" H 7100 2150 50  0001 C CNN
-F 1 "+BATT" H 7114 2475 50  0000 C CNN
-F 2 "" H 7100 2300 50  0001 C CNN
-F 3 "" H 7100 2300 50  0001 C CNN
-	1    7100 2300
+P 7150 2350
+F 0 "#PWR07" H 7150 2200 50  0001 C CNN
+F 1 "+BATT" H 7164 2525 50  0000 C CNN
+F 2 "" H 7150 2350 50  0001 C CNN
+F 3 "" H 7150 2350 50  0001 C CNN
+	1    7150 2350
 	1    0    0    -1
 $EndComp
@@
 CC1101\n\n
 Wire Wire Line
-	8350 2550 8350 2350
-Wire Wire Line
 	8350 1000 7800 1000
 Wire Wire Line
@@
 L SamacSys_Parts:500SSP1S1M6QEA S1
 U 1 1 5BC7E376
-P 7350 2450
-F 0 "S1" V 7704 2578 50  0000 L CNN
-F 1 "500SSP1S1M6QEA" V 7900 2600 50  0000 L CNN
-F 2 "SamacSys_Parts:500SSP1S1M6QEA" H 8000 2550 50  0001 L CNN
-F 3 "https://www.e-switch.com/system/asset/product_line/data_sheet/115/500.pdf" H 8000 2450 50  0001 L CNN
-F 4 "Slide Switches SPDT RA SLIDE PC MNT" H 8000 2350 50  0001 L CNN "Description"
-F 5 "6" H 8000 2250 50  0001 L CNN "Height"
-F 6 "E-Switch" H 8000 2150 50  0001 L CNN "Manufacturer_Name"
-F 7 "500SSP1S1M6QEA" H 8000 2050 50  0001 L CNN "Manufacturer_Part_Number"
-F 8 "" H 8000 1950 50  0001 L CNN "RS Part Number"
-F 9 "" H 8000 1850 50  0001 L CNN "RS Price/Stock"
-F 10 "500SSP1S1M6QEA" H 8000 1750 50  0001 L CNN "Arrow Part Number"
-F 11 "" H 8000 1650 50  0001 L CNN "Arrow Price/Stock"
-	1    7350 2450
-	0    1    1    0
-$EndComp
-Wire Wire Line
-	7250 3250 7300 3250
-Wire Wire Line
-	7300 3300 7300 3250
-Connection ~ 7300 3250
-Wire Wire Line
-	7300 3250 7350 3250
+P 7350 2850
+F 0 "S1" H 7300 3350 50  0000 L CNN
+F 1 "500SSP1S1M6QEA" H 7300 3250 50  0000 L CNN
+F 2 "SamacSys_Parts:500SSP1S1M6QEA" H 8000 2950 50  0001 L CNN
+F 3 "https://www.e-switch.com/system/asset/product_line/data_sheet/115/500.pdf" H 8000 2850 50  0001 L CNN
+F 4 "Slide Switches SPDT RA SLIDE PC MNT" H 8000 2750 50  0001 L CNN "Description"
+F 5 "6" H 8000 2650 50  0001 L CNN "Height"
+F 6 "E-Switch" H 8000 2550 50  0001 L CNN "Manufacturer_Name"
+F 7 "500SSP1S1M6QEA" H 8000 2450 50  0001 L CNN "Manufacturer_Part_Number"
+F 8 "" H 8000 2350 50  0001 L CNN "RS Part Number"
+F 9 "" H 8000 2250 50  0001 L CNN "RS Price/Stock"
+F 10 "500SSP1S1M6QEA" H 8000 2150 50  0001 L CNN "Arrow Part Number"
+F 11 "" H 8000 2050 50  0001 L CNN "Arrow Price/Stock"
+	1    7350 2850
+	1    0    0    -1
+$EndComp
+Wire Wire Line
+	7300 3100 7350 3100
+Wire Wire Line
+	7350 3150 7350 3100
+Connection ~ 7350 3100
+Wire Wire Line
+	7350 3100 7400 3100
 $Comp
 L power:GND #PWR011
@@
 Connection ~ 8700 2750
 Wire Wire Line
-	7100 2300 7100 2400
-Wire Wire Line
-	7100 2400 7150 2400
-Wire Wire Line
-	7150 2400 7150 2450
-Wire Wire Line
-	7250 2450 7250 2350
-Wire Wire Line
-	7250 2350 8350 2350
-Connection ~ 8350 2350
-Wire Wire Line
-	8350 2350 8350 1000
+	7150 2350 7150 2800
+Wire Wire Line
+	8350 1000 8350 2550
+Wire Wire Line
+	8350 2550 7650 2550
+Wire Wire Line
+	7650 2550 7650 2700
+Connection ~ 8350 2550
+Wire Wire Line
+	7650 2700 7550 2700
 $EndSCHEMATC
