File: Hardware/Satelite/PCB_A/CC1101.sch (KiCad schematic (older format))
At the start: 18 parts

Commit message: Más modificaciones al esquema del PCB_A
Parts:
- gave numbers to parts that had none: 18
Changed lines of the file:
@@
 $EndDescr
 $Comp
-L AXTEC_IC:CC1101 U?
+L AXTEC_IC:CC1101 U4
 U 1 1 5B9A80AC
 P 3950 3400
-F 0 "U?" H 4350 4050 50  0000 L CNN
+F 0 "U4" H 4350 4050 50  0000 L CNN
 F 1 "CC1101" H 4200 3950 50  0000 L CNN
 F 2 "" H 3650 3450 50  0001 C CNN
@@
 SI
 $Comp
-L power:GND #PWR?
+L power:GND #PWR032
 U 1 1 5B9A819D
 P 3850 4150
-F 0 "#PWR?" H 3850 3900 50  0001 C CNN
+F 0 "#PWR032" H 3850 3900 50  0001 C CNN
 F 1 "GND" H 3855 3977 50  0000 C CNN
 F 2 "" H 3850 4150 50  0001 C CNN
@@
 $EndBitmap
 $Comp
-L Device:C_Small C?
+L Device:C_Small C14
 U 1 1 5B9B43C5
 P 7650 3650
-F 0 "C?" H 7450 3650 50  0000 L CNN
+F 0 "C14" H 7450 3650 50  0000 L CNN
 F 1 "n.a" H 7450 3600 50  0000 L CNN
 F 2 "" H 7650 3650 50  0001 C CNN
@@
 $EndComp
 $Comp
-L Device:R R?
+L Device:R R13
 U 1 1 5B9B44A8
 P 7400 3500
-F 0 "R?" V 7500 3500 50  0000 L CNN
+F 0 "R13" V 7500 3500 50  0000 L CNN
 F 1 "0R" V 7300 3500 50  0000 L CNN
 F 2 "" V 7330 3500 50  0001 C CNN
@@
 $EndComp
 $Comp
-L Device:L L?
+L Device:L L1
 U 1 1 5B9B4522
 P 8400 3500
-F 0 "L?" V 8500 3500 50  0000 L CNN
+F 0 "L1" V 8500 3500 50  0000 L CNN
 F 1 "12nH" V 8350 3400 50  0000 L CNN
 F 2 "" H 8400 3500 50  0001 C CNN
@@
 $EndComp
 $Comp
-L Device:C_Small C?
+L Device:C_Small C6
 U 1 1 5B9B4631
 P 3100 3800
-F 0 "C?" H 3192 3846 50  0000 L CNN
+F 0 "C6" H 3192 3846 50  0000 L CNN
 F 1 "100nF" H 3192 3755 50  0000 L CNN
 F 2 "" H 3100 3800 50  0001 C CNN
@@
 $EndComp
 $Comp
-L Device:C_Small C?
+L Device:C_Small C11
 U 1 1 5B9B4701
 P 4650 3800
-F 0 "C?" H 4742 3846 50  0000 L CNN
+F 0 "C11" H 4742 3846 50  0000 L CNN
 F 1 "100nF" H 4742 3755 50  0000 L CNN
 F 2 "" H 4650 3800 50  0001 C CNN
@@
 $EndComp
 $Comp
-L Device:C_Small C?
+L Device:C_Small C12
 U 1 1 5B9B475E
 P 5050 3400
-F 0 "C?" H 5150 3400 50  0000 L CNN
+F 0 "C12" H 5150 3400 50  0000 L CNN
 F 1 "100nF" H 5100 3300 50  0000 L CNN
 F 2 "" H 5050 3400 50  0001 C CNN
@@
 $EndComp
 $Comp
-L Device:C_Small C?
+L Device:C_Small C13
 U 1 1 5B9B4786
 P 5450 3400
-F 0 "C?" H 5600 3400 50  0000 L CNN
+F 0 "C13" H 5600 3400 50  0000 L CNN
 F 1 "100nF" H 5550 3300 50  0000 L CNN
 F 2 "" H 5450 3400 50  0001 C CNN
@@
 $EndComp
 $Comp
-L Device:C_Small C?
+L Device:C_Small C5
 U 1 1 5B9B48E2
 P 2700 3800
-F 0 "C?" H 2600 3750 50  0000 R CNN
+F 0 "C5" H 2600 3750 50  0000 R CNN
 F 1 "100nF" H 2600 3850 50  0000 R CNN
 F 2 "" H 2700 3800 50  0001 C CNN
@@
 $EndComp
 $Comp
-L Device:C_Small C?
+L Device:C_Small C7
 U 1 1 5B9B4930
 P 3650 2450
-F 0 "C?" H 3800 2400 50  0000 R CNN
+F 0 "C7" H 3800 2400 50  0000 R CNN
 F 1 "100nF" H 3950 2500 50  0000 R CNN
 F 2 "" H 3650 2450 50  0001 C CNN
@@
 $EndComp
 $Comp
-L power:+3V3 #PWR?
+L power:+3V3 #PWR029
 U 1 1 5B9B505D
 P 2700 3400
-F 0 "#PWR?" H 2700 3250 50  0001 C CNN
+F 0 "#PWR029" H 2700 3250 50  0001 C CNN
 F 1 "+3V3" H 2715 3573 50  0000 C CNN
 F 2 "" H 2700 3400 50  0001 C CNN
@@
 	3100 3600 3100 3700
 $Comp
-L power:GND #PWR?
+L power:GND #PWR030
 U 1 1 5B9B53D0
 P 2700 4150
-F 0 "#PWR?" H 2700 3900 50  0001 C CNN
+F 0 "#PWR030" H 2700 3900 50  0001 C CNN
 F 1 "GND" H 2705 3977 50  0000 C CNN
 F 2 "" H 2700 4150 50  0001 C CNN
@@
 $EndComp
 $Comp
-L power:GND #PWR?
+L power:GND #PWR031
 U 1 1 5B9B53EF
 P 3100 4150
-F 0 "#PWR?" H 3100 3900 50  0001 C CNN
+F 0 "#PWR031" H 3100 3900 50  0001 C CNN
 F 1 "GND" H 3105 3977 50  0000 C CNN
 F 2 "" H 3100 4150 50  0001 C CNN
@@
 	2700 3900 2700 4150
 $Comp
-L power:GND #PWR?
+L power:GND #PWR041
 U 1 1 5B9B5925
 P 4650 3950
-F 0 "#PWR?" H 4650 3700 50  0001 C CNN
+F 0 "#PWR041" H 4650 3700 50  0001 C CNN
 F 1 "GND" H 4655 3777 50  0000 C CNN
 F 2 "" H 4650 3950 50  0001 C CNN
@@
 	4650 3600 4650 3700
 $Comp
-L Device:R R?
+L Device:R R12
 U 1 1 5B9B5CA8
 P 4050 2500
-F 0 "R?" H 4120 2546 50  0000 L CNN
+F 0 "R12" H 4120 2546 50  0000 L CNN
 F 1 "56k" H 4120 2455 50  0000 L CNN
 F 2 "" V 3980 2500 50  0001 C CNN
@@
 	4050 2800 4050 2650
 $Comp
-L power:GND #PWR?
+L power:GND #PWR039
 U 1 1 5B9B5F96
 P 4550 2450
-F 0 "#PWR?" H 4550 2200 50  0001 C CNN
+F 0 "#PWR039" H 4550 2200 50  0001 C CNN
 F 1 "GND" H 4555 2277 50  0000 C CNN
 F 2 "" H 4550 2450 50  0001 C CNN
@@
 Connection ~ 4050 2300
 $Comp
-L power:+3V3 #PWR?
+L power:+3V3 #PWR033
 U 1 1 5B9B68A5
 P 3950 2200
-F 0 "#PWR?" H 3950 2050 50  0001 C CNN
+F 0 "#PWR033" H 3950 2050 50  0001 C CNN
 F 1 "+3V3" H 3965 2373 50  0000 C CNN
 F 2 "" H 3950 2200 50  0001 C CNN
@@
 	4650 3300 4650 3200
 $Comp
-L power:+3V3 #PWR?
+L power:+3V3 #PWR040
 U 1 1 5B9B89E5
 P 4650 3050
-F 0 "#PWR?" H 4650 2900 50  0001 C CNN
+F 0 "#PWR040" H 4650 2900 50  0001 C CNN
 F 1 "+3V3" H 4665 3223 50  0000 C CNN
 F 2 "" H 4650 3050 50  0001 C CNN
@@
 	5450 3300 5450 3200
 $Comp
-L power:GND #PWR?
+L power:GND #PWR042
 U 1 1 5B9BA176
 P 5050 3600
-F 0 "#PWR?" H 5050 3350 50  0001 C CNN
+F 0 "#PWR042" H 5050 3350 50  0001 C CNN
 F 1 "GND" H 5055 3427 50  0000 C CNN
 F 2 "" H 5050 3600 50  0001 C CNN
@@
 $EndComp
 $Comp
-L power:GND #PWR?
+L power:GND #PWR043
 U 1 1 5B9BA197
 P 5450 3600
-F 0 "#PWR?" H 5450 3350 50  0001 C CNN
+F 0 "#PWR043" H 5450 3350 50  0001 C CNN
 F 1 "GND" H 5455 3427 50  0000 C CNN
 F 2 "" H 5450 3600 50  0001 C CNN
@@
 	4550 3500 4750 3500
 $Comp
-L power:+3V3 #PWR?
+L power:+3V3 #PWR037
 U 1 1 5B9BC629
 P 4450 4150
-F 0 "#PWR?" H 4450 4000 50  0001 C CNN
+F 0 "#PWR037" H 4450 4000 50  0001 C CNN
 F 1 "+3V3" H 4465 4323 50  0000 C CNN
 F 2 "" H 4450 4150 50  0001 C CNN
@@
 	4050 4000 4050 4200
 $Comp
-L Device:C_Small C?
+L Device:C_Small C10
 U 1 1 5B9BEE8E
 P 4450 4350
-F 0 "C?" H 4542 4396 50  0000 L CNN
+F 0 "C10" H 4542 4396 50  0000 L CNN
 F 1 "100nF" H 4542 4305 50  0000 L CNN
 F 2 "" H 4450 4350 50  0001 C CNN
@@
 $EndComp
 $Comp
-L power:GND #PWR?
+L power:GND #PWR038
 U 1 1 5B9BEEBE
 P 4450 4500
-F 0 "#PWR?" H 4450 4250 50  0001 C CNN
+F 0 "#PWR038" H 4450 4250 50  0001 C CNN
 F 1 "GND" H 4455 4327 50  0000 C CNN
 F 2 "" H 4450 4500 50  0001 C CNN
@@
 $EndComp
 $Comp
-L Device:Crystal_GND2 Y?
+L Device:Crystal_GND2 Y1
 U 1 1 5B9C0407
 P 4150 4500
-F 0 "Y?" H 4150 4768 50  0000 C CNN
+F 0 "Y1" H 4150 4768 50  0000 C CNN
 F 1 "26MHz" H 4150 4677 50  0000 C CNN
 F 2 "" H 4150 4500 50  0001 C CNN
@@
 	4350 4500 4300 4500
 $Comp
-L Device:C_Small C?
+L Device:C_Small C8
 U 1 1 5B9C4C05
 P 3950 4800
-F 0 "C?" H 3800 4850 50  0000 L CNN
+F 0 "C8" H 3800 4850 50  0000 L CNN
 F 1 "15pF" H 3700 4750 50  0000 L CNN
 F 2 "" H 3950 4800 50  0001 C CNN
@@
 $EndComp
 $Comp
-L Device:C_Small C?
+L Device:C_Small C9
 U 1 1 5B9C4C3F
 P 4350 4800
-F 0 "C?" H 4442 4846 50  0000 L CNN
+F 0 "C9" H 4442 4846 50  0000 L CNN
 F 1 "15pF" H 4442 4755 50  0000 L CNN
 F 2 "" H 4350 4800 50  0001 C CNN
@@
 Connection ~ 4350 4500
 $Comp
-L power:GND #PWR?
+L power:GND #PWR035
 U 1 1 5B9C69B0
 P 4150 4950
-F 0 "#PWR?" H 4150 4700 50  0001 C CNN
+F 0 "#PWR035" H 4150 4700 50  0001 C CNN
 F 1 "GND" H 4155 4777 50  0000 C CNN
 F 2 "" H 4150 4950 50  0001 C CNN
@@
 	4350 4950 4350 4900
 $Comp
-L power:GND #PWR?
+L power:GND #PWR034
 U 1 1 5B9C8C28
 P 3950 4950
-F 0 "#PWR?" H 3950 4700 50  0001 C CNN
+F 0 "#PWR034" H 3950 4700 50  0001 C CNN
 F 1 "GND" H 3955 4777 50  0000 C CNN
 F 2 "" H 3950 4950 50  0001 C CNN
@@
 $EndComp
 $Comp
-L power:GND #PWR?
+L power:GND #PWR036
 U 1 1 5B9C8C51
 P 4350 4950
-F 0 "#PWR?" H 4350 4700 50  0001 C CNN
+F 0 "#PWR036" H 4350 4700 50  0001 C CNN
 F 1 "GND" H 4355 4777 50  0000 C CNN
 F 2 "" H 4350 4950 50  0001 C CNN
@@
 	4650 3300 5050 3300
 $Comp
-L AXTEC_IC:0915BM15A0001 U?
+L AXTEC_IC:0915BM15A0001 U5
 U 1 1 5B9AD529
 P 6600 3400
-F 0 "U?" H 6600 3765 50  0000 C CNN
+F 0 "U5" H 6600 3765 50  0000 C CNN
 F 1 "0915BM15A0001" H 6600 3674 50  0000 C CNN
 F 2 "" H 6350 3400 50  0001 C CNN
@@
 	7000 3300 7100 3300
 $Comp
-L power:GND #PWR?
+L power:GND #PWR044
 U 1 1 5B9AFA28
 P 6100 3600
-F 0 "#PWR?" H 6100 3350 50  0001 C CNN
+F 0 "#PWR044" H 6100 3350 50  0001 C CNN
 F 1 "GND" H 6105 3427 50  0000 C CNN
 F 2 "" H 6100 3600 50  0001 C CNN
@@
 Connection ~ 6100 3500
 $Comp
-L power:GND #PWR?
+L power:GND #PWR045
 U 1 1 5B9B345A
 P 7100 3600
-F 0 "#PWR?" H 7100 3350 50  0001 C CNN
+F 0 "#PWR045" H 7100 3350 50  0001 C CNN
 F 1 "GND" H 7105 3427 50  0000 C CNN
 F 2 "" H 7100 3600 50  0001 C CNN
@@
 $EndComp
 $Comp
-L Device:R R?
+L Device:R R14
 U 1 1 5B9B73AA
 P 7900 3500
-F 0 "R?" V 8000 3500 50  0000 L CNN
+F 0 "R14" V 8000 3500 50  0000 L CNN
 F 1 "0R" V 7800 3500 50  0000 L CNN
 F 2 "" V 7830 3500 50  0001 C CNN
@@
 $EndComp
 $Comp
-L Device:C_Small C?
+L Device:C_Small C15
 U 1 1 5B9B73EA
 P 8150 3650
-F 0 "C?" H 7950 3650 50  0000 L CNN
+F 0 "C15" H 7950 3650 50  0000 L CNN
 F 1 "n.a" H 7950 3600 50  0000 L CNN
 F 2 "" H 8150 3650 50  0001 C CNN
@@
 	7000 3500 7250 3500
 $Comp
-L power:GND #PWR?
+L power:GND #PWR046
 U 1 1 5B9C151D
 P 7650 3800
-F 0 "#PWR?" H 7650 3550 50  0001 C CNN
+F 0 "#PWR046" H 7650 3550 50  0001 C CNN
 F 1 "GND" H 7655 3627 50  0000 C CNN
 F 2 "" H 7650 3800 50  0001 C CNN
@@
 $EndComp
 $Comp
-L power:GND #PWR?
+L power:GND #PWR047
 U 1 1 5B9C1582
 P 8150 3800
-F 0 "#PWR?" H 8150 3550 50  0001 C CNN
+F 0 "#PWR047" H 8150 3550 50  0001 C CNN
 F 1 "GND" H 8155 3627 50  0000 C CNN
 F 2 "" H 8150 3800 50  0001 C CNN

Commit message: Completado esquema PCB_B. Mejoras en esquemas de PCB_A.
Connections:
- net labels added: CS
Changed lines of the file:
@@
 Text HLabel 3150 3100 0    50   Input ~ 0
 SI
-$Comp
-L power:GND #PWR032
-U 1 1 5B9A819D
-P 3850 4150
-F 0 "#PWR032" H 3850 3900 50  0001 C CNN
-F 1 "GND" H 3855 3977 50  0000 C CNN
-F 2 "" H 3850 4150 50  0001 C CNN
-F 3 "" H 3850 4150 50  0001 C CNN
-	1    3850 4150
-	1    0    0    -1
-$EndComp
-Wire Wire Line
-	3850 4150 3850 4000
 Text HLabel 8750 3500 2    50   BiDi ~ 0
 ANT
@@
 Wire Wire Line
 	4450 4450 4450 4500
+Text HLabel 3850 4200 3    50   Input ~ 0
+CS
+Wire Wire Line
+	3850 4200 3850 4000
 $EndSCHEMATC

Commit message: PCB_A correciones, netlist y footprints
Parts:
- removed C15: n.a, symbol Device:C_Small
- removed R12: 56k, symbol Device:R
- removed R13, R14: 0R, symbol Device:R
- removed U4: CC1101, symbol AXTEC_IC:CC1101
- removed U5: 0915BM15A0001, symbol AXTEC_IC:0915BM15A0001
- removed Y1: 26MHz, symbol Device:Crystal_GND2
- added C4: 100nF, Capacitor_SMD:C_0603_1608Metric, symbol Device:C_Small
- added R10, R9: 0R, Resistor_SMD:R_0402_1005Metric, symbol Device:R
- added R8: 56k, Resistor_SMD:R_0603_1608Metric_Pad1.05x0.95mm_HandSolder, symbol Device:R
- added U2: CC1101RGP, SamacSys_Parts:QFN50P400X400X100-21N-D, symbol SamacSys_Parts:CC1101RGP
- added U3: 0915BM15A0001E, SamacSys_Parts:0915BM15A0001E, symbol SamacSys_Parts:0915BM15A0001E
- added Y1: 26 MHz, Crystal:Crystal_SMD_2520-4Pin_2.5x2.0mm, symbol Device:Crystal_GND24
- C10, C11, C12, C5, C6: footprint (none) -> Capacitor_SMD:C_0603_1608Metric; Dielectric (none) -> X7R; Manufacturer Part Number (none) -> EMK107B7104KAHT; Voltage (none) -> 16V
- C13: value 100nF -> n.a; footprint (none) -> Capacitor_SMD:C_0402_1005Metric
- C14: footprint (none) -> Capacitor_SMD:C_0402_1005Metric
- C7: value 100nF -> 18pF; footprint (none) -> Capacitor_SMD:C_0603_1608Metric; Dielectric (none) -> NP0; Manufacturer Part Number (none) -> VJ0603A180KXQPW1BC; Voltage (none) -> 10V
- C8: value 15pF -> 18pF; footprint (none) -> Capacitor_SMD:C_0603_1608Metric; Dielectric (none) -> NP0; Manufacturer Part Number (none) -> VJ0603A180KXQPW1BC; Voltage (none) -> 10V
- C9: value 15pF -> 100nF; footprint (none) -> Capacitor_SMD:C_0603_1608Metric; Dielectric (none) -> X7R; Manufacturer Part Number (none) -> EMK107B7104KAHT; Voltage (none) -> 16V
- L1: footprint (none) -> Inductor_SMD:L_0402_1005Metric; Manufacturer Part Number (none) -> L-07C12NJV6
Connections:
- net labels added: +3V3_Internal
- net labels removed: +3V3, CS
