File: Hardware/Satelite/PCB_A/GPS.sch (KiCad schematic (older format))
At the start: 8 parts

Commit message: Más modificaciones al esquema del PCB_A
Parts:
- C4: renamed from C?; value 100nF -> 1uF
- gave numbers to parts that had none: 7
Changed lines of the file:
@@
 $EndDescr
 $Comp
-L AXTEC_IC:A2235-H U?
+L AXTEC_IC:A2235-H U3
 U 1 1 5BAD46BE
 P 5650 3250
-F 0 "U?" H 5700 3965 50  0000 C CNN
+F 0 "U3" H 5700 3965 50  0000 C CNN
 F 1 "A2235-H" H 5700 3874 50  0000 C CNN
 F 2 "AXTEC:A2235-H" H 5200 4150 50  0001 C CNN
@@
 P 4100 3400
 AR Path="/5BA17F9C/5BAD7E11" Ref="R?"  Part="1"
-AR Path="/5BA1A7F9/5BAD7E11" Ref="R?"  Part="1"
-F 0 "R?" V 4200 3400 50  0000 L CNN
+AR Path="/5BA1A7F9/5BAD7E11" Ref="R8"  Part="1"
+F 0 "R8" V 4200 3400 50  0000 L CNN
 F 1 "10k" V 4000 3400 50  0000 L CNN
 F 2 "" V 4030 3400 50  0001 C CNN
@@
 	4100 3600 4100 3550
 $Comp
-L power:GND #PWR?
+L power:GND #PWR026
 U 1 1 5BAD7F7A
 P 5650 4350
-F 0 "#PWR?" H 5650 4100 50  0001 C CNN
+F 0 "#PWR026" H 5650 4100 50  0001 C CNN
 F 1 "GND" H 5655 4177 50  0000 C CNN
 F 2 "" H 5650 4350 50  0001 C CNN
@@
 P 4100 2650
 AR Path="/5BA17F9C/5BAD804E" Ref="R?"  Part="1"
-AR Path="/5BA1A7F9/5BAD804E" Ref="R?"  Part="1"
-F 0 "R?" V 4200 2650 50  0000 L CNN
+AR Path="/5BA1A7F9/5BAD804E" Ref="R7"  Part="1"
+F 0 "R7" V 4200 2650 50  0000 L CNN
 F 1 "10k" V 4000 2650 50  0000 L CNN
 F 2 "" V 4030 2650 50  0001 C CNN
@@
 P 4100 2500
 AR Path="/5BA17F9C/5BAD9CFC" Ref="#PWR?"  Part="1"
-AR Path="/5BA1A7F9/5BAD9CFC" Ref="#PWR?"  Part="1"
-F 0 "#PWR?" H 4100 2350 50  0001 C CNN
+AR Path="/5BA1A7F9/5BAD9CFC" Ref="#PWR025"  Part="1"
+F 0 "#PWR025" H 4100 2350 50  0001 C CNN
 F 1 "+3V3" H 4115 2673 50  0000 C CNN
 F 2 "" H 4100 2500 50  0001 C CNN
@@
 P 7250 3500
 AR Path="/5BA17F9C/5BADA56C" Ref="R?"  Part="1"
-AR Path="/5BA1A7F9/5BADA56C" Ref="R?"  Part="1"
-F 0 "R?" V 7350 3500 50  0000 L CNN
+AR Path="/5BA1A7F9/5BADA56C" Ref="R9"  Part="1"
+F 0 "R9" V 7350 3500 50  0000 L CNN
 F 1 "10k" V 7150 3500 50  0000 L CNN
 F 2 "" V 7180 3500 50  0001 C CNN
@@
 P 7550 3500
 AR Path="/5BA17F9C/5BADA5CC" Ref="R?"  Part="1"
-AR Path="/5BA1A7F9/5BADA5CC" Ref="R?"  Part="1"
-F 0 "R?" V 7650 3500 50  0000 L CNN
+AR Path="/5BA1A7F9/5BADA5CC" Ref="R10"  Part="1"
+F 0 "R10" V 7650 3500 50  0000 L CNN
 F 1 "10k" V 7450 3500 50  0000 L CNN
 F 2 "" V 7480 3500 50  0001 C CNN
@@
 	7550 3200 7550 3350
 $Comp
-L power:GND #PWR?
+L power:GND #PWR027
 U 1 1 5BADABD5
 P 7250 3650
-F 0 "#PWR?" H 7250 3400 50  0001 C CNN
+F 0 "#PWR027" H 7250 3400 50  0001 C CNN
 F 1 "GND" H 7255 3477 50  0000 C CNN
 F 2 "" H 7250 3650 50  0001 C CNN
@@
 P 3100 2500
 AR Path="/5BA17F9C/5BADC174" Ref="#PWR?"  Part="1"
-AR Path="/5BA1A7F9/5BADC174" Ref="#PWR?"  Part="1"
-F 0 "#PWR?" H 3100 2350 50  0001 C CNN
+AR Path="/5BA1A7F9/5BADC174" Ref="#PWR022"  Part="1"
+F 0 "#PWR022" H 3100 2350 50  0001 C CNN
 F 1 "+3V3" H 3115 2673 50  0000 C CNN
 F 2 "" H 3100 2500 50  0001 C CNN
@@
 P 3500 3200
 AR Path="/5BA17F9C/5BADD1F1" Ref="C?"  Part="1"
-AR Path="/5BA1A7F9/5BADD1F1" Ref="C?"  Part="1"
-F 0 "C?" H 3650 3200 50  0000 L CNN
-F 1 "100nF" H 3600 3100 50  0000 L CNN
+AR Path="/5BA1A7F9/5BADD1F1" Ref="C4"  Part="1"
+F 0 "C4" H 3650 3200 50  0000 L CNN
+F 1 "1uF" H 3600 3100 50  0000 L CNN
 F 2 "" H 3500 3200 50  0001 C CNN
 F 3 "~" H 3500 3200 50  0001 C CNN
@@
 $EndComp
 $Comp
-L power:GND #PWR?
+L power:GND #PWR024
 U 1 1 5BADD72A
 P 3500 3450
-F 0 "#PWR?" H 3500 3200 50  0001 C CNN
+F 0 "#PWR024" H 3500 3200 50  0001 C CNN
 F 1 "GND" H 3505 3277 50  0000 C CNN
 F 2 "" H 3500 3450 50  0001 C CNN
@@
 P 3100 3200
 AR Path="/5BA17F9C/5BADE1B6" Ref="C?"  Part="1"
-AR Path="/5BA1A7F9/5BADE1B6" Ref="C?"  Part="1"
-F 0 "C?" H 3250 3200 50  0000 L CNN
+AR Path="/5BA1A7F9/5BADE1B6" Ref="C3"  Part="1"
+F 0 "C3" H 3250 3200 50  0000 L CNN
 F 1 "100nF" H 3200 3100 50  0000 L CNN
 F 2 "" H 3100 3200 50  0001 C CNN
@@
 	3100 3300 3100 3450
 $Comp
-L power:GND #PWR?
+L power:GND #PWR023
 U 1 1 5BADEDE8
 P 3100 3450
-F 0 "#PWR?" H 3100 3200 50  0001 C CNN
+F 0 "#PWR023" H 3100 3200 50  0001 C CNN
 F 1 "GND" H 3105 3277 50  0000 C CNN
 F 2 "" H 3100 3450 50  0001 C CNN
@@
 P 8200 3500
 AR Path="/5BA17F9C/5BAE0532" Ref="R?"  Part="1"
-AR Path="/5BA1A7F9/5BAE0532" Ref="R?"  Part="1"
-F 0 "R?" V 8300 3500 50  0000 L CNN
+AR Path="/5BA1A7F9/5BAE0532" Ref="R11"  Part="1"
+F 0 "R11" V 8300 3500 50  0000 L CNN
 F 1 "10k" V 8100 3500 50  0000 L CNN
 F 2 "" V 8130 3500 50  0001 C CNN
@@
 	8200 3000 8200 3350
 $Comp
-L power:GND #PWR?
+L power:GND #PWR028
 U 1 1 5BAE0C54
 P 8200 3650
-F 0 "#PWR?" H 8200 3400 50  0001 C CNN
+F 0 "#PWR028" H 8200 3400 50  0001 C CNN
 F 1 "GND" H 8205 3477 50  0000 C CNN
 F 2 "" H 8200 3650 50  0001 C CNN

Commit message: PCB_A correciones, netlist y footprints
Parts:
- C2: renamed from C3; footprint (none) -> Capacitor_SMD:C_0603_1608Metric_Pad1.05x0.95mm_HandSolder
- C3: renamed from C4; footprint (none) -> Capacitor_SMD:C_0603_1608Metric_Pad1.05x0.95mm_HandSolder
- R3: renamed from R7; footprint (none) -> Resistor_SMD:R_0603_1608Metric_Pad1.05x0.95mm_HandSolder
- R4: renamed from R8; footprint (none) -> Resistor_SMD:R_0603_1608Metric_Pad1.05x0.95mm_HandSolder
- R5: renamed from R9; footprint (none) -> Resistor_SMD:R_0603_1608Metric_Pad1.05x0.95mm_HandSolder
- R6: renamed from R10; footprint (none) -> Resistor_SMD:R_0603_1608Metric_Pad1.05x0.95mm_HandSolder
- R7: renamed from R11; footprint (none) -> Resistor_SMD:R_0603_1608Metric_Pad1.05x0.95mm_HandSolder
- renumbered U3 to U1
Connections:
- net labels added: +3V3_Internal
- net labels removed: +3V3
- wire segments 40 -> 41
Changed lines of the file:
@@
 $EndDescr
 $Comp
-L AXTEC_IC:A2235-H U3
+L AXTEC_IC:A2235-H U1
 U 1 1 5BAD46BE
 P 5650 3250
-F 0 "U3" H 5700 3965 50  0000 C CNN
+F 0 "U1" H 5700 3965 50  0000 C CNN
 F 1 "A2235-H" H 5700 3874 50  0000 C CNN
 F 2 "AXTEC:A2235-H" H 5200 4150 50  0001 C CNN
@@
 P 4100 3400
 AR Path="/5BA17F9C/5BAD7E11" Ref="R?"  Part="1"
-AR Path="/5BA1A7F9/5BAD7E11" Ref="R8"  Part="1"
-F 0 "R8" V 4200 3400 50  0000 L CNN
+AR Path="/5BA1A7F9/5BAD7E11" Ref="R4"  Part="1"
+F 0 "R4" V 4200 3400 50  0000 L CNN
 F 1 "10k" V 4000 3400 50  0000 L CNN
-F 2 "" V 4030 3400 50  0001 C CNN
+F 2 "Resistor_SMD:R_0603_1608Metric_Pad1.05x0.95mm_HandSolder" V 4030 3400 50  0001 C CNN
 F 3 "~" H 4100 3400 50  0001 C CNN
 	1    4100 3400
@@
 	4100 3600 4100 3550
 $Comp
-L power:GND #PWR026
+L power:GND #PWR022
 U 1 1 5BAD7F7A
 P 5650 4350
-F 0 "#PWR026" H 5650 4100 50  0001 C CNN
+F 0 "#PWR022" H 5650 4100 50  0001 C CNN
 F 1 "GND" H 5655 4177 50  0000 C CNN
 F 2 "" H 5650 4350 50  0001 C CNN
@@
 P 4100 2650
 AR Path="/5BA17F9C/5BAD804E" Ref="R?"  Part="1"
-AR Path="/5BA1A7F9/5BAD804E" Ref="R7"  Part="1"
-F 0 "R7" V 4200 2650 50  0000 L CNN
+AR Path="/5BA1A7F9/5BAD804E" Ref="R3"  Part="1"
+F 0 "R3" V 4200 2650 50  0000 L CNN
 F 1 "10k" V 4000 2650 50  0000 L CNN
-F 2 "" V 4030 2650 50  0001 C CNN
+F 2 "Resistor_SMD:R_0603_1608Metric_Pad1.05x0.95mm_HandSolder" V 4030 2650 50  0001 C CNN
 F 3 "~" H 4100 2650 50  0001 C CNN
 	1    4100 2650
@@
 Wire Wire Line
 	4700 2800 4100 2800
-$Comp
-L power:+3V3 #PWR?
-U 1 1 5BAD9CFC
-P 4100 2500
-AR Path="/5BA17F9C/5BAD9CFC" Ref="#PWR?"  Part="1"
-AR Path="/5BA1A7F9/5BAD9CFC" Ref="#PWR025"  Part="1"
-F 0 "#PWR025" H 4100 2350 50  0001 C CNN
-F 1 "+3V3" H 4115 2673 50  0000 C CNN
-F 2 "" H 4100 2500 50  0001 C CNN
-F 3 "" H 4100 2500 50  0001 C CNN
-	1    4100 2500
-	1    0    0    -1
-$EndComp
 Wire Wire Line
 	4700 3300 4600 3300
@@
 P 7250 3500
 AR Path="/5BA17F9C/5BADA56C" Ref="R?"  Part="1"
-AR Path="/5BA1A7F9/5BADA56C" Ref="R9"  Part="1"
-F 0 "R9" V 7350 3500 50  0000 L CNN
+AR Path="/5BA1A7F9/5BADA56C" Ref="R5"  Part="1"
+F 0 "R5" V 7350 3500 50  0000 L CNN
 F 1 "10k" V 7150 3500 50  0000 L CNN
-F 2 "" V 7180 3500 50  0001 C CNN
+F 2 "Resistor_SMD:R_0603_1608Metric_Pad1.05x0.95mm_HandSolder" V 7180 3500 50  0001 C CNN
 F 3 "~" H 7250 3500 50  0001 C CNN
 	1    7250 3500
@@
 P 7550 3500
 AR Path="/5BA17F9C/5BADA5CC" Ref="R?"  Part="1"
-AR Path="/5BA1A7F9/5BADA5CC" Ref="R10"  Part="1"
-F 0 "R10" V 7650 3500 50  0000 L CNN
+AR Path="/5BA1A7F9/5BADA5CC" Ref="R6"  Part="1"
+F 0 "R6" V 7650 3500 50  0000 L CNN
 F 1 "10k" V 7450 3500 50  0000 L CNN
-F 2 "" V 7480 3500 50  0001 C CNN
+F 2 "Resistor_SMD:R_0603_1608Metric_Pad1.05x0.95mm_HandSolder" V 7480 3500 50  0001 C CNN
 F 3 "~" H 7550 3500 50  0001 C CNN
 	1    7550 3500
@@
 	7550 3200 7550 3350
 $Comp
-L power:GND #PWR027
+L power:GND #PWR023
 U 1 1 5BADABD5
 P 7250 3650
-F 0 "#PWR027" H 7250 3400 50  0001 C CNN
+F 0 "#PWR023" H 7250 3400 50  0001 C CNN
 F 1 "GND" H 7255 3477 50  0000 C CNN
 F 2 "" H 7250 3650 50  0001 C CNN
@@
 TX
 $Comp
-L power:+3V3 #PWR?
-U 1 1 5BADC174
-P 3100 2500
-AR Path="/5BA17F9C/5BADC174" Ref="#PWR?"  Part="1"
-AR Path="/5BA1A7F9/5BADC174" Ref="#PWR022"  Part="1"
-F 0 "#PWR022" H 3100 2350 50  0001 C CNN
-F 1 "+3V3" H 3115 2673 50  0000 C CNN
-F 2 "" H 3100 2500 50  0001 C CNN
-F 3 "" H 3100 2500 50  0001 C CNN
-	1    3100 2500
-	1    0    0    -1
-$EndComp
-$Comp
 L Device:C_Small C?
 U 1 1 5BADD1F1
 P 3500 3200
 AR Path="/5BA17F9C/5BADD1F1" Ref="C?"  Part="1"
-AR Path="/5BA1A7F9/5BADD1F1" Ref="C4"  Part="1"
-F 0 "C4" H 3650 3200 50  0000 L CNN
+AR Path="/5BA1A7F9/5BADD1F1" Ref="C3"  Part="1"
+F 0 "C3" H 3650 3200 50  0000 L CNN
 F 1 "1uF" H 3600 3100 50  0000 L CNN
-F 2 "" H 3500 3200 50  0001 C CNN
+F 2 "Capacitor_SMD:C_0603_1608Metric_Pad1.05x0.95mm_HandSolder" H 3500 3200 50  0001 C CNN
 F 3 "~" H 3500 3200 50  0001 C CNN
 	1    3500 3200
@@
 $EndComp
 $Comp
-L power:GND #PWR024
+L power:GND #PWR020
 U 1 1 5BADD72A
 P 3500 3450
-F 0 "#PWR024" H 3500 3200 50  0001 C CNN
+F 0 "#PWR020" H 3500 3200 50  0001 C CNN
 F 1 "GND" H 3505 3277 50  0000 C CNN
 F 2 "" H 3500 3450 50  0001 C CNN
@@
 P 3100 3200
 AR Path="/5BA17F9C/5BADE1B6" Ref="C?"  Part="1"
-AR Path="/5BA1A7F9/5BADE1B6" Ref="C3"  Part="1"
-F 0 "C3" H 3250 3200 50  0000 L CNN
+AR Path="/5BA1A7F9/5BADE1B6" Ref="C2"  Part="1"
+F 0 "C2" H 3250 3200 50  0000 L CNN
 F 1 "100nF" H 3200 3100 50  0000 L CNN
-F 2 "" H 3100 3200 50  0001 C CNN
+F 2 "Capacitor_SMD:C_0603_1608Metric_Pad1.05x0.95mm_HandSolder" H 3100 3200 50  0001 C CNN
 F 3 "~" H 3100 3200 50  0001 C CNN
 	1    3100 3200
@@
 	3100 3300 3100 3450
 $Comp
-L power:GND #PWR023
+L power:GND #PWR019
 U 1 1 5BADEDE8
 P 3100 3450
-F 0 "#PWR023" H 3100 3200 50  0001 C CNN
+F 0 "#PWR019" H 3100 3200 50  0001 C CNN
 F 1 "GND" H 3105 3277 50  0000 C CNN
 F 2 "" H 3100 3450 50  0001 C CNN
@@
 	3500 3000 4700 3000
 Connection ~ 3500 3000
-Wire Wire Line
-	3100 3000 3100 2500
 Connection ~ 3100 3000
 $Comp
@@
 P 8200 3500
 AR Path="/5BA17F9C/5BAE0532" Ref="R?"  Part="1"
-AR Path="/5BA1A7F9/5BAE0532" Ref="R11"  Part="1"
-F 0 "R11" V 8300 3500 50  0000 L CNN
+AR Path="/5BA1A7F9/5BAE0532" Ref="R7"  Part="1"
+F 0 "R7" V 8300 3500 50  0000 L CNN
 F 1 "10k" V 8100 3500 50  0000 L CNN
-F 2 "" V 8130 3500 50  0001 C CNN
+F 2 "Resistor_SMD:R_0603_1608Metric_Pad1.05x0.95mm_HandSolder" V 8130 3500 50  0001 C CNN
 F 3 "~" H 8200 3500 50  0001 C CNN
 	1    8200 3500
@@
 	8200 3000 8200 3350
 $Comp
-L power:GND #PWR028
+L power:GND #PWR024
 U 1 1 5BAE0C54
 P 8200 3650
-F 0 "#PWR028" H 8200 3400 50  0001 C CNN
+F 0 "#PWR024" H 8200 3400 50  0001 C CNN
 F 1 "GND" H 8205 3477 50  0000 C CNN
 F 2 "" H 8200 3650 50  0001 C CNN
@@
 	1    0    0    -1
 $EndComp
+$Comp
+L AXTEC_IC:+3V3_Internal #PWR?
+U 1 1 5BCA70ED
+P 3100 2450
+AR Path="/5BCA70ED" Ref="#PWR?"  Part="1"
+AR Path="/5BA1A7F9/5BCA70ED" Ref="#PWR18"  Part="1"
+F 0 "#PWR18" H 3100 2850 50  0001 C CNN
+F 1 "+3V3_Internal" H 3085 2623 50  0000 C CNN
+F 2 "" H 3100 2450 50  0001 C CNN
+F 3 "" H 3100 2450 50  0001 C CNN
+	1    3100 2450
+	1    0    0    -1
+$EndComp
+$Comp
+L AXTEC_IC:+3V3_Internal #PWR?
+U 1 1 5BCA7823
+P 4100 2450
+AR Path="/5BCA7823" Ref="#PWR?"  Part="1"
+AR Path="/5BA1A7F9/5BCA7823" Ref="#PWR21"  Part="1"
+F 0 "#PWR21" H 4100 2850 50  0001 C CNN
+F 1 "+3V3_Internal" H 4085 2623 50  0000 C CNN
+F 2 "" H 4100 2450 50  0001 C CNN
+F 3 "" H 4100 2450 50  0001 C CNN
+	1    4100 2450
+	1    0    0    -1
+$EndComp
+Wire Wire Line
+	4100 2450 4100 2500
+Wire Wire Line
+	3100 2450 3100 3000
 $EndSCHEMATC
