File: Hardware/Satelite/PCB_B/PCB_B.sch (KiCad schematic (older format))
At the start: 0 parts

Commit message: Agregado esquemas de sensores a PCB_B
Parts:
- added J? (x5): Conn_02x02_Counter_Clockwise, symbol Connector_Generic:Conn_02x02_Counter_Clockwise
- added U?: STM32F401RETx, Package_QFP:LQFP-64_10x10mm_P0.5mm, symbol MCU_ST_STM32F4:STM32F401RETx
Connections:
- net labels added: +3V3, CHG, CHG_DISABLE, GND, GPOUT, GPS_TX, ISET, P1, P2, SCLK, SDI, SDO, S_GLOBO, S_PARACAIDAS, VBUS, VBat, VBat_I_SENSE
- wire segments 0 -> 35

Commit message: Fuente de 3.3V interna
Parts:
- added C? (x2): 1uF, symbol Device:C_Small
- added C?: 100nF, symbol Device:C_Small
- added IC?: MIC5323-3.3YD5_TR, SOT95P280X100-5N, symbol SamacSys_Parts:MIC5323-3.3YD5_TR
Connections:
- net labels added: +BATT, 3V3_INT
- net labels removed: VBat
- wire segments 35 -> 52
Other:
- moved on the sheet: U?
Changed lines of the file:
@@
 	9850 950  9300 950
 Wire Wire Line
-	9850 1050 9300 1050
-Wire Wire Line
 	10350 950  10900 950
 Wire Wire Line
@@
 Wire Wire Line
 	10350 3250 10900 3250
-Text Label 9400 950  0    50   ~ 0
-VBat
-Text Label 9400 1050 0    50   ~ 0
-VBUS
 $Comp
 L power:GND #PWR?
@@
 L MCU_ST_STM32F4:STM32F401RETx U?
 U 1 1 5BB6D45B
-P 5650 3000
-F 0 "U?" H 5600 4878 50  0000 C CNN
-F 1 "STM32F401RETx" H 5600 4787 50  0000 C CNN
-F 2 "Package_QFP:LQFP-64_10x10mm_P0.5mm" H 5050 1300 50  0001 R CNN
-F 3 "http://www.st.com/st-web-ui/static/active/en/resource/technical/document/datasheet/DM00102166.pdf" H 5650 3000 50  0001 C CNN
-	1    5650 3000
+P 6600 3200
+F 0 "U?" H 6550 5078 50  0000 C CNN
+F 1 "STM32F401RETx" H 6550 4987 50  0000 C CNN
+F 2 "Package_QFP:LQFP-64_10x10mm_P0.5mm" H 6000 1500 50  0001 R CNN
+F 3 "http://www.st.com/st-web-ui/static/active/en/resource/technical/document/datasheet/DM00102166.pdf" H 6600 3200 50  0001 C CNN
+	1    6600 3200
 	1    0    0    -1
 $EndComp
@@
 EndData
 $EndBitmap
+$Comp
+L SamacSys_Parts:MIC5323-3.3YD5_TR IC?
+U 1 1 5BB7621F
+P 1450 6900
+F 0 "IC?" H 2000 7165 50  0000 C CNN
+F 1 "MIC5323-3.3YD5_TR" H 2000 7074 50  0000 C CNN
+F 2 "SOT95P280X100-5N" H 2400 7000 50  0001 L CNN
+F 3 "http://ww1.microchip.com/downloads/en/DeviceDoc/MIC5323.pdf" H 2400 6900 50  0001 L CNN
+F 4 "Micrel MIC5323-3.3YD5 TR, LDO Voltage Regulator, 300mA, 3.3 V 2%, 2.65  5.5 Vin, 5-Pin TSOT-23" H 2400 6800 50  0001 L CNN "Description"
+F 5 "1" H 2400 6700 50  0001 L CNN "Height"
+F 6 "Micrel" H 2400 6600 50  0001 L CNN "Manufacturer_Name"
+F 7 "MIC5323-3.3YD5 TR" H 2400 6500 50  0001 L CNN "Manufacturer_Part_Number"
+F 8 "8855996P" H 2400 6400 50  0001 L CNN "RS Part Number"
+F 9 "http://uk.rs-online.com/web/p/products/8855996P" H 2400 6300 50  0001 L CNN "RS Price/Stock"
+F 10 "MIC5323-3.3YD5 TR" H 2400 6200 50  0001 L CNN "Arrow Part Number"
+F 11 "http://uk.rs-online.com/web/p/products/8855996P" H 2400 6100 50  0001 L CNN "Arrow Price/Stock"
+	1    1450 6900
+	1    0    0    -1
+$EndComp
+$Comp
+L Device:C_Small C?
+U 1 1 5BB76226
+P 850 7050
+AR Path="/5BB122CA/5BB76226" Ref="C?"  Part="1"
+AR Path="/5BB12371/5BB76226" Ref="C?"  Part="1"
+AR Path="/5BB123AC/5BB76226" Ref="C?"  Part="1"
+AR Path="/5BB76226" Ref="C?"  Part="1"
+F 0 "C?" H 758 7004 50  0000 R CNN
+F 1 "1uF" H 758 7095 50  0000 R CNN
+F 2 "" H 850 7050 50  0001 C CNN
+F 3 "~" H 850 7050 50  0001 C CNN
+	1    850  7050
+	-1   0    0    1
+$EndComp
+Wire Wire Line
+	1450 6900 1350 6900
+Wire Wire Line
+	850  6900 850  6950
+$Comp
+L power:GND #PWR?
+U 1 1 5BB772C4
+P 850 7350
+F 0 "#PWR?" H 850 7100 50  0001 C CNN
+F 1 "GND" H 855 7177 50  0000 C CNN
+F 2 "" H 850 7350 50  0001 C CNN
+F 3 "" H 850 7350 50  0001 C CNN
+	1    850  7350
+	1    0    0    -1
+$EndComp
+$Comp
+L power:GND #PWR?
+U 1 1 5BB772E6
+P 1200 7350
+F 0 "#PWR?" H 1200 7100 50  0001 C CNN
+F 1 "GND" H 1205 7177 50  0000 C CNN
+F 2 "" H 1200 7350 50  0001 C CNN
+F 3 "" H 1200 7350 50  0001 C CNN
+	1    1200 7350
+	1    0    0    -1
+$EndComp
+Wire Wire Line
+	1200 7350 1200 7000
+Wire Wire Line
+	1200 7000 1450 7000
+Wire Wire Line
+	850  7350 850  7150
+Wire Wire Line
+	1450 7100 1350 7100
+Wire Wire Line
+	1350 7100 1350 6900
+Connection ~ 1350 6900
+Wire Wire Line
+	1350 6900 850  6900
+$Comp
+L Device:C_Small C?
+U 1 1 5BB79007
+P 2750 7150
+AR Path="/5BB122CA/5BB79007" Ref="C?"  Part="1"
+AR Path="/5BB12371/5BB79007" Ref="C?"  Part="1"
+AR Path="/5BB123AC/5BB79007" Ref="C?"  Part="1"
+AR Path="/5BB79007" Ref="C?"  Part="1"
+F 0 "C?" H 2658 7104 50  0000 R CNN
+F 1 "100nF" H 2658 7195 50  0000 R CNN
+F 2 "" H 2750 7150 50  0001 C CNN
+F 3 "~" H 2750 7150 50  0001 C CNN
+	1    2750 7150
+	-1   0    0    1
+$EndComp
+$Comp
+L power:GND #PWR?
+U 1 1 5BB79C3E
+P 2750 7350
+F 0 "#PWR?" H 2750 7100 50  0001 C CNN
+F 1 "GND" H 2755 7177 50  0000 C CNN
+F 2 "" H 2750 7350 50  0001 C CNN
+F 3 "" H 2750 7350 50  0001 C CNN
+	1    2750 7350
+	1    0    0    -1
+$EndComp
+Wire Wire Line
+	2750 7250 2750 7350
+Wire Wire Line
+	2750 7050 2750 6900
+Wire Wire Line
+	2750 6900 2550 6900
+Wire Wire Line
+	2550 7000 3200 7000
+$Comp
+L Device:C_Small C?
+U 1 1 5BB7D925
+P 3200 7150
+AR Path="/5BB122CA/5BB7D925" Ref="C?"  Part="1"
+AR Path="/5BB12371/5BB7D925" Ref="C?"  Part="1"
+AR Path="/5BB123AC/5BB7D925" Ref="C?"  Part="1"
+AR Path="/5BB7D925" Ref="C?"  Part="1"
+F 0 "C?" H 3108 7104 50  0000 R CNN
+F 1 "1uF" H 3108 7195 50  0000 R CNN
+F 2 "" H 3200 7150 50  0001 C CNN
+F 3 "~" H 3200 7150 50  0001 C CNN
+	1    3200 7150
+	-1   0    0    1
+$EndComp
+Wire Wire Line
+	3200 7050 3200 7000
+$Comp
+L power:GND #PWR?
+U 1 1 5BB7E63C
+P 3200 7350
+F 0 "#PWR?" H 3200 7100 50  0001 C CNN
+F 1 "GND" H 3205 7177 50  0000 C CNN
+F 2 "" H 3200 7350 50  0001 C CNN
+F 3 "" H 3200 7350 50  0001 C CNN
+	1    3200 7350
+	1    0    0    -1
+$EndComp
+Wire Wire Line
+	3200 7350 3200 7250
+$Comp
+L power:+BATT #PWR?
+U 1 1 5BB7F55C
+P 9300 900
+F 0 "#PWR?" H 9300 750 50  0001 C CNN
+F 1 "+BATT" H 9315 1073 50  0000 C CNN
+F 2 "" H 9300 900 50  0001 C CNN
+F 3 "" H 9300 900 50  0001 C CNN
+	1    9300 900
+	1    0    0    -1
+$EndComp
+Wire Wire Line
+	9300 950  9300 900
+$Comp
+L power:VBUS #PWR?
+U 1 1 5BB802DA
+P 9000 900
+F 0 "#PWR?" H 9000 750 50  0001 C CNN
+F 1 "VBUS" H 9015 1073 50  0000 C CNN
+F 2 "" H 9000 900 50  0001 C CNN
+F 3 "" H 9000 900 50  0001 C CNN
+	1    9000 900
+	1    0    0    -1
+$EndComp
+Wire Wire Line
+	9000 1050 9000 900
+Wire Wire Line
+	9000 1050 9850 1050
+$Comp
+L power:+BATT #PWR?
+U 1 1 5BB81112
+P 850 6750
+F 0 "#PWR?" H 850 6600 50  0001 C CNN
+F 1 "+BATT" H 865 6923 50  0000 C CNN
+F 2 "" H 850 6750 50  0001 C CNN
+F 3 "" H 850 6750 50  0001 C CNN
+	1    850  6750
+	1    0    0    -1
+$EndComp
+Wire Wire Line
+	850  6750 850  6900
+Connection ~ 850  6900
+Text Label 2900 7000 0    50   ~ 0
+3V3_INT
 $EndSCHEMATC

Commit message: Esquemas de fuentes de 5V y 3.3V del satélite
Connections:
- net labels added: +3V3_Internal
- net labels removed: 3V3_INT
- wire segments 52 -> 53
Changed lines of the file:
@@
 F2 "VBAT" I R 1850 4300 50
 F3 "CTRL" I R 1850 4400 50
-F4 "3V3" I R 1850 4700 50
+F4 "5V" I R 1850 4700 50
 F5 "ISENSE" O R 1850 4600 50
 $EndSheet
@@
 	850  6750 850  6900
 Connection ~ 850  6900
-Text Label 2900 7000 0    50   ~ 0
-3V3_INT
+Wire Wire Line
+	3200 6800 3200 7000
+Connection ~ 3200 7000
+$Comp
+L AXTEC_IC:+3V3_Internal #PWR?
+U 1 1 5BBB29E5
+P 3200 6800
+F 0 "#PWR?" H 3200 7200 50  0001 C CNN
+F 1 "+3V3_Internal" H 3185 6973 50  0000 C CNN
+F 2 "" H 3200 6800 50  0001 C CNN
+F 3 "" H 3200 6800 50  0001 C CNN
+	1    3200 6800
+	1    0    0    -1
+$EndComp
 $EndSCHEMATC

Commit message: Completado esquema PCB_B. Mejoras en esquemas de PCB_A.
Parts:
- removed J? (x5): Conn_02x02_Counter_Clockwise, symbol Connector_Generic:Conn_02x02_Counter_Clockwise
- added C? (x2): 1uF, symbol Device:C_Small
- added C? (x2): 4.3pF, symbol Device:C_Small
- added C? (x2): 20pF, symbol Device:C_Small
- added C? (x2): 4.7uF, symbol Device:C_Small
- added C? (x9): 100nF, symbol Device:C_Small
- added IC?: BQ24392RSER, RSE(R-PUQFN-N10), symbol SamacSys_Parts:BQ24392RSER
- added IC?: MCP1501T-33E_CHY, SOT95P270X145-6N, symbol SamacSys_Parts:MCP1501T-33E_CHY
- added IC?: TXB0304RUTR, RUT(R-PUQFN-N12), symbol SamacSys_Parts:TXB0304RUTR
- added J?: USB_B_Micro, symbol Connector:USB_B_Micro
- added J?: Conn_01x06, symbol Connector_Generic:Conn_01x06
- added J? (x2): Conn_01x10, Connector_PinHeader_1.27mm:PinHeader_1x10_P1.27mm_Vertical, symbol Connector_Generic:Conn_01x10
- added J? (x2): Conn_01x10, symbol Connector_Generic:Conn_01x10
- added U?: TCA9802DGKR, SOP65P490X110-8N, symbol SamacSys_Parts:TCA9802DGKR
- added Y?: LFXTAL016178, LFXTAL016178_1, symbol SamacSys_Parts:LFXTAL016178
- added Y?: Crystal, symbol Device:Crystal
Connections:
- net labels added: +5V, +VREF, 3V_ENABLE, 3V_I_SENSE, 3V_V_SENSE, 5V_ENABLE, 5V_I_SENSE, 5V_V_SENSE, CHG_ALLOWED, CHG_DETECT, CS, D+, D-, EXT_CS, EXT_SCLK, EXT_SDI, EXT_SDO, I2C_EN, NRST, SCL_CHG, SCL_EXT, SDA_CHG, SDA_EXT, SPI_BUFFER_EN, SWCLK, SWDIO, SWO, SW_OPEN
- net labels removed: P2
- wire segments 53 -> 266
Other:
- note added: "+VREF ADC"
- note added: "Alimentación externa e interna"
- note added: "Buffer I2C"
- note added: "Buffer SPI"
- note added: "Conectores para PCB_A"
- note added: "Conectores para PCB_B"
- note added: "Header \nprogramación"
- note added: "Sensores"
- note added: "USB y detección de cargador"
- moved on the sheet: U?

Commit message: Finalizado esquema de PCB_C
Parts:
- removed J?: Conn_01x10, symbol Connector_Generic:Conn_01x10
- added J?: Conn_01x10, Connector_PinHeader_1.27mm:PinHeader_1x10_P1.27mm_Vertical, symbol Connector_Generic:Conn_01x10
- added R? (x4): 10K, symbol Device:R
Connections:
- wire segments 266 -> 275
Changed lines of the file:
@@
 Text Label 7500 5650 2    50   ~ 0
 SDA
-Wire Wire Line
-	7750 5650 7300 5650
-Wire Wire Line
-	9050 3950 9450 3950
 Text Label 9300 3950 2    50   ~ 0
 SCL
-Wire Wire Line
-	9050 5550 9500 5550
 Text Label 9150 5550 0    50   ~ 0
 SDA_CHG
-Wire Wire Line
-	9050 5450 9500 5450
 Text Label 9150 5450 0    50   ~ 0
 SCL_CHG
@@
 	13150 3700 13150 3750
 $Comp
-L Connector_Generic:Conn_01x10 J?
-U 1 1 5C6421BB
-P 15400 3900
-F 0 "J?" H 15479 3892 50  0000 L CNN
-F 1 "Conn_01x10" H 15479 3800 50  0000 L CNN
-F 2 "" H 15400 3900 50  0001 C CNN
-F 3 "~" H 15400 3900 50  0001 C CNN
-	1    15400 3900
-	1    0    0    -1
-$EndComp
-$Comp
 L power:+3V3 #PWR?
 U 1 1 5C6531A4
@@
 Wire Wire Line
 	15150 3400 15150 3500
+$Comp
+L Connector_Generic:Conn_01x10 J?
+U 1 1 5BBF74AE
+P 15400 3900
+F 0 "J?" H 15479 3892 50  0000 L CNN
+F 1 "Conn_01x10" H 15479 3800 50  0000 L CNN
+F 2 "Connector_PinHeader_1.27mm:PinHeader_1x10_P1.27mm_Vertical" H 15400 3900 50  0001 C CNN
+F 3 "https://www.mouser.com/datasheet/2/181/M50-353-1100851.pdf" H 15400 3900 50  0001 C CNN
+F 4 "M50-3531042" H 15400 3900 50  0001 C CNN "Manufacturer Part Number"
+	1    15400 3900
+	1    0    0    -1
+$EndComp
+$Comp
+L Device:R R?
+U 1 1 5BC0B03C
+P 10100 3550
+F 0 "R?" H 10170 3596 50  0000 L CNN
+F 1 "10K" H 10170 3504 50  0000 L CNN
+F 2 "" V 10030 3550 50  0001 C CNN
+F 3 "~" H 10100 3550 50  0001 C CNN
+	1    10100 3550
+	1    0    0    -1
+$EndComp
+Wire Wire Line
+	10100 3950 10100 3700
+Wire Wire Line
+	9050 3950 10100 3950
+$Comp
+L AXTEC_IC:+3V3_Internal #PWR?
+U 1 1 5BC1DDE1
+P 10100 3400
+F 0 "#PWR?" H 10100 3800 50  0001 C CNN
+F 1 "+3V3_Internal" H 10085 3573 50  0000 C CNN
+F 2 "" H 10100 3400 50  0001 C CNN
+F 3 "" H 10100 3400 50  0001 C CNN
+	1    10100 3400
+	1    0    0    -1
+$EndComp
+$Comp
+L Device:R R?
+U 1 1 5BC1DEA5
+P 6650 5350
+F 0 "R?" H 6720 5396 50  0000 L CNN
+F 1 "10K" H 6720 5304 50  0000 L CNN
+F 2 "" V 6580 5350 50  0001 C CNN
+F 3 "~" H 6650 5350 50  0001 C CNN
+	1    6650 5350
+	1    0    0    -1
+$EndComp
+Wire Wire Line
+	6650 5500 6650 5650
+Wire Wire Line
+	6650 5650 7750 5650
+$Comp
+L AXTEC_IC:+3V3_Internal #PWR?
+U 1 1 5BC307DD
+P 6650 5200
+F 0 "#PWR?" H 6650 5600 50  0001 C CNN
+F 1 "+3V3_Internal" H 6635 5373 50  0000 C CNN
+F 2 "" H 6650 5200 50  0001 C CNN
+F 3 "" H 6650 5200 50  0001 C CNN
+	1    6650 5200
+	1    0    0    -1
+$EndComp
+$Comp
+L Device:R R?
+U 1 1 5BC3149F
+P 10000 5200
+F 0 "R?" H 10070 5246 50  0000 L CNN
+F 1 "10K" H 10070 5154 50  0000 L CNN
+F 2 "" V 9930 5200 50  0001 C CNN
+F 3 "~" H 10000 5200 50  0001 C CNN
+	1    10000 5200
+	1    0    0    -1
+$EndComp
+$Comp
+L Device:R R?
+U 1 1 5BC316A8
+P 10400 5200
+F 0 "R?" H 10470 5246 50  0000 L CNN
+F 1 "10K" H 10470 5154 50  0000 L CNN
+F 2 "" V 10330 5200 50  0001 C CNN
+F 3 "~" H 10400 5200 50  0001 C CNN
+	1    10400 5200
+	1    0    0    -1
+$EndComp
+Wire Wire Line
+	10000 5450 10000 5350
+Wire Wire Line
+	9050 5450 10000 5450
+Wire Wire Line
+	10400 5550 10400 5350
+Wire Wire Line
+	9050 5550 10400 5550
+$Comp
+L AXTEC_IC:+3V3_Internal #PWR?
+U 1 1 5BC56B17
+P 10200 4900
+F 0 "#PWR?" H 10200 5300 50  0001 C CNN
+F 1 "+3V3_Internal" H 10185 5073 50  0000 C CNN
+F 2 "" H 10200 4900 50  0001 C CNN
+F 3 "" H 10200 4900 50  0001 C CNN
+	1    10200 4900
+	1    0    0    -1
+$EndComp
+Wire Wire Line
+	10000 5050 10000 4950
+Wire Wire Line
+	10000 4950 10200 4950
+Wire Wire Line
+	10200 4950 10200 4900
+Wire Wire Line
+	10400 5050 10400 4950
+Wire Wire Line
+	10400 4950 10200 4950
+Connection ~ 10200 4950
 $EndSCHEMATC

Commit message: Agregado de más pines de expansión al conector interno del satélite
Parts:
- added J?: Conn_01x10, Connector_PinHeader_1.27mm:PinHeader_1x10_P1.27mm_Vertical, symbol Connector_Generic:Conn_01x10
Connections:
- net labels added: IO0, IO1, IO2, IO3, IO4, IO5, IO6
- wire segments 275 -> 296

Commit message: Cambio de MCU supervisor de F4 a F3 y agregado de protecciones
Parts:
- removed C?: 4.7uF, symbol Device:C_Small
- removed C?: 1uF, symbol Device:C_Small
- removed C?: 100nF, symbol Device:C_Small
- removed IC?: MIC5323-3.3YD5_TR, SOT95P280X100-5N, symbol SamacSys_Parts:MIC5323-3.3YD5_TR
- removed IC?: TXB0304RUTR, RUT(R-PUQFN-N12), symbol SamacSys_Parts:TXB0304RUTR
- removed J? (x3): Conn_01x10, Connector_PinHeader_1.27mm:PinHeader_1x10_P1.27mm_Vertical, symbol Connector_Generic:Conn_01x10
- removed R? (x2): 10K, symbol Device:R
- removed U?: STM32F401RETx, Package_QFP:LQFP-64_10x10mm_P0.5mm, symbol MCU_ST_STM32F4:STM32F401RETx
- added C? (x5): 100nF, symbol Device:C_Small
- added J? (x3): Conn_01x10, Connector_PinHeader_1.27mm:PinHeader_1x10_P1.27mm_Vertical, symbol Connector_Generic:Conn_01x10
- added Q? (x2): SSM3J338R,LF, SamacSys_Parts:SSM3J332RLFT, symbol SamacSys_Parts:SSM3J338R,LF
- added R? (x4): 10K, symbol Device:R
- added U? (x3): NTB0104BQ,115, NTB0104BQ115, symbol SamacSys_Parts:NTB0104BQ,115
- added U?: MIC5323-3.3YD5_TR, SOT95P280X100-5N, symbol SamacSys_Parts:MIC5323-3.3YD5_TR
- added U?: STM32F303RETx, Package_QFP:LQFP-64_10x10mm_P0.5mm, symbol MCU_ST_STM32F3:STM32F303RETx
Connections:
- net labels added: ENABLE_3V3_IO, ENABLE_5V_IO, EXT_IO0, EXT_IO1, EXT_IO2, EXT_IO3, EXT_IO4, EXT_IO5, EXT_IO6, IO_A_EN, IO_B_EN, VDD
- wire segments 296 -> 363
Other:
- note added: "Buffer IO_A"
- note added: "Buffer IO_B"
- note added: "Selección de tensión IO"

Commit message: Agregado jumper para pin BOOT0 y capacitores para los pines de comparadores
Parts:
- added C? (x3): 100nF, symbol Device:C_Small
- added J?: JUMPER, symbol Connector_Generic:Conn_01x03
Connections:
- wire segments 363 -> 372
Changed lines of the file:
@@
 F 3 "~" H 5800 5700 50  0001 C CNN
 	1    5800 5700
-	0    -1   -1   0
+	0    1    -1   0
 $EndComp
 Wire Wire Line
@@
 VBat_I_SENSE
 Wire Wire Line
-	8900 5150 8250 5150
-Wire Wire Line
 	6850 4050 6100 4050
 Wire Wire Line
@@
 L Device:R R?
 U 1 1 5BC0B03C
-P 10100 2850
-F 0 "R?" H 10170 2896 50  0000 L CNN
-F 1 "10K" H 10170 2804 50  0000 L CNN
-F 2 "" V 10030 2850 50  0001 C CNN
-F 3 "~" H 10100 2850 50  0001 C CNN
-	1    10100 2850
-	1    0    0    -1
-$EndComp
-Wire Wire Line
-	10100 3250 10100 3000
+P 10150 2850
+F 0 "R?" H 10220 2896 50  0000 L CNN
+F 1 "10K" H 10220 2804 50  0000 L CNN
+F 2 "" V 10080 2850 50  0001 C CNN
+F 3 "~" H 10150 2850 50  0001 C CNN
+	1    10150 2850
+	1    0    0    -1
+$EndComp
+Wire Wire Line
+	10150 3250 10150 3000
 $Comp
 L AXTEC_IC:+3V3_Internal #PWR?
 U 1 1 5BC1DDE1
-P 10300 2500
-F 0 "#PWR?" H 10300 2900 50  0001 C CNN
-F 1 "+3V3_Internal" H 10285 2673 50  0000 C CNN
-F 2 "" H 10300 2500 50  0001 C CNN
-F 3 "" H 10300 2500 50  0001 C CNN
-	1    10300 2500
+P 10150 2450
+F 0 "#PWR?" H 10150 2850 50  0001 C CNN
+F 1 "+3V3_Internal" H 10135 2623 50  0000 C CNN
+F 2 "" H 10150 2450 50  0001 C CNN
+F 3 "" H 10150 2450 50  0001 C CNN
+	1    10150 2450
 	1    0    0    -1
 $EndComp
@@
 $EndComp
 Wire Wire Line
-	10300 2550 10500 2550
+	10150 2550 10500 2550
 Wire Wire Line
 	10500 2550 10500 2700
 Wire Wire Line
-	10300 2550 10100 2550
-Wire Wire Line
-	10100 2550 10100 2700
-Connection ~ 10300 2550
-Wire Wire Line
-	10300 2500 10300 2550
+	10150 2550 10150 2700
+Connection ~ 10150 2550
+Wire Wire Line
+	10150 2450 10150 2550
 Wire Wire Line
 	10500 3000 10500 3350
@@
 F 3 "~" H 9850 2850 50  0001 C CNN
 	1    9850 2850
-	-1   0    0    -1
+	1    0    0    -1
 $EndComp
 Wire Wire Line
@@
 	9850 2700 9850 2550
 Wire Wire Line
-	9850 2550 10100 2550
-Connection ~ 10100 2550
+	9850 2550 10150 2550
 Wire Wire Line
 	6850 5350 6550 5350
@@
 	8250 3150 9850 3150
 Wire Wire Line
-	8250 3250 10100 3250
+	8250 3250 10150 3250
 Wire Wire Line
 	8250 3350 10500 3350
 Text Label 8350 2450 0    50   ~ 0
 3V_I_SENSE
-Wire Wire Line
-	8250 2450 8900 2450
-Wire Wire Line
-	8250 4050 8900 4050
 Text Label 8350 4050 0    50   ~ 0
 5V_I_SENSE
@@
 Wire Wire Line
 	15300 4800 14900 4800
+$Comp
+L Connector_Generic:Conn_01x03 J?
+U 1 1 5E51E963
+P 6150 2950
+F 0 "J?" V 6350 2950 50  0000 C CNN
+F 1 "JUMPER" V 6250 2950 50  0000 C CNN
+F 2 "" H 6150 2950 50  0001 C CNN
+F 3 "~" H 6150 2950 50  0001 C CNN
+	1    6150 2950
+	-1   0    0    1
+$EndComp
+Wire Wire Line
+	6350 2950 6700 2950
+Wire Wire Line
+	6700 2950 6700 2550
+Wire Wire Line
+	6700 2550 6850 2550
+$Comp
+L AXTEC_IC:+3V3_Internal #PWR?
+U 1 1 5E58E4CE
+P 6400 2750
+F 0 "#PWR?" H 6400 3150 50  0001 C CNN
+F 1 "+3V3_Internal" H 6385 2923 50  0000 C CNN
+F 2 "" H 6400 2750 50  0001 C CNN
+F 3 "" H 6400 2750 50  0001 C CNN
+	1    6400 2750
+	1    0    0    -1
+$EndComp
+Wire Wire Line
+	6400 2750 6400 2850
+Wire Wire Line
+	6400 2850 6350 2850
+$Comp
+L power:GND #PWR?
+U 1 1 5E5B466E
+P 6400 3100
+F 0 "#PWR?" H 6400 2850 50  0001 C CNN
+F 1 "GND" H 6405 2927 50  0000 C CNN
+F 2 "" H 6400 3100 50  0001 C CNN
+F 3 "" H 6400 3100 50  0001 C CNN
+	1    6400 3100
+	-1   0    0    -1
+$EndComp
+Wire Wire Line
+	6350 3050 6400 3050
+Wire Wire Line
+	6400 3050 6400 3100
+$Comp
+L Device:C_Small C?
+U 1 1 5E5DB995
+P 9100 5300
+AR Path="/5BB122CA/5E5DB995" Ref="C?"  Part="1"
+AR Path="/5BB12371/5E5DB995" Ref="C?"  Part="1"
+AR Path="/5BB123AC/5E5DB995" Ref="C?"  Part="1"
+AR Path="/5E5DB995" Ref="C?"  Part="1"
+F 0 "C?" H 9008 5254 50  0000 R CNN
+F 1 "100nF" H 9008 5345 50  0000 R CNN
+F 2 "" H 9100 5300 50  0001 C CNN
+F 3 "~" H 9100 5300 50  0001 C CNN
+	1    9100 5300
+	-1   0    0    1
+$EndComp
+Wire Wire Line
+	9100 5150 9100 5200
+Wire Wire Line
+	8250 5150 9100 5150
+$Comp
+L power:GND #PWR?
+U 1 1 5E629CB7
+P 9100 5400
+F 0 "#PWR?" H 9100 5150 50  0001 C CNN
+F 1 "GND" H 9104 5226 50  0000 C CNN
+F 2 "" H 9100 5400 50  0001 C CNN
+F 3 "" H 9100 5400 50  0001 C CNN
+	1    9100 5400
+	1    0    0    -1
+$EndComp
+$Comp
+L Device:C_Small C?
+U 1 1 5E629D24
+P 9100 4200
+AR Path="/5BB122CA/5E629D24" Ref="C?"  Part="1"
+AR Path="/5BB12371/5E629D24" Ref="C?"  Part="1"
+AR Path="/5BB123AC/5E629D24" Ref="C?"  Part="1"
+AR Path="/5E629D24" Ref="C?"  Part="1"
+F 0 "C?" H 9008 4154 50  0000 R CNN
+F 1 "100nF" H 9008 4245 50  0000 R CNN
+F 2 "" H 9100 4200 50  0001 C CNN
+F 3 "~" H 9100 4200 50  0001 C CNN
+	1    9100 4200
+	-1   0    0    1
+$EndComp
+Wire Wire Line
+	8250 4050 9100 4050
+Wire Wire Line
+	9100 4050 9100 4100
+$Comp
+L power:GND #PWR?
+U 1 1 5E677B4C
+P 9100 4300
+F 0 "#PWR?" H 9100 4050 50  0001 C CNN
+F 1 "GND" H 9104 4126 50  0000 C CNN
+F 2 "" H 9100 4300 50  0001 C CNN
+F 3 "" H 9100 4300 50  0001 C CNN
+	1    9100 4300
+	1    0    0    -1
+$EndComp
+$Comp
+L Device:C_Small C?
+U 1 1 5E677BBB
+P 9100 2600
+AR Path="/5BB122CA/5E677BBB" Ref="C?"  Part="1"
+AR Path="/5BB12371/5E677BBB" Ref="C?"  Part="1"
+AR Path="/5BB123AC/5E677BBB" Ref="C?"  Part="1"
+AR Path="/5E677BBB" Ref="C?"  Part="1"
+F 0 "C?" H 9008 2554 50  0000 R CNN
+F 1 "100nF" H 9008 2645 50  0000 R CNN
+F 2 "" H 9100 2600 50  0001 C CNN
+F 3 "~" H 9100 2600 50  0001 C CNN
+	1    9100 2600
+	-1   0    0    1
+$EndComp
+Wire Wire Line
+	9100 2450 9100 2500
+Wire Wire Line
+	8250 2450 9100 2450
+$Comp
+L power:GND #PWR?
+U 1 1 5E6ECD86
+P 9100 2700
+F 0 "#PWR?" H 9100 2450 50  0001 C CNN
+F 1 "GND" H 9104 2526 50  0000 C CNN
+F 2 "" H 9100 2700 50  0001 C CNN
+F 3 "" H 9100 2700 50  0001 C CNN
+	1    9100 2700
+	1    0    0    -1
+$EndComp
 $EndSCHEMATC
