File: Hardware/Satelite/PCB_B/PCB_B.sch (KiCad schematic (older format))
At the start: 51 parts

Commit message: Nuevos PCB_B y PCB_C
Parts:
- removed C? (x3): 1uF, symbol Device:C_Small
- removed C? (x17): 100nF, symbol Device:C_Small
- removed C? (x2): 4.3pF, symbol Device:C_Small
- removed C? (x2): 20pF, symbol Device:C_Small
- removed C?: 4.7uF, symbol Device:C_Small
- removed IC?: BQ24392RSER, RSE(R-PUQFN-N10), symbol SamacSys_Parts:BQ24392RSER
- removed IC?: MCP1501T-33E_CHY, SOT95P270X145-6N, symbol SamacSys_Parts:MCP1501T-33E_CHY
- removed J?: USB_B_Micro, symbol Connector:USB_B_Micro
- removed J?: Conn_01x06, symbol Connector_Generic:Conn_01x06
- removed J? (x4): Conn_01x10, Connector_PinHeader_1.27mm:PinHeader_1x10_P1.27mm_Vertical, symbol Connector_Generic:Conn_01x10
- removed J?: Conn_01x10, symbol Connector_Generic:Conn_01x10
- removed J?: JUMPER, symbol Connector_Generic:Conn_01x03
- removed Q? (x2): SSM3J338R,LF, SamacSys_Parts:SSM3J332RLFT, symbol SamacSys_Parts:SSM3J338R,LF
- removed R? (x6): 10K, symbol Device:R
- removed U? (x3): NTB0104BQ,115, NTB0104BQ115, symbol SamacSys_Parts:NTB0104BQ,115
- removed U?: TCA9802DGKR, SOP65P490X110-8N, symbol SamacSys_Parts:TCA9802DGKR
- removed U?: MIC5323-3.3YD5_TR, SOT95P280X100-5N, symbol SamacSys_Parts:MIC5323-3.3YD5_TR
- removed U?: STM32F303RETx, Package_QFP:LQFP-64_10x10mm_P0.5mm, symbol MCU_ST_STM32F3:STM32F303RETx
- removed Y?: LFXTAL016178, LFXTAL016178_1, symbol SamacSys_Parts:LFXTAL016178
- removed Y?: Crystal, symbol Device:Crystal
- added C? (x2): 2.2uF, symbol Device:C_Small
- added C?: 100nF, symbol Device:C_Small
- added J? (x5): Conn_01x10, Connector_PinHeader_1.27mm:PinHeader_1x10_P1.27mm_Vertical, symbol Connector_Generic:Conn_01x10
- added U?: MIC5323-3.3YD5_TR, SOT95P280X100-5N, symbol SamacSys_Parts:MIC5323-3.3YD5_TR
Connections:
- net labels added: BATT_INTERNO, I_SENSE_3V3, I_SENSE_5V, I_SENSE_BATT, V_SENSE_3V3, V_SENSE_5V
- net labels removed: +VREF, 3V_ENABLE, 3V_I_SENSE, 3V_V_SENSE, 5V_ENABLE, 5V_I_SENSE, 5V_V_SENSE, ACC_INT, CHG_ALLOWED, CHG_DETECT, D+, D-, ENABLE_3V3_IO, ENABLE_5V_IO, EXT_CS, EXT_IO0, EXT_IO1, EXT_IO2, EXT_IO3, EXT_IO4, EXT_IO5, EXT_IO6, EXT_SCLK, EXT_SDI, EXT_SDO, GYRO_INT, I2C_EN, IO0, IO1, IO2, IO3, IO4, IO5, IO6, IO_A_EN, IO_B_EN, MAG_INT, NRST, SCL_CHG, SCL_EXT, SDA_CHG, SDA_EXT, SPI_BUFFER_EN, SWCLK, SWDIO, SWO, SW_OPEN, VBat_I_SENSE, VDD
- wire segments 372 -> 103
Other:
- note added: "Administración de Batería"
- note added: "Conectores a PCB_A"
- note added: "Conectores a PCB_C"
- note added: "Regulador Interno"
- note added: "Reguladores"
- note removed: "+VREF ADC"
- note removed: "Alimentación externa e interna"
- note removed: "Buffer I2C"
- note removed: "Buffer IO_A"
- note removed: "Buffer IO_B"
- note removed: "Buffer SPI"
- note removed: "Conectores para PCB_A"
- note removed: "Conectores para PCB_B"
- note removed: "Header \nprogramación"
- note removed: "Selección de tensión IO"
- note removed: "Sensores"
- note removed: "USB y detección de cargador"

Commit message: Agregados agujeros de montajes
Parts:
- added H? (x3): MountingHole_Pad, symbol Mechanical:MountingHole_Pad
Changed lines of the file:
@@
 EESchema Schematic File Version 4
+LIBS:PCB_B-cache
 EELAYER 26 0
 EELAYER END
@@
 Wire Wire Line
 	10200 4150 10200 3750
+$Comp
+L Mechanical:MountingHole_Pad H?
+U 1 1 5C3A9049
+P 3600 2850
+F 0 "H?" H 3700 2901 50  0000 L CNN
+F 1 "MountingHole_Pad" H 3700 2809 50  0000 L CNN
+F 2 "" H 3600 2850 50  0001 C CNN
+F 3 "~" H 3600 2850 50  0001 C CNN
+	1    3600 2850
+	1    0    0    -1
+$EndComp
+$Comp
+L power:GND #PWR?
+U 1 1 5C3A916B
+P 3600 2950
+F 0 "#PWR?" H 3600 2700 50  0001 C CNN
+F 1 "GND" H 3604 2776 50  0000 C CNN
+F 2 "" H 3600 2950 50  0001 C CNN
+F 3 "" H 3600 2950 50  0001 C CNN
+	1    3600 2950
+	1    0    0    -1
+$EndComp
+$Comp
+L Mechanical:MountingHole_Pad H?
+U 1 1 5C3A91AE
+P 3600 3350
+F 0 "H?" H 3700 3401 50  0000 L CNN
+F 1 "MountingHole_Pad" H 3700 3309 50  0000 L CNN
+F 2 "" H 3600 3350 50  0001 C CNN
+F 3 "~" H 3600 3350 50  0001 C CNN
+	1    3600 3350
+	1    0    0    -1
+$EndComp
+$Comp
+L power:GND #PWR?
+U 1 1 5C3A91B5
+P 3600 3450
+F 0 "#PWR?" H 3600 3200 50  0001 C CNN
+F 1 "GND" H 3604 3276 50  0000 C CNN
+F 2 "" H 3600 3450 50  0001 C CNN
+F 3 "" H 3600 3450 50  0001 C CNN
+	1    3600 3450
+	1    0    0    -1
+$EndComp
+$Comp
+L Mechanical:MountingHole_Pad H?
+U 1 1 5C3AC283
+P 3600 3850
+F 0 "H?" H 3700 3901 50  0000 L CNN
+F 1 "MountingHole_Pad" H 3700 3809 50  0000 L CNN
+F 2 "" H 3600 3850 50  0001 C CNN
+F 3 "~" H 3600 3850 50  0001 C CNN
+	1    3600 3850
+	1    0    0    -1
+$EndComp
+$Comp
+L power:GND #PWR?
+U 1 1 5C3AC28A
+P 3600 3950
+F 0 "#PWR?" H 3600 3700 50  0001 C CNN
+F 1 "GND" H 3604 3776 50  0000 C CNN
+F 2 "" H 3600 3950 50  0001 C CNN
+F 3 "" H 3600 3950 50  0001 C CNN
+	1    3600 3950
+	1    0    0    -1
+$EndComp
 $EndSCHEMATC

Commit message: Nuevo conector interno para conexión entre PCB_C y PCB_B
Parts:
- removed J? (x5): Conn_01x10, Connector_PinHeader_1.27mm:PinHeader_1x10_P1.27mm_Vertical, symbol Connector_Generic:Conn_01x10
- added J?: Conector_PCB_A-B, symbol AXTEC_IC:Conector_PCB_A-B
- added J?: Conector_PCB_B-C, symbol AXTEC_IC:Conector_PCB_B-C
Connections:
- wire segments 103 -> 98

Commit message: Generación de 5V separados para alimentación de los servos
Parts:
- added C? (x2): 10uF, symbol Device:C_Small
- added IC?: MCP1642B-50I_MS, SOP65P490X110-8N, symbol SamacSys_Parts:MCP1642B-50I_MS
- added L?: 4.7uH, ~, symbol Device:L_Core_Iron
Connections:
- net labels added: SERVOS_5V
- wire segments 98 -> 121
Other:
- note added: "Regulador Interno 3V3"
- note added: "Regulador Servos 5V"
- note removed: "Regulador Interno"

Commit message: Agregado MH_CanSat a PCB_B
Parts:
- removed H? (x3): MountingHole_Pad, symbol Mechanical:MountingHole_Pad
- added MH?: MH_CanSat, symbol AXTEC_IC:MH_CanSat
Connections:
- wire segments 121 -> 127
Other:
- note added: "Agujeros de montaje\n"
Changed lines of the file:
@@
 Conectores a PCB_C
-$Comp
-L Mechanical:MountingHole_Pad H?
-U 1 1 5C3A9049
-P 3600 2850
-F 0 "H?" H 3700 2901 50  0000 L CNN
-F 1 "MountingHole_Pad" H 3700 2809 50  0000 L CNN
-F 2 "" H 3600 2850 50  0001 C CNN
-F 3 "~" H 3600 2850 50  0001 C CNN
-	1    3600 2850
-	1    0    0    -1
-$EndComp
-$Comp
-L power:GND #PWR?
-U 1 1 5C3A916B
-P 3600 2950
-F 0 "#PWR?" H 3600 2700 50  0001 C CNN
-F 1 "GND" H 3604 2776 50  0000 C CNN
-F 2 "" H 3600 2950 50  0001 C CNN
-F 3 "" H 3600 2950 50  0001 C CNN
-	1    3600 2950
-	1    0    0    -1
-$EndComp
-$Comp
-L Mechanical:MountingHole_Pad H?
-U 1 1 5C3A91AE
-P 3600 3350
-F 0 "H?" H 3700 3401 50  0000 L CNN
-F 1 "MountingHole_Pad" H 3700 3309 50  0000 L CNN
-F 2 "" H 3600 3350 50  0001 C CNN
-F 3 "~" H 3600 3350 50  0001 C CNN
-	1    3600 3350
-	1    0    0    -1
-$EndComp
-$Comp
-L power:GND #PWR?
-U 1 1 5C3A91B5
-P 3600 3450
-F 0 "#PWR?" H 3600 3200 50  0001 C CNN
-F 1 "GND" H 3604 3276 50  0000 C CNN
-F 2 "" H 3600 3450 50  0001 C CNN
-F 3 "" H 3600 3450 50  0001 C CNN
-	1    3600 3450
-	1    0    0    -1
-$EndComp
-$Comp
-L Mechanical:MountingHole_Pad H?
-U 1 1 5C3AC283
-P 3600 3850
-F 0 "H?" H 3700 3901 50  0000 L CNN
-F 1 "MountingHole_Pad" H 3700 3809 50  0000 L CNN
-F 2 "" H 3600 3850 50  0001 C CNN
-F 3 "~" H 3600 3850 50  0001 C CNN
-	1    3600 3850
-	1    0    0    -1
-$EndComp
-$Comp
-L power:GND #PWR?
-U 1 1 5C3AC28A
-P 3600 3950
-F 0 "#PWR?" H 3600 3700 50  0001 C CNN
-F 1 "GND" H 3604 3776 50  0000 C CNN
-F 2 "" H 3600 3950 50  0001 C CNN
-F 3 "" H 3600 3950 50  0001 C CNN
-	1    3600 3950
-	1    0    0    -1
-$EndComp
 $Comp
 L AXTEC_IC:Conector_PCB_A-B J?
@@
 Wire Wire Line
 	8400 1500 8950 1500
+$Comp
+L AXTEC_IC:MH_CanSat MH?
+U 1 1 5BC80D4F
+P 1550 1450
+F 0 "MH?" H 1828 1565 50  0000 L CNN
+F 1 "MH_CanSat" H 1828 1474 50  0000 L CNN
+F 2 "" H 1550 1450 50  0001 C CNN
+F 3 "" H 1550 1450 50  0001 C CNN
+	1    1550 1450
+	1    0    0    -1
+$EndComp
+$Comp
+L power:GND #PWR?
+U 1 1 5BC80DF0
+P 1550 1650
+AR Path="/5BB6C3A1/5BC80DF0" Ref="#PWR?"  Part="1"
+AR Path="/5BB6C83B/5BC80DF0" Ref="#PWR?"  Part="1"
+AR Path="/5BC14C3C/5BC80DF0" Ref="#PWR?"  Part="1"
+AR Path="/5BC80DF0" Ref="#PWR?"  Part="1"
+F 0 "#PWR?" H 1550 1400 50  0001 C CNN
+F 1 "GND" H 1555 1477 50  0000 C CNN
+F 2 "" H 1550 1650 50  0001 C CNN
+F 3 "" H 1550 1650 50  0001 C CNN
+	1    1550 1650
+	1    0    0    -1
+$EndComp
+Wire Wire Line
+	1400 1550 1400 1600
+Wire Wire Line
+	1400 1600 1550 1600
+Wire Wire Line
+	1700 1600 1700 1550
+Wire Wire Line
+	1550 1550 1550 1600
+Connection ~ 1550 1600
+Wire Wire Line
+	1550 1600 1700 1600
+Wire Wire Line
+	1550 1650 1550 1600
+Text Notes 700  800  0    118  ~ 0
+Agujeros de montaje\n
+Wire Notes Line
+	550  550  2700 550
+Wire Notes Line
+	2700 550  2700 2400
+Wire Notes Line
+	2700 2400 550  2400
+Wire Notes Line
+	550  2400 550  550
 $EndSCHEMATC

Commit message: Footprints para PCB_B
Parts:
- removed C?: 2.2uF, symbol Device:C_Small
- removed C?: 10uF, symbol Device:C_Small
- added C?: 2.2uF, Capacitor_SMD:C_0805_2012Metric_Pad1.15x1.40mm_HandSolder, symbol Device:C_Small
- added C?: 10uF, Capacitor_SMD:C_0805_2012Metric_Pad1.15x1.40mm_HandSolder, symbol Device:C_Small
- C?: footprint (none) -> Capacitor_SMD:C_0805_2012Metric_Pad1.15x1.40mm_HandSolder; Manufacturer Part Number (none) -> LMK212B7225KG-T
- C?: footprint (none) -> Capacitor_SMD:C_0603_1608Metric_Pad1.05x0.95mm_HandSolder; Manufacturer Part Number (none) -> EMK107B7104KAHT
- C?: footprint (none) -> Capacitor_SMD:C_0805_2012Metric_Pad1.15x1.40mm_HandSolder; Manufacturer Part Number (none) -> C2012X7R1A106M125AC
- J?: footprint (none) -> AXTEC:Conector_PCB_A-B
- L?: footprint ~ -> AXTEC:SRN3010TA-4R7M
Changed lines of the file:
@@
 F 0 "C?" H 8258 5954 50  0000 R CNN
 F 1 "2.2uF" H 8258 6045 50  0000 R CNN
-F 2 "" H 8350 6000 50  0001 C CNN
+F 2 "Capacitor_SMD:C_0805_2012Metric_Pad1.15x1.40mm_HandSolder" H 8350 6000 50  0001 C CNN
 F 3 "~" H 8350 6000 50  0001 C CNN
 F 4 "10V" H 8350 6000 50  0001 C CNN "Voltage"
+F 5 "LMK212B7225KG-T" H 8350 6000 50  0001 C CNN "Manufacturer Part Number"
 	1    8350 6000
 	-1   0    0    1
@@
 Wire Wire Line
 	9350 6000 9350 6200
-$Comp
-L Device:C_Small C?
-U 1 1 5BC1EB06
-P 10300 6050
-AR Path="/5BB122CA/5BC1EB06" Ref="C?"  Part="1"
-AR Path="/5BB12371/5BC1EB06" Ref="C?"  Part="1"
-AR Path="/5BB123AC/5BC1EB06" Ref="C?"  Part="1"
-AR Path="/5BB6C3A1/5BC1EB06" Ref="C?"  Part="1"
-AR Path="/5BB6C83B/5BC1EB06" Ref="C?"  Part="1"
-AR Path="/5BC14C3C/5BC1EB06" Ref="C?"  Part="1"
-AR Path="/5BC1EB06" Ref="C?"  Part="1"
-F 0 "C?" H 10208 6004 50  0000 R CNN
-F 1 "2.2uF" H 10208 6095 50  0000 R CNN
-F 2 "" H 10300 6050 50  0001 C CNN
-F 3 "~" H 10300 6050 50  0001 C CNN
-F 4 "10V" H 10300 6050 50  0001 C CNN "Voltage"
-	1    10300 6050
-	-1   0    0    1
-$EndComp
 Wire Wire Line
 	10300 5600 10300 5700
@@
 F 0 "C?" H 9758 6004 50  0000 R CNN
 F 1 "100nF" H 9758 6095 50  0000 R CNN
-F 2 "" H 9850 6050 50  0001 C CNN
+F 2 "Capacitor_SMD:C_0603_1608Metric_Pad1.05x0.95mm_HandSolder" H 9850 6050 50  0001 C CNN
 F 3 "~" H 9850 6050 50  0001 C CNN
 F 4 "10V" H 9850 6050 50  0001 C CNN "Voltage"
+F 5 "EMK107B7104KAHT" H 9850 6050 50  0001 C CNN "Manufacturer Part Number"
 	1    9850 6050
 	-1   0    0    1
@@
 F 0 "J?" H 9650 2067 50  0000 C CNN
 F 1 "Conector_PCB_A-B" H 9650 1975 50  0000 C CNN
-F 2 "" H 9250 1950 50  0001 C CNN
+F 2 "AXTEC:Conector_PCB_A-B" H 9250 1950 50  0001 C CNN
 F 3 "" H 9250 1950 50  0001 C CNN
 	1    9500 1500
@@
 F 0 "C?" H 6808 6054 50  0000 R CNN
 F 1 "10uF" H 6808 6145 50  0000 R CNN
-F 2 "" H 6900 6100 50  0001 C CNN
+F 2 "Capacitor_SMD:C_0805_2012Metric_Pad1.15x1.40mm_HandSolder" H 6900 6100 50  0001 C CNN
 F 3 "~" H 6900 6100 50  0001 C CNN
 F 4 "10V" H 6900 6100 50  0001 C CNN "Voltage"
+F 5 "C2012X7R1A106M125AC" H 6900 6100 50  0001 C CNN "Manufacturer Part Number"
 	1    6900 6100
 	-1   0    0    1
@@
 F 0 "L?" H 5109 5704 50  0000 R CNN
 F 1 "4.7uH" H 5109 5795 50  0000 R CNN
-F 2 "~" H 5150 5750 50  0001 C CNN
+F 2 "AXTEC:SRN3010TA-4R7M" H 5150 5750 50  0001 C CNN
 F 3 "~" H 5150 5750 50  0001 C CNN
 F 4 "SRN3010TA-4R7M" V 5150 5750 50  0001 C CNN "Manufacturer Part Number"
@@
 	1    0    0    -1
 $EndComp
-$Comp
-L Device:C_Small C?
-U 1 1 5C2EB009
-P 4750 5850
-AR Path="/5BB122CA/5C2EB009" Ref="C?"  Part="1"
-AR Path="/5BB12371/5C2EB009" Ref="C?"  Part="1"
-AR Path="/5BB123AC/5C2EB009" Ref="C?"  Part="1"
-AR Path="/5BB6C3A1/5C2EB009" Ref="C?"  Part="1"
-AR Path="/5BB6C83B/5C2EB009" Ref="C?"  Part="1"
-AR Path="/5BC14C3C/5C2EB009" Ref="C?"  Part="1"
-AR Path="/5C2EB009" Ref="C?"  Part="1"
-F 0 "C?" H 4658 5804 50  0000 R CNN
-F 1 "10uF" H 4658 5895 50  0000 R CNN
-F 2 "" H 4750 5850 50  0001 C CNN
-F 3 "~" H 4750 5850 50  0001 C CNN
-F 4 "10V" H 4750 5850 50  0001 C CNN "Voltage"
-	1    4750 5850
-	-1   0    0    1
-$EndComp
 Wire Wire Line
 	4750 5600 4750 5750
@@
 Wire Notes Line
 	550  2400 550  550
+$Comp
+L Device:C_Small C?
+U 1 1 5C68C1F1
+P 10300 6050
+AR Path="/5BB122CA/5C68C1F1" Ref="C?"  Part="1"
+AR Path="/5BB12371/5C68C1F1" Ref="C?"  Part="1"
+AR Path="/5BB123AC/5C68C1F1" Ref="C?"  Part="1"
+AR Path="/5BB6C3A1/5C68C1F1" Ref="C?"  Part="1"
+AR Path="/5BB6C83B/5C68C1F1" Ref="C?"  Part="1"
+AR Path="/5BC14C3C/5C68C1F1" Ref="C?"  Part="1"
+AR Path="/5C68C1F1" Ref="C?"  Part="1"
+F 0 "C?" H 10208 6004 50  0000 R CNN
+F 1 "2.2uF" H 10208 6095 50  0000 R CNN
+F 2 "Capacitor_SMD:C_0805_2012Metric_Pad1.15x1.40mm_HandSolder" H 10300 6050 50  0001 C CNN
+F 3 "~" H 10300 6050 50  0001 C CNN
+F 4 "10V" H 10300 6050 50  0001 C CNN "Voltage"
+F 5 "LMK212B7225KG-T" H 10300 6050 50  0001 C CNN "Manufacturer Part Number"
+	1    10300 6050
+	-1   0    0    1
+$EndComp
+$Comp
+L Device:C_Small C?
+U 1 1 5C68C592
+P 4750 5850
+AR Path="/5BB122CA/5C68C592" Ref="C?"  Part="1"
+AR Path="/5BB12371/5C68C592" Ref="C?"  Part="1"
+AR Path="/5BB123AC/5C68C592" Ref="C?"  Part="1"
+AR Path="/5BB6C3A1/5C68C592" Ref="C?"  Part="1"
+AR Path="/5BB6C83B/5C68C592" Ref="C?"  Part="1"
+AR Path="/5BC14C3C/5C68C592" Ref="C?"  Part="1"
+AR Path="/5C68C592" Ref="C?"  Part="1"
+F 0 "C?" H 4658 5804 50  0000 R CNN
+F 1 "10uF" H 4658 5895 50  0000 R CNN
+F 2 "Capacitor_SMD:C_0805_2012Metric_Pad1.15x1.40mm_HandSolder" H 4750 5850 50  0001 C CNN
+F 3 "~" H 4750 5850 50  0001 C CNN
+F 4 "10V" H 4750 5850 50  0001 C CNN "Voltage"
+F 5 "C2012X7R1A106M125AC" H 4750 5850 50  0001 C CNN "Manufacturer Part Number"
+	1    4750 5850
+	-1   0    0    1
+$EndComp
 $EndSCHEMATC

Commit message: Enumeración de esquema de PCB_B
Parts:
- MH1: renamed from MH?; footprint (none) -> AXTEC:MH_CanSat
- gave numbers to parts that had none: 10

Commit message: PCB inicial para PCB_B y footprint de conector entre los PCB B-C (WIP)
Parts:
- J1: footprint (none) -> AXTEC:Conector_PCB_B-C
Changed lines of the file:
@@
 F 0 "J1" H 9050 4167 50  0000 C CNN
 F 1 "Conector_PCB_B-C" H 9050 4075 50  0000 C CNN
-F 2 "" H 8950 4200 50  0001 C CNN
+F 2 "AXTEC:Conector_PCB_B-C" H 8950 4200 50  0001 C CNN
 F 3 "" H 8950 4200 50  0001 C CNN
 	1    9050 3450
