File: Hardware/Satelite/PCB_B/Power 3V3.sch (KiCad schematic (older format))
At the start: 0 parts

Commit message: Esquemas de fuentes de 5V y 3.3V del satélite
Parts:
- added C? (x2): 10uF, symbol Device:C_Small
- added C? (x2): 1uF, symbol Device:C_Small
- added C?: 100n, symbol Device:C_Small
- added L?: 1uH, Inductor_SMD:L_0805_2012Metric_Pad1.15x1.40mm_HandSolder, symbol Device:L_Core_Iron
- added R?: 120m, Resistor_SMD:R_1206_3216Metric_Pad1.42x1.75mm_HandSolder, symbol Device:R
- added R? (x2): 50R, Resistor_SMD:R_1206_3216Metric_Pad1.42x1.75mm_HandSolder, symbol Device:R
- added U?: ADP2108AUJ-3.3, Package_TO_SOT_SMD:TSOT-23-5, symbol Regulator_Switching:ADP2108AUJ-3.3
- added U?: INA194, Package_TO_SOT_SMD:SOT-23-5, symbol Amplifier_Current:INA194
Connections:
- net labels added: +3V3_Internal, 3V3, CTRL, GND, ISENSE, VBAT
- wire segments 0 -> 38

Commit message: Completado esquema PCB_B. Mejoras en esquemas de PCB_A.
Parts:
- added C?: 1uF, symbol Device:C_Small
- added C? (x2): 100n, symbol Device:C_Small
- added R?: 2k, Resistor_SMD:R_1206_3216Metric_Pad1.42x1.75mm_HandSolder, symbol Device:R
- added R?: 130k, Resistor_SMD:R_1206_3216Metric_Pad1.42x1.75mm_HandSolder, symbol Device:R
- added U?: MCP6001-OT, Package_TO_SOT_SMD:SOT-23-5, symbol Amplifier_Operational:MCP6001-OT
Connections:
- net labels added: VSENSE
- wire segments 38 -> 57
Other:
- note added: "fc = 808 Hz"
- moved on the sheet: U?

Commit message: Footprints para PCB_B
Parts:
- removed C? (x2): 10uF, symbol Device:C_Small
- removed C? (x2): 1uF, symbol Device:C_Small
- removed C? (x3): 100n, symbol Device:C_Small
- added C? (x2): 10uF, Capacitor_SMD:C_0805_2012Metric_Pad1.15x1.40mm_HandSolder, symbol Device:C_Small
- added C? (x3): 100nF, Capacitor_SMD:C_0603_1608Metric_Pad1.05x0.95mm_HandSolder, symbol Device:C_Small
- added C? (x2): 1uF, Capacitor_SMD:C_0603_1608Metric_Pad1.05x0.95mm_HandSolder, symbol Device:C_Small
- C?: footprint (none) -> Capacitor_SMD:C_0603_1608Metric_Pad1.05x0.95mm_HandSolder; Manufacturer Part Number (none) -> LMK107B7105MA-T
- R? (x2): value 50R -> 51R; footprint Resistor_SMD:R_1206_3216Metric_Pad1.42x1.75mm_HandSolder -> Resistor_SMD:R_0603_1608Metric_Pad1.05x0.95mm_HandSolder; Manufacturer Part Number KRL1632E-M-R120-F-T5 -> AC0603FR-0751RL
- R?: footprint Resistor_SMD:R_1206_3216Metric_Pad1.42x1.75mm_HandSolder -> Resistor_SMD:R_0603_1608Metric_Pad1.05x0.95mm_HandSolder; Manufacturer Part Number KRL1632E-M-R120-F-T5 -> RC0603FR-102KL
- R?: footprint Resistor_SMD:R_1206_3216Metric_Pad1.42x1.75mm_HandSolder -> Resistor_SMD:R_0603_1608Metric_Pad1.05x0.95mm_HandSolder; Manufacturer Part Number KRL1632E-M-R120-F-T5 -> RC0603FR-07150KL
Other:
- note added: "fc = 795 Hz"
- note removed: "fc = 808 Hz"

Commit message: Enumeración de esquema de PCB_B
Parts:
- gave numbers to parts that had none: 17

Commit message: PCB B WIP
Connections:
- wire segments 57 -> 58
Other:
- moved on the sheet: U3
