File: Hardware/Satelite/PCB_B/Power 3V3.sch (KiCad schematic (older format))
At the start: 17 parts, among them U2 ADP2108AUJ-3.3, U3 INA194, U4 MCP6001-OT

Commit message: Revert "PCB B WIP"
This reverts commit 7e9720afefe395d959b0157ab5be25ebb8bd8a98.
Connections:
- wire segments 58 -> 57
Other:
- moved on the sheet: U3

Commit message: Numeros de parte para PCB_B
Parts:
- R5: value 130k -> 150k
- U2: Manufacturer Part Number (none) -> ADP2108AUJZ-3.3-R7
- U3: Manufacturer Part Number (none) -> INA194AIDBVR
- U4: Manufacturer Part Number (none) -> MCP6001T-I/OT
Changed lines of the file:
@@
 F 2 "Package_TO_SOT_SMD:TSOT-23-5" H 4700 4150 50  0001 L CNN
 F 3 "http://www.analog.com/media/en/technical-documentation/data-sheets/ADP2108.pdf" H 4400 4050 50  0001 C CNN
+F 4 "ADP2108AUJZ-3.3-R7" H 4650 4400 50  0001 C CNN "Manufacturer Part Number"
 	1    4650 4400
 	1    0    0    -1
@@
 F 2 "Package_TO_SOT_SMD:SOT-23-5" H 5600 2500 50  0001 C CNN
 F 3 "http://www.ti.com/lit/ds/symlink/ina193.pdf" H 5600 2500 50  0001 C CNN
+F 4 "INA194AIDBVR" V 5600 2500 50  0001 C CNN "Manufacturer Part Number"
 	1    5600 2500
 	0    -1   -1   0
@@
 AR Path="/5BC14C3C/5C2719F0" Ref="R?"  Part="1"
 F 0 "R5" H 6630 4908 50  0000 R CNN
-F 1 "130k" H 6630 5000 50  0000 R CNN
+F 1 "150k" H 6630 5000 50  0000 R CNN
 F 2 "Resistor_SMD:R_0603_1608Metric_Pad1.05x0.95mm_HandSolder" V 6630 5000 50  0001 C CNN
 F 3 "~" H 6700 5000 50  0001 C CNN
@@
 F 2 "Package_TO_SOT_SMD:SOT-23-5" H 7900 4650 50  0001 L CNN
 F 3 "http://ww1.microchip.com/downloads/en/DeviceDoc/21733j.pdf" H 8000 5050 50  0001 C CNN
+F 4 "MCP6001T-I/OT" H 8000 4850 50  0001 C CNN "Manufacturer Part Number"
 	1    8000 4850
 	1    0    0    -1

Commit message: Cambios en el valor del divisor resistivo de la fuente de 3.3V y en el filtro anti-aliasing de tensión de la fuente de 5V
Parts:
- R4: value 2k -> 6k8; Manufacturer Part Number RC0603FR-102KL -> RC0603FR-076K8L
Other:
- note added: "fc = 234 Hz"
- note removed: "fc = 795 Hz"
Changed lines of the file:
@@
 AR Path="/5BC14C3C/5C270D6B" Ref="R?"  Part="1"
 F 0 "R4" H 6630 4408 50  0000 R CNN
-F 1 "2k" H 6630 4500 50  0000 R CNN
+F 1 "6k8" H 6630 4500 50  0000 R CNN
 F 2 "Resistor_SMD:R_0603_1608Metric_Pad1.05x0.95mm_HandSolder" V 6630 4500 50  0001 C CNN
 F 3 "~" H 6700 4500 50  0001 C CNN
 F 4 "1%" H 6630 4592 50  0000 R CNN "Tolerance"
-F 5 "RC0603FR-102KL" V 6700 4500 50  0001 C CNN "Manufacturer Part Number"
+F 5 "RC0603FR-076K8L" V 6700 4500 50  0001 C CNN "Manufacturer Part Number"
 	1    6700 4500
 	-1   0    0    1
@@
 	7050 5200 7050 5100
 Text Notes 6600 5550 0    50   ~ 0
-fc = 795 Hz
+fc = 234 Hz
 $Comp
 L Device:C_Small C?
