File: Hardware/Satelite/PCB_B/Power 5V.sch (KiCad schematic (older format))
At the start: 0 parts

Commit message: Esquemas de fuentes de 5V y 3.3V del satélite
Parts:
- added C? (x2): 10uF, symbol Device:C_Small
- added C? (x2): 1uF, symbol Device:C_Small
- added C?: 100n, symbol Device:C_Small
- added IC?: MCP1642B-50I_MS, SOP65P490X110-8N, symbol SamacSys_Parts:MCP1642B-50I_MS
- added L?: 4.7uH, ~, symbol Device:L_Core_Iron
- added R?: 200m, Resistor_SMD:R_1206_3216Metric_Pad1.42x1.75mm_HandSolder, symbol Device:R
- added R? (x2): 50R, Resistor_SMD:R_1206_3216Metric_Pad1.42x1.75mm_HandSolder, symbol Device:R
- added U?: INA194, Package_TO_SOT_SMD:SOT-23-5, symbol Amplifier_Current:INA194
Connections:
- net labels added: +3V3_Internal, 5V, CTRL, GND, ISENSE, VBAT
- wire segments 0 -> 45

Commit message: Completado esquema PCB_B. Mejoras en esquemas de PCB_A.
Parts:
- added C?: 1uF, symbol Device:C_Small
- added C?: 100n, symbol Device:C_Small
- added C?: 10n, symbol Device:C_Small
- added R?: 30k, Resistor_SMD:R_1206_3216Metric_Pad1.42x1.75mm_HandSolder, symbol Device:R
- added R?: 56k, Resistor_SMD:R_1206_3216Metric_Pad1.42x1.75mm_HandSolder, symbol Device:R
- added U?: MCP6001-OT, Package_TO_SOT_SMD:SOT-23-5, symbol Amplifier_Operational:MCP6001-OT
Connections:
- net labels added: VSENSE
- wire segments 45 -> 64
Other:
- note added: "fc = 815 Hz"
Changed lines of the file:
@@
 Text HLabel 2950 4100 0    50   Input ~ 0
 VBAT
-Text HLabel 7000 4400 2    50   Output ~ 0
+Text HLabel 7600 4400 2    50   Output ~ 0
 5V
 Wire Wire Line
@@
 Wire Wire Line
 	6500 4400 6750 4400
-Wire Wire Line
-	7000 4400 6750 4400
 Connection ~ 6750 4400
 $Comp
@@
 Wire Wire Line
 	3500 4100 4050 4100
+$Comp
+L Device:R R?
+U 1 1 5C27BA5D
+P 7250 4600
+AR Path="/5BB6C3A1/5C27BA5D" Ref="R?"  Part="1"
+AR Path="/5BB6C83B/5C27BA5D" Ref="R?"  Part="1"
+F 0 "R?" H 7180 4508 50  0000 R CNN
+F 1 "30k" H 7180 4600 50  0000 R CNN
+F 2 "Resistor_SMD:R_1206_3216Metric_Pad1.42x1.75mm_HandSolder" V 7180 4600 50  0001 C CNN
+F 3 "~" H 7250 4600 50  0001 C CNN
+F 4 "1%" H 7180 4692 50  0000 R CNN "Tolerance"
+F 5 "KRL1632E-M-R120-F-T5" V 7250 4600 50  0001 C CNN "Manufacturer Part Number"
+	1    7250 4600
+	-1   0    0    1
+$EndComp
+Wire Wire Line
+	7250 4450 7250 4400
+Wire Wire Line
+	7250 4400 7600 4400
+$Comp
+L Device:R R?
+U 1 1 5C27BA6A
+P 7250 5100
+AR Path="/5BB6C3A1/5C27BA6A" Ref="R?"  Part="1"
+AR Path="/5BB6C83B/5C27BA6A" Ref="R?"  Part="1"
+F 0 "R?" H 7180 5008 50  0000 R CNN
+F 1 "56k" H 7180 5100 50  0000 R CNN
+F 2 "Resistor_SMD:R_1206_3216Metric_Pad1.42x1.75mm_HandSolder" V 7180 5100 50  0001 C CNN
+F 3 "~" H 7250 5100 50  0001 C CNN
+F 4 "1%" H 7180 5192 50  0000 R CNN "Tolerance"
+F 5 "KRL1632E-M-R120-F-T5" V 7250 5100 50  0001 C CNN "Manufacturer Part Number"
+	1    7250 5100
+	-1   0    0    1
+$EndComp
+$Comp
+L power:GND #PWR?
+U 1 1 5C27BA72
+P 7250 5300
+AR Path="/5BB6C3A1/5C27BA72" Ref="#PWR?"  Part="1"
+AR Path="/5BB6C83B/5C27BA72" Ref="#PWR?"  Part="1"
+F 0 "#PWR?" H 7250 5050 50  0001 C CNN
+F 1 "GND" H 7255 5127 50  0000 C CNN
+F 2 "" H 7250 5300 50  0001 C CNN
+F 3 "" H 7250 5300 50  0001 C CNN
+	1    7250 5300
+	1    0    0    -1
+$EndComp
+Wire Wire Line
+	7250 5250 7250 5300
+Text HLabel 9300 4950 2    50   Output ~ 0
+VSENSE
+$Comp
+L Amplifier_Operational:MCP6001-OT U?
+U 1 1 5C27BA7C
+P 8500 4950
+AR Path="/5BB6C3A1/5C27BA7C" Ref="U?"  Part="1"
+AR Path="/5BB6C83B/5C27BA7C" Ref="U?"  Part="1"
+F 0 "U?" H 8550 4750 50  0000 L CNN
+F 1 "MCP6001-OT" H 8550 4650 50  0000 L CNN
+F 2 "Package_TO_SOT_SMD:SOT-23-5" H 8400 4750 50  0001 L CNN
+F 3 "http://ww1.microchip.com/downloads/en/DeviceDoc/21733j.pdf" H 8500 5150 50  0001 C CNN
+	1    8500 4950
+	1    0    0    -1
+$EndComp
+$Comp
+L AXTEC_IC:+3V3_Internal #PWR?
+U 1 1 5C27BA83
+P 8400 4150
+AR Path="/5BB6C3A1/5C27BA83" Ref="#PWR?"  Part="1"
+AR Path="/5BB6C83B/5C27BA83" Ref="#PWR?"  Part="1"
+F 0 "#PWR?" H 8400 4550 50  0001 C CNN
+F 1 "+3V3_Internal" H 8385 4323 50  0000 C CNN
+F 2 "" H 8400 4150 50  0001 C CNN
+F 3 "" H 8400 4150 50  0001 C CNN
+	1    8400 4150
+	1    0    0    -1
+$EndComp
+$Comp
+L Device:C_Small C?
+U 1 1 5C27BA8A
+P 8600 4350
+AR Path="/5BB122CA/5C27BA8A" Ref="C?"  Part="1"
+AR Path="/5BB12371/5C27BA8A" Ref="C?"  Part="1"
+AR Path="/5BB123AC/5C27BA8A" Ref="C?"  Part="1"
+AR Path="/5BB6C3A1/5C27BA8A" Ref="C?"  Part="1"
+AR Path="/5BB6C83B/5C27BA8A" Ref="C?"  Part="1"
+F 0 "C?" H 8508 4304 50  0000 R CNN
+F 1 "1uF" H 8508 4395 50  0000 R CNN
+F 2 "" H 8600 4350 50  0001 C CNN
+F 3 "~" H 8600 4350 50  0001 C CNN
+F 4 "10V" H 8600 4350 50  0001 C CNN "Voltage"
+	1    8600 4350
+	-1   0    0    1
+$EndComp
+$Comp
+L Device:C_Small C?
+U 1 1 5C27BA92
+P 8950 4350
+AR Path="/5BB122CA/5C27BA92" Ref="C?"  Part="1"
+AR Path="/5BB12371/5C27BA92" Ref="C?"  Part="1"
+AR Path="/5BB123AC/5C27BA92" Ref="C?"  Part="1"
+AR Path="/5BB6C3A1/5C27BA92" Ref="C?"  Part="1"
+AR Path="/5BB6C83B/5C27BA92" Ref="C?"  Part="1"
+F 0 "C?" H 8858 4304 50  0000 R CNN
+F 1 "100n" H 8858 4395 50  0000 R CNN
+F 2 "" H 8950 4350 50  0001 C CNN
+F 3 "~" H 8950 4350 50  0001 C CNN
+F 4 "10V" H 8950 4350 50  0001 C CNN "Voltage"
+	1    8950 4350
+	-1   0    0    1
+$EndComp
+Wire Wire Line
+	8200 5050 7850 5050
+Wire Wire Line
+	7850 5500 9150 5500
+Wire Wire Line
+	9150 5500 9150 4950
+Wire Wire Line
+	9150 4950 8800 4950
+$Comp
+L power:GND #PWR?
+U 1 1 5C27BA9E
+P 8400 5250
+AR Path="/5BB6C3A1/5C27BA9E" Ref="#PWR?"  Part="1"
+AR Path="/5BB6C83B/5C27BA9E" Ref="#PWR?"  Part="1"
+F 0 "#PWR?" H 8400 5000 50  0001 C CNN
+F 1 "GND" H 8405 5077 50  0000 C CNN
+F 2 "" H 8400 5250 50  0001 C CNN
+F 3 "" H 8400 5250 50  0001 C CNN
+	1    8400 5250
+	1    0    0    -1
+$EndComp
+Wire Wire Line
+	8400 4150 8400 4250
+Wire Wire Line
+	8950 4250 8600 4250
+Connection ~ 8400 4250
+Wire Wire Line
+	8400 4250 8400 4650
+Connection ~ 8600 4250
+Wire Wire Line
+	8600 4250 8400 4250
+$Comp
+L power:GND #PWR?
+U 1 1 5C27BAAA
+P 8600 4450
+AR Path="/5BB6C3A1/5C27BAAA" Ref="#PWR?"  Part="1"
+AR Path="/5BB6C83B/5C27BAAA" Ref="#PWR?"  Part="1"
+F 0 "#PWR?" H 8600 4200 50  0001 C CNN
+F 1 "GND" H 8605 4277 50  0000 C CNN
+F 2 "" H 8600 4450 50  0001 C CNN
+F 3 "" H 8600 4450 50  0001 C CNN
+	1    8600 4450
+	1    0    0    -1
+$EndComp
+$Comp
+L power:GND #PWR?
+U 1 1 5C27BAB0
+P 8950 4450
+AR Path="/5BB6C3A1/5C27BAB0" Ref="#PWR?"  Part="1"
+AR Path="/5BB6C83B/5C27BAB0" Ref="#PWR?"  Part="1"
+F 0 "#PWR?" H 8950 4200 50  0001 C CNN
+F 1 "GND" H 8955 4277 50  0000 C CNN
+F 2 "" H 8950 4450 50  0001 C CNN
+F 3 "" H 8950 4450 50  0001 C CNN
+	1    8950 4450
+	1    0    0    -1
+$EndComp
+Wire Wire Line
+	9300 4950 9150 4950
+Connection ~ 9150 4950
+Connection ~ 7250 4400
+Wire Wire Line
+	6750 4400 7250 4400
+Wire Wire Line
+	7250 4750 7250 4850
+Wire Wire Line
+	7850 5050 7850 5500
+Wire Wire Line
+	7250 4850 7550 4850
+Connection ~ 7250 4850
+Wire Wire Line
+	7250 4850 7250 4950
+$Comp
+L Device:C_Small C?
+U 1 1 5C2825F0
+P 7550 5100
+AR Path="/5BB122CA/5C2825F0" Ref="C?"  Part="1"
+AR Path="/5BB12371/5C2825F0" Ref="C?"  Part="1"
+AR Path="/5BB123AC/5C2825F0" Ref="C?"  Part="1"
+AR Path="/5BB6C3A1/5C2825F0" Ref="C?"  Part="1"
+AR Path="/5BB6C83B/5C2825F0" Ref="C?"  Part="1"
+F 0 "C?" H 7458 5054 50  0000 R CNN
+F 1 "10n" H 7458 5145 50  0000 R CNN
+F 2 "" H 7550 5100 50  0001 C CNN
+F 3 "~" H 7550 5100 50  0001 C CNN
+F 4 "10V" H 7550 5100 50  0001 C CNN "Voltage"
+	1    7550 5100
+	-1   0    0    1
+$EndComp
+Wire Wire Line
+	7550 5000 7550 4850
+Connection ~ 7550 4850
+Wire Wire Line
+	7550 4850 8200 4850
+$Comp
+L power:GND #PWR?
+U 1 1 5C283540
+P 7550 5300
+AR Path="/5BB6C3A1/5C283540" Ref="#PWR?"  Part="1"
+AR Path="/5BB6C83B/5C283540" Ref="#PWR?"  Part="1"
+F 0 "#PWR?" H 7550 5050 50  0001 C CNN
+F 1 "GND" H 7555 5127 50  0000 C CNN
+F 2 "" H 7550 5300 50  0001 C CNN
+F 3 "" H 7550 5300 50  0001 C CNN
+	1    7550 5300
+	1    0    0    -1
+$EndComp
+Wire Wire Line
+	7550 5300 7550 5200
+Text Notes 7150 5700 0    50   ~ 0
+fc = 815 Hz
 $EndSCHEMATC

Commit message: Nuevos PCB_B y PCB_C
Connections:
- wire segments 64 -> 63
Changed lines of the file:
@@
 EESchema Schematic File Version 4
-LIBS:PCB_B-cache
 EELAYER 26 0
 EELAYER END
 $Descr A4 11693 8268
 encoding utf-8
-Sheet 6 6
+Sheet 3 6
 Title ""
 Date ""
@@
 AR Path="/5BB6C3A1/5BBB58E1" Ref="C?"  Part="1"
 AR Path="/5BB6C83B/5BBB58E1" Ref="C?"  Part="1"
+AR Path="/5BC14C3C/5BBB58E1" Ref="C?"  Part="1"
 F 0 "C?" H 3008 4304 50  0000 R CNN
 F 1 "10uF" H 3008 4395 50  0000 R CNN
@@
 AR Path="/5BB6C3A1/5BBB58EA" Ref="#PWR?"  Part="1"
 AR Path="/5BB6C83B/5BBB58EA" Ref="#PWR?"  Part="1"
+AR Path="/5BC14C3C/5BBB58EA" Ref="#PWR?"  Part="1"
 F 0 "#PWR?" H 3100 4350 50  0001 C CNN
 F 1 "GND" H 3105 4427 50  0000 C CNN
@@
 AR Path="/5BB6C3A1/5BBB58F9" Ref="C?"  Part="1"
 AR Path="/5BB6C83B/5BBB58F9" Ref="C?"  Part="1"
+AR Path="/5BC14C3C/5BBB58F9" Ref="C?"  Part="1"
 F 0 "C?" H 6658 4554 50  0000 R CNN
 F 1 "10uF" H 6658 4645 50  0000 R CNN
@@
 AR Path="/5BB6C3A1/5BBB5901" Ref="L?"  Part="1"
 AR Path="/5BB6C83B/5BBB5901" Ref="L?"  Part="1"
+AR Path="/5BC14C3C/5BBB5901" Ref="L?"  Part="1"
 F 0 "L?" H 3459 4204 50  0000 R CNN
 F 1 "4.7uH" H 3459 4295 50  0000 R CNN
@@
 AR Path="/5BB6C3A1/5BBB590A" Ref="#PWR?"  Part="1"
 AR Path="/5BB6C83B/5BBB590A" Ref="#PWR?"  Part="1"
+AR Path="/5BC14C3C/5BBB590A" Ref="#PWR?"  Part="1"
 F 0 "#PWR?" H 6750 4650 50  0001 C CNN
 F 1 "GND" H 6755 4727 50  0000 C CNN
@@
 Text HLabel 5400 4100 2    50   Input ~ 0
 CTRL
-Wire Wire Line
-	6500 4600 6500 4400
 Connection ~ 6500 4400
 Wire Wire Line
@@
 AR Path="/5BB6C3A1/5BBB591E" Ref="U?"  Part="1"
 AR Path="/5BB6C83B/5BBB591E" Ref="U?"  Part="1"
+AR Path="/5BC14C3C/5BBB591E" Ref="U?"  Part="1"
 F 0 "U?" V 6296 2259 50  0000 R CNN
 F 1 "INA194" V 6205 2259 50  0000 R CNN
@@
 AR Path="/5BB6C3A1/5BBB5927" Ref="R?"  Part="1"
 AR Path="/5BB6C83B/5BBB5927" Ref="R?"  Part="1"
+AR Path="/5BC14C3C/5BBB5927" Ref="R?"  Part="1"
 F 0 "R?" V 5953 4400 50  0000 C CNN
 F 1 "200m" V 6044 4400 50  0000 C CNN
@@
 AR Path="/5BB6C3A1/5BBB5931" Ref="R?"  Part="1"
 AR Path="/5BB6C83B/5BBB5931" Ref="R?"  Part="1"
+AR Path="/5BC14C3C/5BBB5931" Ref="R?"  Part="1"
 F 0 "R?" H 5930 3709 50  0000 R CNN
 F 1 "50R" H 5930 3800 50  0000 R CNN
@@
 AR Path="/5BB6C3A1/5BBB593A" Ref="R?"  Part="1"
 AR Path="/5BB6C83B/5BBB593A" Ref="R?"  Part="1"
+AR Path="/5BC14C3C/5BBB593A" Ref="R?"  Part="1"
 F 0 "R?" H 6430 3709 50  0000 R CNN
 F 1 "50R" H 6430 3800 50  0000 R CNN
@@
 AR Path="/5BB6C3A1/5BBB5946" Ref="C?"  Part="1"
 AR Path="/5BB6C83B/5BBB5946" Ref="C?"  Part="1"
+AR Path="/5BC14C3C/5BBB5946" Ref="C?"  Part="1"
 F 0 "C?" H 6158 3254 50  0000 R CNN
 F 1 "1uF" H 6158 3345 50  0000 R CNN
@@
 AR Path="/5BB6C3A1/5BBB5959" Ref="#PWR?"  Part="1"
 AR Path="/5BB6C83B/5BBB5959" Ref="#PWR?"  Part="1"
+AR Path="/5BC14C3C/5BBB5959" Ref="#PWR?"  Part="1"
 F 0 "#PWR?" H 5100 3000 50  0001 C CNN
 F 1 "+3V3_Internal" H 5085 2773 50  0000 C CNN
@@
 AR Path="/5BB6C3A1/5BBB5960" Ref="C?"  Part="1"
 AR Path="/5BB6C83B/5BBB5960" Ref="C?"  Part="1"
+AR Path="/5BC14C3C/5BBB5960" Ref="C?"  Part="1"
 F 0 "C?" H 5508 2854 50  0000 R CNN
 F 1 "1uF" H 5508 2945 50  0000 R CNN
@@
 AR Path="/5BB6C3A1/5BBB5968" Ref="C?"  Part="1"
 AR Path="/5BB6C83B/5BBB5968" Ref="C?"  Part="1"
+AR Path="/5BC14C3C/5BBB5968" Ref="C?"  Part="1"
 F 0 "C?" H 5158 2854 50  0000 R CNN
 F 1 "100n" H 5158 2945 50  0000 R CNN
@@
 AR Path="/5BB6C3A1/5BBB5977" Ref="#PWR?"  Part="1"
 AR Path="/5BB6C83B/5BBB5977" Ref="#PWR?"  Part="1"
+AR Path="/5BC14C3C/5BBB5977" Ref="#PWR?"  Part="1"
 F 0 "#PWR?" H 5250 2750 50  0001 C CNN
 F 1 "GND" H 5255 2827 50  0000 C CNN
@@
 AR Path="/5BB6C3A1/5BBB597D" Ref="#PWR?"  Part="1"
 AR Path="/5BB6C83B/5BBB597D" Ref="#PWR?"  Part="1"
+AR Path="/5BC14C3C/5BBB597D" Ref="#PWR?"  Part="1"
 F 0 "#PWR?" H 5600 2750 50  0001 C CNN
 F 1 "GND" H 5605 2827 50  0000 C CNN
@@
 AR Path="/5BB6C3A1/5BBB5983" Ref="#PWR?"  Part="1"
 AR Path="/5BB6C83B/5BBB5983" Ref="#PWR?"  Part="1"
+AR Path="/5BC14C3C/5BBB5983" Ref="#PWR?"  Part="1"
 F 0 "#PWR?" H 6800 2700 50  0001 C CNN
 F 1 "GND" H 6805 2777 50  0000 C CNN
@@
 AR Path="/5BB6C3A1/5BBB7A9F" Ref="#PWR?"  Part="1"
 AR Path="/5BB6C83B/5BBB7A9F" Ref="#PWR?"  Part="1"
+AR Path="/5BC14C3C/5BBB7A9F" Ref="#PWR?"  Part="1"
 F 0 "#PWR?" H 3850 4000 50  0001 C CNN
 F 1 "GND" H 3855 4077 50  0000 C CNN
@@
 AR Path="/5BB6C3A1/5C27BA5D" Ref="R?"  Part="1"
 AR Path="/5BB6C83B/5C27BA5D" Ref="R?"  Part="1"
+AR Path="/5BC14C3C/5C27BA5D" Ref="R?"  Part="1"
 F 0 "R?" H 7180 4508 50  0000 R CNN
 F 1 "30k" H 7180 4600 50  0000 R CNN
@@
 AR Path="/5BB6C3A1/5C27BA6A" Ref="R?"  Part="1"
 AR Path="/5BB6C83B/5C27BA6A" Ref="R?"  Part="1"
+AR Path="/5BC14C3C/5C27BA6A" Ref="R?"  Part="1"
 F 0 "R?" H 7180 5008 50  0000 R CNN
 F 1 "56k" H 7180 5100 50  0000 R CNN
@@
 AR Path="/5BB6C3A1/5C27BA72" Ref="#PWR?"  Part="1"
 AR Path="/5BB6C83B/5C27BA72" Ref="#PWR?"  Part="1"
+AR Path="/5BC14C3C/5C27BA72" Ref="#PWR?"  Part="1"
 F 0 "#PWR?" H 7250 5050 50  0001 C CNN
 F 1 "GND" H 7255 5127 50  0000 C CNN
@@
 AR Path="/5BB6C3A1/5C27BA7C" Ref="U?"  Part="1"
 AR Path="/5BB6C83B/5C27BA7C" Ref="U?"  Part="1"
+AR Path="/5BC14C3C/5C27BA7C" Ref="U?"  Part="1"
 F 0 "U?" H 8550 4750 50  0000 L CNN
 F 1 "MCP6001-OT" H 8550 4650 50  0000 L CNN
@@
 AR Path="/5BB6C3A1/5C27BA83" Ref="#PWR?"  Part="1"
 AR Path="/5BB6C83B/5C27BA83" Ref="#PWR?"  Part="1"
+AR Path="/5BC14C3C/5C27BA83" Ref="#PWR?"  Part="1"
 F 0 "#PWR?" H 8400 4550 50  0001 C CNN
 F 1 "+3V3_Internal" H 8385 4323 50  0000 C CNN
@@
 AR Path="/5BB6C3A1/5C27BA8A" Ref="C?"  Part="1"
 AR Path="/5BB6C83B/5C27BA8A" Ref="C?"  Part="1"
+AR Path="/5BC14C3C/5C27BA8A" Ref="C?"  Part="1"
 F 0 "C?" H 8508 4304 50  0000 R CNN
 F 1 "1uF" H 8508 4395 50  0000 R CNN
@@
 AR Path="/5BB6C3A1/5C27BA92" Ref="C?"  Part="1"
 AR Path="/5BB6C83B/5C27BA92" Ref="C?"  Part="1"
+AR Path="/5BC14C3C/5C27BA92" Ref="C?"  Part="1"
 F 0 "C?" H 8858 4304 50  0000 R CNN
 F 1 "100n" H 8858 4395 50  0000 R CNN
@@
 AR Path="/5BB6C3A1/5C27BA9E" Ref="#PWR?"  Part="1"
 AR Path="/5BB6C83B/5C27BA9E" Ref="#PWR?"  Part="1"
+AR Path="/5BC14C3C/5C27BA9E" Ref="#PWR?"  Part="1"
 F 0 "#PWR?" H 8400 5000 50  0001 C CNN
 F 1 "GND" H 8405 5077 50  0000 C CNN
@@
 AR Path="/5BB6C3A1/5C27BAAA" Ref="#PWR?"  Part="1"
 AR Path="/5BB6C83B/5C27BAAA" Ref="#PWR?"  Part="1"
+AR Path="/5BC14C3C/5C27BAAA" Ref="#PWR?"  Part="1"
 F 0 "#PWR?" H 8600 4200 50  0001 C CNN
 F 1 "GND" H 8605 4277 50  0000 C CNN
@@
 AR Path="/5BB6C3A1/5C27BAB0" Ref="#PWR?"  Part="1"
 AR Path="/5BB6C83B/5C27BAB0" Ref="#PWR?"  Part="1"
+AR Path="/5BC14C3C/5C27BAB0" Ref="#PWR?"  Part="1"
 F 0 "#PWR?" H 8950 4200 50  0001 C CNN
 F 1 "GND" H 8955 4277 50  0000 C CNN
@@
 AR Path="/5BB6C3A1/5C2825F0" Ref="C?"  Part="1"
 AR Path="/5BB6C83B/5C2825F0" Ref="C?"  Part="1"
+AR Path="/5BC14C3C/5C2825F0" Ref="C?"  Part="1"
 F 0 "C?" H 7458 5054 50  0000 R CNN
 F 1 "10n" H 7458 5145 50  0000 R CNN
@@
 AR Path="/5BB6C3A1/5C283540" Ref="#PWR?"  Part="1"
 AR Path="/5BB6C83B/5C283540" Ref="#PWR?"  Part="1"
+AR Path="/5BC14C3C/5C283540" Ref="#PWR?"  Part="1"
 F 0 "#PWR?" H 7550 5050 50  0001 C CNN
 F 1 "GND" H 7555 5127 50  0000 C CNN

Commit message: Footprints para PCB_B
Parts:
- removed C? (x2): 10uF, symbol Device:C_Small
- removed C? (x3): 1uF, symbol Device:C_Small
- removed C? (x2): 100n, symbol Device:C_Small
- removed R? (x2): 50R, Resistor_SMD:R_1206_3216Metric_Pad1.42x1.75mm_HandSolder, symbol Device:R
- added C? (x3): 1uF, Capacitor_SMD:C_0603_1608Metric_Pad1.05x0.95mm_HandSolder, symbol Device:C_Small
- added C? (x2): 100nF, Capacitor_SMD:C_0603_1608Metric_Pad1.05x0.95mm_HandSolder, symbol Device:C_Small
- added C? (x2): 10uF, Capacitor_SMD:C_0805_2012Metric_Pad1.15x1.40mm_HandSolder, symbol Device:C_Small
- added R? (x2): 51R, Resistor_SMD:R_0603_1608Metric_Pad1.05x0.95mm_HandSolder, symbol Device:R
- C?: footprint (none) -> Capacitor_SMD:C_0603_1608Metric_Pad1.05x0.95mm_HandSolder; Manufacturer Part Number (none) -> 06033C103K4T2A
- L?: footprint ~ -> AXTEC:SRN3010TA-4R7M
- R?: value 30k -> 22k; footprint Resistor_SMD:R_1206_3216Metric_Pad1.42x1.75mm_HandSolder -> Resistor_SMD:R_0603_1608Metric_Pad1.05x0.95mm_HandSolder; Manufacturer Part Number KRL1632E-M-R120-F-T5 -> RC0603FR-1322KL
- R?: value 56k -> 39k; footprint Resistor_SMD:R_1206_3216Metric_Pad1.42x1.75mm_HandSolder -> Resistor_SMD:R_0603_1608Metric_Pad1.05x0.95mm_HandSolder; Manufacturer Part Number KRL1632E-M-R120-F-T5 -> RC0603FR-1339KL
Other:
- note added: "fc = 723 Hz"
- note removed: "fc = 815 Hz"

Commit message: Enumeración de esquema de PCB_B
Parts:
- gave numbers to parts that had none: 17

Commit message: PCB B WIP
Parts:
- IC2: footprint SOP65P490X110-8N -> SamacSys_Parts:SOP65P490X110-8N
Changed lines of the file:
@@
 F 0 "IC2" H 5700 4365 50  0000 C CNN
 F 1 "MCP1642B-50I_MS" H 5700 4274 50  0000 C CNN
-F 2 "SOP65P490X110-8N" H 6100 4200 50  0001 L CNN
+F 2 "SamacSys_Parts:SOP65P490X110-8N" H 6100 4200 50  0001 L CNN
 F 3 "http://ww1.microchip.com/downloads/en/DeviceDoc/20005253A.pdf" H 6100 4100 50  0001 L CNN
 F 4 "Switching Voltage Regulators Step-up DC/DC Reg 1 MHz, 1.6A, 5Vout" H 6100 4000 50  0001 L CNN "Description"

Commit message: Revert "PCB B WIP"
This reverts commit 7e9720afefe395d959b0157ab5be25ebb8bd8a98.
Parts:
- IC2: footprint SamacSys_Parts:SOP65P490X110-8N -> SOP65P490X110-8N
Changed lines of the file:
@@
 F 0 "IC2" H 5700 4365 50  0000 C CNN
 F 1 "MCP1642B-50I_MS" H 5700 4274 50  0000 C CNN
-F 2 "SamacSys_Parts:SOP65P490X110-8N" H 6100 4200 50  0001 L CNN
+F 2 "SOP65P490X110-8N" H 6100 4200 50  0001 L CNN
 F 3 "http://ww1.microchip.com/downloads/en/DeviceDoc/20005253A.pdf" H 6100 4100 50  0001 L CNN
 F 4 "Switching Voltage Regulators Step-up DC/DC Reg 1 MHz, 1.6A, 5Vout" H 6100 4000 50  0001 L CNN "Description"
