File: Hardware/Satelite/PCB_B/Power 5V.sch (KiCad schematic (older format))
At the start: 17 parts, among them IC2 MCP1642B-50I_MS, U5 INA194, U6 MCP6001-OT

Commit message: Numeros de parte para PCB_B
Parts:
- IC2: Manufacturer Part Number (none) -> MCP1642B-50I/MS; Manufacturer_Part_Number MCP1642B-50I/MS -> (none)
- U5: Manufacturer Part Number (none) -> INA194AIDBVR
- U6: Manufacturer Part Number (none) -> MCP6001T-I/OT
Changed lines of the file:
@@
 F 2 "Package_TO_SOT_SMD:SOT-23-5" H 6250 2600 50  0001 C CNN
 F 3 "http://www.ti.com/lit/ds/symlink/ina193.pdf" H 6250 2600 50  0001 C CNN
+F 4 "INA194AIDBVR" V 6250 2600 50  0001 C CNN "Manufacturer Part Number"
 	1    6250 2600
 	0    -1   -1   0
@@
 F 5 "1.1" H 6100 3900 50  0001 L CNN "Height"
 F 6 "Microchip" H 6100 3800 50  0001 L CNN "Manufacturer_Name"
-F 7 "MCP1642B-50I/MS" H 6100 3700 50  0001 L CNN "Manufacturer_Part_Number"
-F 8 "" H 6100 3600 50  0001 L CNN "RS Part Number"
-F 9 "" H 6100 3500 50  0001 L CNN "RS Price/Stock"
-F 10 "70567327" H 6100 3400 50  0001 L CNN "Allied_Number"
-F 11 "https://www.alliedelec.com/microchip-technology-inc-mcp1642b-50i-ms/70567327/" H 6100 3300 50  0001 L CNN "Allied Price/Stock"
-F 12 "MCP1642B-50I/MS" H 6100 3200 50  0001 L CNN "Arrow Part Number"
-F 13 "https://www.arrow.com/en/products/mcp1642b-50ims/microchip-technology" H 6100 3100 50  0001 L CNN "Arrow Price/Stock"
+F 7 "MCP1642B-50I/MS" H 6100 3700 50  0001 L CNN "Manufacturer Part Number"
+F 8 "70567327" H 6100 3400 50  0001 L CNN "Allied_Number"
+F 9 "https://www.alliedelec.com/microchip-technology-inc-mcp1642b-50i-ms/70567327/" H 6100 3300 50  0001 L CNN "Allied Price/Stock"
+F 10 "MCP1642B-50I/MS" H 6100 3200 50  0001 L CNN "Arrow Part Number"
+F 11 "https://www.arrow.com/en/products/mcp1642b-50ims/microchip-technology" H 6100 3100 50  0001 L CNN "Arrow Price/Stock"
 	1    5150 4100
 	-1   0    0    -1
@@
 F 2 "Package_TO_SOT_SMD:SOT-23-5" H 8400 4750 50  0001 L CNN
 F 3 "http://ww1.microchip.com/downloads/en/DeviceDoc/21733j.pdf" H 8500 5150 50  0001 C CNN
+F 4 "MCP6001T-I/OT" H 8500 4950 50  0001 C CNN "Manufacturer Part Number"
 	1    8500 4950
 	1    0    0    -1

Commit message: Cambios en el valor del divisor resistivo de la fuente de 3.3V y en el filtro anti-aliasing de tensión de la fuente de 5V
Parts:
- C19: value 10n -> 100n; Manufacturer Part Number 06033C103K4T2A -> EMK107B7104KAHT
Other:
- note added: "fc = 113 Hz"
- note removed: "fc = 723 Hz"
Changed lines of the file:
@@
 AR Path="/5BC14C3C/5C2825F0" Ref="C19"  Part="1"
 F 0 "C19" H 7458 5054 50  0000 R CNN
-F 1 "10n" H 7458 5145 50  0000 R CNN
+F 1 "100n" H 7458 5145 50  0000 R CNN
 F 2 "Capacitor_SMD:C_0603_1608Metric_Pad1.05x0.95mm_HandSolder" H 7550 5100 50  0001 C CNN
 F 3 "~" H 7550 5100 50  0001 C CNN
 F 4 "10V" H 7550 5100 50  0001 C CNN "Voltage"
-F 5 "06033C103K4T2A" H 7550 5100 50  0001 C CNN "Manufacturer Part Number"
+F 5 "EMK107B7104KAHT" H 7550 5100 50  0001 C CNN "Manufacturer Part Number"
 	1    7550 5100
 	-1   0    0    1
@@
 	7550 5300 7550 5200
 Text Notes 7150 5700 0    50   ~ 0
-fc = 723 Hz
+fc = 113 Hz
 $Comp
 L Device:C_Small C?
