File: Hardware/Satelite/PCB_B/Cargador de batería.sch (KiCad schematic (older format))
At the start: 6 parts, among them U2 BQ24091DGQT

Commit message: Nuevos PCB_B y PCB_C
Parts:
- renumbered C1 to C?, C2 to C?, R4 to R?, R5 to R?, R6 to R?, U2 to U?
Connections:
- net labels added: VBAT, VIN
- net labels removed: VBUS, VBat+
Changed lines of the file:
@@
 EESchema Schematic File Version 4
-LIBS:PCB_A-cache
 EELAYER 26 0
 EELAYER END
 $Descr A4 11693 8268
 encoding utf-8
-Sheet 2 6
+Sheet 6 6
 Title ""
 Date ""
@@
 $EndDescr
 $Comp
-L SamacSys_Parts:BQ24091DGQT U2
+L SamacSys_Parts:BQ24091DGQT U?
 U 1 1 5BAD7302
 P 5250 3550
-F 0 "U2" H 5900 3815 50  0000 C CNN
+F 0 "U?" H 5900 3815 50  0000 C CNN
 F 1 "BQ24091DGQT" H 5900 3724 50  0000 C CNN
 F 2 "SamacSys_Parts:SOP50P490X110-11N" H 6400 3650 50  0001 L CNN
@@
 $EndComp
 Text HLabel 3550 3550 0    50   Input ~ 0
-VBUS
+VIN
 Text HLabel 7250 3950 2    50   Input ~ 0
 ISET
-Text HLabel 7250 3650 2    50   Output ~ 0
-VBat+
+Text HLabel 7250 3650 2    50   BiDi ~ 0
+VBAT
 $Comp
 L Device:C_Small C?
@@
 AR Path="/5BA17F9C/5BAD793D" Ref="C?"  Part="1"
 AR Path="/5BA1A7F9/5BAD793D" Ref="C?"  Part="1"
-AR Path="/5BA1A77A/5BAD793D" Ref="C1"  Part="1"
-F 0 "C1" H 4050 4050 50  0000 L CNN
+AR Path="/5BA1A77A/5BAD793D" Ref="C?"  Part="1"
+AR Path="/5BC300BF/5BAD793D" Ref="C?"  Part="1"
+F 0 "C?" H 4050 4050 50  0000 L CNN
 F 1 "1uF" H 4000 3950 50  0000 L CNN
 F 2 "" H 3900 4050 50  0001 C CNN
@@
 P 3900 4300
 AR Path="/5BA1A7F9/5BAD7944" Ref="#PWR?"  Part="1"
-AR Path="/5BA1A77A/5BAD7944" Ref="#PWR015"  Part="1"
-F 0 "#PWR015" H 3900 4050 50  0001 C CNN
+AR Path="/5BA1A77A/5BAD7944" Ref="#PWR?"  Part="1"
+AR Path="/5BC300BF/5BAD7944" Ref="#PWR?"  Part="1"
+F 0 "#PWR?" H 3900 4050 50  0001 C CNN
 F 1 "GND" H 3905 4127 50  0000 C CNN
 F 2 "" H 3900 4300 50  0001 C CNN
@@
 AR Path="/5BA17F9C/5BAD7C51" Ref="R?"  Part="1"
 AR Path="/5BA1A7F9/5BAD7C51" Ref="R?"  Part="1"
-AR Path="/5BA1A77A/5BAD7C51" Ref="R4"  Part="1"
-F 0 "R4" V 4450 4100 50  0000 L CNN
+AR Path="/5BA1A77A/5BAD7C51" Ref="R?"  Part="1"
+AR Path="/5BC300BF/5BAD7C51" Ref="R?"  Part="1"
+F 0 "R?" V 4450 4100 50  0000 L CNN
 F 1 "1k8" V 4250 4100 50  0000 L CNN
 F 2 "" V 4280 4100 50  0001 C CNN
@@
 P 4350 4300
 AR Path="/5BA1A7F9/5BAD7E3B" Ref="#PWR?"  Part="1"
-AR Path="/5BA1A77A/5BAD7E3B" Ref="#PWR016"  Part="1"
-F 0 "#PWR016" H 4350 4050 50  0001 C CNN
+AR Path="/5BA1A77A/5BAD7E3B" Ref="#PWR?"  Part="1"
+AR Path="/5BC300BF/5BAD7E3B" Ref="#PWR?"  Part="1"
+F 0 "#PWR?" H 4350 4050 50  0001 C CNN
 F 1 "GND" H 4355 4127 50  0000 C CNN
 F 2 "" H 4350 4300 50  0001 C CNN
@@
 P 4600 4300
 AR Path="/5BA1A7F9/5BAD7F3D" Ref="#PWR?"  Part="1"
-AR Path="/5BA1A77A/5BAD7F3D" Ref="#PWR017"  Part="1"
-F 0 "#PWR017" H 4600 4050 50  0001 C CNN
+AR Path="/5BA1A77A/5BAD7F3D" Ref="#PWR?"  Part="1"
+AR Path="/5BC300BF/5BAD7F3D" Ref="#PWR?"  Part="1"
+F 0 "#PWR?" H 4600 4050 50  0001 C CNN
 F 1 "GND" H 4605 4127 50  0000 C CNN
 F 2 "" H 4600 4300 50  0001 C CNN
@@
 AR Path="/5BA17F9C/5BAD7FE1" Ref="R?"  Part="1"
 AR Path="/5BA1A7F9/5BAD7FE1" Ref="R?"  Part="1"
-AR Path="/5BA1A77A/5BAD7FE1" Ref="R5"  Part="1"
-F 0 "R5" V 4900 4100 50  0000 L CNN
+AR Path="/5BA1A77A/5BAD7FE1" Ref="R?"  Part="1"
+AR Path="/5BC300BF/5BAD7FE1" Ref="R?"  Part="1"
+F 0 "R?" V 4900 4100 50  0000 L CNN
 F 1 "2k" V 4700 4100 50  0000 L CNN
 F 2 "" V 4730 4100 50  0001 C CNN
@@
 P 4800 4300
 AR Path="/5BA1A7F9/5BAD80E4" Ref="#PWR?"  Part="1"
-AR Path="/5BA1A77A/5BAD80E4" Ref="#PWR018"  Part="1"
-F 0 "#PWR018" H 4800 4050 50  0001 C CNN
+AR Path="/5BA1A77A/5BAD80E4" Ref="#PWR?"  Part="1"
+AR Path="/5BC300BF/5BAD80E4" Ref="#PWR?"  Part="1"
+F 0 "#PWR?" H 4800 4050 50  0001 C CNN
 F 1 "GND" H 4805 4127 50  0000 C CNN
 F 2 "" H 4800 4300 50  0001 C CNN
@@
 AR Path="/5BA17F9C/5BAD840C" Ref="R?"  Part="1"
 AR Path="/5BA1A7F9/5BAD840C" Ref="R?"  Part="1"
-AR Path="/5BA1A77A/5BAD840C" Ref="R6"  Part="1"
-F 0 "R6" V 7900 4100 50  0000 L CNN
+AR Path="/5BA1A77A/5BAD840C" Ref="R?"  Part="1"
+AR Path="/5BC300BF/5BAD840C" Ref="R?"  Part="1"
+F 0 "R?" V 7900 4100 50  0000 L CNN
 F 1 "100k" V 7700 4100 50  0000 L CNN
 F 2 "" V 7730 4100 50  0001 C CNN
@@
 P 7800 4300
 AR Path="/5BA1A7F9/5BAD8415" Ref="#PWR?"  Part="1"
-AR Path="/5BA1A77A/5BAD8415" Ref="#PWR021"  Part="1"
-F 0 "#PWR021" H 7800 4050 50  0001 C CNN
+AR Path="/5BA1A77A/5BAD8415" Ref="#PWR?"  Part="1"
+AR Path="/5BC300BF/5BAD8415" Ref="#PWR?"  Part="1"
+F 0 "#PWR?" H 7800 4050 50  0001 C CNN
 F 1 "GND" H 7805 4127 50  0000 C CNN
 F 2 "" H 7800 4300 50  0001 C CNN
@@
 P 6800 4300
 AR Path="/5BA1A7F9/5BAD886E" Ref="#PWR?"  Part="1"
-AR Path="/5BA1A77A/5BAD886E" Ref="#PWR019"  Part="1"
-F 0 "#PWR019" H 6800 4050 50  0001 C CNN
+AR Path="/5BA1A77A/5BAD886E" Ref="#PWR?"  Part="1"
+AR Path="/5BC300BF/5BAD886E" Ref="#PWR?"  Part="1"
+F 0 "#PWR?" H 6800 4050 50  0001 C CNN
 F 1 "GND" H 6805 4127 50  0000 C CNN
 F 2 "" H 6800 4300 50  0001 C CNN
@@
 AR Path="/5BA17F9C/5BAF1DFA" Ref="C?"  Part="1"
 AR Path="/5BA1A7F9/5BAF1DFA" Ref="C?"  Part="1"
-AR Path="/5BA1A77A/5BAF1DFA" Ref="C2"  Part="1"
-F 0 "C2" H 7150 4150 50  0000 L CNN
+AR Path="/5BA1A77A/5BAF1DFA" Ref="C?"  Part="1"
+AR Path="/5BC300BF/5BAF1DFA" Ref="C?"  Part="1"
+F 0 "C?" H 7150 4150 50  0000 L CNN
 F 1 "1uF" H 7100 4050 50  0000 L CNN
 F 2 "" H 7000 4150 50  0001 C CNN
@@
 P 7000 4300
 AR Path="/5BA1A7F9/5BAF219B" Ref="#PWR?"  Part="1"
-AR Path="/5BA1A77A/5BAF219B" Ref="#PWR020"  Part="1"
-F 0 "#PWR020" H 7000 4050 50  0001 C CNN
+AR Path="/5BA1A77A/5BAF219B" Ref="#PWR?"  Part="1"
+AR Path="/5BC300BF/5BAF219B" Ref="#PWR?"  Part="1"
+F 0 "#PWR?" H 7000 4050 50  0001 C CNN
 F 1 "GND" H 7005 4127 50  0000 C CNN
 F 2 "" H 7000 4300 50  0001 C CNN

Commit message: Footprints para PCB_B
Parts:
- removed C? (x2): 1uF, symbol Device:C_Small
- removed R?: 1k8, symbol Device:R
- removed R?: 2k, symbol Device:R
- added C? (x2): 1uF, Capacitor_SMD:C_0603_1608Metric_Pad1.05x0.95mm_HandSolder, symbol Device:C_Small
- added R?: 2k, Resistor_SMD:R_0603_1608Metric_Pad1.05x0.95mm_HandSolder, symbol Device:R
- added R?: 1k8, Resistor_SMD:R_0603_1608Metric_Pad1.05x0.95mm_HandSolder, symbol Device:R
- R?: footprint (none) -> Resistor_SMD:R_0603_1608Metric_Pad1.05x0.95mm_HandSolder
Changed lines of the file:
@@
 VBAT
-$Comp
-L Device:C_Small C?
-U 1 1 5BAD793D
-P 3900 4050
-AR Path="/5BA17F9C/5BAD793D" Ref="C?"  Part="1"
-AR Path="/5BA1A7F9/5BAD793D" Ref="C?"  Part="1"
-AR Path="/5BA1A77A/5BAD793D" Ref="C?"  Part="1"
-AR Path="/5BC300BF/5BAD793D" Ref="C?"  Part="1"
-F 0 "C?" H 4050 4050 50  0000 L CNN
-F 1 "1uF" H 4000 3950 50  0000 L CNN
-F 2 "" H 3900 4050 50  0001 C CNN
-F 3 "~" H 3900 4050 50  0001 C CNN
-	1    3900 4050
-	1    0    0    -1
-$EndComp
 $Comp
 L power:GND #PWR?
@@
 Wire Wire Line
 	7250 3950 6550 3950
-$Comp
-L Device:R R?
-U 1 1 5BAD7C51
-P 4350 4100
-AR Path="/5BA17F9C/5BAD7C51" Ref="R?"  Part="1"
-AR Path="/5BA1A7F9/5BAD7C51" Ref="R?"  Part="1"
-AR Path="/5BA1A77A/5BAD7C51" Ref="R?"  Part="1"
-AR Path="/5BC300BF/5BAD7C51" Ref="R?"  Part="1"
-F 0 "R?" V 4450 4100 50  0000 L CNN
-F 1 "1k8" V 4250 4100 50  0000 L CNN
-F 2 "" V 4280 4100 50  0001 C CNN
-F 3 "~" H 4350 4100 50  0001 C CNN
-	1    4350 4100
-	-1   0    0    1
-$EndComp
 Wire Wire Line
 	3900 3550 5250 3550
@@
 Text Notes 5350 4300 0    50   ~ 0
 Corriente de carga a 300mA
-$Comp
-L Device:R R?
-U 1 1 5BAD7FE1
-P 4800 4100
-AR Path="/5BA17F9C/5BAD7FE1" Ref="R?"  Part="1"
-AR Path="/5BA1A7F9/5BAD7FE1" Ref="R?"  Part="1"
-AR Path="/5BA1A77A/5BAD7FE1" Ref="R?"  Part="1"
-AR Path="/5BC300BF/5BAD7FE1" Ref="R?"  Part="1"
-F 0 "R?" V 4900 4100 50  0000 L CNN
-F 1 "2k" V 4700 4100 50  0000 L CNN
-F 2 "" V 4730 4100 50  0001 C CNN
-F 3 "~" H 4800 4100 50  0001 C CNN
-	1    4800 4100
-	-1   0    0    1
-$EndComp
 Wire Wire Line
 	4800 4300 4800 4250
@@
 F 0 "R?" V 7900 4100 50  0000 L CNN
 F 1 "100k" V 7700 4100 50  0000 L CNN
-F 2 "" V 7730 4100 50  0001 C CNN
+F 2 "Resistor_SMD:R_0603_1608Metric_Pad1.05x0.95mm_HandSolder" V 7730 4100 50  0001 C CNN
 F 3 "~" H 7800 4100 50  0001 C CNN
 	1    7800 4100
@@
 Wire Wire Line
 	6800 3550 6800 4300
-$Comp
-L Device:C_Small C?
-U 1 1 5BAF1DFA
-P 7000 4150
-AR Path="/5BA17F9C/5BAF1DFA" Ref="C?"  Part="1"
-AR Path="/5BA1A7F9/5BAF1DFA" Ref="C?"  Part="1"
-AR Path="/5BA1A77A/5BAF1DFA" Ref="C?"  Part="1"
-AR Path="/5BC300BF/5BAF1DFA" Ref="C?"  Part="1"
-F 0 "C?" H 7150 4150 50  0000 L CNN
-F 1 "1uF" H 7100 4050 50  0000 L CNN
-F 2 "" H 7000 4150 50  0001 C CNN
-F 3 "~" H 7000 4150 50  0001 C CNN
-	1    7000 4150
-	1    0    0    -1
-$EndComp
 Wire Wire Line
 	7000 3650 7000 4050
@@
 Wire Wire Line
 	7000 4250 7000 4300
+$Comp
+L Device:C_Small C?
+U 1 1 5C6A0401
+P 3900 4050
+AR Path="/5BB122CA/5C6A0401" Ref="C?"  Part="1"
+AR Path="/5BB12371/5C6A0401" Ref="C?"  Part="1"
+AR Path="/5BB123AC/5C6A0401" Ref="C?"  Part="1"
+AR Path="/5BB6C3A1/5C6A0401" Ref="C?"  Part="1"
+AR Path="/5BC13C37/5C6A0401" Ref="C?"  Part="1"
+AR Path="/5BC14C3C/5C6A0401" Ref="C?"  Part="1"
+AR Path="/5BC300BF/5C6A0401" Ref="C?"  Part="1"
+F 0 "C?" H 3808 4004 50  0000 R CNN
+F 1 "1uF" H 3808 4095 50  0000 R CNN
+F 2 "Capacitor_SMD:C_0603_1608Metric_Pad1.05x0.95mm_HandSolder" H 3900 4050 50  0001 C CNN
+F 3 "~" H 3900 4050 50  0001 C CNN
+F 4 "10V" H 3900 4050 50  0001 C CNN "Voltage"
+F 5 "LMK107B7105MA-T" H 3900 4050 50  0001 C CNN "Manufacturer Part Number"
+	1    3900 4050
+	-1   0    0    1
+$EndComp
+$Comp
+L Device:C_Small C?
+U 1 1 5C6A063E
+P 7000 4150
+AR Path="/5BB122CA/5C6A063E" Ref="C?"  Part="1"
+AR Path="/5BB12371/5C6A063E" Ref="C?"  Part="1"
+AR Path="/5BB123AC/5C6A063E" Ref="C?"  Part="1"
+AR Path="/5BB6C3A1/5C6A063E" Ref="C?"  Part="1"
+AR Path="/5BC13C37/5C6A063E" Ref="C?"  Part="1"
+AR Path="/5BC14C3C/5C6A063E" Ref="C?"  Part="1"
+AR Path="/5BC300BF/5C6A063E" Ref="C?"  Part="1"
+F 0 "C?" H 6908 4104 50  0000 R CNN
+F 1 "1uF" H 6908 4195 50  0000 R CNN
+F 2 "Capacitor_SMD:C_0603_1608Metric_Pad1.05x0.95mm_HandSolder" H 7000 4150 50  0001 C CNN
+F 3 "~" H 7000 4150 50  0001 C CNN
+F 4 "10V" H 7000 4150 50  0001 C CNN "Voltage"
+F 5 "LMK107B7105MA-T" H 7000 4150 50  0001 C CNN "Manufacturer Part Number"
+	1    7000 4150
+	-1   0    0    1
+$EndComp
+$Comp
+L Device:R R?
+U 1 1 5C6A0A52
+P 4800 4100
+AR Path="/5BC13C37/5C6A0A52" Ref="R?"  Part="1"
+AR Path="/5BC14C3C/5C6A0A52" Ref="R?"  Part="1"
+AR Path="/5BC300BF/5C6A0A52" Ref="R?"  Part="1"
+F 0 "R?" H 4730 4008 50  0000 R CNN
+F 1 "2k" H 4730 4100 50  0000 R CNN
+F 2 "Resistor_SMD:R_0603_1608Metric_Pad1.05x0.95mm_HandSolder" V 4730 4100 50  0001 C CNN
+F 3 "~" H 4800 4100 50  0001 C CNN
+F 4 "1%" H 4730 4192 50  0000 R CNN "Tolerance"
+F 5 "RC0603FR-102KL" V 4800 4100 50  0001 C CNN "Manufacturer Part Number"
+	1    4800 4100
+	-1   0    0    1
+$EndComp
+$Comp
+L Device:R R?
+U 1 1 5C6A0C34
+P 4350 4100
+AR Path="/5BC13C37/5C6A0C34" Ref="R?"  Part="1"
+AR Path="/5BC14C3C/5C6A0C34" Ref="R?"  Part="1"
+AR Path="/5BC300BF/5C6A0C34" Ref="R?"  Part="1"
+F 0 "R?" H 4280 4008 50  0000 R CNN
+F 1 "1k8" H 4280 4100 50  0000 R CNN
+F 2 "Resistor_SMD:R_0603_1608Metric_Pad1.05x0.95mm_HandSolder" V 4280 4100 50  0001 C CNN
+F 3 "~" H 4350 4100 50  0001 C CNN
+F 4 "1%" H 4280 4192 50  0000 R CNN "Tolerance"
+F 5 "RC0603FR-071K8L" V 4350 4100 50  0001 C CNN "Manufacturer Part Number"
+	1    4350 4100
+	-1   0    0    1
+$EndComp
 $EndSCHEMATC

Commit message: Enumeración de esquema de PCB_B
Parts:
- gave numbers to parts that had none: 6
Changed lines of the file:
@@
 $EndDescr
 $Comp
-L SamacSys_Parts:BQ24091DGQT U?
+L SamacSys_Parts:BQ24091DGQT U8
 U 1 1 5BAD7302
 P 5250 3550
-F 0 "U?" H 5900 3815 50  0000 C CNN
+F 0 "U8" H 5900 3815 50  0000 C CNN
 F 1 "BQ24091DGQT" H 5900 3724 50  0000 C CNN
 F 2 "SamacSys_Parts:SOP50P490X110-11N" H 6400 3650 50  0001 L CNN
@@
 AR Path="/5BA1A7F9/5BAD7944" Ref="#PWR?"  Part="1"
 AR Path="/5BA1A77A/5BAD7944" Ref="#PWR?"  Part="1"
-AR Path="/5BC300BF/5BAD7944" Ref="#PWR?"  Part="1"
-F 0 "#PWR?" H 3900 4050 50  0001 C CNN
+AR Path="/5BC300BF/5BAD7944" Ref="#PWR0148"  Part="1"
+F 0 "#PWR0148" H 3900 4050 50  0001 C CNN
 F 1 "GND" H 3905 4127 50  0000 C CNN
 F 2 "" H 3900 4300 50  0001 C CNN
@@
 AR Path="/5BA1A7F9/5BAD7E3B" Ref="#PWR?"  Part="1"
 AR Path="/5BA1A77A/5BAD7E3B" Ref="#PWR?"  Part="1"
-AR Path="/5BC300BF/5BAD7E3B" Ref="#PWR?"  Part="1"
-F 0 "#PWR?" H 4350 4050 50  0001 C CNN
+AR Path="/5BC300BF/5BAD7E3B" Ref="#PWR0149"  Part="1"
+F 0 "#PWR0149" H 4350 4050 50  0001 C CNN
 F 1 "GND" H 4355 4127 50  0000 C CNN
 F 2 "" H 4350 4300 50  0001 C CNN
@@
 AR Path="/5BA1A7F9/5BAD7F3D" Ref="#PWR?"  Part="1"
 AR Path="/5BA1A77A/5BAD7F3D" Ref="#PWR?"  Part="1"
-AR Path="/5BC300BF/5BAD7F3D" Ref="#PWR?"  Part="1"
-F 0 "#PWR?" H 4600 4050 50  0001 C CNN
+AR Path="/5BC300BF/5BAD7F3D" Ref="#PWR0150"  Part="1"
+F 0 "#PWR0150" H 4600 4050 50  0001 C CNN
 F 1 "GND" H 4605 4127 50  0000 C CNN
 F 2 "" H 4600 4300 50  0001 C CNN
@@
 AR Path="/5BA1A7F9/5BAD80E4" Ref="#PWR?"  Part="1"
 AR Path="/5BA1A77A/5BAD80E4" Ref="#PWR?"  Part="1"
-AR Path="/5BC300BF/5BAD80E4" Ref="#PWR?"  Part="1"
-F 0 "#PWR?" H 4800 4050 50  0001 C CNN
+AR Path="/5BC300BF/5BAD80E4" Ref="#PWR0151"  Part="1"
+F 0 "#PWR0151" H 4800 4050 50  0001 C CNN
 F 1 "GND" H 4805 4127 50  0000 C CNN
 F 2 "" H 4800 4300 50  0001 C CNN
@@
 AR Path="/5BA1A7F9/5BAD840C" Ref="R?"  Part="1"
 AR Path="/5BA1A77A/5BAD840C" Ref="R?"  Part="1"
-AR Path="/5BC300BF/5BAD840C" Ref="R?"  Part="1"
-F 0 "R?" V 7900 4100 50  0000 L CNN
+AR Path="/5BC300BF/5BAD840C" Ref="R16"  Part="1"
+F 0 "R16" V 7900 4100 50  0000 L CNN
 F 1 "100k" V 7700 4100 50  0000 L CNN
 F 2 "Resistor_SMD:R_0603_1608Metric_Pad1.05x0.95mm_HandSolder" V 7730 4100 50  0001 C CNN
@@
 AR Path="/5BA1A7F9/5BAD8415" Ref="#PWR?"  Part="1"
 AR Path="/5BA1A77A/5BAD8415" Ref="#PWR?"  Part="1"
-AR Path="/5BC300BF/5BAD8415" Ref="#PWR?"  Part="1"
-F 0 "#PWR?" H 7800 4050 50  0001 C CNN
+AR Path="/5BC300BF/5BAD8415" Ref="#PWR0152"  Part="1"
+F 0 "#PWR0152" H 7800 4050 50  0001 C CNN
 F 1 "GND" H 7805 4127 50  0000 C CNN
 F 2 "" H 7800 4300 50  0001 C CNN
@@
 AR Path="/5BA1A7F9/5BAD886E" Ref="#PWR?"  Part="1"
 AR Path="/5BA1A77A/5BAD886E" Ref="#PWR?"  Part="1"
-AR Path="/5BC300BF/5BAD886E" Ref="#PWR?"  Part="1"
-F 0 "#PWR?" H 6800 4050 50  0001 C CNN
+AR Path="/5BC300BF/5BAD886E" Ref="#PWR0153"  Part="1"
+F 0 "#PWR0153" H 6800 4050 50  0001 C CNN
 F 1 "GND" H 6805 4127 50  0000 C CNN
 F 2 "" H 6800 4300 50  0001 C CNN
@@
 AR Path="/5BA1A7F9/5BAF219B" Ref="#PWR?"  Part="1"
 AR Path="/5BA1A77A/5BAF219B" Ref="#PWR?"  Part="1"
-AR Path="/5BC300BF/5BAF219B" Ref="#PWR?"  Part="1"
-F 0 "#PWR?" H 7000 4050 50  0001 C CNN
+AR Path="/5BC300BF/5BAF219B" Ref="#PWR0154"  Part="1"
+F 0 "#PWR0154" H 7000 4050 50  0001 C CNN
 F 1 "GND" H 7005 4127 50  0000 C CNN
 F 2 "" H 7000 4300 50  0001 C CNN
@@
 AR Path="/5BC13C37/5C6A0401" Ref="C?"  Part="1"
 AR Path="/5BC14C3C/5C6A0401" Ref="C?"  Part="1"
-AR Path="/5BC300BF/5C6A0401" Ref="C?"  Part="1"
-F 0 "C?" H 3808 4004 50  0000 R CNN
+AR Path="/5BC300BF/5C6A0401" Ref="C25"  Part="1"
+F 0 "C25" H 3808 4004 50  0000 R CNN
 F 1 "1uF" H 3808 4095 50  0000 R CNN
 F 2 "Capacitor_SMD:C_0603_1608Metric_Pad1.05x0.95mm_HandSolder" H 3900 4050 50  0001 C CNN
@@
 AR Path="/5BC13C37/5C6A063E" Ref="C?"  Part="1"
 AR Path="/5BC14C3C/5C6A063E" Ref="C?"  Part="1"
-AR Path="/5BC300BF/5C6A063E" Ref="C?"  Part="1"
-F 0 "C?" H 6908 4104 50  0000 R CNN
+AR Path="/5BC300BF/5C6A063E" Ref="C26"  Part="1"
+F 0 "C26" H 6908 4104 50  0000 R CNN
 F 1 "1uF" H 6908 4195 50  0000 R CNN
 F 2 "Capacitor_SMD:C_0603_1608Metric_Pad1.05x0.95mm_HandSolder" H 7000 4150 50  0001 C CNN
@@
 AR Path="/5BC13C37/5C6A0A52" Ref="R?"  Part="1"
 AR Path="/5BC14C3C/5C6A0A52" Ref="R?"  Part="1"
-AR Path="/5BC300BF/5C6A0A52" Ref="R?"  Part="1"
-F 0 "R?" H 4730 4008 50  0000 R CNN
+AR Path="/5BC300BF/5C6A0A52" Ref="R15"  Part="1"
+F 0 "R15" H 4730 4008 50  0000 R CNN
 F 1 "2k" H 4730 4100 50  0000 R CNN
 F 2 "Resistor_SMD:R_0603_1608Metric_Pad1.05x0.95mm_HandSolder" V 4730 4100 50  0001 C CNN
@@
 AR Path="/5BC13C37/5C6A0C34" Ref="R?"  Part="1"
 AR Path="/5BC14C3C/5C6A0C34" Ref="R?"  Part="1"
-AR Path="/5BC300BF/5C6A0C34" Ref="R?"  Part="1"
-F 0 "R?" H 4280 4008 50  0000 R CNN
+AR Path="/5BC300BF/5C6A0C34" Ref="R14"  Part="1"
+F 0 "R14" H 4280 4008 50  0000 R CNN
 F 1 "1k8" H 4280 4100 50  0000 R CNN
 F 2 "Resistor_SMD:R_0603_1608Metric_Pad1.05x0.95mm_HandSolder" V 4280 4100 50  0001 C CNN

Commit message: Numeros de parte para PCB_B
Parts:
- R16: Manufacturer Part Number (none) -> RC0603JR-07100KL
Changed lines of the file:
@@
 F 2 "Resistor_SMD:R_0603_1608Metric_Pad1.05x0.95mm_HandSolder" V 7730 4100 50  0001 C CNN
 F 3 "~" H 7800 4100 50  0001 C CNN
+F 4 "RC0603JR-07100KL" V 7800 4100 50  0001 C CNN "Manufacturer Part Number"
 	1    7800 4100
 	-1   0    0    1

Commit message: Agregada R pull-up faltante en PCB_B
Parts:
- added R22: 100k, Resistor_SMD:R_0603_1608Metric_Pad1.05x0.95mm_HandSolder, symbol Device:R
Connections:
- net labels added: +3V3_Internal
- wire segments 24 -> 26
Changed lines of the file:
@@
 CHG
 Wire Wire Line
-	6550 3850 7250 3850
+	6550 3850 7150 3850
 $Comp
 L Device:R R?
@@
 	-1   0    0    1
 $EndComp
+$Comp
+L Device:R R?
+U 1 1 5C2818A5
+P 7150 3350
+AR Path="/5BA17F9C/5C2818A5" Ref="R?"  Part="1"
+AR Path="/5BA1A7F9/5C2818A5" Ref="R?"  Part="1"
+AR Path="/5BA1A77A/5C2818A5" Ref="R?"  Part="1"
+AR Path="/5BC300BF/5C2818A5" Ref="R22"  Part="1"
+F 0 "R22" V 7250 3350 50  0000 L CNN
+F 1 "100k" V 7050 3350 50  0000 L CNN
+F 2 "Resistor_SMD:R_0603_1608Metric_Pad1.05x0.95mm_HandSolder" V 7080 3350 50  0001 C CNN
+F 3 "~" H 7150 3350 50  0001 C CNN
+F 4 "RC0603JR-07100KL" V 7150 3350 50  0001 C CNN "Manufacturer Part Number"
+	1    7150 3350
+	-1   0    0    1
+$EndComp
+Wire Wire Line
+	7150 3500 7150 3850
+Connection ~ 7150 3850
+Wire Wire Line
+	7150 3850 7250 3850
+$Comp
+L AXTEC_IC:+3V3_Internal #PWR?
+U 1 1 5C286F2A
+P 7150 3200
+AR Path="/5BB6C3A1/5C286F2A" Ref="#PWR?"  Part="1"
+AR Path="/5BB6C83B/5C286F2A" Ref="#PWR?"  Part="1"
+AR Path="/5BC14C3C/5C286F2A" Ref="#PWR?"  Part="1"
+AR Path="/5C286F2A" Ref="#PWR?"  Part="1"
+AR Path="/5BC300BF/5C286F2A" Ref="#PWR11"  Part="1"
+F 0 "#PWR11" H 7150 3600 50  0001 C CNN
+F 1 "+3V3_Internal" H 7135 3373 50  0000 C CNN
+F 2 "" H 7150 3200 50  0001 C CNN
+F 3 "" H 7150 3200 50  0001 C CNN
+	1    7150 3200
+	1    0    0    -1
+$EndComp
 $EndSCHEMATC
