File: Hardware/Satelite/PCB_B/Fuel Gauge.sch (KiCad schematic (older format))
At the start: 7 parts, among them U6 BQ27441DRZR-G1A

Commit message: Nuevos PCB_B y PCB_C
Parts:
- renumbered C17 to C?, R17 to R?, R16 to R?, R15 to R?, R18 to R?, U6 to U?
Connections:
- net labels added: VBAT
- net labels removed: VBat+
Changed lines of the file:
@@
 EESchema Schematic File Version 4
-LIBS:PCB_A-cache
 EELAYER 26 0
 EELAYER END
@@
 $EndDescr
 $Comp
-L Battery_Management:BQ27441DRZR-G1A U6
+L Battery_Management:BQ27441DRZR-G1A U?
 U 1 1 5BB27F17
 P 5900 3700
-F 0 "U6" H 5900 4367 50  0000 C CNN
+F 0 "U?" H 5900 4367 50  0000 C CNN
 F 1 "BQ27441DRZR-G1A" H 5900 4276 50  0000 C CNN
 F 2 "Package_SON:Texas_S-PDSO-N12" H 6150 3150 50  0001 L CNN
@@
 AR Path="/5BA1A7F9/5BB28170" Ref="#PWR?"  Part="1"
 AR Path="/5BA1A77A/5BB28170" Ref="#PWR?"  Part="1"
-AR Path="/5BB1631B/5BB28170" Ref="#PWR0102"  Part="1"
-F 0 "#PWR0102" H 5900 4400 50  0001 C CNN
+AR Path="/5BB1631B/5BB28170" Ref="#PWR?"  Part="1"
+AR Path="/5BC28DAC/5BB28170" Ref="#PWR?"  Part="1"
+F 0 "#PWR?" H 5900 4400 50  0001 C CNN
 F 1 "GND" H 5905 4477 50  0000 C CNN
 F 2 "" H 5900 4650 50  0001 C CNN
@@
 P 4750 2700
 AR Path="/5BA17F9C/5BB29A49" Ref="#PWR?"  Part="1"
-AR Path="/5BB1631B/5BB29A49" Ref="#PWR0103"  Part="1"
-F 0 "#PWR0103" H 4750 2550 50  0001 C CNN
+AR Path="/5BB1631B/5BB29A49" Ref="#PWR?"  Part="1"
+AR Path="/5BC28DAC/5BB29A49" Ref="#PWR?"  Part="1"
+F 0 "#PWR?" H 4750 2550 50  0001 C CNN
 F 1 "+3V3" H 4765 2873 50  0000 C CNN
 F 2 "" H 4750 2700 50  0001 C CNN
@@
 AR Path="/5BA1A77A/5BB5738A" Ref="R?"  Part="1"
 AR Path="/5BB5738A" Ref="R?"  Part="1"
-AR Path="/5BB1631B/5BB5738A" Ref="R17"  Part="1"
-F 0 "R17" V 5150 4350 50  0000 L CNN
+AR Path="/5BB1631B/5BB5738A" Ref="R?"  Part="1"
+AR Path="/5BC28DAC/5BB5738A" Ref="R?"  Part="1"
+F 0 "R?" V 5150 4350 50  0000 L CNN
 F 1 "10k" V 4950 4350 50  0000 L CNN
 F 2 "" V 4980 4350 50  0001 C CNN
@@
 AR Path="/5BA1A7F9/5BB573CA" Ref="#PWR?"  Part="1"
 AR Path="/5BA1A77A/5BB573CA" Ref="#PWR?"  Part="1"
-AR Path="/5BB1631B/5BB573CA" Ref="#PWR0104"  Part="1"
-F 0 "#PWR0104" H 5050 4400 50  0001 C CNN
+AR Path="/5BB1631B/5BB573CA" Ref="#PWR?"  Part="1"
+AR Path="/5BC28DAC/5BB573CA" Ref="#PWR?"  Part="1"
+F 0 "#PWR?" H 5050 4400 50  0001 C CNN
 F 1 "GND" H 5055 4477 50  0000 C CNN
 F 2 "" H 5050 4650 50  0001 C CNN
@@
 AR Path="/5BA1A77A/5BB57404" Ref="R?"  Part="1"
 AR Path="/5BB57404" Ref="R?"  Part="1"
-AR Path="/5BB1631B/5BB57404" Ref="R16"  Part="1"
-F 0 "R16" V 5150 2950 50  0000 L CNN
+AR Path="/5BB1631B/5BB57404" Ref="R?"  Part="1"
+AR Path="/5BC28DAC/5BB57404" Ref="R?"  Part="1"
+F 0 "R?" V 5150 2950 50  0000 L CNN
 F 1 "10k" V 4950 2950 50  0000 L CNN
 F 2 "" V 4980 2950 50  0001 C CNN
@@
 Text HLabel 4200 3600 0    50   Input ~ 0
 SCL
-Text HLabel 3550 5050 0    50   Input ~ 0
-VBat+
+Text HLabel 3550 5050 0    50   BiDi ~ 0
+VBAT
 $Comp
 L Device:R R?
@@
 AR Path="/5BA1A77A/5BB59022" Ref="R?"  Part="1"
 AR Path="/5BB59022" Ref="R?"  Part="1"
-AR Path="/5BB1631B/5BB59022" Ref="R15"  Part="1"
-F 0 "R15" V 4850 2950 50  0000 L CNN
+AR Path="/5BB1631B/5BB59022" Ref="R?"  Part="1"
+AR Path="/5BC28DAC/5BB59022" Ref="R?"  Part="1"
+F 0 "R?" V 4850 2950 50  0000 L CNN
 F 1 "10k" V 4650 2950 50  0000 L CNN
 F 2 "" V 4680 2950 50  0001 C CNN
@@
 P 5050 2700
 AR Path="/5BA17F9C/5BB59119" Ref="#PWR?"  Part="1"
-AR Path="/5BB1631B/5BB59119" Ref="#PWR0105"  Part="1"
-F 0 "#PWR0105" H 5050 2550 50  0001 C CNN
+AR Path="/5BB1631B/5BB59119" Ref="#PWR?"  Part="1"
+AR Path="/5BC28DAC/5BB59119" Ref="#PWR?"  Part="1"
+F 0 "#PWR?" H 5050 2550 50  0001 C CNN
 F 1 "+3V3" H 5065 2873 50  0000 C CNN
 F 2 "" H 5050 2700 50  0001 C CNN
@@
 AR Path="/5BA1A77A/5BB59286" Ref="R?"  Part="1"
 AR Path="/5BB59286" Ref="R?"  Part="1"
-AR Path="/5BB1631B/5BB59286" Ref="R18"  Part="1"
-F 0 "R18" V 7250 3000 50  0000 L CNN
+AR Path="/5BB1631B/5BB59286" Ref="R?"  Part="1"
+AR Path="/5BC28DAC/5BB59286" Ref="R?"  Part="1"
+F 0 "R?" V 7250 3000 50  0000 L CNN
 F 1 "10k" V 7050 3000 50  0000 L CNN
 F 2 "" V 7080 3000 50  0001 C CNN
@@
 P 7150 2700
 AR Path="/5BA17F9C/5BB593CD" Ref="#PWR?"  Part="1"
-AR Path="/5BB1631B/5BB593CD" Ref="#PWR0106"  Part="1"
-F 0 "#PWR0106" H 7150 2550 50  0001 C CNN
+AR Path="/5BB1631B/5BB593CD" Ref="#PWR?"  Part="1"
+AR Path="/5BC28DAC/5BB593CD" Ref="#PWR?"  Part="1"
+F 0 "#PWR?" H 7150 2550 50  0001 C CNN
 F 1 "+3V3" H 7165 2873 50  0000 C CNN
 F 2 "" H 7150 2700 50  0001 C CNN
@@
 AR Path="/5BA1A77A/5BB5956D" Ref="C?"  Part="1"
 AR Path="/5BB5956D" Ref="C?"  Part="1"
-AR Path="/5BB1631B/5BB5956D" Ref="C17"  Part="1"
-F 0 "C17" H 6800 3950 50  0000 L CNN
+AR Path="/5BB1631B/5BB5956D" Ref="C?"  Part="1"
+AR Path="/5BC28DAC/5BB5956D" Ref="C?"  Part="1"
+F 0 "C?" H 6800 3950 50  0000 L CNN
 F 1 "0.47uF" H 6750 3850 50  0000 L CNN
 F 2 "" H 6650 3950 50  0001 C CNN
@@
 AR Path="/5BA1A7F9/5BB59DD4" Ref="#PWR?"  Part="1"
 AR Path="/5BA1A77A/5BB59DD4" Ref="#PWR?"  Part="1"
-AR Path="/5BB1631B/5BB59DD4" Ref="#PWR0107"  Part="1"
-F 0 "#PWR0107" H 6650 3800 50  0001 C CNN
+AR Path="/5BB1631B/5BB59DD4" Ref="#PWR?"  Part="1"
+AR Path="/5BC28DAC/5BB59DD4" Ref="#PWR?"  Part="1"
+F 0 "#PWR?" H 6650 3800 50  0001 C CNN
 F 1 "GND" H 6655 3877 50  0000 C CNN
 F 2 "" H 6650 4050 50  0001 C CNN
@@
 AR Path="/5BB5A45B" Ref="R?"  Part="1"
 AR Path="/5BB1631B/5BB5A45B" Ref="R?"  Part="1"
+AR Path="/5BC28DAC/5BB5A45B" Ref="R?"  Part="1"
 F 0 "R?" V 4550 5050 50  0000 L CNN
 F 1 "10m" V 4350 5050 50  0000 L CNN

Commit message: Nuevo conector interno para conexión entre PCB_C y PCB_B
Connections:
- net labels added: +3V3_Internal
- net labels removed: +3V3
- wire segments 32 -> 37
Changed lines of the file:
@@
 $Descr A4 11693 8268
 encoding utf-8
-Sheet 5 6
+Sheet 6 6
 Title ""
 Date ""
@@
 F 3 "" H 5900 4650 50  0001 C CNN
 	1    5900 4650
-	1    0    0    -1
-$EndComp
-$Comp
-L power:+3V3 #PWR?
-U 1 1 5BB29A49
-P 4750 2700
-AR Path="/5BA17F9C/5BB29A49" Ref="#PWR?"  Part="1"
-AR Path="/5BB1631B/5BB29A49" Ref="#PWR?"  Part="1"
-AR Path="/5BC28DAC/5BB29A49" Ref="#PWR?"  Part="1"
-F 0 "#PWR?" H 4750 2550 50  0001 C CNN
-F 1 "+3V3" H 4765 2873 50  0000 C CNN
-F 2 "" H 4750 2700 50  0001 C CNN
-F 3 "" H 4750 2700 50  0001 C CNN
-	1    4750 2700
 	1    0    0    -1
 $EndComp
@@
 	5050 3600 5300 3600
 $Comp
-L power:+3V3 #PWR?
-U 1 1 5BB59119
-P 5050 2700
-AR Path="/5BA17F9C/5BB59119" Ref="#PWR?"  Part="1"
-AR Path="/5BB1631B/5BB59119" Ref="#PWR?"  Part="1"
-AR Path="/5BC28DAC/5BB59119" Ref="#PWR?"  Part="1"
-F 0 "#PWR?" H 5050 2550 50  0001 C CNN
-F 1 "+3V3" H 5065 2873 50  0000 C CNN
-F 2 "" H 5050 2700 50  0001 C CNN
-F 3 "" H 5050 2700 50  0001 C CNN
-	1    5050 2700
-	1    0    0    -1
-$EndComp
-Wire Wire Line
-	5050 2800 5050 2700
-Wire Wire Line
-	4750 2700 4750 2800
-$Comp
 L Device:R R?
 U 1 1 5BB59286
-P 7150 3000
+P 7300 3450
 AR Path="/5BA17F9C/5BB59286" Ref="R?"  Part="1"
 AR Path="/5BA1A7F9/5BB59286" Ref="R?"  Part="1"
@@
 AR Path="/5BB1631B/5BB59286" Ref="R?"  Part="1"
 AR Path="/5BC28DAC/5BB59286" Ref="R?"  Part="1"
-F 0 "R?" V 7250 3000 50  0000 L CNN
-F 1 "10k" V 7050 3000 50  0000 L CNN
-F 2 "" V 7080 3000 50  0001 C CNN
-F 3 "~" H 7150 3000 50  0001 C CNN
-	1    7150 3000
-	1    0    0    -1
-$EndComp
-Wire Wire Line
-	7150 3150 7150 3700
-Wire Wire Line
-	7150 3700 6500 3700
-$Comp
-L power:+3V3 #PWR?
-U 1 1 5BB593CD
-P 7150 2700
-AR Path="/5BA17F9C/5BB593CD" Ref="#PWR?"  Part="1"
-AR Path="/5BB1631B/5BB593CD" Ref="#PWR?"  Part="1"
-AR Path="/5BC28DAC/5BB593CD" Ref="#PWR?"  Part="1"
-F 0 "#PWR?" H 7150 2550 50  0001 C CNN
-F 1 "+3V3" H 7165 2873 50  0000 C CNN
-F 2 "" H 7150 2700 50  0001 C CNN
-F 3 "" H 7150 2700 50  0001 C CNN
-	1    7150 2700
-	1    0    0    -1
-$EndComp
-Wire Wire Line
-	7150 2700 7150 2850
+F 0 "R?" V 7400 3450 50  0000 L CNN
+F 1 "10k" V 7200 3450 50  0000 L CNN
+F 2 "" V 7230 3450 50  0001 C CNN
+F 3 "~" H 7300 3450 50  0001 C CNN
+	1    7300 3450
+	1    0    0    -1
+$EndComp
+Wire Wire Line
+	7300 3600 7300 4150
+Wire Wire Line
+	7300 3150 7300 3300
 $Comp
 L Device:C_Small C?
 U 1 1 5BB5956D
-P 6650 3950
+P 6800 3550
 AR Path="/5BA17F9C/5BB5956D" Ref="C?"  Part="1"
 AR Path="/5BA1A7F9/5BB5956D" Ref="C?"  Part="1"
@@
 AR Path="/5BB1631B/5BB5956D" Ref="C?"  Part="1"
 AR Path="/5BC28DAC/5BB5956D" Ref="C?"  Part="1"
-F 0 "C?" H 6800 3950 50  0000 L CNN
-F 1 "0.47uF" H 6750 3850 50  0000 L CNN
-F 2 "" H 6650 3950 50  0001 C CNN
-F 3 "~" H 6650 3950 50  0001 C CNN
-	1    6650 3950
-	1    0    0    -1
-$EndComp
-Wire Wire Line
-	6500 3400 6650 3400
-Wire Wire Line
-	6650 3400 6650 3850
+F 0 "C?" H 6950 3550 50  0000 L CNN
+F 1 "0.47uF" H 6900 3450 50  0000 L CNN
+F 2 "" H 6800 3550 50  0001 C CNN
+F 3 "~" H 6800 3550 50  0001 C CNN
+	1    6800 3550
+	1    0    0    -1
+$EndComp
 $Comp
 L power:GND #PWR?
 U 1 1 5BB59DD4
-P 6650 4050
+P 6800 3650
 AR Path="/5BA1A7F9/5BB59DD4" Ref="#PWR?"  Part="1"
 AR Path="/5BA1A77A/5BB59DD4" Ref="#PWR?"  Part="1"
 AR Path="/5BB1631B/5BB59DD4" Ref="#PWR?"  Part="1"
 AR Path="/5BC28DAC/5BB59DD4" Ref="#PWR?"  Part="1"
-F 0 "#PWR?" H 6650 3800 50  0001 C CNN
-F 1 "GND" H 6655 3877 50  0000 C CNN
-F 2 "" H 6650 4050 50  0001 C CNN
-F 3 "" H 6650 4050 50  0001 C CNN
-	1    6650 4050
-	1    0    0    -1
-$EndComp
-Wire Wire Line
-	7150 3700 7500 3700
-Connection ~ 7150 3700
-Text HLabel 7500 3700 2    50   Output ~ 0
+F 0 "#PWR?" H 6800 3400 50  0001 C CNN
+F 1 "GND" H 6805 3477 50  0000 C CNN
+F 2 "" H 6800 3650 50  0001 C CNN
+F 3 "" H 6800 3650 50  0001 C CNN
+	1    6800 3650
+	1    0    0    -1
+$EndComp
+Wire Wire Line
+	7300 4150 7650 4150
+Text HLabel 7650 4150 2    50   Output ~ 0
 GPOUT
 Wire Wire Line
@@
 Text HLabel 5350 5050 2    50   BiDi ~ 0
 SYS
+$Comp
+L AXTEC_IC:+3V3_Internal #PWR?
+U 1 1 5BD19F65
+P 7300 3150
+AR Path="/5BD19F65" Ref="#PWR?"  Part="1"
+AR Path="/5BC28DAC/5BD19F65" Ref="#PWR?"  Part="1"
+F 0 "#PWR?" H 7300 3550 50  0001 C CNN
+F 1 "+3V3_Internal" H 7285 3325 50  0000 C CNN
+F 2 "" H 7300 3150 50  0001 C CNN
+F 3 "" H 7300 3150 50  0001 C CNN
+	1    7300 3150
+	1    0    0    -1
+$EndComp
+$Comp
+L AXTEC_IC:+3V3_Internal #PWR?
+U 1 1 5BD1A8BA
+P 4900 2600
+AR Path="/5BD1A8BA" Ref="#PWR?"  Part="1"
+AR Path="/5BC28DAC/5BD1A8BA" Ref="#PWR?"  Part="1"
+F 0 "#PWR?" H 4900 3000 50  0001 C CNN
+F 1 "+3V3_Internal" H 4885 2775 50  0000 C CNN
+F 2 "" H 4900 2600 50  0001 C CNN
+F 3 "" H 4900 2600 50  0001 C CNN
+	1    4900 2600
+	1    0    0    -1
+$EndComp
+Wire Wire Line
+	4750 2650 4900 2650
+Wire Wire Line
+	5050 2650 5050 2800
+Wire Wire Line
+	4750 2650 4750 2800
+Wire Wire Line
+	4900 2600 4900 2650
+Connection ~ 4900 2650
+Wire Wire Line
+	4900 2650 5050 2650
+Wire Wire Line
+	6800 3400 6800 3450
+Wire Wire Line
+	6500 3400 6800 3400
+Wire Wire Line
+	7300 4150 6600 4150
+Wire Wire Line
+	6600 4150 6600 3700
+Wire Wire Line
+	6600 3700 6500 3700
+Connection ~ 7300 4150
 $EndSCHEMATC

Commit message: Footprints para PCB_B
Parts:
- removed R? (x3): 10k, symbol Device:R
- added R? (x3): 10k, Capacitor_SMD:C_0603_1608Metric_Pad1.05x0.95mm_HandSolder, symbol Device:R
- C?: footprint (none) -> Capacitor_SMD:C_0603_1608Metric_Pad1.05x0.95mm_HandSolder; Manufacturer Part Number (none) -> 885012206024
- R?: footprint (none) -> Capacitor_SMD:C_0603_1608Metric_Pad1.05x0.95mm_HandSolder
- R?: footprint (none) -> Resistor_SMD:R_2512_6332Metric_Pad1.52x3.35mm_HandSolder; Manufacturer Part Number (none) -> KRL3264-C-R010-F-T1
Changed lines of the file:
@@
-	1    0    0    -1
-$EndComp
-$Comp
-L Device:R R?
-U 1 1 5BB5738A
-P 5050 4350
-AR Path="/5BA17F9C/5BB5738A" Ref="R?"  Part="1"
-AR Path="/5BA1A7F9/5BB5738A" Ref="R?"  Part="1"
-AR Path="/5BA1A77A/5BB5738A" Ref="R?"  Part="1"
-AR Path="/5BB5738A" Ref="R?"  Part="1"
-AR Path="/5BB1631B/5BB5738A" Ref="R?"  Part="1"
-AR Path="/5BC28DAC/5BB5738A" Ref="R?"  Part="1"
-F 0 "R?" V 5150 4350 50  0000 L CNN
-F 1 "10k" V 4950 4350 50  0000 L CNN
-F 2 "" V 4980 4350 50  0001 C CNN
-F 3 "~" H 5050 4350 50  0001 C CNN
-	1    5050 4350
 	1    0    0    -1
 $EndComp
@@
 Wire Wire Line
 	5050 4650 5050 4500
-$Comp
-L Device:R R?
-U 1 1 5BB57404
-P 5050 2950
-AR Path="/5BA17F9C/5BB57404" Ref="R?"  Part="1"
-AR Path="/5BA1A7F9/5BB57404" Ref="R?"  Part="1"
-AR Path="/5BA1A77A/5BB57404" Ref="R?"  Part="1"
-AR Path="/5BB57404" Ref="R?"  Part="1"
-AR Path="/5BB1631B/5BB57404" Ref="R?"  Part="1"
-AR Path="/5BC28DAC/5BB57404" Ref="R?"  Part="1"
-F 0 "R?" V 5150 2950 50  0000 L CNN
-F 1 "10k" V 4950 2950 50  0000 L CNN
-F 2 "" V 4980 2950 50  0001 C CNN
-F 3 "~" H 5050 2950 50  0001 C CNN
-	1    5050 2950
-	1    0    0    -1
-$EndComp
 Wire Wire Line
 	5300 3500 4750 3500
@@
 F 0 "R?" V 4850 2950 50  0000 L CNN
 F 1 "10k" V 4650 2950 50  0000 L CNN
-F 2 "" V 4680 2950 50  0001 C CNN
+F 2 "Capacitor_SMD:C_0603_1608Metric_Pad1.05x0.95mm_HandSolder" V 4680 2950 50  0001 C CNN
 F 3 "~" H 4750 2950 50  0001 C CNN
 	1    4750 2950
@@
 Wire Wire Line
 	5050 3600 5300 3600
-$Comp
-L Device:R R?
-U 1 1 5BB59286
-P 7300 3450
-AR Path="/5BA17F9C/5BB59286" Ref="R?"  Part="1"
-AR Path="/5BA1A7F9/5BB59286" Ref="R?"  Part="1"
-AR Path="/5BA1A77A/5BB59286" Ref="R?"  Part="1"
-AR Path="/5BB59286" Ref="R?"  Part="1"
-AR Path="/5BB1631B/5BB59286" Ref="R?"  Part="1"
-AR Path="/5BC28DAC/5BB59286" Ref="R?"  Part="1"
-F 0 "R?" V 7400 3450 50  0000 L CNN
-F 1 "10k" V 7200 3450 50  0000 L CNN
-F 2 "" V 7230 3450 50  0001 C CNN
-F 3 "~" H 7300 3450 50  0001 C CNN
-	1    7300 3450
-	1    0    0    -1
-$EndComp
 Wire Wire Line
 	7300 3600 7300 4150
@@
 F 0 "C?" H 6950 3550 50  0000 L CNN
 F 1 "0.47uF" H 6900 3450 50  0000 L CNN
-F 2 "" H 6800 3550 50  0001 C CNN
+F 2 "Capacitor_SMD:C_0603_1608Metric_Pad1.05x0.95mm_HandSolder" H 6800 3550 50  0001 C CNN
 F 3 "~" H 6800 3550 50  0001 C CNN
+F 4 "885012206024" H 6800 3550 50  0001 C CNN "Manufacturer Part Number"
 	1    6800 3550
 	1    0    0    -1
@@
 F 0 "R?" V 4550 5050 50  0000 L CNN
 F 1 "10m" V 4350 5050 50  0000 L CNN
-F 2 "" V 4380 5050 50  0001 C CNN
+F 2 "Resistor_SMD:R_2512_6332Metric_Pad1.52x3.35mm_HandSolder" V 4380 5050 50  0001 C CNN
 F 3 "~" H 4450 5050 50  0001 C CNN
 F 4 "1%" V 4450 5050 50  0000 C CNN "Tolerance"
+F 5 "KRL3264-C-R010-F-T1" V 4450 5050 50  0001 C CNN "Manufacturer Part Number"
 	1    4450 5050
 	0    1    1    0
@@
 	6600 3700 6500 3700
 Connection ~ 7300 4150
+$Comp
+L Device:R R?
+U 1 1 5C69F6F3
+P 5050 2950
+AR Path="/5BA17F9C/5C69F6F3" Ref="R?"  Part="1"
+AR Path="/5BA1A7F9/5C69F6F3" Ref="R?"  Part="1"
+AR Path="/5BA1A77A/5C69F6F3" Ref="R?"  Part="1"
+AR Path="/5C69F6F3" Ref="R?"  Part="1"
+AR Path="/5BB1631B/5C69F6F3" Ref="R?"  Part="1"
+AR Path="/5BC28DAC/5C69F6F3" Ref="R?"  Part="1"
+F 0 "R?" V 5150 2950 50  0000 L CNN
+F 1 "10k" V 4950 2950 50  0000 L CNN
+F 2 "Capacitor_SMD:C_0603_1608Metric_Pad1.05x0.95mm_HandSolder" V 4980 2950 50  0001 C CNN
+F 3 "~" H 5050 2950 50  0001 C CNN
+	1    5050 2950
+	1    0    0    -1
+$EndComp
+$Comp
+L Device:R R?
+U 1 1 5C69F715
+P 5050 4350
+AR Path="/5BA17F9C/5C69F715" Ref="R?"  Part="1"
+AR Path="/5BA1A7F9/5C69F715" Ref="R?"  Part="1"
+AR Path="/5BA1A77A/5C69F715" Ref="R?"  Part="1"
+AR Path="/5C69F715" Ref="R?"  Part="1"
+AR Path="/5BB1631B/5C69F715" Ref="R?"  Part="1"
+AR Path="/5BC28DAC/5C69F715" Ref="R?"  Part="1"
+F 0 "R?" V 5150 4350 50  0000 L CNN
+F 1 "10k" V 4950 4350 50  0000 L CNN
+F 2 "Capacitor_SMD:C_0603_1608Metric_Pad1.05x0.95mm_HandSolder" V 4980 4350 50  0001 C CNN
+F 3 "~" H 5050 4350 50  0001 C CNN
+	1    5050 4350
+	1    0    0    -1
+$EndComp
+$Comp
+L Device:R R?
+U 1 1 5C69F74F
+P 7300 3450
+AR Path="/5BA17F9C/5C69F74F" Ref="R?"  Part="1"
+AR Path="/5BA1A7F9/5C69F74F" Ref="R?"  Part="1"
+AR Path="/5BA1A77A/5C69F74F" Ref="R?"  Part="1"
+AR Path="/5C69F74F" Ref="R?"  Part="1"
+AR Path="/5BB1631B/5C69F74F" Ref="R?"  Part="1"
+AR Path="/5BC28DAC/5C69F74F" Ref="R?"  Part="1"
+F 0 "R?" V 7400 3450 50  0000 L CNN
+F 1 "10k" V 7200 3450 50  0000 L CNN
+F 2 "Capacitor_SMD:C_0603_1608Metric_Pad1.05x0.95mm_HandSolder" V 7230 3450 50  0001 C CNN
+F 3 "~" H 7300 3450 50  0001 C CNN
+	1    7300 3450
+	1    0    0    -1
+$EndComp
 $EndSCHEMATC

Commit message: Enumeración de esquema de PCB_B
Parts:
- gave numbers to parts that had none: 7
Changed lines of the file:
@@
 $EndDescr
 $Comp
-L Battery_Management:BQ27441DRZR-G1A U?
+L Battery_Management:BQ27441DRZR-G1A U9
 U 1 1 5BB27F17
 P 5900 3700
-F 0 "U?" H 5900 4367 50  0000 C CNN
+F 0 "U9" H 5900 4367 50  0000 C CNN
 F 1 "BQ27441DRZR-G1A" H 5900 4276 50  0000 C CNN
 F 2 "Package_SON:Texas_S-PDSO-N12" H 6150 3150 50  0001 L CNN
@@
 AR Path="/5BA1A77A/5BB28170" Ref="#PWR?"  Part="1"
 AR Path="/5BB1631B/5BB28170" Ref="#PWR?"  Part="1"
-AR Path="/5BC28DAC/5BB28170" Ref="#PWR?"  Part="1"
-F 0 "#PWR?" H 5900 4400 50  0001 C CNN
+AR Path="/5BC28DAC/5BB28170" Ref="#PWR0155"  Part="1"
+F 0 "#PWR0155" H 5900 4400 50  0001 C CNN
 F 1 "GND" H 5905 4477 50  0000 C CNN
 F 2 "" H 5900 4650 50  0001 C CNN
@@
 AR Path="/5BA1A77A/5BB573CA" Ref="#PWR?"  Part="1"
 AR Path="/5BB1631B/5BB573CA" Ref="#PWR?"  Part="1"
-AR Path="/5BC28DAC/5BB573CA" Ref="#PWR?"  Part="1"
-F 0 "#PWR?" H 5050 4400 50  0001 C CNN
+AR Path="/5BC28DAC/5BB573CA" Ref="#PWR0156"  Part="1"
+F 0 "#PWR0156" H 5050 4400 50  0001 C CNN
 F 1 "GND" H 5055 4477 50  0000 C CNN
 F 2 "" H 5050 4650 50  0001 C CNN
@@
 AR Path="/5BB59022" Ref="R?"  Part="1"
 AR Path="/5BB1631B/5BB59022" Ref="R?"  Part="1"
-AR Path="/5BC28DAC/5BB59022" Ref="R?"  Part="1"
-F 0 "R?" V 4850 2950 50  0000 L CNN
+AR Path="/5BC28DAC/5BB59022" Ref="R18"  Part="1"
+F 0 "R18" V 4850 2950 50  0000 L CNN
 F 1 "10k" V 4650 2950 50  0000 L CNN
 F 2 "Capacitor_SMD:C_0603_1608Metric_Pad1.05x0.95mm_HandSolder" V 4680 2950 50  0001 C CNN
@@
 AR Path="/5BB5956D" Ref="C?"  Part="1"
 AR Path="/5BB1631B/5BB5956D" Ref="C?"  Part="1"
-AR Path="/5BC28DAC/5BB5956D" Ref="C?"  Part="1"
-F 0 "C?" H 6950 3550 50  0000 L CNN
+AR Path="/5BC28DAC/5BB5956D" Ref="C27"  Part="1"
+F 0 "C27" H 6950 3550 50  0000 L CNN
 F 1 "0.47uF" H 6900 3450 50  0000 L CNN
 F 2 "Capacitor_SMD:C_0603_1608Metric_Pad1.05x0.95mm_HandSolder" H 6800 3550 50  0001 C CNN
@@
 AR Path="/5BA1A77A/5BB59DD4" Ref="#PWR?"  Part="1"
 AR Path="/5BB1631B/5BB59DD4" Ref="#PWR?"  Part="1"
-AR Path="/5BC28DAC/5BB59DD4" Ref="#PWR?"  Part="1"
-F 0 "#PWR?" H 6800 3400 50  0001 C CNN
+AR Path="/5BC28DAC/5BB59DD4" Ref="#PWR0157"  Part="1"
+F 0 "#PWR0157" H 6800 3400 50  0001 C CNN
 F 1 "GND" H 6805 3477 50  0000 C CNN
 F 2 "" H 6800 3650 50  0001 C CNN
@@
 AR Path="/5BB5A45B" Ref="R?"  Part="1"
 AR Path="/5BB1631B/5BB5A45B" Ref="R?"  Part="1"
-AR Path="/5BC28DAC/5BB5A45B" Ref="R?"  Part="1"
-F 0 "R?" V 4550 5050 50  0000 L CNN
+AR Path="/5BC28DAC/5BB5A45B" Ref="R17"  Part="1"
+F 0 "R17" V 4550 5050 50  0000 L CNN
 F 1 "10m" V 4350 5050 50  0000 L CNN
 F 2 "Resistor_SMD:R_2512_6332Metric_Pad1.52x3.35mm_HandSolder" V 4380 5050 50  0001 C CNN
@@
 P 7300 3150
 AR Path="/5BD19F65" Ref="#PWR?"  Part="1"
-AR Path="/5BC28DAC/5BD19F65" Ref="#PWR?"  Part="1"
-F 0 "#PWR?" H 7300 3550 50  0001 C CNN
+AR Path="/5BC28DAC/5BD19F65" Ref="#PWR10"  Part="1"
+F 0 "#PWR10" H 7300 3550 50  0001 C CNN
 F 1 "+3V3_Internal" H 7285 3325 50  0000 C CNN
 F 2 "" H 7300 3150 50  0001 C CNN
@@
 P 4900 2600
 AR Path="/5BD1A8BA" Ref="#PWR?"  Part="1"
-AR Path="/5BC28DAC/5BD1A8BA" Ref="#PWR?"  Part="1"
-F 0 "#PWR?" H 4900 3000 50  0001 C CNN
+AR Path="/5BC28DAC/5BD1A8BA" Ref="#PWR9"  Part="1"
+F 0 "#PWR9" H 4900 3000 50  0001 C CNN
 F 1 "+3V3_Internal" H 4885 2775 50  0000 C CNN
 F 2 "" H 4900 2600 50  0001 C CNN
@@
 AR Path="/5C69F6F3" Ref="R?"  Part="1"
 AR Path="/5BB1631B/5C69F6F3" Ref="R?"  Part="1"
-AR Path="/5BC28DAC/5C69F6F3" Ref="R?"  Part="1"
-F 0 "R?" V 5150 2950 50  0000 L CNN
+AR Path="/5BC28DAC/5C69F6F3" Ref="R19"  Part="1"
+F 0 "R19" V 5150 2950 50  0000 L CNN
 F 1 "10k" V 4950 2950 50  0000 L CNN
 F 2 "Capacitor_SMD:C_0603_1608Metric_Pad1.05x0.95mm_HandSolder" V 4980 2950 50  0001 C CNN
@@
 AR Path="/5C69F715" Ref="R?"  Part="1"
 AR Path="/5BB1631B/5C69F715" Ref="R?"  Part="1"
-AR Path="/5BC28DAC/5C69F715" Ref="R?"  Part="1"
-F 0 "R?" V 5150 4350 50  0000 L CNN
+AR Path="/5BC28DAC/5C69F715" Ref="R20"  Part="1"
+F 0 "R20" V 5150 4350 50  0000 L CNN
 F 1 "10k" V 4950 4350 50  0000 L CNN
 F 2 "Capacitor_SMD:C_0603_1608Metric_Pad1.05x0.95mm_HandSolder" V 4980 4350 50  0001 C CNN
@@
 AR Path="/5C69F74F" Ref="R?"  Part="1"
 AR Path="/5BB1631B/5C69F74F" Ref="R?"  Part="1"
-AR Path="/5BC28DAC/5C69F74F" Ref="R?"  Part="1"
-F 0 "R?" V 7400 3450 50  0000 L CNN
+AR Path="/5BC28DAC/5C69F74F" Ref="R21"  Part="1"
+F 0 "R21" V 7400 3450 50  0000 L CNN
 F 1 "10k" V 7200 3450 50  0000 L CNN
 F 2 "Capacitor_SMD:C_0603_1608Metric_Pad1.05x0.95mm_HandSolder" V 7230 3450 50  0001 C CNN
