File: Hardware/EstacionTerrena/EstacionTerrena.kicad_pcb (KiCad board)
At the start: 2 copper layers, 40 x 30 mm, 38 parts, among them J1 5-1814832-1, J2 USB_B_Micro, U1 TPD2E2U06, U2 MIC5323-3.3YD5_TR, U3 MCP2210, U4 CC1101RGP, U5 0915BM15A0001E, Y1 12MHz, Y2 26 MHz

Commit message: PCB de estación terrena
Parts:
- H1, H2, H3, H4: value MountingHole -> MountingHole_Pad
- J2, U1, U3: moved to F.Cu
- moved R1 37.1 mm to (30.8, 6.80), turned to 180 degrees
- moved C5 35.8 mm to (11.0, 9.70), turned to 180 degrees
- moved C7 34.6 mm to (12.9, 22.1), turned to 180 degrees
- moved C6 34.0 mm to (12.9, 20.4), turned to 180 degrees
- moved C8 33.9 mm to (17.1, 14.8), turned to 90 degrees
- moved C13 33.8 mm to (22.2, 15.7), turned to 90 degrees
- moved R4 32.9 mm to (18.7, 14.8), turned to 270 degrees
- moved C14 32.0 mm to (20.5, 15.7), turned to 90 degrees
- moved C12 29.2 mm to (19.2, 24.5)
- moved C9 29.1 mm to (14.9, 27.2), turned to 90 degrees
- moved D2 29.0 mm to (3.62, 21.1)
- moved C16 28.6 mm to (27.6, 16.2), turned to 90 degrees
- moved D1 28.2 mm to (27.3, 8.07)
- moved R6 27.7 mm to (27.2, 18.1)
- moved R3 27.0 mm to (17.2, 11.5), turned to 180 degrees
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Connections:
- H1 pad 1: (no net) -> GND
- H2 pad 1: (no net) -> GND
- H3 pad 1: (no net) -> GND
- H4 pad 1: (no net) -> GND
Routing:
- net +3V3: track 2.64 -> 126.9 mm, vias 0 -> 6
- net GND: track 5.79 -> 55.1 mm, vias 4 -> 30
- net +5V: track 7.36 -> 36.5 mm
- net /USBaSPI/D-: track 0.00 -> 22.0 mm
- net /USBaSPI/GP0: track 0.00 -> 22.0 mm, vias 0 -> 2
- net /USBaSPI/SCK: track 0.00 -> 21.1 mm
- net /USBaSPI/MISO: track 0.00 -> 20.5 mm
- net /USBaSPI/MOSI: track 0.00 -> 20.3 mm
- net /USBaSPI/D+: track 0.00 -> 17.6 mm
- net Net-(C9-Pad1): track 0.00 -> 10.5 mm
- net Net-(C10-Pad1): track 0.00 -> 9.21 mm
- net Net-(R3-Pad2): track 0.00 -> 8.89 mm
- net /CC1101/ANT: track 0.00 -> 7.31 mm
- net Net-(U3-Pad3): track 0.00 -> 4.31 mm
- net Net-(U3-Pad2): track 0.00 -> 4.25 mm
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- added copper zone on B.Cu, net GND
