File: Hardware/EstacionTerrena/USBaSPI.sch (KiCad schematic (older format))
At the start: 10 parts, among them J1 USB_B_Micro, U1 MIC5323-3.3YD5, U2 MCP2210, Y1 Crystal_GND2

Commit message: Esquema de estación terrena casi terminado. falta revision.
Parts:
- added D1, D2: LED, symbol Device:LED
- added R2, R3: 100, symbol Device:R
- added U4: TPD2E2U06, Package_TO_SOT_SMD:SOT-543, symbol Power_Protection:TPD2E2U06
- Y1: value Crystal_GND2 -> 12MHz
Connections:
- net labels added: GP0
- wire segments 48 -> 58

Commit message: Correciones en esquema de estacion terrena y agrege descripciones a libs
Parts:
- R2, R3: value 100 -> 220
Changed lines of the file:
@@
 P 3750 5300
 F 0 "R2" H 3820 5346 50  0000 L CNN
-F 1 "100" H 3820 5255 50  0000 L CNN
+F 1 "220" H 3820 5255 50  0000 L CNN
 F 2 "" V 3680 5300 50  0001 C CNN
 F 3 "~" H 3750 5300 50  0001 C CNN
@@
 P 4250 5300
 F 0 "R3" H 4320 5346 50  0000 L CNN
-F 1 "100" H 4320 5255 50  0000 L CNN
+F 1 "220" H 4320 5255 50  0000 L CNN
 F 2 "" V 4180 5300 50  0001 C CNN
 F 3 "~" H 4250 5300 50  0001 C CNN

Commit message: Asignados footprints a esquema de estación terrena
Parts:
- removed R1: 10K, symbol Device:R
- removed U1: MIC5323-3.3YD5, symbol AXTEC_IC:MIC5323-3.3YD5
- added R2: 220, Resistor_SMD:R_0603_1608Metric_Pad1.05x0.95mm_HandSolder, symbol Device:R
- added U2: MIC5323-3.3YD5_TR, SOT95P280X100-5N, symbol SamacSys_Parts:MIC5323-3.3YD5_TR
- C1, C3: footprint (none) -> Capacitor_SMD:C_0805_2012Metric; Dielectric (none) -> X7R; Manufacturer Part Number (none) -> LMK212B7225KG-T; Voltage (none) -> 10V
- C2, C4: value 0.1uF -> 100nF; footprint (none) -> Capacitor_SMD:C_0603_1608Metric; Dielectric (none) -> X7R; Manufacturer Part Number (none) -> EMK107B7104KAHT; Voltage (none) -> 16V
- C5: footprint (none) -> Capacitor_SMD:C_0603_1608Metric; Dielectric (none) -> X7R; Manufacturer Part Number (none) -> EMK107B7104KAHT; Voltage (none) -> 10V
- D1: value LED -> Verde; footprint (none) -> LED_SMD:LED_0603_1608Metric; Manufacturer Part Number (none) -> 150060VS75000
- D2: value LED -> Rojo; footprint (none) -> LED_SMD:LED_0603_1608Metric; Manufacturer Part Number (none) -> 150060RS75000
- J2: renamed from J1; footprint (none) -> Connector_USB:USB_Micro-B_Molex-105017-0001
- R1: renamed from R2; footprint (none) -> Resistor_SMD:R_0603_1608Metric_Pad1.05x0.95mm_HandSolder
- R3: value 220 -> 10k; footprint (none) -> Resistor_SMD:R_0603_1608Metric_Pad1.05x0.95mm_HandSolder
- U3: renamed from U2; footprint (none) -> Package_SO:SSOP-20_5.3x7.2mm_P0.65mm; Manufacturer Part Number (none) -> MCP2210-I/SS
- Y1: footprint (none) -> Crystal:Resonator_SMD_muRata_CSTxExxV-3Pin_3.0x1.1mm; Manufacturer Part Number (none) -> CSTNE12M0GH5L000R0
- renumbered U4 to U1

Commit message: PCB inicial para estación terrena
Parts:
- U1: footprint Package_TO_SOT_SMD:SOT-543 -> Package_TO_SOT_SMD:SOT-553; Manufacturer Part Number (none) -> TPD2E2U06DRLR
Changed lines of the file:
@@
 F 0 "U1" H 2600 4500 50  0000 L CNN
 F 1 "TPD2E2U06" H 2400 4400 50  0000 L CNN
-F 2 "Package_TO_SOT_SMD:SOT-543" H 1800 3900 50  0001 C CNN
+F 2 "Package_TO_SOT_SMD:SOT-553" H 1800 3900 50  0001 C CNN
 F 3 "http://www.ti.com/lit/ds/symlink/tpd2e2u06.pdf" H 2400 4350 50  0001 C CNN
+F 4 "TPD2E2U06DRLR" H 2600 4150 50  0001 C CNN "Manufacturer Part Number"
 	1    2600 4150
 	1    0    0    -1

Commit message: Más progreso en PCB estación terrena
Connections:
- wire segments 58 -> 59
Changed lines of the file:
@@
 	1    0    0    -1
 $EndComp
+Text Label 2100 4250 0    50   ~ 0
+D-
 Text Label 2100 4050 0    50   ~ 0
-D-
-Text Label 2100 4250 0    50   ~ 0
 D+
 Wire Wire Line
@@
 	1    0    0    -1
 $EndComp
+Text Label 3000 4250 0    50   ~ 0
+D-
+Wire Wire Line
+	2900 4250 3000 4250
 $EndSCHEMATC

Commit message: Footprints para PCB_C
Parts:
- C5: Manufacturer Part Number EMK107B7104KAHT -> LMK107B7105MA-T
- J2: Manufacturer Part Number (none) -> 105017-0001
Changed lines of the file:
@@
 F 2 "Connector_USB:USB_Micro-B_Molex-105017-0001" H 1300 4100 50  0001 C CNN
 F 3 "https://www.molex.com/webdocs/datasheets/pdf/en-us/1050170001_IO_CONNECTORS.pdf" H 1300 4100 50  0001 C CNN
+F 4 "105017-0001" H 1150 4150 50  0001 C CNN "Manufacturer Part Number"
 	1    1150 4150
 	1    0    0    -1
@@
 F 4 "X7R" H 9250 4500 50  0001 C CNN "Dielectric"
 F 5 "10V" H 9250 4500 50  0001 C CNN "Voltage"
-F 6 "EMK107B7104KAHT" H 9250 4500 50  0001 C CNN "Manufacturer Part Number"
+F 6 "LMK107B7105MA-T" H 9250 4500 50  0001 C CNN "Manufacturer Part Number"
 	1    9250 4500
 	1    0    0    -1

Commit message: Numeros de parte para estación terrena. Capacitores de 15pF para cristal de CC1101 (en lugar de 18pF).
Parts:
- R1, R2: Manufacturer Part Number (none) -> RC0603FR-07220RL
- R3: Manufacturer Part Number (none) -> RC0603JR-0710KL
Changed lines of the file:
@@
 F 2 "Resistor_SMD:R_0603_1608Metric_Pad1.05x0.95mm_HandSolder" V 3680 5300 50  0001 C CNN
 F 3 "~" H 3750 5300 50  0001 C CNN
+F 4 "RC0603FR-07220RL" H 3750 5300 50  0001 C CNN "Manufacturer Part Number"
 	1    3750 5300
 	1    0    0    -1
@@
 F 2 "Resistor_SMD:R_0603_1608Metric_Pad1.05x0.95mm_HandSolder" V 4180 5300 50  0001 C CNN
 F 3 "~" H 4250 5300 50  0001 C CNN
+F 4 "RC0603FR-07220RL" H 4250 5300 50  0001 C CNN "Manufacturer Part Number"
 	1    4250 5300
 	1    0    0    -1
@@
 F 2 "Resistor_SMD:R_0603_1608Metric_Pad1.05x0.95mm_HandSolder" V 7280 3850 50  0001 C CNN
 F 3 "~" H 7350 3850 50  0001 C CNN
+F 4 "RC0603JR-0710KL" H 7350 3850 50  0001 C CNN "Manufacturer Part Number"
 	1    7350 3850
 	1    0    0    -1
