File: Hardware/EstacionTerrena/USBaSPI.sch (KiCad schematic (older format))
At the start: 17 parts, among them J2 USB_B_Micro, U1 TPD2E2U06, U2 MIC5323-3.3YD5_TR, U3 MCP2210, Y1 12MHz

Commit message: Cambios de logos en esquemas
Parts:
- U2: symbol SamacSys_Parts:MIC5323-3.3YD5_TR -> EstacionTerrena-rescue:MIC5323-3.3YD5_TR-SamacSys_Parts
- U3: symbol AXTEC_IC:MCP2210 -> EstacionTerrena-rescue:MCP2210-AXTEC_IC
