File: Hardware/EstacionTerrena/EstacionTerrena.sch (KiCad schematic (older format))
At the start: 10 parts, among them J1 5-1814832-1

Commit message: Cambios de logos en esquemas
Parts:
- J1: symbol SamacSys_Parts:5-1814832-1 -> EstacionTerrena-rescue:5-1814832-1-SamacSys_Parts
