File: Hardware/EstacionTerrena/CC1101.sch (KiCad schematic (older format))
At the start: 19 parts, among them U4 CC1101RGP, U5 0915BM15A0001E, Y2 26 MHz

Commit message: Cambios de logos en esquemas
Parts:
- U4: symbol SamacSys_Parts:CC1101RGP -> EstacionTerrena-rescue:CC1101RGP-SamacSys_Parts
- U5: symbol SamacSys_Parts:0915BM15A0001E -> EstacionTerrena-rescue:0915BM15A0001E-SamacSys_Parts
