File: Hardware/Satelite/PCB_D/PCB_D.sch (KiCad schematic (older format))
At the start: 22 parts

Commit message: Eliminado conector interno del PCB D
Parts:
- removed J? (x3): Conn_01x10, Connector_PinHeader_1.27mm:PinHeader_1x10_P1.27mm_Vertical, symbol Connector_Generic:Conn_01x10
Connections:
- net labels removed: GPIO0, GPIO1, GPIO2, GPIO3, GPIO4, GPIO5, GPIO6, GPS_TX, VBUS
- wire segments 159 -> 107
Other:
- note removed: "Conectores de PCB_B"

Commit message: Agregados agujeros de montajes
Parts:
- added H? (x3): MountingHole_Pad, symbol Mechanical:MountingHole_Pad
Changed lines of the file:
@@
+	1    0    0    -1
+$EndComp
+$Comp
+L Mechanical:MountingHole_Pad H?
+U 1 1 5C39553A
+P 5750 4750
+F 0 "H?" H 5850 4801 50  0000 L CNN
+F 1 "MountingHole_Pad" H 5850 4709 50  0000 L CNN
+F 2 "" H 5750 4750 50  0001 C CNN
+F 3 "~" H 5750 4750 50  0001 C CNN
+	1    5750 4750
+	1    0    0    -1
+$EndComp
+$Comp
+L power:GND #PWR?
+U 1 1 5C395636
+P 5750 4850
+F 0 "#PWR?" H 5750 4600 50  0001 C CNN
+F 1 "GND" H 5754 4676 50  0000 C CNN
+F 2 "" H 5750 4850 50  0001 C CNN
+F 3 "" H 5750 4850 50  0001 C CNN
+	1    5750 4850
+	1    0    0    -1
+$EndComp
+$Comp
+L Mechanical:MountingHole_Pad H?
+U 1 1 5C39569B
+P 5750 5250
+F 0 "H?" H 5850 5301 50  0000 L CNN
+F 1 "MountingHole_Pad" H 5850 5209 50  0000 L CNN
+F 2 "" H 5750 5250 50  0001 C CNN
+F 3 "~" H 5750 5250 50  0001 C CNN
+	1    5750 5250
+	1    0    0    -1
+$EndComp
+$Comp
+L power:GND #PWR?
+U 1 1 5C3956A2
+P 5750 5350
+F 0 "#PWR?" H 5750 5100 50  0001 C CNN
+F 1 "GND" H 5754 5176 50  0000 C CNN
+F 2 "" H 5750 5350 50  0001 C CNN
+F 3 "" H 5750 5350 50  0001 C CNN
+	1    5750 5350
+	1    0    0    -1
+$EndComp
+$Comp
+L Mechanical:MountingHole_Pad H?
+U 1 1 5C39971C
+P 5750 5750
+F 0 "H?" H 5850 5801 50  0000 L CNN
+F 1 "MountingHole_Pad" H 5850 5709 50  0000 L CNN
+F 2 "" H 5750 5750 50  0001 C CNN
+F 3 "~" H 5750 5750 50  0001 C CNN
+	1    5750 5750
+	1    0    0    -1
+$EndComp
+$Comp
+L power:GND #PWR?
+U 1 1 5C399723
+P 5750 5850
+F 0 "#PWR?" H 5750 5600 50  0001 C CNN
+F 1 "GND" H 5754 5676 50  0000 C CNN
+F 2 "" H 5750 5850 50  0001 C CNN
+F 3 "" H 5750 5850 50  0001 C CNN
+	1    5750 5850
 	1    0    0    -1
 $EndComp

Commit message: Nuevo conector de expansión
Parts:
- removed J? (x7): Conn_02x02_Counter_Clockwise, Connector_PinHeader_2.54mm:PinHeader_2x02_P2.54mm_Vertical, symbol Connector_Generic:Conn_02x02_Counter_Clockwise
- added J? (x4): Conn_01x06, Connector_PinHeader_2.54mm:PinHeader_1x06_P2.54mm_Vertical, symbol Connector_Generic:Conn_01x06
Connections:
- net labels removed: CS, SCLK
- wire segments 107 -> 103
Other:
- moved on the sheet: U?

Commit message: Modificado conector expansión en PCB_D
Parts:
- removed H? (x3): MountingHole_Pad, symbol Mechanical:MountingHole_Pad
- removed J? (x4): Conn_01x06, Connector_PinHeader_2.54mm:PinHeader_1x06_P2.54mm_Vertical, symbol Connector_Generic:Conn_01x06
- added J?: Conector_Expansion_CanSat, AXTEC:Conector_Expansion_CanSat, symbol AXTEC_IC:Conector_Expansion_CanSat
Connections:
- wire segments 103 -> 107
Other:
- note added: "Arduino uno"
- note added: "Conector de expansión\n"
- note removed: "Conector de expansión"
- moved on the sheet: U?

Commit message: Agregado ICSP para PCB_D y header de pines no usados.
Parts:
- added D1: Verde, LED_SMD:LED_0603_1608Metric, symbol Device:LED
- added D2: Rojo, LED_SMD:LED_0603_1608Metric, symbol Device:LED
- added J1: Conn_01x04, symbol Connector_Generic:Conn_01x04
- added J3: Conn_02x03_Odd_Even, symbol Connector_Generic:Conn_02x03_Odd_Even
- added R4, R5: 220, Resistor_SMD:R_0603_1608Metric_Pad1.05x0.95mm_HandSolder, symbol Device:R
- gave numbers to parts that had none: 13
Connections:
- net labels added: RST
- wire segments 107 -> 132

Commit message: PCB_D agregado LED para blink + boton reset. Creado netlist
Parts:
- added D1: Amarillo, LED_SMD:LED_0603_1608Metric, symbol Device:LED
- added R4: 220, Resistor_SMD:R_0805_2012Metric_Pad1.15x1.40mm_HandSolder, symbol Device:R
- added SW1: RESET, Button_Switch_SMD:SW_SPST_PTS645, symbol Switch:SW_Push
- C1, C2, C3, C4, C5: footprint (none) -> Capacitor_SMD:C_0805_2012Metric_Pad1.15x1.40mm_HandSolder
- J1: footprint (none) -> Connector_PinHeader_2.54mm:PinHeader_1x04_P2.54mm_Vertical
- J3: footprint (none) -> Connector_PinHeader_2.54mm:PinHeader_2x03_P2.54mm_Vertical
- J4: footprint (none) -> Connector_USB:USB_Micro-B_Molex-105017-0001
- R1, R2, R3: footprint (none) -> Resistor_SMD:R_0805_2012Metric_Pad1.15x1.40mm_HandSolder
- R5: renamed from R4; footprint Resistor_SMD:R_0603_1608Metric_Pad1.05x0.95mm_HandSolder -> Resistor_SMD:R_0805_2012Metric_Pad1.15x1.40mm_HandSolder
- R6: renamed from R5; footprint Resistor_SMD:R_0603_1608Metric_Pad1.05x0.95mm_HandSolder -> Resistor_SMD:R_0805_2012Metric_Pad1.15x1.40mm_HandSolder
- U2: footprint CSTNE16M0V530000R0 -> SamacSys_Parts:CSTNE16M0V530000R0
- renumbered D1 to D2, D2 to D3
Connections:
- wire segments 132 -> 139
Changed lines of the file:
@@
 F 0 "J4" H 9920 4541 50  0000 R CNN
 F 1 "USB_B_Micro" H 9920 4449 50  0000 R CNN
-F 2 "" H 10300 4500 50  0001 C CNN
+F 2 "Connector_USB:USB_Micro-B_Molex-105017-0001" H 10300 4500 50  0001 C CNN
 F 3 "~" H 10300 4500 50  0001 C CNN
 	1    10150 4550
@@
 F 0 "C4" H 9092 3496 50  0000 L CNN
 F 1 "100n" H 9092 3404 50  0000 L CNN
-F 2 "" H 9000 3450 50  0001 C CNN
+F 2 "Capacitor_SMD:C_0805_2012Metric_Pad1.15x1.40mm_HandSolder" H 9000 3450 50  0001 C CNN
 F 3 "~" H 9000 3450 50  0001 C CNN
 	1    9000 3450
@@
 $EndComp
 $Comp
-L power:GND #PWR017
+L power:GND #PWR018
 U 1 1 5BBD9911
 P 9000 3550
-F 0 "#PWR017" H 9000 3300 50  0001 C CNN
+F 0 "#PWR018" H 9000 3300 50  0001 C CNN
 F 1 "GND" H 9004 3376 50  0000 C CNN
 F 2 "" H 9000 3550 50  0001 C CNN
@@
 	9850 4650 9450 4650
 $Comp
-L power:GND #PWR019
+L power:GND #PWR020
 U 1 1 5BBDE393
 P 10150 5100
-F 0 "#PWR019" H 10150 4850 50  0001 C CNN
+F 0 "#PWR020" H 10150 4850 50  0001 C CNN
 F 1 "GND" H 10154 4926 50  0000 C CNN
 F 2 "" H 10150 5100 50  0001 C CNN
@@
 $EndComp
 $Comp
-L power:GND #PWR016
+L power:GND #PWR017
 U 1 1 5BBDE3C1
 P 8750 5850
-F 0 "#PWR016" H 8750 5600 50  0001 C CNN
+F 0 "#PWR017" H 8750 5600 50  0001 C CNN
 F 1 "GND" H 8754 5676 50  0000 C CNN
 F 2 "" H 8750 5850 50  0001 C CNN
@@
 F 0 "C5" H 9492 3496 50  0000 L CNN
 F 1 "4.7uF" H 9492 3404 50  0000 L CNN
-F 2 "" H 9400 3450 50  0001 C CNN
+F 2 "Capacitor_SMD:C_0805_2012Metric_Pad1.15x1.40mm_HandSolder" H 9400 3450 50  0001 C CNN
 F 3 "~" H 9400 3450 50  0001 C CNN
 	1    9400 3450
@@
 	9400 3350 9750 3350
 $Comp
-L power:GND #PWR018
+L power:GND #PWR019
 U 1 1 5BBE96DA
 P 9400 3550
-F 0 "#PWR018" H 9400 3300 50  0001 C CNN
+F 0 "#PWR019" H 9400 3300 50  0001 C CNN
 F 1 "GND" H 9404 3376 50  0000 C CNN
 F 2 "" H 9400 3550 50  0001 C CNN
@@
 F 0 "R3" V 3800 6400 50  0000 C CNN
 F 1 "1k" V 3584 6400 50  0000 C CNN
-F 2 "" V 3630 6400 50  0001 C CNN
+F 2 "Resistor_SMD:R_0805_2012Metric_Pad1.15x1.40mm_HandSolder" V 3630 6400 50  0001 C CNN
 F 3 "~" H 3700 6400 50  0001 C CNN
 	1    3700 6400
@@
 F 0 "C3" V 3670 6200 50  0000 C CNN
 F 1 "100n" V 3762 6200 50  0000 C CNN
-F 2 "" H 3900 6200 50  0001 C CNN
+F 2 "Capacitor_SMD:C_0805_2012Metric_Pad1.15x1.40mm_HandSolder" H 3900 6200 50  0001 C CNN
 F 3 "~" H 3900 6200 50  0001 C CNN
 	1    3900 6200
@@
 F 0 "R2" H 3480 5954 50  0000 R CNN
 F 1 "10k" H 3480 6046 50  0000 R CNN
-F 2 "" V 3480 6000 50  0001 C CNN
+F 2 "Resistor_SMD:R_0805_2012Metric_Pad1.15x1.40mm_HandSolder" V 3480 6000 50  0001 C CNN
 F 3 "~" H 3550 6000 50  0001 C CNN
 	1    3550 6000
@@
 F 0 "C1" H 2358 4054 50  0000 R CNN
 F 1 "100n" H 2358 4146 50  0000 R CNN
-F 2 "" H 2450 4100 50  0001 C CNN
+F 2 "Capacitor_SMD:C_0805_2012Metric_Pad1.15x1.40mm_HandSolder" H 2450 4100 50  0001 C CNN
 F 3 "~" H 2450 4100 50  0001 C CNN
 	1    2450 4100
@@
 F 0 "C2" H 2758 4054 50  0000 R CNN
 F 1 "1uF" H 2758 4146 50  0000 R CNN
-F 2 "" H 2850 4100 50  0001 C CNN
+F 2 "Capacitor_SMD:C_0805_2012Metric_Pad1.15x1.40mm_HandSolder" H 2850 4100 50  0001 C CNN
 F 3 "~" H 2850 4100 50  0001 C CNN
 	1    2850 4100
@@
 	2450 4000 2450 3900
 $Comp
-L power:GND #PWR08
+L power:GND #PWR09
 U 1 1 5BC1C1FC
 P 2450 4200
-F 0 "#PWR08" H 2450 3950 50  0001 C CNN
+F 0 "#PWR09" H 2450 3950 50  0001 C CNN
 F 1 "GND" H 2454 4026 50  0000 C CNN
 F 2 "" H 2450 4200 50  0001 C CNN
@@
 F 0 "R1" V 3500 6500 50  0000 C CNN
 F 1 "1k" V 3284 6500 50  0000 C CNN
-F 2 "" V 3330 6500 50  0001 C CNN
+F 2 "Resistor_SMD:R_0805_2012Metric_Pad1.15x1.40mm_HandSolder" V 3330 6500 50  0001 C CNN
 F 3 "~" H 3400 6500 50  0001 C CNN
 	1    3400 6500
@@
 F 0 "U2" V 4750 6100 50  0000 L CNN
 F 1 "CSTNE16M0V530000R0" V 4650 5350 50  0000 L CNN
-F 2 "CSTNE16M0V530000R0" H 4650 6350 50  0001 L CNN
+F 2 "SamacSys_Parts:CSTNE16M0V530000R0" H 4650 6350 50  0001 L CNN
 F 3 "https://www.murata.com/en-eu/products/productdata/8801162231838/SPEC-CSTNE16M0V530000R0.pdf?1519875007000" H 4650 6250 50  0001 L CNN
 F 4 "Resonators 16.0000MHz 15pF SMD CHP Resntr" H 4650 6150 50  0001 L CNN "Description"
@@
 $EndComp
 $Comp
-L power:+5V #PWR02
+L power:+5V #PWR01
 U 1 1 5BC634E8
 P 850 2100
-F 0 "#PWR02" H 850 1950 50  0001 C CNN
+F 0 "#PWR01" H 850 1950 50  0001 C CNN
 F 1 "+5V" H 864 2275 50  0000 C CNN
 F 2 "" H 850 2100 50  0001 C CNN
@@
 	1700 2750 1700 2650
 $Comp
-L power:GND #PWR09
+L power:GND #PWR08
 U 1 1 5BC634FC
 P 2450 3100
-F 0 "#PWR09" H 2450 2850 50  0001 C CNN
+F 0 "#PWR08" H 2450 2850 50  0001 C CNN
 F 1 "GND" H 2454 2926 50  0000 C CNN
 F 2 "" H 2450 3100 50  0001 C CNN
@@
 F 0 "J3" H 5050 6067 50  0000 C CNN
 F 1 "Conn_02x03_Odd_Even" H 5050 5976 50  0000 C CNN
-F 2 "" H 5000 5750 50  0001 C CNN
+F 2 "Connector_PinHeader_2.54mm:PinHeader_2x03_P2.54mm_Vertical" H 5000 5750 50  0001 C CNN
 F 3 "~" H 5000 5750 50  0001 C CNN
 	1    5000 5750
@@
 	5300 5850 5500 5850
 $Comp
-L power:GND #PWR013
+L power:GND #PWR015
 U 1 1 5BC64733
 P 5500 5850
-F 0 "#PWR013" H 5500 5600 50  0001 C CNN
+F 0 "#PWR015" H 5500 5600 50  0001 C CNN
 F 1 "GND" H 5504 5676 50  0000 C CNN
 F 2 "" H 5500 5850 50  0001 C CNN
@@
 $EndComp
 $Comp
-L power:+5V #PWR014
+L power:+5V #PWR016
 U 1 1 5BC64784
 P 5550 5600
-F 0 "#PWR014" H 5550 5450 50  0001 C CNN
+F 0 "#PWR016" H 5550 5450 50  0001 C CNN
 F 1 "+5V" H 5564 5775 50  0000 C CNN
 F 2 "" H 5550 5600 50  0001 C CNN
@@
 F 0 "J1" H 720 4475 50  0000 C CNN
 F 1 "Conn_01x04" H 720 4566 50  0000 C CNN
-F 2 "" H 800 4900 50  0001 C CNN
+F 2 "Connector_PinHeader_2.54mm:PinHeader_1x04_P2.54mm_Vertical" H 800 4900 50  0001 C CNN
 F 3 "~" H 800 4900 50  0001 C CNN
 	1    800  4900
@@
 	1200 5000 1500 5000
 $Comp
-L power:GND #PWR01
+L power:GND #PWR02
 U 1 1 5BC7DF22
 P 1050 5050
-F 0 "#PWR01" H 1050 4800 50  0001 C CNN
+F 0 "#PWR02" H 1050 4800 50  0001 C CNN
 F 1 "GND" H 1054 4876 50  0000 C CNN
 F 2 "" H 1050 5050 50  0001 C CNN
@@
 P 6800 4650
 AR Path="/5B9997DB/5BC47B07" Ref="R?"  Part="1"
-AR Path="/5BC47B07" Ref="R4"  Part="1"
-F 0 "R4" H 6870 4696 50  0000 L CNN
+AR Path="/5BC47B07" Ref="R5"  Part="1"
+F 0 "R5" H 6870 4696 50  0000 L CNN
 F 1 "220" H 6870 4605 50  0000 L CNN
-F 2 "Resistor_SMD:R_0603_1608Metric_Pad1.05x0.95mm_HandSolder" V 6730 4650 50  0001 C CNN
+F 2 "Resistor_SMD:R_0805_2012Metric_Pad1.15x1.40mm_HandSolder" V 6730 4650 50  0001 C CNN
 F 3 "~" H 6800 4650 50  0001 C CNN
 	1    6800 4650
@@
 P 6800 5000
 AR Path="/5B9997DB/5BC47B16" Ref="D?"  Part="1"
-AR Path="/5BC47B16" Ref="D1"  Part="1"
-F 0 "D1" V 6838 4883 50  0000 R CNN
+AR Path="/5BC47B16" Ref="D2"  Part="1"
+F 0 "D2" V 6838 4883 50  0000 R CNN
 F 1 "Verde" V 6747 4883 50  0000 R CNN
 F 2 "LED_SMD:LED_0603_1608Metric" H 6800 5000 50  0001 C CNN
@@
 P 7300 4650
 AR Path="/5B9997DB/5BC47B2F" Ref="R?"  Part="1"
-AR Path="/5BC47B2F" Ref="R5"  Part="1"
-F 0 "R5" H 7370 4696 50  0000 L CNN
+AR Path="/5BC47B2F" Ref="R6"  Part="1"
+F 0 "R6" H 7370 4696 50  0000 L CNN
 F 1 "220" H 7370 4605 50  0000 L CNN
-F 2 "Resistor_SMD:R_0603_1608Metric_Pad1.05x0.95mm_HandSolder" V 7230 4650 50  0001 C CNN
+F 2 "Resistor_SMD:R_0805_2012Metric_Pad1.15x1.40mm_HandSolder" V 7230 4650 50  0001 C CNN
 F 3 "~" H 7300 4650 50  0001 C CNN
 	1    7300 4650
@@
 P 7300 5000
 AR Path="/5B9997DB/5BC47B37" Ref="D?"  Part="1"
-AR Path="/5BC47B37" Ref="D2"  Part="1"
-F 0 "D2" V 7338 4883 50  0000 R CNN
+AR Path="/5BC47B37" Ref="D3"  Part="1"
+F 0 "D3" V 7338 4883 50  0000 R CNN
 F 1 "Rojo" V 7247 4883 50  0000 R CNN
 F 2 "LED_SMD:LED_0603_1608Metric" H 7300 5000 50  0001 C CNN
@@
 	0    -1   -1   0
 $EndComp
-$Comp
-L power:+5V #PWR015
-U 1 1 5BC4D86D
-P 7050 4350
-F 0 "#PWR015" H 7050 4200 50  0001 C CNN
-F 1 "+5V" H 7064 4525 50  0000 C CNN
-F 2 "" H 7050 4350 50  0001 C CNN
-F 3 "" H 7050 4350 50  0001 C CNN
-	1    7050 4350
-	1    0    0    -1
-$EndComp
 Wire Wire Line
 	6800 4450 7050 4450
 Wire Wire Line
 	7300 4450 7300 4500
-Wire Wire Line
-	7050 4350 7050 4450
 Connection ~ 7050 4450
 Wire Wire Line
@@
 Wire Notes Line
 	10900 2650 10900 6200
+Wire Wire Line
+	7050 3350 8850 3350
+Wire Wire Line
+	7050 3350 7050 4450
+Connection ~ 8850 3350
+$Comp
+L Device:R R?
+U 1 1 5BC90912
+P 4900 6500
+AR Path="/5B9997DB/5BC90912" Ref="R?"  Part="1"
+AR Path="/5BC90912" Ref="R4"  Part="1"
+F 0 "R4" H 4970 6546 50  0000 L CNN
+F 1 "220" H 4970 6455 50  0000 L CNN
+F 2 "Resistor_SMD:R_0805_2012Metric_Pad1.15x1.40mm_HandSolder" V 4830 6500 50  0001 C CNN
+F 3 "~" H 4900 6500 50  0001 C CNN
+	1    4900 6500
+	1    0    0    -1
+$EndComp
+Wire Wire Line
+	4900 6300 4900 6350
+$Comp
+L Device:LED D?
+U 1 1 5BC9091B
+P 4900 6850
+AR Path="/5B9997DB/5BC9091B" Ref="D?"  Part="1"
+AR Path="/5BC9091B" Ref="D1"  Part="1"
+F 0 "D1" V 4938 6733 50  0000 R CNN
+F 1 "Amarillo" V 4847 6733 50  0000 R CNN
+F 2 "LED_SMD:LED_0603_1608Metric" H 4900 6850 50  0001 C CNN
+F 3 "~" H 4900 6850 50  0001 C CNN
+F 4 "150060VS75000" V 4900 6850 50  0001 C CNN "Manufacturer Part Number"
+	1    4900 6850
+	0    -1   -1   0
+$EndComp
+Wire Wire Line
+	4900 6700 4900 6650
+$Comp
+L power:GND #PWR013
+U 1 1 5BC96C3C
+P 4900 7100
+F 0 "#PWR013" H 4900 6850 50  0001 C CNN
+F 1 "GND" H 4904 6926 50  0000 C CNN
+F 2 "" H 4900 7100 50  0001 C CNN
+F 3 "" H 4900 7100 50  0001 C CNN
+	1    4900 7100
+	1    0    0    -1
+$EndComp
+Wire Wire Line
+	4900 7100 4900 7000
+Text Label 4900 6300 0    50   ~ 0
+SCK
+$Comp
+L Switch:SW_Push SW1
+U 1 1 5BC9E574
+P 5050 4500
+F 0 "SW1" H 5050 4785 50  0000 C CNN
+F 1 "RESET" H 5050 4694 50  0000 C CNN
+F 2 "Button_Switch_SMD:SW_SPST_PTS645" H 5050 4700 50  0001 C CNN
+F 3 "" H 5050 4700 50  0001 C CNN
+	1    5050 4500
+	1    0    0    -1
+$EndComp
+$Comp
+L power:GND #PWR014
+U 1 1 5BC9E63E
+P 5350 4550
+F 0 "#PWR014" H 5350 4300 50  0001 C CNN
+F 1 "GND" H 5354 4376 50  0000 C CNN
+F 2 "" H 5350 4550 50  0001 C CNN
+F 3 "" H 5350 4550 50  0001 C CNN
+	1    5350 4550
+	1    0    0    -1
+$EndComp
+Wire Wire Line
+	5250 4500 5350 4500
+Wire Wire Line
+	5350 4500 5350 4550
+Wire Wire Line
+	4850 4500 4700 4500
+Text Label 4700 4500 0    50   ~ 0
+RST
 $EndSCHEMATC

Commit message: PCB_D Terminada
Parts:
- removed J1: Conn_01x04, Connector_PinHeader_2.54mm:PinHeader_1x04_P2.54mm_Vertical, symbol Connector_Generic:Conn_01x04
- removed SW1: RESET, Button_Switch_SMD:SW_SPST_PTS645, symbol Switch:SW_Push
- added J1: Conn_01x03, Connector_PinHeader_2.54mm:PinHeader_1x03_P2.54mm_Vertical, symbol Connector_Generic:Conn_01x03
Connections:
- wire segments 139 -> 132
Changed lines of the file:
@@
 	3550 6200 3550 6150
 $Comp
-L power:+5V #PWR011
+L power:+5V #PWR012
 U 1 1 5BC1151B
 P 3550 5850
-F 0 "#PWR011" H 3550 5700 50  0001 C CNN
+F 0 "#PWR012" H 3550 5700 50  0001 C CNN
 F 1 "+5V" H 3564 6025 50  0000 C CNN
 F 2 "" H 3550 5850 50  0001 C CNN
@@
 	2450 4000 2450 3900
 $Comp
-L power:GND #PWR09
+L power:GND #PWR010
 U 1 1 5BC1C1FC
 P 2450 4200
-F 0 "#PWR09" H 2450 3950 50  0001 C CNN
+F 0 "#PWR010" H 2450 3950 50  0001 C CNN
 F 1 "GND" H 2454 4026 50  0000 C CNN
 F 2 "" H 2450 4200 50  0001 C CNN
@@
 $EndComp
 $Comp
-L power:GND #PWR010
+L power:GND #PWR011
 U 1 1 5BC1C21F
 P 2850 4200
-F 0 "#PWR010" H 2850 3950 50  0001 C CNN
+F 0 "#PWR011" H 2850 3950 50  0001 C CNN
 F 1 "GND" H 2854 4026 50  0000 C CNN
 F 2 "" H 2850 4200 50  0001 C CNN
@@
 	2100 4350 2100 3900
 $Comp
-L power:+5V #PWR06
+L power:+5V #PWR07
 U 1 1 5BC1E466
 P 2100 3850
-F 0 "#PWR06" H 2100 3700 50  0001 C CNN
+F 0 "#PWR07" H 2100 3700 50  0001 C CNN
 F 1 "+5V" H 2114 4025 50  0000 C CNN
 F 2 "" H 2100 3850 50  0001 C CNN
@@
 	2100 3850 2100 3900
 $Comp
-L power:GND #PWR07
+L power:GND #PWR08
 U 1 1 5BC2080C
 P 2100 7450
-F 0 "#PWR07" H 2100 7200 50  0001 C CNN
+F 0 "#PWR08" H 2100 7200 50  0001 C CNN
 F 1 "GND" H 2104 7276 50  0000 C CNN
 F 2 "" H 2100 7450 50  0001 C CNN
@@
 	3350 5500 3500 5500
 $Comp
-L power:GND #PWR012
+L power:GND #PWR013
 U 1 1 5BCA5EC3
 P 3800 5400
-F 0 "#PWR012" H 3800 5150 50  0001 C CNN
+F 0 "#PWR013" H 3800 5150 50  0001 C CNN
 F 1 "GND" H 3804 5226 50  0000 C CNN
 F 2 "" H 3800 5400 50  0001 C CNN
@@
 	1800 1400 1600 1400
 $Comp
-L power:+BATT #PWR04
+L power:+BATT #PWR05
 U 1 1 5BC634DC
 P 1350 2100
-F 0 "#PWR04" H 1350 1950 50  0001 C CNN
+F 0 "#PWR05" H 1350 1950 50  0001 C CNN
 F 1 "+BATT" H 1364 2275 50  0000 C CNN
 F 2 "" H 1350 2100 50  0001 C CNN
@@
 $EndComp
 $Comp
-L power:GND #PWR05
+L power:GND #PWR06
 U 1 1 5BC634EE
 P 1700 2850
-F 0 "#PWR05" H 1700 2600 50  0001 C CNN
+F 0 "#PWR06" H 1700 2600 50  0001 C CNN
 F 1 "GND" H 1704 2676 50  0000 C CNN
 F 2 "" H 1700 2850 50  0001 C CNN
@@
 	1700 2750 1700 2650
 $Comp
-L power:GND #PWR08
+L power:GND #PWR09
 U 1 1 5BC634FC
 P 2450 3100
-F 0 "#PWR08" H 2450 2850 50  0001 C CNN
+F 0 "#PWR09" H 2450 2850 50  0001 C CNN
 F 1 "GND" H 2454 2926 50  0000 C CNN
 F 2 "" H 2450 3100 50  0001 C CNN
@@
 MOSI
 $Comp
-L Connector_Generic:Conn_01x04 J1
-U 1 1 5BC69750
-P 800 4900
-F 0 "J1" H 720 4475 50  0000 C CNN
-F 1 "Conn_01x04" H 720 4566 50  0000 C CNN
-F 2 "Connector_PinHeader_2.54mm:PinHeader_1x04_P2.54mm_Vertical" H 800 4900 50  0001 C CNN
-F 3 "~" H 800 4900 50  0001 C CNN
-	1    800  4900
-	-1   0    0    1
-$EndComp
-Wire Wire Line
-	1500 4700 1000 4700
-Wire Wire Line
-	1500 4900 1250 4900
-Wire Wire Line
-	1250 4900 1250 4800
-Wire Wire Line
-	1250 4800 1000 4800
-Wire Wire Line
-	1000 4900 1200 4900
-Wire Wire Line
-	1200 4900 1200 5000
-Wire Wire Line
-	1200 5000 1500 5000
-$Comp
 L power:GND #PWR02
 U 1 1 5BC7DF22
-P 1050 5050
-F 0 "#PWR02" H 1050 4800 50  0001 C CNN
-F 1 "GND" H 1054 4876 50  0000 C CNN
-F 2 "" H 1050 5050 50  0001 C CNN
-F 3 "" H 1050 5050 50  0001 C CNN
-	1    1050 5050
-	1    0    0    -1
-$EndComp
-Wire Wire Line
-	1000 5000 1050 5000
-Wire Wire Line
-	1050 5000 1050 5050
+P 1050 4950
+F 0 "#PWR02" H 1050 4700 50  0001 C CNN
+F 1 "GND" H 1054 4776 50  0000 C CNN
+F 2 "" H 1050 4950 50  0001 C CNN
+F 3 "" H 1050 4950 50  0001 C CNN
+	1    1050 4950
+	1    0    0    -1
+$EndComp
 $Comp
 L Device:R R?
@@
 	4900 6700 4900 6650
 $Comp
-L power:GND #PWR013
+L power:GND #PWR014
 U 1 1 5BC96C3C
 P 4900 7100
-F 0 "#PWR013" H 4900 6850 50  0001 C CNN
+F 0 "#PWR014" H 4900 6850 50  0001 C CNN
 F 1 "GND" H 4904 6926 50  0000 C CNN
 F 2 "" H 4900 7100 50  0001 C CNN
@@
 SCK
 $Comp
-L Switch:SW_Push SW1
-U 1 1 5BC9E574
-P 5050 4500
-F 0 "SW1" H 5050 4785 50  0000 C CNN
-F 1 "RESET" H 5050 4694 50  0000 C CNN
-F 2 "Button_Switch_SMD:SW_SPST_PTS645" H 5050 4700 50  0001 C CNN
-F 3 "" H 5050 4700 50  0001 C CNN
-	1    5050 4500
-	1    0    0    -1
-$EndComp
-$Comp
-L power:GND #PWR014
-U 1 1 5BC9E63E
-P 5350 4550
-F 0 "#PWR014" H 5350 4300 50  0001 C CNN
-F 1 "GND" H 5354 4376 50  0000 C CNN
-F 2 "" H 5350 4550 50  0001 C CNN
-F 3 "" H 5350 4550 50  0001 C CNN
-	1    5350 4550
-	1    0    0    -1
-$EndComp
-Wire Wire Line
-	5250 4500 5350 4500
-Wire Wire Line
-	5350 4500 5350 4550
-Wire Wire Line
-	4850 4500 4700 4500
-Text Label 4700 4500 0    50   ~ 0
-RST
+L Connector_Generic:Conn_01x03 J1
+U 1 1 5BC51AA7
+P 800 4700
+F 0 "J1" H 720 4375 50  0000 C CNN
+F 1 "Conn_01x03" H 720 4466 50  0000 C CNN
+F 2 "Connector_PinHeader_2.54mm:PinHeader_1x03_P2.54mm_Vertical" H 800 4700 50  0001 C CNN
+F 3 "~" H 800 4700 50  0001 C CNN
+	1    800  4700
+	-1   0    0    1
+$EndComp
+Wire Wire Line
+	1000 4800 1050 4800
+Wire Wire Line
+	1050 4800 1050 4950
+$Comp
+L power:+5V #PWR04
+U 1 1 5BC577AC
+P 1150 4550
+F 0 "#PWR04" H 1150 4400 50  0001 C CNN
+F 1 "+5V" H 1164 4725 50  0000 C CNN
+F 2 "" H 1150 4550 50  0001 C CNN
+F 3 "" H 1150 4550 50  0001 C CNN
+	1    1150 4550
+	1    0    0    -1
+$EndComp
+Wire Wire Line
+	1000 4600 1150 4600
+Wire Wire Line
+	1150 4600 1150 4550
+Wire Wire Line
+	1000 4700 1500 4700
 $EndSCHEMATC
