File: Hardware/Satelite/PCB_D/PCB_D.sch (KiCad schematic (older format))
At the start: 21 parts, among them J1 Conn_01x03, J2 Conector_Expansion_CanSat, J3 Conn_02x03_Odd_Even, J4 USB_B_Micro, U1 ATmega328P-AU, U2 CSTNE16M0V530000R0, U3 FT231XS

Commit message: PCB_D agregado MH_CanSat y conector expansion por separado
Parts:
- added MH1: MH_CanSat, AXTEC:MH_CanSat, symbol AXTEC_IC:MH_CanSat
Other:
- note added: "Agujeros de montaje\n"
Changed lines of the file:
@@
 	3550 6200 3550 6150
 $Comp
-L power:+5V #PWR012
+L power:+5V #PWR011
 U 1 1 5BC1151B
 P 3550 5850
-F 0 "#PWR012" H 3550 5700 50  0001 C CNN
+F 0 "#PWR011" H 3550 5700 50  0001 C CNN
 F 1 "+5V" H 3564 6025 50  0000 C CNN
 F 2 "" H 3550 5850 50  0001 C CNN
@@
 	2450 4000 2450 3900
 $Comp
-L power:GND #PWR010
+L power:GND #PWR09
 U 1 1 5BC1C1FC
 P 2450 4200
-F 0 "#PWR010" H 2450 3950 50  0001 C CNN
+F 0 "#PWR09" H 2450 3950 50  0001 C CNN
 F 1 "GND" H 2454 4026 50  0000 C CNN
 F 2 "" H 2450 4200 50  0001 C CNN
@@
 $EndComp
 $Comp
-L power:GND #PWR011
+L power:GND #PWR010
 U 1 1 5BC1C21F
 P 2850 4200
-F 0 "#PWR011" H 2850 3950 50  0001 C CNN
+F 0 "#PWR010" H 2850 3950 50  0001 C CNN
 F 1 "GND" H 2854 4026 50  0000 C CNN
 F 2 "" H 2850 4200 50  0001 C CNN
@@
 	3350 5500 3500 5500
 $Comp
-L power:GND #PWR013
+L power:GND #PWR012
 U 1 1 5BCA5EC3
 P 3800 5400
-F 0 "#PWR013" H 3800 5150 50  0001 C CNN
+F 0 "#PWR012" H 3800 5150 50  0001 C CNN
 F 1 "GND" H 3804 5226 50  0000 C CNN
 F 2 "" H 3800 5400 50  0001 C CNN
@@
 	1700 2750 1700 2650
 $Comp
-L power:GND #PWR09
+L power:GND #PWR014
 U 1 1 5BC634FC
-P 2450 3100
-F 0 "#PWR09" H 2450 2850 50  0001 C CNN
-F 1 "GND" H 2454 2926 50  0000 C CNN
-F 2 "" H 2450 3100 50  0001 C CNN
-F 3 "" H 2450 3100 50  0001 C CNN
-	1    2450 3100
-	1    0    0    -1
-$EndComp
-Wire Wire Line
-	2350 3000 2350 3050
-Wire Wire Line
-	2350 3050 2450 3050
-Wire Wire Line
-	2550 3050 2550 3000
-Wire Wire Line
-	2450 3000 2450 3050
-Connection ~ 2450 3050
-Wire Wire Line
-	2450 3050 2550 3050
-Wire Wire Line
-	2450 3100 2450 3050
+P 5350 2550
+F 0 "#PWR014" H 5350 2300 50  0001 C CNN
+F 1 "GND" H 5354 2376 50  0000 C CNN
+F 2 "" H 5350 2550 50  0001 C CNN
+F 3 "" H 5350 2550 50  0001 C CNN
+	1    5350 2550
+	1    0    0    -1
+$EndComp
 Wire Wire Line
 	1350 2100 1800 2100
@@
 Wire Wire Line
 	3100 2750 3300 2750
-Text Notes 1950 1000 0    118  ~ 0
+Text Notes 700  1000 0    118  ~ 0
 Conector de expansión\n
 Wire Notes Line
@@
 	4900 6700 4900 6650
 $Comp
-L power:GND #PWR014
+L power:GND #PWR013
 U 1 1 5BC96C3C
 P 4900 7100
-F 0 "#PWR014" H 4900 6850 50  0001 C CNN
+F 0 "#PWR013" H 4900 6850 50  0001 C CNN
 F 1 "GND" H 4904 6926 50  0000 C CNN
 F 2 "" H 4900 7100 50  0001 C CNN
@@
 Wire Wire Line
 	1000 4700 1500 4700
+$Comp
+L AXTEC_IC:MH_CanSat MH1
+U 1 1 5BC6ACD9
+P 5350 2350
+F 0 "MH1" H 5628 2465 50  0000 L CNN
+F 1 "MH_CanSat" H 5628 2374 50  0000 L CNN
+F 2 "AXTEC:MH_CanSat" H 5350 2350 50  0001 C CNN
+F 3 "" H 5350 2350 50  0001 C CNN
+	1    5350 2350
+	1    0    0    -1
+$EndComp
+Wire Wire Line
+	5200 2450 5200 2500
+Wire Wire Line
+	5200 2500 5350 2500
+Wire Wire Line
+	5500 2500 5500 2450
+Wire Wire Line
+	5350 2550 5350 2500
+Connection ~ 5350 2500
+Wire Wire Line
+	5350 2500 5500 2500
+Wire Wire Line
+	5350 2450 5350 2500
+Wire Notes Line
+	4200 800  4200 3400
+Wire Notes Line
+	4200 3400 6550 3400
+Wire Notes Line
+	6550 3400 6550 800
+Wire Notes Line
+	4200 800  6550 800
+Text Notes 4350 1000 0    118  ~ 0
+Agujeros de montaje\n
 $EndSCHEMATC
