File: Hardware/Satelite/PCB_D/PCB_D.sch (KiCad schematic (older format))
At the start: 22 parts, among them J1 Conn_01x03, J2 Conector_Expansion_CanSat, J3 Conn_02x03_Odd_Even, J4 USB_B_Micro, U1 ATmega328P-AU, U2 CSTNE16M0V530000R0, U3 FT231XS

Commit message: PCB_D arreglado y serigrafias acorde a nueva disposicion de pines del conector de expansion
Connections:
- wire segments 132 -> 134
Changed lines of the file:
@@
 	1    0    0    -1
 $EndComp
-Text Label 1600 1400 0    50   ~ 0
+Text Label 1600 2300 0    50   ~ 0
 MOSI
-Text Label 1600 1500 0    50   ~ 0
+Text Label 1600 2400 0    50   ~ 0
 MISO
-Text Label 1600 1600 0    50   ~ 0
+Text Label 1600 2500 0    50   ~ 0
 SCK
-Text Label 1600 1700 0    50   ~ 0
+Text Label 1600 2600 0    50   ~ 0
 SS
-Text Label 1600 1800 0    50   ~ 0
+Text Label 1600 2700 0    50   ~ 0
 SCL
-Text Label 1600 1900 0    50   ~ 0
+Text Label 1600 2800 0    50   ~ 0
 SDA
 Wire Wire Line
-	1800 1900 1600 1900
-Wire Wire Line
-	1800 1800 1600 1800
-Wire Wire Line
-	1800 1700 1600 1700
-Wire Wire Line
-	1800 1600 1600 1600
-Wire Wire Line
-	1800 1500 1600 1500
-Wire Wire Line
-	1800 1400 1600 1400
+	1800 2800 1600 2800
+Wire Wire Line
+	1800 2700 1600 2700
+Wire Wire Line
+	1800 2600 1600 2600
+Wire Wire Line
+	1800 2500 1600 2500
+Wire Wire Line
+	1800 2400 1600 2400
+Wire Wire Line
+	1800 2300 1600 2300
 $Comp
 L power:+BATT #PWR05
 U 1 1 5BC634DC
-P 1350 2100
-F 0 "#PWR05" H 1350 1950 50  0001 C CNN
-F 1 "+BATT" H 1364 2275 50  0000 C CNN
-F 2 "" H 1350 2100 50  0001 C CNN
-F 3 "" H 1350 2100 50  0001 C CNN
-	1    1350 2100
+P 1700 1400
+F 0 "#PWR05" H 1700 1250 50  0001 C CNN
+F 1 "+BATT" H 1714 1575 50  0000 C CNN
+F 2 "" H 1700 1400 50  0001 C CNN
+F 3 "" H 1700 1400 50  0001 C CNN
+	1    1700 1400
 	1    0    0    -1
 $EndComp
@@
 L power:+3V3 #PWR03
 U 1 1 5BC634E2
-P 1100 2100
-F 0 "#PWR03" H 1100 1950 50  0001 C CNN
-F 1 "+3V3" H 1114 2275 50  0000 C CNN
-F 2 "" H 1100 2100 50  0001 C CNN
-F 3 "" H 1100 2100 50  0001 C CNN
-	1    1100 2100
+P 1450 1400
+F 0 "#PWR03" H 1450 1250 50  0001 C CNN
+F 1 "+3V3" H 1464 1575 50  0000 C CNN
+F 2 "" H 1450 1400 50  0001 C CNN
+F 3 "" H 1450 1400 50  0001 C CNN
+	1    1450 1400
 	1    0    0    -1
 $EndComp
@@
 L power:+5V #PWR01
 U 1 1 5BC634E8
-P 850 2100
-F 0 "#PWR01" H 850 1950 50  0001 C CNN
-F 1 "+5V" H 864 2275 50  0000 C CNN
-F 2 "" H 850 2100 50  0001 C CNN
-F 3 "" H 850 2100 50  0001 C CNN
-	1    850  2100
+P 1200 1400
+F 0 "#PWR01" H 1200 1250 50  0001 C CNN
+F 1 "+5V" H 1214 1575 50  0000 C CNN
+F 2 "" H 1200 1400 50  0001 C CNN
+F 3 "" H 1200 1400 50  0001 C CNN
+	1    1200 1400
 	1    0    0    -1
 $EndComp
@@
 L power:GND #PWR06
 U 1 1 5BC634EE
-P 1700 2850
-F 0 "#PWR06" H 1700 2600 50  0001 C CNN
-F 1 "GND" H 1704 2676 50  0000 C CNN
-F 2 "" H 1700 2850 50  0001 C CNN
-F 3 "" H 1700 2850 50  0001 C CNN
-	1    1700 2850
-	1    0    0    -1
-$EndComp
-Wire Wire Line
-	1700 2850 1700 2750
-Wire Wire Line
-	1700 2550 1800 2550
-Wire Wire Line
-	1800 2650 1700 2650
-Connection ~ 1700 2650
-Wire Wire Line
-	1700 2650 1700 2550
-Wire Wire Line
-	1800 2750 1700 2750
-Connection ~ 1700 2750
-Wire Wire Line
-	1700 2750 1700 2650
+P 1500 2050
+F 0 "#PWR06" H 1500 1800 50  0001 C CNN
+F 1 "GND" H 1504 1876 50  0000 C CNN
+F 2 "" H 1500 2050 50  0001 C CNN
+F 3 "" H 1500 2050 50  0001 C CNN
+	1    1500 2050
+	1    0    0    -1
+$EndComp
+Wire Wire Line
+	1700 1900 1800 1900
+Wire Wire Line
+	1800 2000 1700 2000
+Connection ~ 1700 2000
+Wire Wire Line
+	1700 2000 1700 1900
+Wire Wire Line
+	1800 2100 1700 2100
+Wire Wire Line
+	1700 2100 1700 2000
 $Comp
 L power:GND #PWR014
@@
 	1    0    0    -1
 $EndComp
-Wire Wire Line
-	1350 2100 1800 2100
-Wire Wire Line
-	1800 2200 1100 2200
-Wire Wire Line
-	1100 2200 1100 2100
-Wire Wire Line
-	1800 2300 850  2300
-Wire Wire Line
-	850  2300 850  2100
 Wire Wire Line
 	3100 1400 3300 1400
@@
 Text Notes 4350 1000 0    118  ~ 0
 Agujeros de montaje\n
+Wire Wire Line
+	1500 2050 1500 2000
+Wire Wire Line
+	1500 2000 1700 2000
+Wire Wire Line
+	1800 1650 1200 1650
+Wire Wire Line
+	1200 1650 1200 1400
+Wire Wire Line
+	1450 1400 1450 1550
+Wire Wire Line
+	1450 1550 1800 1550
+Wire Wire Line
+	1700 1400 1700 1450
+Wire Wire Line
+	1700 1450 1800 1450
 $EndSCHEMATC

Commit message: Numeros de parte para PCB_D
Parts:
- C1, C3, C4: Manufacturer Part Number (none) -> EMK107B7104KAHT
- C2: Manufacturer Part Number (none) -> LMK107B7105MA-T
- C5: Manufacturer Part Number (none) -> GRM21BR71A475KE51K
- J4: Manufacturer Part Number (none) -> 105017-0001

Commit message: Correciones en PCB D
Parts:
- added D4: LL4148, Diode_SMD:D_MiniMELF, symbol Diode:LL4148
Connections:
- wire segments 134 -> 136
Changed lines of the file:
@@
 	10900 800  10900 4350
-Wire Wire Line
-	7050 1500 8850 1500
 Wire Wire Line
 	7050 1500 7050 2600
@@
 Wire Wire Line
 	1700 1450 1800 1450
+$Comp
+L power:+5V #PWR021
+U 1 1 5BE24D5E
+P 7500 1250
+F 0 "#PWR021" H 7500 1100 50  0001 C CNN
+F 1 "+5V" H 7514 1425 50  0000 C CNN
+F 2 "" H 7500 1250 50  0001 C CNN
+F 3 "" H 7500 1250 50  0001 C CNN
+	1    7500 1250
+	1    0    0    -1
+$EndComp
+Wire Wire Line
+	7050 1500 8850 1500
+Wire Wire Line
+	7350 1250 7500 1250
+Wire Wire Line
+	7050 1250 7050 1500
+Connection ~ 7050 1500
+$Comp
+L Diode:LL4148 D4
+U 1 1 5BE5040B
+P 7200 1250
+F 0 "D4" H 7200 1034 50  0000 C CNN
+F 1 "LL4148" H 7200 1125 50  0000 C CNN
+F 2 "Diode_SMD:D_MiniMELF" H 7200 1075 50  0001 C CNN
+F 3 "http://www.vishay.com/docs/85557/ll4148.pdf" H 7200 1250 50  0001 C CNN
+	1    7200 1250
+	-1   0    0    1
+$EndComp
 $EndSCHEMATC

Commit message: Numeros de parte para PCB_D
Parts:
- added JP1: BOM_Jumper, AXTEC:Empty_Footprint, symbol AXTEC_IC:BOM_Jumper
- added M1 (x2), M2 (x2), M3 (x2): Spacer, AXTEC:Empty_Footprint, symbol AXTEC_IC:Spacer
- C1, C2, C3, C4: footprint Capacitor_SMD:C_0805_2012Metric_Pad1.15x1.40mm_HandSolder -> Capacitor_SMD:C_0603_1608Metric_Pad1.05x0.95mm_HandSolder
- D1: value Amarillo -> Verde
- D4: Manufacturer Part Number (none) -> LL4148-GS08
- J1: Manufacturer Part Number (none) -> 61300311121
- J2: Manufacturer Part Number (none) -> SSQ-106-03-T-S; Quantity (none) -> 4
- J3: Manufacturer Part Number (none) -> TSM-103-03-T-DV
- R1, R3: Manufacturer Part Number (none) -> RC0603JR-071KL
- R2: Manufacturer Part Number (none) -> RC0603JR-0710KL
- R4, R5, R6: footprint Resistor_SMD:R_0805_2012Metric_Pad1.15x1.40mm_HandSolder -> Resistor_SMD:R_0603_1608Metric_Pad1.05x0.95mm_HandSolder; Manufacturer Part Number (none) -> RC0603JR-13220RL
- U1: Manufacturer Part Number (none) -> ATMEGA328P-AU
- U3: Manufacturer Part Number (none) -> FT231XS-U
Other:
- note added: "Mecánica"
- moved on the sheet: U1

Commit message: Numeros de parte para PCB_E
Parts:
- removed M1, M2, M3: Spacer, AXTEC:Empty_Footprint, symbol AXTEC_IC:Spacer
Other:
- note removed: "Mecánica"
Changed lines of the file:
@@
-	1    0    0    -1
-$EndComp
-$Comp
-L AXTEC_IC:Spacer M1
-U 1 1 5C302141
-P 9300 5900
-F 0 "M1" H 9379 5893 50  0000 L CNN
-F 1 "Spacer" H 9379 5801 50  0000 L CNN
-F 2 "AXTEC:Empty_Footprint" H 9200 6050 50  0001 C CNN
-F 3 "https://www.mouser.com/datasheet/2/181/R30-301-1135805.pdf" H 9300 6150 50  0001 C CNN
-F 4 "R30-3011002" H 9379 5755 50  0001 L CNN "Manufacturer Part Number"
-	1    9300 5900
-	1    0    0    -1
-$EndComp
-$Comp
-L AXTEC_IC:Spacer M2
-U 1 1 5C3025E5
-P 9850 5900
-F 0 "M2" H 9929 5893 50  0000 L CNN
-F 1 "Spacer" H 9929 5801 50  0000 L CNN
-F 2 "AXTEC:Empty_Footprint" H 9750 6050 50  0001 C CNN
-F 3 "https://www.mouser.com/datasheet/2/181/R30-301-1135805.pdf" H 9850 6150 50  0001 C CNN
-F 4 "R30-3011002" H 9929 5755 50  0001 L CNN "Manufacturer Part Number"
-	1    9850 5900
-	1    0    0    -1
-$EndComp
-$Comp
-L AXTEC_IC:Spacer M3
-U 1 1 5C30263D
-P 10400 5900
-F 0 "M3" H 10479 5893 50  0000 L CNN
-F 1 "Spacer" H 10479 5801 50  0000 L CNN
-F 2 "AXTEC:Empty_Footprint" H 10300 6050 50  0001 C CNN
-F 3 "https://www.mouser.com/datasheet/2/181/R30-301-1135805.pdf" H 10400 6150 50  0001 C CNN
-F 4 "R30-3011002" H 10479 5755 50  0001 L CNN "Manufacturer Part Number"
-	1    10400 5900
 	1    0    0    -1
 $EndComp
 Wire Notes Line
-	10900 4400 10900 6500
-Wire Notes Line
 	10900 6500 8950 6500
-Wire Notes Line
-	8950 6500 8950 4400
-Wire Notes Line
-	8950 4400 10900 4400
-Text Notes 9550 4650 0    118  ~ 0
-Mecánica
 $Comp
 L AXTEC_IC:BOM_Jumper JP1
 U 1 1 5C31B4FD
-P 9900 5150
-F 0 "JP1" H 10064 5224 50  0000 L CNN
-F 1 "BOM_Jumper" H 10064 5132 50  0000 L CNN
-F 2 "AXTEC:Empty_Footprint" H 9900 5250 50  0001 C CNN
-F 3 "" H 9900 5250 50  0001 C CNN
-F 4 "M7581-05" H 10064 5040 50  0000 L CNN "Manufacturer Part Number"
-	1    9900 5150
+P 5300 3100
+F 0 "JP1" H 5464 3174 50  0000 L CNN
+F 1 "BOM_Jumper" H 5464 3082 50  0000 L CNN
+F 2 "AXTEC:Empty_Footprint" H 5300 3200 50  0001 C CNN
+F 3 "" H 5300 3200 50  0001 C CNN
+F 4 "M7581-05" H 5464 2990 50  0000 L CNN "Manufacturer Part Number"
+	1    5300 3100
 	1    0    0    -1
 $EndComp

Commit message: Agregado boton de reset para Arduino en PCB_D
Parts:
- added SW1: Reset Switch, Button_Switch_THT:SW_PUSH_6mm, symbol Switch:SW_Push
Connections:
- wire segments 136 -> 139
Changed lines of the file:
@@
 	1    0    0    -1
 $EndComp
+$Comp
+L Switch:SW_Push SW1
+U 1 1 5BE70135
+P 4650 4500
+F 0 "SW1" H 4650 4787 50  0000 C CNN
+F 1 "Reset Switch" H 4650 4695 50  0000 C CNN
+F 2 "Button_Switch_THT:SW_PUSH_6mm" H 4650 4700 50  0001 C CNN
+F 3 "" H 4650 4700 50  0001 C CNN
+F 4 "FSM18JH" H 4650 4500 50  0001 C CNN "Manufacturer Part Number"
+	1    4650 4500
+	1    0    0    -1
+$EndComp
+Text Label 4200 4500 0    50   ~ 0
+RST
+Wire Wire Line
+	4450 4500 4200 4500
+$Comp
+L power:GND #PWR?
+U 1 1 5BE769FE
+P 5050 4600
+F 0 "#PWR?" H 5050 4350 50  0001 C CNN
+F 1 "GND" H 5054 4426 50  0000 C CNN
+F 2 "" H 5050 4600 50  0001 C CNN
+F 3 "" H 5050 4600 50  0001 C CNN
+	1    5050 4600
+	1    0    0    -1
+$EndComp
+Wire Wire Line
+	4850 4500 5050 4500
+Wire Wire Line
+	5050 4500 5050 4600
 $EndSCHEMATC

Commit message: Encapsulado 0603 en lugar de 0805 para las resistencias en PCB_D
Parts:
- R1, R2, R3: footprint Resistor_SMD:R_0805_2012Metric_Pad1.15x1.40mm_HandSolder -> Resistor_SMD:R_0603_1608Metric_Pad1.05x0.95mm_HandSolder
Changed lines of the file:
@@
 F 0 "R3" V 3850 6400 50  0000 C CNN
 F 1 "1k" V 3634 6400 50  0000 C CNN
-F 2 "Resistor_SMD:R_0805_2012Metric_Pad1.15x1.40mm_HandSolder" V 3680 6400 50  0001 C CNN
+F 2 "Resistor_SMD:R_0603_1608Metric_Pad1.05x0.95mm_HandSolder" V 3680 6400 50  0001 C CNN
 F 3 "~" H 3750 6400 50  0001 C CNN
 F 4 "RC0603JR-071KL" V 3750 6400 50  0001 C CNN "Manufacturer Part Number"
@@
 F 0 "R2" H 3530 5954 50  0000 R CNN
 F 1 "10k" H 3530 6046 50  0000 R CNN
-F 2 "Resistor_SMD:R_0805_2012Metric_Pad1.15x1.40mm_HandSolder" V 3530 6000 50  0001 C CNN
+F 2 "Resistor_SMD:R_0603_1608Metric_Pad1.05x0.95mm_HandSolder" V 3530 6000 50  0001 C CNN
 F 3 "~" H 3600 6000 50  0001 C CNN
 F 4 "RC0603JR-0710KL" H 3600 6000 50  0001 C CNN "Manufacturer Part Number"
@@
 F 0 "R1" V 3550 6500 50  0000 C CNN
 F 1 "1k" V 3334 6500 50  0000 C CNN
-F 2 "Resistor_SMD:R_0805_2012Metric_Pad1.15x1.40mm_HandSolder" V 3380 6500 50  0001 C CNN
+F 2 "Resistor_SMD:R_0603_1608Metric_Pad1.05x0.95mm_HandSolder" V 3380 6500 50  0001 C CNN
 F 3 "~" H 3450 6500 50  0001 C CNN
 F 4 "RC0603JR-071KL" V 3450 6500 50  0001 C CNN "Manufacturer Part Number"
@@
 	4450 4500 4200 4500
 $Comp
-L power:GND #PWR?
+L power:GND #PWR0101
 U 1 1 5BE769FE
 P 5050 4600
-F 0 "#PWR?" H 5050 4350 50  0001 C CNN
+F 0 "#PWR0101" H 5050 4350 50  0001 C CNN
 F 1 "GND" H 5054 4426 50  0000 C CNN
 F 2 "" H 5050 4600 50  0001 C CNN

Commit message: Agregado TPD2E2U06 a PCB D
Parts:
- added U4: TPD2E2U06, SamacSys_Parts:SOT95P280X100-5N, symbol Power_Protection:TPD2E2U06
Connections:
- net labels added: D+, D-
- wire segments 139 -> 142
Changed lines of the file:
@@
 Wire Wire Line
 	5050 4500 5050 4600
+$Comp
+L Power_Protection:TPD2E2U06 U4
+U 1 1 5BE4E800
+P 10150 3750
+F 0 "U4" H 10400 3850 50  0000 L CNN
+F 1 "TPD2E2U06" H 10400 3750 50  0000 L CNN
+F 2 "SamacSys_Parts:SOT95P280X100-5N" H 9350 3500 50  0001 C CNN
+F 3 "http://www.ti.com/lit/ds/symlink/tpd2e2u06.pdf" H 9950 3950 50  0001 C CNN
+	1    10150 3750
+	1    0    0    -1
+$EndComp
+$Comp
+L power:GND #PWR022
+U 1 1 5BE4E903
+P 10150 4100
+F 0 "#PWR022" H 10150 3850 50  0001 C CNN
+F 1 "GND" H 10154 3926 50  0000 C CNN
+F 2 "" H 10150 4100 50  0001 C CNN
+F 3 "" H 10150 4100 50  0001 C CNN
+	1    10150 4100
+	1    0    0    -1
+$EndComp
+Wire Wire Line
+	10150 4100 10150 4050
+Text Label 9650 2700 0    50   ~ 0
+D+
+Text Label 9650 2800 0    50   ~ 0
+D-
+Wire Wire Line
+	9850 3650 9700 3650
+Wire Wire Line
+	9850 3850 9700 3850
+Text Label 9700 3850 0    50   ~ 0
+D+
+Text Label 9700 3650 0    50   ~ 0
+D-
 $EndSCHEMATC
