File: Hardware/Satelite/PCB_E/PCB_E.kicad_pcb (KiCad board)
At the start: 2 copper layers, 47 x 47 mm, 16 parts, among them J1 Conn_02x02_Counter_Clockwise, J10 Conn_02x04_Odd_Even, J11 Conn_02x04_Odd_Even, J12 Conector_Expansion_CanSat, J13 Conn_01x06, J14 Conn_01x06, J15 Conn_01x06, J2 Conn_02x02_Counter_Clockwise, J3 Conn_02x02_Counter_Clockwise, J4 Conn_02x04_Odd_Even, J5 Conn_02x04_Odd_Even, J6 Conn_02x04_Odd_Even, J7 Conn_02x04_Odd_Even, J8 Conn_02x04_Odd_Even, J9 Conn_02x04_Odd_Even

Commit message: PCB_E corregido
Parts:
- moved J15 1.56 mm to (-13.5, -6.35)
- moved J10 0.50 mm to (-2.45, 7.75)
- moved J11 0.50 mm to (-7.66, 7.75)
- moved J5 0.50 mm to (-5.03, -0.63)
- moved J6 0.50 mm to (7.95, 7.75)
- moved J7 0.50 mm to (0.17, -0.63)
- moved J8 0.50 mm to (2.75, 7.75)
- moved J9 0.50 mm to (5.37, -0.63)
- moved J4 0.50 mm to (-10.2, -0.65)
Connections:
- J12 pad 13: /MOSI -> +BATT
- J12 pad 14: /MISO -> +3V3
- J12 pad 15: /SCK -> +5V
- J12 pad 16: /SS -> GND
- J12 pad 17: /SCL -> GND
- J12 pad 18: /SDA -> GND
- J12 pad 19: +BATT -> /MOSI
- J12 pad 20: +3V3 -> /MISO
- J12 pad 21: +5V -> /SCK
- J12 pad 22: GND -> /SS
- J12 pad 23: GND -> /SCL
- J12 pad 24: GND -> /SDA
Routing:
- net /SCK: track 3.70 -> 14.4 mm
- net /MISO: track 3.70 -> 14.4 mm
- net /SS: track 3.70 -> 13.7 mm
- net /SDA: track 3.70 -> 13.7 mm
- net /SCL: track 3.70 -> 13.7 mm
- net /MOSI: track 3.70 -> 13.7 mm
- net +5V: track 42.6 -> 37.4 mm
- net +3V3: track 32.5 -> 29.7 mm
- net +BATT: track 30.4 -> 28.5 mm
- net GND: track 126.2 -> 125.6 mm
Other:
- net class Alimentacion: trace_width 0.8 -> 0.6
