File: Hardware/Satelite/PCB_E/PCB_E.sch (KiCad schematic (older format))
At the start: 29 parts, among them J1 Conn_02x14_Odd_Even, J10 Conn_02x05_Counter_Clockwise, J11 Conn_02x05_Counter_Clockwise, J12 Conn_02x05_Counter_Clockwise, J13 Conn_02x05_Counter_Clockwise, J14 Conn_02x05_Counter_Clockwise, J15 Conn_02x05_Counter_Clockwise, J16 Conn_01x08, J17 Conn_01x04, J18 Conn_01x04, J19 Conn_01x02, J2 Conn_02x14_Odd_Even, J20 Conn_02x02_Counter_Clockwise, J21 Conn_02x02_Counter_Clockwise, J22 Conn_02x02_Counter_Clockwise, J23 Conn_02x02_Counter_Clockwise, J24 Conn_02x02_Counter_Clockwise, J25 Conn_02x02_Counter_Clockwise, J26 Conn_02x02_Counter_Clockwise, J3 Conn_02x14_Odd_Even, J4 Conn_02x05_Counter_Clockwise, J5 Conn_02x05_Counter_Clockwise, J6 Conn_02x05_Counter_Clockwise, J7 Conn_02x05_Counter_Clockwise, J8 Conn_02x05_Counter_Clockwise, J9 Conn_02x05_Counter_Clockwise

Commit message: PCB_E modificado conector de expansion y PCB WIP
Parts:
- removed J1, J2, J3: Conn_02x14_Odd_Even, Connector_PinHeader_2.54mm:PinHeader_2x14_P2.54mm_Vertical, symbol Connector_Generic:Conn_02x14_Odd_Even
- removed J10, J11, J12, J13, J14, J15, J4, J5, J6, J7, J8, J9: Conn_02x05_Counter_Clockwise, Connector_PinSocket_2.54mm:PinSocket_2x05_P2.54mm_Vertical, symbol Connector_Generic:Conn_02x05_Counter_Clockwise
- removed J16: Conn_01x08, Connector_PinHeader_2.54mm:PinHeader_1x08_P2.54mm_Vertical, symbol Connector_Generic:Conn_01x08
- removed J17, J18: Conn_01x04, Connector_PinHeader_2.54mm:PinHeader_1x04_P2.54mm_Vertical, symbol Connector_Generic:Conn_01x04
- removed J19: Conn_01x02, Connector_PinHeader_2.54mm:PinHeader_1x02_P2.54mm_Vertical, symbol Connector_Generic:Conn_01x02
- removed J20, J21, J22, J23, J24, J25, J26: Conn_02x02_Counter_Clockwise, Connector_PinHeader_2.54mm:PinHeader_2x02_P2.54mm_Vertical, symbol Connector_Generic:Conn_02x02_Counter_Clockwise
- added J1, J2, J3: Conn_02x02_Counter_Clockwise, Connector_PinSocket_2.54mm:PinSocket_2x02_P2.54mm_Vertical, symbol Connector_Generic:Conn_02x02_Counter_Clockwise
- added J10, J11, J4, J5, J6, J7, J8, J9: Conn_02x04_Odd_Even, Connector_PinSocket_2.54mm:PinSocket_2x04_P2.54mm_Vertical, symbol Connector_Generic:Conn_02x04_Odd_Even
- added J12, J13, J14, J15, J16, J17, J18: Conn_01x06, Connector_PinHeader_2.54mm:PinHeader_1x06_P2.54mm_Vertical, symbol Connector_Generic:Conn_01x06
Connections:
- net labels added: SCK, SS
- net labels removed: CS, SCLK
- wire segments 263 -> 124

Commit message: Mejoras en esquematico PCB_E
Other:
- note added: "Alimentación\n"
- note added: "Conectores internos"
- note added: "Conexiones Auxiliares\n"
- note added: "Montaje"
- moved on the sheet: J1, J12, J13, J14, J15, J16, J17, J18, J2, J3

Commit message: PCB_E terminado
Parts:
- removed J14, J16, J17, J18: Conn_01x06, Connector_PinHeader_2.54mm:PinHeader_1x06_P2.54mm_Vertical, symbol Connector_Generic:Conn_01x06
- removed MH1, MH2, MH3: MountingHole_Pad, MountingHole:MountingHole_3.2mm_M3_Pad, symbol Mechanical:MountingHole_Pad
- added J12: Conector_Expansion_CanSat, AXTEC:Conector_Expansion_CanSat, symbol AXTEC_IC:Conector_Expansion_CanSat
- renumbered J12 to J13, J15 to J14, J13 to J15
Connections:
- wire segments 124 -> 125
Other:
- note added: "Conector de expansión\n"
- note removed: "Conector de expansión"
- note removed: "Montaje"
- moved on the sheet: J1, J13, J14, J15, J2, J3

Commit message: PCB_E con  MH_CanSat y Conector externo nuevo
Parts:
- added MH1: MH_CanSat, AXTEC:MH_CanSat, symbol AXTEC_IC:MH_CanSat
Other:
- note added: "Agujeros de montaje"
Changed lines of the file:
@@
 Text Label 9450 2700 0    50   ~ 0
 AD3
-$Comp
-L AXTEC_IC:Conector_Expansion_CanSat J12
-U 1 1 5BC5ED90
-P 8750 1900
-F 0 "J12" H 8800 2750 50  0000 C CNN
-F 1 "Conector_Expansion_CanSat" H 8750 2650 50  0000 C CNN
-F 2 "AXTEC:Conector_Expansion_CanSat" H 8750 2400 50  0001 C CNN
-F 3 "" H 8750 2400 50  0001 C CNN
-	1    8750 1900
-	1    0    0    -1
-$EndComp
 Text Label 7900 1350 0    50   ~ 0
 MOSI
@@
 	8100 1350 7900 1350
 $Comp
-L power:+BATT #PWR09
+L power:+BATT #PWR010
 U 1 1 5BC88F35
 P 7650 2050
-F 0 "#PWR09" H 7650 1900 50  0001 C CNN
+F 0 "#PWR010" H 7650 1900 50  0001 C CNN
 F 1 "+BATT" H 7664 2225 50  0000 C CNN
 F 2 "" H 7650 2050 50  0001 C CNN
@@
 $EndComp
 $Comp
-L power:+3V3 #PWR08
+L power:+3V3 #PWR09
 U 1 1 5BC88F45
 P 7400 2050
-F 0 "#PWR08" H 7400 1900 50  0001 C CNN
+F 0 "#PWR09" H 7400 1900 50  0001 C CNN
 F 1 "+3V3" H 7414 2225 50  0000 C CNN
 F 2 "" H 7400 2050 50  0001 C CNN
@@
 $EndComp
 $Comp
-L power:+5V #PWR07
+L power:+5V #PWR08
 U 1 1 5BC88F4D
 P 7150 2050
-F 0 "#PWR07" H 7150 1900 50  0001 C CNN
+F 0 "#PWR08" H 7150 1900 50  0001 C CNN
 F 1 "+5V" H 7164 2225 50  0000 C CNN
 F 2 "" H 7150 2050 50  0001 C CNN
@@
 $EndComp
 $Comp
-L power:GND #PWR010
+L power:GND #PWR011
 U 1 1 5BC88F55
 P 8000 2800
-F 0 "#PWR010" H 8000 2550 50  0001 C CNN
+F 0 "#PWR011" H 8000 2550 50  0001 C CNN
 F 1 "GND" H 8004 2626 50  0000 C CNN
 F 2 "" H 8000 2800 50  0001 C CNN
@@
 	8000 2700 8000 2600
 $Comp
-L power:GND #PWR011
+L power:GND #PWR07
 U 1 1 5BC9E797
-P 8750 3050
-F 0 "#PWR011" H 8750 2800 50  0001 C CNN
-F 1 "GND" H 8754 2876 50  0000 C CNN
-F 2 "" H 8750 3050 50  0001 C CNN
-F 3 "" H 8750 3050 50  0001 C CNN
-	1    8750 3050
+P 5250 4850
+F 0 "#PWR07" H 5250 4600 50  0001 C CNN
+F 1 "GND" H 5254 4676 50  0000 C CNN
+F 2 "" H 5250 4850 50  0001 C CNN
+F 3 "" H 5250 4850 50  0001 C CNN
+	1    5250 4850
 	1    0    0    -1
 $EndComp
-Wire Wire Line
-	8650 2950 8650 3000
-Wire Wire Line
-	8650 3000 8750 3000
-Wire Wire Line
-	8850 3000 8850 2950
-Wire Wire Line
-	8750 2950 8750 3000
-Connection ~ 8750 3000
-Wire Wire Line
-	8750 3000 8850 3000
-Wire Wire Line
-	8750 3050 8750 3000
 Wire Wire Line
 	7650 2050 8100 2050
@@
 Text Label 9650 4700 0    50   ~ 0
 IO7
+$Comp
+L AXTEC_IC:Conector_Expansion_CanSat J12
+U 1 1 5BC62CAE
+P 8750 1900
+F 0 "J12" H 9143 2765 50  0000 C CNN
+F 1 "Conector_Expansion_CanSat" H 9143 2674 50  0000 C CNN
+F 2 "AXTEC:Conector_Expansion_CanSat" H 8750 2400 50  0001 C CNN
+F 3 "" H 8750 2400 50  0001 C CNN
+	1    8750 1900
+	1    0    0    -1
+$EndComp
+$Comp
+L AXTEC_IC:MH_CanSat MH1
+U 1 1 5BC69FBC
+P 5250 4650
+F 0 "MH1" H 5528 4765 50  0000 L CNN
+F 1 "MH_CanSat" H 5528 4674 50  0000 L CNN
+F 2 "AXTEC:MH_CanSat" H 5250 4650 50  0001 C CNN
+F 3 "" H 5250 4650 50  0001 C CNN
+	1    5250 4650
+	1    0    0    -1
+$EndComp
+Wire Wire Line
+	5100 4750 5100 4800
+Wire Wire Line
+	5100 4800 5250 4800
+Wire Wire Line
+	5400 4800 5400 4750
+Wire Wire Line
+	5250 4750 5250 4800
+Connection ~ 5250 4800
+Wire Wire Line
+	5250 4800 5400 4800
+Wire Wire Line
+	5250 4850 5250 4800
+Wire Notes Line
+	4150 3900 4150 5200
+Wire Notes Line
+	4150 5200 6450 5200
+Wire Notes Line
+	6450 5200 6450 3900
+Wire Notes Line
+	6450 3900 4150 3900
+Text Notes 4450 4150 0    118  ~ 0
+Agujeros de montaje
 $EndSCHEMATC

Commit message: PCB_E corregido
Changed lines of the file:
@@
 Text Label 9450 2700 0    50   ~ 0
 AD3
-Text Label 7900 1350 0    50   ~ 0
+Text Label 7850 2250 0    50   ~ 0
 MOSI
-Text Label 7900 1450 0    50   ~ 0
+Text Label 7850 2350 0    50   ~ 0
 MISO
-Text Label 7900 1550 0    50   ~ 0
+Text Label 7850 2450 0    50   ~ 0
 SCK
-Text Label 7900 1650 0    50   ~ 0
+Text Label 7850 2550 0    50   ~ 0
 SS
-Text Label 7900 1750 0    50   ~ 0
+Text Label 7850 2650 0    50   ~ 0
 SCL
-Text Label 7900 1850 0    50   ~ 0
+Text Label 7850 2750 0    50   ~ 0
 SDA
-Wire Wire Line
-	8100 1850 7900 1850
-Wire Wire Line
-	8100 1750 7900 1750
-Wire Wire Line
-	8100 1650 7900 1650
-Wire Wire Line
-	8100 1550 7900 1550
-Wire Wire Line
-	8100 1450 7900 1450
-Wire Wire Line
-	8100 1350 7900 1350
 $Comp
-L power:+BATT #PWR010
+L power:+BATT #PWR011
 U 1 1 5BC88F35
+P 8000 1400
+F 0 "#PWR011" H 8000 1250 50  0001 C CNN
+F 1 "+BATT" H 8014 1575 50  0000 C CNN
+F 2 "" H 8000 1400 50  0001 C CNN
+F 3 "" H 8000 1400 50  0001 C CNN
+	1    8000 1400
+	1    0    0    -1
+$EndComp
+$Comp
+L power:+3V3 #PWR010
+U 1 1 5BC88F45
+P 7750 1400
+F 0 "#PWR010" H 7750 1250 50  0001 C CNN
+F 1 "+3V3" H 7764 1575 50  0000 C CNN
+F 2 "" H 7750 1400 50  0001 C CNN
+F 3 "" H 7750 1400 50  0001 C CNN
+	1    7750 1400
+	1    0    0    -1
+$EndComp
+$Comp
+L power:+5V #PWR08
+U 1 1 5BC88F4D
+P 7500 1400
+F 0 "#PWR08" H 7500 1250 50  0001 C CNN
+F 1 "+5V" H 7514 1575 50  0000 C CNN
+F 2 "" H 7500 1400 50  0001 C CNN
+F 3 "" H 7500 1400 50  0001 C CNN
+	1    7500 1400
+	1    0    0    -1
+$EndComp
+$Comp
+L power:GND #PWR09
+U 1 1 5BC88F55
 P 7650 2050
-F 0 "#PWR010" H 7650 1900 50  0001 C CNN
-F 1 "+BATT" H 7664 2225 50  0000 C CNN
+F 0 "#PWR09" H 7650 1800 50  0001 C CNN
+F 1 "GND" H 7654 1876 50  0000 C CNN
 F 2 "" H 7650 2050 50  0001 C CNN
 F 3 "" H 7650 2050 50  0001 C CNN
@@
 	1    0    0    -1
 $EndComp
-$Comp
-L power:+3V3 #PWR09
-U 1 1 5BC88F45
-P 7400 2050
-F 0 "#PWR09" H 7400 1900 50  0001 C CNN
-F 1 "+3V3" H 7414 2225 50  0000 C CNN
-F 2 "" H 7400 2050 50  0001 C CNN
-F 3 "" H 7400 2050 50  0001 C CNN
-	1    7400 2050
-	1    0    0    -1
-$EndComp
-$Comp
-L power:+5V #PWR08
-U 1 1 5BC88F4D
-P 7150 2050
-F 0 "#PWR08" H 7150 1900 50  0001 C CNN
-F 1 "+5V" H 7164 2225 50  0000 C CNN
-F 2 "" H 7150 2050 50  0001 C CNN
-F 3 "" H 7150 2050 50  0001 C CNN
-	1    7150 2050
-	1    0    0    -1
-$EndComp
-$Comp
-L power:GND #PWR011
-U 1 1 5BC88F55
-P 8000 2800
-F 0 "#PWR011" H 8000 2550 50  0001 C CNN
-F 1 "GND" H 8004 2626 50  0000 C CNN
-F 2 "" H 8000 2800 50  0001 C CNN
-F 3 "" H 8000 2800 50  0001 C CNN
-	1    8000 2800
-	1    0    0    -1
-$EndComp
-Wire Wire Line
-	8000 2800 8000 2700
-Wire Wire Line
-	8000 2500 8100 2500
-Wire Wire Line
-	8100 2600 8000 2600
-Connection ~ 8000 2600
-Wire Wire Line
-	8000 2600 8000 2500
-Wire Wire Line
-	8100 2700 8000 2700
-Connection ~ 8000 2700
-Wire Wire Line
-	8000 2700 8000 2600
 $Comp
 L power:GND #PWR07
@@
 $EndComp
 Wire Wire Line
-	7650 2050 8100 2050
+	7750 1500 7750 1400
 Wire Wire Line
-	8100 2150 7400 2150
-Wire Wire Line
-	7400 2150 7400 2050
-Wire Wire Line
-	8100 2250 7150 2250
-Wire Wire Line
-	7150 2250 7150 2050
+	7500 1600 7500 1400
 Wire Wire Line
 	9400 1350 9600 1350
@@
 IO7
 $Comp
-L AXTEC_IC:Conector_Expansion_CanSat J12
-U 1 1 5BC62CAE
-P 8750 1900
-F 0 "J12" H 9143 2765 50  0000 C CNN
-F 1 "Conector_Expansion_CanSat" H 9143 2674 50  0000 C CNN
-F 2 "AXTEC:Conector_Expansion_CanSat" H 8750 2400 50  0001 C CNN
-F 3 "" H 8750 2400 50  0001 C CNN
-	1    8750 1900
-	1    0    0    -1
-$EndComp
-$Comp
 L AXTEC_IC:MH_CanSat MH1
 U 1 1 5BC69FBC
@@
 Text Notes 4450 4150 0    118  ~ 0
 Agujeros de montaje
+$Comp
+L AXTEC_IC:Conector_Expansion_CanSat J12
+U 1 1 5BC6ED70
+P 8750 1900
+F 0 "J12" H 9143 2765 50  0000 C CNN
+F 1 "Conector_Expansion_CanSat" H 9143 2674 50  0000 C CNN
+F 2 "AXTEC:Conector_Expansion_CanSat" H 8750 2400 50  0001 C CNN
+F 3 "" H 8750 2400 50  0001 C CNN
+	1    8750 1900
+	1    0    0    -1
+$EndComp
+Wire Wire Line
+	8100 2750 7850 2750
+Wire Wire Line
+	8100 2650 7850 2650
+Wire Wire Line
+	8100 2550 7850 2550
+Wire Wire Line
+	8100 2450 7850 2450
+Wire Wire Line
+	8100 2350 7850 2350
+Wire Wire Line
+	7850 2250 8100 2250
+Wire Wire Line
+	8100 1400 8000 1400
+Wire Wire Line
+	8100 1500 7750 1500
+Wire Wire Line
+	8100 1600 7500 1600
+Wire Wire Line
+	7650 2050 8050 2050
+Wire Wire Line
+	8100 1850 8050 1850
+Wire Wire Line
+	8050 1850 8050 1950
+Connection ~ 8050 2050
+Wire Wire Line
+	8050 2050 8100 2050
+Wire Wire Line
+	8100 1950 8050 1950
+Connection ~ 8050 1950
+Wire Wire Line
+	8050 1950 8050 2050
 $EndSCHEMATC

Commit message: Numeros de parte para PCB_E
Parts:
- added M1, M2, M3: Spacer, AXTEC:Empty_Footprint, symbol AXTEC_IC:Spacer
- J12: Manufacturer Part Number (none) -> SSQ-106-03-T-S; Quantity (none) -> 4
Other:
- moved on the sheet: J12
Changed lines of the file:
@@
 Text Label 9650 4100 0    50   ~ 0
 IO5
-Text Label 9450 1950 0    50   ~ 0
+Text Label 9450 2150 0    50   ~ 0
 IO6
 Wire Wire Line
@@
 Wire Wire Line
 	9600 5100 10050 5100
-Text Label 9450 2050 0    50   ~ 0
+Text Label 9450 2250 0    50   ~ 0
 IO7
 Text Label 9650 4800 0    50   ~ 0
@@
 EndData
 $EndBitmap
-Text Label 9450 1350 0    50   ~ 0
+Text Label 9450 1550 0    50   ~ 0
 IO0
-Text Label 9450 1450 0    50   ~ 0
+Text Label 9450 1650 0    50   ~ 0
 IO1
-Text Label 9450 1550 0    50   ~ 0
+Text Label 9450 1750 0    50   ~ 0
 IO2
-Text Label 9450 1650 0    50   ~ 0
+Text Label 9450 1850 0    50   ~ 0
 IO3
-Text Label 9450 1750 0    50   ~ 0
+Text Label 9450 1950 0    50   ~ 0
 IO4
-Text Label 9450 1850 0    50   ~ 0
+Text Label 9450 2050 0    50   ~ 0
 IO5
-Text Label 9450 2400 0    50   ~ 0
+Text Label 9450 2600 0    50   ~ 0
 AD0
-Text Label 9450 2500 0    50   ~ 0
+Text Label 9450 2700 0    50   ~ 0
 AD1
-Text Label 9450 2600 0    50   ~ 0
+Text Label 9450 2800 0    50   ~ 0
 AD2
-Text Label 9450 2700 0    50   ~ 0
+Text Label 9450 2900 0    50   ~ 0
 AD3
-Text Label 7850 2250 0    50   ~ 0
+Text Label 7850 2450 0    50   ~ 0
 MOSI
-Text Label 7850 2350 0    50   ~ 0
+Text Label 7850 2550 0    50   ~ 0
 MISO
-Text Label 7850 2450 0    50   ~ 0
+Text Label 7850 2650 0    50   ~ 0
 SCK
-Text Label 7850 2550 0    50   ~ 0
+Text Label 7850 2750 0    50   ~ 0
 SS
-Text Label 7850 2650 0    50   ~ 0
+Text Label 7850 2850 0    50   ~ 0
 SCL
-Text Label 7850 2750 0    50   ~ 0
+Text Label 7850 2950 0    50   ~ 0
 SDA
 $Comp
 L power:+BATT #PWR011
 U 1 1 5BC88F35
-P 8000 1400
-F 0 "#PWR011" H 8000 1250 50  0001 C CNN
-F 1 "+BATT" H 8014 1575 50  0000 C CNN
-F 2 "" H 8000 1400 50  0001 C CNN
-F 3 "" H 8000 1400 50  0001 C CNN
-	1    8000 1400
+P 8000 1600
+F 0 "#PWR011" H 8000 1450 50  0001 C CNN
+F 1 "+BATT" H 8014 1775 50  0000 C CNN
+F 2 "" H 8000 1600 50  0001 C CNN
+F 3 "" H 8000 1600 50  0001 C CNN
+	1    8000 1600
 	1    0    0    -1
 $EndComp
@@
 L power:+3V3 #PWR010
 U 1 1 5BC88F45
-P 7750 1400
-F 0 "#PWR010" H 7750 1250 50  0001 C CNN
-F 1 "+3V3" H 7764 1575 50  0000 C CNN
-F 2 "" H 7750 1400 50  0001 C CNN
-F 3 "" H 7750 1400 50  0001 C CNN
-	1    7750 1400
+P 7750 1600
+F 0 "#PWR010" H 7750 1450 50  0001 C CNN
+F 1 "+3V3" H 7764 1775 50  0000 C CNN
+F 2 "" H 7750 1600 50  0001 C CNN
+F 3 "" H 7750 1600 50  0001 C CNN
+	1    7750 1600
 	1    0    0    -1
 $EndComp
@@
 L power:+5V #PWR08
 U 1 1 5BC88F4D
-P 7500 1400
-F 0 "#PWR08" H 7500 1250 50  0001 C CNN
-F 1 "+5V" H 7514 1575 50  0000 C CNN
-F 2 "" H 7500 1400 50  0001 C CNN
-F 3 "" H 7500 1400 50  0001 C CNN
-	1    7500 1400
+P 7500 1600
+F 0 "#PWR08" H 7500 1450 50  0001 C CNN
+F 1 "+5V" H 7514 1775 50  0000 C CNN
+F 2 "" H 7500 1600 50  0001 C CNN
+F 3 "" H 7500 1600 50  0001 C CNN
+	1    7500 1600
 	1    0    0    -1
 $EndComp
@@
 L power:GND #PWR09
 U 1 1 5BC88F55
-P 7650 2050
-F 0 "#PWR09" H 7650 1800 50  0001 C CNN
-F 1 "GND" H 7654 1876 50  0000 C CNN
-F 2 "" H 7650 2050 50  0001 C CNN
-F 3 "" H 7650 2050 50  0001 C CNN
-	1    7650 2050
+P 7650 2250
+F 0 "#PWR09" H 7650 2000 50  0001 C CNN
+F 1 "GND" H 7654 2076 50  0000 C CNN
+F 2 "" H 7650 2250 50  0001 C CNN
+F 3 "" H 7650 2250 50  0001 C CNN
+	1    7650 2250
 	1    0    0    -1
 $EndComp
@@
 $EndComp
 Wire Wire Line
-	7750 1500 7750 1400
-Wire Wire Line
-	7500 1600 7500 1400
-Wire Wire Line
-	9400 1350 9600 1350
-Wire Wire Line
-	9400 1450 9600 1450
+	7750 1700 7750 1600
+Wire Wire Line
+	7500 1800 7500 1600
 Wire Wire Line
 	9400 1550 9600 1550
@@
 	9400 2050 9600 2050
 Wire Wire Line
-	9400 2400 9600 2400
-Wire Wire Line
-	9400 2500 9600 2500
+	9400 2150 9600 2150
+Wire Wire Line
+	9400 2250 9600 2250
 Wire Wire Line
 	9400 2600 9600 2600
 Wire Wire Line
 	9400 2700 9600 2700
+Wire Wire Line
+	9400 2800 9600 2800
+Wire Wire Line
+	9400 2900 9600 2900
 Text Notes 7750 950  0    118  ~ 0
 Conector de expansión\n
@@
 	5250 4850 5250 4800
 Wire Notes Line
-	4150 3900 4150 5200
-Wire Notes Line
-	4150 5200 6450 5200
-Wire Notes Line
-	6450 5200 6450 3900
+	4150 3900 4150 5900
+Wire Notes Line
+	4150 5900 6450 5900
+Wire Notes Line
+	6450 5900 6450 3900
 Wire Notes Line
 	6450 3900 4150 3900
@@
 L AXTEC_IC:Conector_Expansion_CanSat J12
 U 1 1 5BC6ED70
-P 8750 1900
-F 0 "J12" H 9143 2765 50  0000 C CNN
-F 1 "Conector_Expansion_CanSat" H 9143 2674 50  0000 C CNN
-F 2 "AXTEC:Conector_Expansion_CanSat" H 8750 2400 50  0001 C CNN
-F 3 "" H 8750 2400 50  0001 C CNN
-	1    8750 1900
-	1    0    0    -1
-$EndComp
+P 8750 2100
+F 0 "J12" H 8300 3000 50  0000 C CNN
+F 1 "Conector_Expansion_CanSat" H 8750 2900 50  0000 C CNN
+F 2 "AXTEC:Conector_Expansion_CanSat" H 8750 2600 50  0001 C CNN
+F 3 "" H 8750 2600 50  0001 C CNN
+F 4 "SSQ-106-03-T-S" H 8750 2100 50  0001 C CNN "Manufacturer Part Number"
+F 5 "4" H 8750 2100 50  0001 C CNN "Quantity"
+	1    8750 2100
+	1    0    0    -1
+$EndComp
+Wire Wire Line
+	8100 2950 7850 2950
+Wire Wire Line
+	8100 2850 7850 2850
 Wire Wire Line
 	8100 2750 7850 2750
@@
 	8100 2550 7850 2550
 Wire Wire Line
-	8100 2450 7850 2450
-Wire Wire Line
-	8100 2350 7850 2350
-Wire Wire Line
-	7850 2250 8100 2250
-Wire Wire Line
-	8100 1400 8000 1400
-Wire Wire Line
-	8100 1500 7750 1500
-Wire Wire Line
-	8100 1600 7500 1600
-Wire Wire Line
-	7650 2050 8050 2050
-Wire Wire Line
-	8100 1850 8050 1850
-Wire Wire Line
-	8050 1850 8050 1950
-Connection ~ 8050 2050
-Wire Wire Line
-	8050 2050 8100 2050
-Wire Wire Line
-	8100 1950 8050 1950
-Connection ~ 8050 1950
-Wire Wire Line
-	8050 1950 8050 2050
+	7850 2450 8100 2450
+Wire Wire Line
+	8100 1600 8000 1600
+Wire Wire Line
+	8100 1700 7750 1700
+Wire Wire Line
+	8100 1800 7500 1800
+Wire Wire Line
+	7650 2250 8050 2250
+Wire Wire Line
+	8100 2050 8050 2050
+Wire Wire Line
+	8050 2050 8050 2150
+Connection ~ 8050 2250
+Wire Wire Line
+	8050 2250 8100 2250
+Wire Wire Line
+	8100 2150 8050 2150
+Connection ~ 8050 2150
+Wire Wire Line
+	8050 2150 8050 2250
+$Comp
+L AXTEC_IC:Spacer M1
+U 1 1 5C332544
+P 4400 5450
+F 0 "M1" H 4479 5443 50  0000 L CNN
+F 1 "Spacer" H 4479 5351 50  0000 L CNN
+F 2 "AXTEC:Empty_Footprint" H 4300 5600 50  0001 C CNN
+F 3 "https://www.mouser.com/datasheet/2/181/R30-301-1135805.pdf" H 4400 5700 50  0001 C CNN
+F 4 "R30-3011002" H 4479 5305 50  0001 L CNN "Manufacturer Part Number"
+	1    4400 5450
+	1    0    0    -1
+$EndComp
+$Comp
+L AXTEC_IC:Spacer M2
+U 1 1 5C332635
+P 5250 5450
+F 0 "M2" H 5329 5443 50  0000 L CNN
+F 1 "Spacer" H 5329 5351 50  0000 L CNN
+F 2 "AXTEC:Empty_Footprint" H 5150 5600 50  0001 C CNN
+F 3 "https://www.mouser.com/datasheet/2/181/R30-301-1135805.pdf" H 5250 5700 50  0001 C CNN
+F 4 "R30-3011002" H 5329 5305 50  0001 L CNN "Manufacturer Part Number"
+	1    5250 5450
+	1    0    0    -1
+$EndComp
+$Comp
+L AXTEC_IC:Spacer M3
+U 1 1 5C332687
+P 6000 5450
+F 0 "M3" H 6079 5443 50  0000 L CNN
+F 1 "Spacer" H 6079 5351 50  0000 L CNN
+F 2 "AXTEC:Empty_Footprint" H 5900 5600 50  0001 C CNN
+F 3 "https://www.mouser.com/datasheet/2/181/R30-301-1135805.pdf" H 6000 5700 50  0001 C CNN
+F 4 "R30-3011002" H 6079 5305 50  0001 L CNN "Manufacturer Part Number"
+	1    6000 5450
+	1    0    0    -1
+$EndComp
 $EndSCHEMATC

Commit message: Modificaciones en PCB_E y nuevas serigrafias
Parts:
- removed J10, J11, J4, J5, J6, J7, J8, J9: Conn_02x04_Odd_Even, Connector_PinSocket_2.54mm:PinSocket_2x04_P2.54mm_Vertical, symbol Connector_Generic:Conn_02x04_Odd_Even
- removed J13: Conn_01x06, Connector_PinHeader_2.54mm:PinHeader_1x06_P2.54mm_Vertical, symbol Connector_Generic:Conn_01x06
- added J4, J5, J6, J7: Conn_02x10_Odd_Even, Connector_PinSocket_2.54mm:PinSocket_2x10_P2.54mm_Vertical, symbol Connector_Generic:Conn_02x10_Odd_Even
- added J8: Conn_01x04, Connector_PinHeader_2.54mm:PinHeader_1x04_P2.54mm_Vertical, symbol Connector_Generic:Conn_01x04
Connections:
- wire segments 125 -> 75

Commit message: BOM y corrección de numero de partes en PCB_E
Parts:
- J14, J15: Manufacturer Part Number SSW-106-03-T-S -> (none)
Changed lines of the file:
@@
 F 2 "Connector_PinHeader_2.54mm:PinHeader_1x06_P2.54mm_Vertical" H 10250 5750 50  0001 C CNN
 F 3 "https://www.mouser.com/datasheet/2/527/ssw_sm-1370305.pdf" H 10250 5750 50  0001 C CNN
-F 4 "SSW-106-03-T-S" H 10250 5750 50  0001 C CNN "Manufacturer Part Number"
 	1    10250 5750
 	1    0    0    -1
@@
 F 2 "Connector_PinHeader_2.54mm:PinHeader_1x06_P2.54mm_Vertical" H 10250 4800 50  0001 C CNN
 F 3 "https://www.mouser.com/datasheet/2/527/ssw_sm-1370305.pdf" H 10250 4800 50  0001 C CNN
-F 4 "SSW-106-03-T-S" H 10250 4800 50  0001 C CNN "Manufacturer Part Number"
 	1    10250 4800
 	1    0    0    -1
