File: Hardware/Satelite/PCB_E/PCB_E.sch (KiCad schematic (older format))
At the start: 14 parts, among them J1 Conn_02x02_Counter_Clockwise, J12 Conector_Expansion_CanSat, J14 Conn_01x06, J15 Conn_01x06, J2 Conn_02x02_Counter_Clockwise, J3 Conn_02x02_Counter_Clockwise, J4 Conn_02x10_Odd_Even, J5 Conn_02x10_Odd_Even, J6 Conn_02x10_Odd_Even, J7 Conn_02x10_Odd_Even, M1 Spacer, M2 Spacer, M3 Spacer

Commit message: Añadida información faltante en rótulos de los esquemas
Parts:
- added J8: Conn_01x06, Connector_PinHeader_2.54mm:PinHeader_1x06_P2.54mm_Vertical, symbol Connector_Generic:Conn_01x06
Connections:
- wire segments 75 -> 77
Changed lines of the file:
@@
 encoding utf-8
 Sheet 1 1
-Title ""
-Date ""
-Rev ""
+Title "PCB_E"
+Date "2019-01-19"
+Rev "1.0.0"
 Comp ""
 Comment1 ""
@@
 Vbus
 $Comp
-L Graphic:Logo_Open_Hardware_Large #LOGO?
+L Graphic:Logo_Open_Hardware_Large #LOGO1
 U 1 1 5C333B8B
 P 1200 7200
-F 0 "#LOGO?" H 1200 7700 50  0001 C CNN
+F 0 "#LOGO1" H 1200 7700 50  0001 C CNN
 F 1 "Logo_Open_Hardware_Large" H 1200 6800 50  0001 C CNN
 F 2 "" H 1200 7200 50  0001 C CNN
@@
 	1    0    0    -1
 $EndComp
+$Comp
+L Connector_Generic:Conn_01x06 J8
+U 1 1 5C5B02DA
+P 10250 3800
+F 0 "J8" H 9850 3400 50  0000 L CNN
+F 1 "Conn_01x06" H 9850 3300 50  0000 L CNN
+F 2 "Connector_PinHeader_2.54mm:PinHeader_1x06_P2.54mm_Vertical" H 10250 3800 50  0001 C CNN
+F 3 "https://www.mouser.com/datasheet/2/527/ssw_sm-1370305.pdf" H 10250 3800 50  0001 C CNN
+	1    10250 3800
+	1    0    0    -1
+$EndComp
+Wire Wire Line
+	10050 4000 9600 4000
+Wire Wire Line
+	10050 4100 9600 4100
+Text Label 9650 4000 0    50   ~ 0
+IO4
+Text Label 9650 4100 0    50   ~ 0
+IO5
 $EndSCHEMATC
