File: Hardware/Satelite/PCB_C/PCB_C.sch (KiCad schematic (older format))
At the start: 52 parts

Commit message: Eliminado label no usado
Connections:
- net labels removed: EXT_IO7
Changed lines of the file:
@@
 Text Label 13750 4150 0    50   ~ 0
 EXT_IO6
-Text Label 13750 4050 0    50   ~ 0
-EXT_IO7
 Text Label 14400 4700 0    50   ~ 0
 EXT_SDO

Commit message: Agregados agujeros de montajes
Parts:
- added H? (x3): MountingHole_Pad, symbol Mechanical:MountingHole_Pad
Changed lines of the file:
@@
 Wire Wire Line
 	15250 9450 15250 9500
+$Comp
+L Mechanical:MountingHole_Pad H?
+U 1 1 5C32A6E4
+P 7550 7250
+F 0 "H?" H 7650 7301 50  0000 L CNN
+F 1 "MountingHole_Pad" H 7650 7209 50  0000 L CNN
+F 2 "" H 7550 7250 50  0001 C CNN
+F 3 "~" H 7550 7250 50  0001 C CNN
+	1    7550 7250
+	1    0    0    -1
+$EndComp
+$Comp
+L Mechanical:MountingHole_Pad H?
+U 1 1 5C32AA74
+P 7550 6750
+F 0 "H?" H 7650 6801 50  0000 L CNN
+F 1 "MountingHole_Pad" H 7650 6709 50  0000 L CNN
+F 2 "" H 7550 6750 50  0001 C CNN
+F 3 "~" H 7550 6750 50  0001 C CNN
+	1    7550 6750
+	1    0    0    -1
+$EndComp
+$Comp
+L power:GND #PWR?
+U 1 1 5C32AE7C
+P 7550 6850
+F 0 "#PWR?" H 7550 6600 50  0001 C CNN
+F 1 "GND" H 7554 6676 50  0000 C CNN
+F 2 "" H 7550 6850 50  0001 C CNN
+F 3 "" H 7550 6850 50  0001 C CNN
+	1    7550 6850
+	1    0    0    -1
+$EndComp
+$Comp
+L power:GND #PWR?
+U 1 1 5C32B18F
+P 7550 7350
+F 0 "#PWR?" H 7550 7100 50  0001 C CNN
+F 1 "GND" H 7554 7176 50  0000 C CNN
+F 2 "" H 7550 7350 50  0001 C CNN
+F 3 "" H 7550 7350 50  0001 C CNN
+	1    7550 7350
+	1    0    0    -1
+$EndComp
+$Comp
+L Mechanical:MountingHole_Pad H?
+U 1 1 5C32B252
+P 7550 7750
+F 0 "H?" H 7650 7801 50  0000 L CNN
+F 1 "MountingHole_Pad" H 7650 7709 50  0000 L CNN
+F 2 "" H 7550 7750 50  0001 C CNN
+F 3 "~" H 7550 7750 50  0001 C CNN
+	1    7550 7750
+	1    0    0    -1
+$EndComp
+$Comp
+L power:GND #PWR?
+U 1 1 5C32B259
+P 7550 7850
+F 0 "#PWR?" H 7550 7600 50  0001 C CNN
+F 1 "GND" H 7554 7676 50  0000 C CNN
+F 2 "" H 7550 7850 50  0001 C CNN
+F 3 "" H 7550 7850 50  0001 C CNN
+	1    7550 7850
+	1    0    0    -1
+$EndComp
 $EndSCHEMATC

Commit message: Nuevo conector de expansión
Parts:
- removed J? (x7): Conn_02x02_Counter_Clockwise, Connector_PinHeader_2.54mm:PinHeader_2x02_P2.54mm_Vertical, symbol Connector_Generic:Conn_02x02_Counter_Clockwise
- added J? (x4): Conn_01x06, Connector_PinHeader_2.54mm:PinHeader_1x06_P2.54mm_Vertical, symbol Connector_Generic:Conn_01x06
Connections:
- wire segments 349 -> 345

Commit message: PCB_C: Cambiado conector externo y pequeño arreglo en texto descriptivo
Parts:
- removed H? (x3): MountingHole_Pad, symbol Mechanical:MountingHole_Pad
- removed J? (x4): Conn_01x06, Connector_PinHeader_2.54mm:PinHeader_1x06_P2.54mm_Vertical, symbol Connector_Generic:Conn_01x06
- added J?: Conector_Expansion_CanSat, AXTEC:Conector_Expansion_CanSat, symbol AXTEC_IC:Conector_Expansion_CanSat
Connections:
- wire segments 345 -> 344
Other:
- note added: "Conector de expansión\n"
- note removed: "Conector de expansión"

Commit message: Cambio en el simbolo de SW1 en PCB_A
Parts:
- removed C?: 1uF, symbol Device:C_Small
- added C?: 1uF, Capacitor_SMD:C_0603_1608Metric_Pad1.05x0.95mm_HandSolder, symbol Device:C_Small
Connections:
- wire segments 344 -> 338
Changed lines of the file:
@@
-$EndComp
-$Comp
-L Device:C_Small C?
-U 1 1 5BC3E35C
-P 1150 6000
-AR Path="/5BB122CA/5BC3E35C" Ref="C?"  Part="1"
-AR Path="/5BB12371/5BC3E35C" Ref="C?"  Part="1"
-AR Path="/5BB123AC/5BC3E35C" Ref="C?"  Part="1"
-AR Path="/5BC3E35C" Ref="C?"  Part="1"
-F 0 "C?" H 1058 5954 50  0000 R CNN
-F 1 "1uF" H 1058 6045 50  0000 R CNN
-F 2 "" H 1150 6000 50  0001 C CNN
-F 3 "~" H 1150 6000 50  0001 C CNN
-	1    1150 6000
-	1    0    0    1
 $EndComp
 $Comp
@@
 L power:+BATT #PWR?
 U 1 1 5BCB9E27
-P 13100 4100
-F 0 "#PWR?" H 13100 3950 50  0001 C CNN
-F 1 "+BATT" H 13114 4275 50  0000 C CNN
-F 2 "" H 13100 4100 50  0001 C CNN
-F 3 "" H 13100 4100 50  0001 C CNN
-	1    13100 4100
+P 13250 4100
+F 0 "#PWR?" H 13250 3950 50  0001 C CNN
+F 1 "+BATT" H 13264 4275 50  0000 C CNN
+F 2 "" H 13250 4100 50  0001 C CNN
+F 3 "" H 13250 4100 50  0001 C CNN
+	1    13250 4100
 	1    0    0    -1
 $EndComp
@@
 L power:+3V3 #PWR?
 U 1 1 5BCB9E2D
-P 12850 4100
-F 0 "#PWR?" H 12850 3950 50  0001 C CNN
-F 1 "+3V3" H 12864 4275 50  0000 C CNN
-F 2 "" H 12850 4100 50  0001 C CNN
-F 3 "" H 12850 4100 50  0001 C CNN
-	1    12850 4100
+P 13000 4100
+F 0 "#PWR?" H 13000 3950 50  0001 C CNN
+F 1 "+3V3" H 13014 4275 50  0000 C CNN
+F 2 "" H 13000 4100 50  0001 C CNN
+F 3 "" H 13000 4100 50  0001 C CNN
+	1    13000 4100
 	1    0    0    -1
 $EndComp
@@
 L power:+5V #PWR?
 U 1 1 5BCB9E33
-P 12650 4100
-F 0 "#PWR?" H 12650 3950 50  0001 C CNN
-F 1 "+5V" H 12664 4275 50  0000 C CNN
-F 2 "" H 12650 4100 50  0001 C CNN
-F 3 "" H 12650 4100 50  0001 C CNN
-	1    12650 4100
+P 12800 4100
+F 0 "#PWR?" H 12800 3950 50  0001 C CNN
+F 1 "+5V" H 12814 4275 50  0000 C CNN
+F 2 "" H 12800 4100 50  0001 C CNN
+F 3 "" H 12800 4100 50  0001 C CNN
+	1    12800 4100
 	1    0    0    -1
 $EndComp
@@
 L power:GND #PWR?
 U 1 1 5BCB9E39
-P 13600 4850
-F 0 "#PWR?" H 13600 4600 50  0001 C CNN
-F 1 "GND" H 13604 4676 50  0000 C CNN
-F 2 "" H 13600 4850 50  0001 C CNN
-F 3 "" H 13600 4850 50  0001 C CNN
-	1    13600 4850
-	1    0    0    -1
-$EndComp
-Wire Wire Line
-	13600 4850 13600 4750
-Wire Wire Line
-	13600 4550 13700 4550
-Wire Wire Line
-	13700 4650 13600 4650
-Connection ~ 13600 4650
-Wire Wire Line
-	13600 4650 13600 4550
-Wire Wire Line
-	13700 4750 13600 4750
-Connection ~ 13600 4750
-Wire Wire Line
-	13600 4750 13600 4650
-$Comp
-L power:GND #PWR?
-U 1 1 5BCB9E47
-P 14350 5100
-F 0 "#PWR?" H 14350 4850 50  0001 C CNN
-F 1 "GND" H 14354 4926 50  0000 C CNN
-F 2 "" H 14350 5100 50  0001 C CNN
-F 3 "" H 14350 5100 50  0001 C CNN
-	1    14350 5100
-	1    0    0    -1
-$EndComp
-Wire Wire Line
-	14250 5000 14250 5050
-Wire Wire Line
-	14250 5050 14350 5050
-Wire Wire Line
-	14450 5050 14450 5000
-Wire Wire Line
-	14350 5000 14350 5050
-Connection ~ 14350 5050
-Wire Wire Line
-	14350 5100 14350 5050
-Text Notes 13850 3000 0    118  ~ 0
+P 13750 4850
+F 0 "#PWR?" H 13750 4600 50  0001 C CNN
+F 1 "GND" H 13754 4676 50  0000 C CNN
+F 2 "" H 13750 4850 50  0001 C CNN
+F 3 "" H 13750 4850 50  0001 C CNN
+	1    13750 4850
+	1    0    0    -1
+$EndComp
+Wire Wire Line
+	13750 4850 13750 4750
+Wire Wire Line
+	13750 4550 13850 4550
+Wire Wire Line
+	13850 4650 13750 4650
+Connection ~ 13750 4650
+Wire Wire Line
+	13750 4650 13750 4550
+Wire Wire Line
+	13850 4750 13750 4750
+Connection ~ 13750 4750
+Wire Wire Line
+	13750 4750 13750 4650
+Text Notes 13250 3000 0    118  ~ 0
 Conector de expansión\n
 Wire Notes Line
@@
 Wire Notes Line
 	16000 2800 16000 5400
-Wire Wire Line
-	14350 5050 14450 5050
-Text Label 15050 3400 0    50   ~ 0
+Text Label 15200 3400 0    50   ~ 0
 EXT_IO0
-Text Label 15050 3500 0    50   ~ 0
+Text Label 15200 3500 0    50   ~ 0
 EXT_IO1
-Text Label 15050 3600 0    50   ~ 0
+Text Label 15200 3600 0    50   ~ 0
 EXT_IO2
-Text Label 15050 3700 0    50   ~ 0
+Text Label 15200 3700 0    50   ~ 0
 EXT_IO3
-Text Label 15050 3800 0    50   ~ 0
+Text Label 15200 3800 0    50   ~ 0
 EXT_IO4
-Text Label 15050 3900 0    50   ~ 0
+Text Label 15200 3900 0    50   ~ 0
 EXT_IO5
 Wire Wire Line
-	15000 3400 15450 3400
-Wire Wire Line
-	15000 3500 15450 3500
-Wire Wire Line
-	15000 3600 15450 3600
-Wire Wire Line
-	15000 3700 15450 3700
-Wire Wire Line
-	15000 3800 15450 3800
-Wire Wire Line
-	15000 3900 15450 3900
-Text Label 15050 4000 0    50   ~ 0
+	15150 3400 15600 3400
+Wire Wire Line
+	15150 3500 15600 3500
+Wire Wire Line
+	15150 3600 15600 3600
+Wire Wire Line
+	15150 3700 15600 3700
+Wire Wire Line
+	15150 3800 15600 3800
+Wire Wire Line
+	15150 3900 15600 3900
+Text Label 15200 4000 0    50   ~ 0
 EXT_IO6
 Wire Wire Line
-	15000 4000 15450 4000
+	15150 4000 15600 4000
 $Comp
 L AXTEC_IC:Conector_Expansion_CanSat J?
 U 1 1 5BCB9E14
-P 14350 3950
-F 0 "J?" H 14400 4800 50  0000 C CNN
-F 1 "Conector_Expansion_CanSat" H 14350 4700 50  0000 C CNN
-F 2 "AXTEC:Conector_Expansion_CanSat" H 14350 4450 50  0001 C CNN
-F 3 "" H 14350 4450 50  0001 C CNN
-	1    14350 3950
-	1    0    0    -1
-$EndComp
-Wire Wire Line
-	13250 3400 13700 3400
-Wire Wire Line
-	13700 3500 13250 3500
-Wire Wire Line
-	13700 3600 13250 3600
-Wire Wire Line
-	13250 3700 13700 3700
-Wire Wire Line
-	13250 3800 13700 3800
-Wire Wire Line
-	13250 3900 13700 3900
-Text Label 13300 3400 0    50   ~ 0
+P 14500 3950
+F 0 "J?" H 14550 4800 50  0000 C CNN
+F 1 "Conector_Expansion_CanSat" H 14500 4700 50  0000 C CNN
+F 2 "AXTEC:Conector_Expansion_CanSat" H 14500 4450 50  0001 C CNN
+F 3 "" H 14500 4450 50  0001 C CNN
+	1    14500 3950
+	1    0    0    -1
+$EndComp
+Wire Wire Line
+	13400 3400 13850 3400
+Wire Wire Line
+	13850 3500 13400 3500
+Wire Wire Line
+	13850 3600 13400 3600
+Wire Wire Line
+	13400 3700 13850 3700
+Wire Wire Line
+	13400 3800 13850 3800
+Wire Wire Line
+	13400 3900 13850 3900
+Text Label 13450 3400 0    50   ~ 0
 EXT_SDO
-Text Label 13300 3500 0    50   ~ 0
+Text Label 13450 3500 0    50   ~ 0
 EXT_SDI
-Text Label 13300 3600 0    50   ~ 0
+Text Label 13450 3600 0    50   ~ 0
 EXT_SCLK
-Text Label 13300 3700 0    50   ~ 0
+Text Label 13450 3700 0    50   ~ 0
 EXT_CS
-Text Label 13300 3800 0    50   ~ 0
+Text Label 13450 3800 0    50   ~ 0
 SCL_EXT
-Text Label 13300 3900 0    50   ~ 0
+Text Label 13450 3900 0    50   ~ 0
 SDA_EXT
 Wire Wire Line
-	12650 4300 13700 4300
-Wire Wire Line
-	12650 4300 12650 4100
-Wire Wire Line
-	12850 4100 12850 4200
-Wire Wire Line
-	12850 4200 13700 4200
-Wire Wire Line
-	13100 4100 13700 4100
+	12800 4300 13850 4300
+Wire Wire Line
+	12800 4300 12800 4100
+Wire Wire Line
+	13000 4100 13000 4200
+Wire Wire Line
+	13000 4200 13850 4200
+Wire Wire Line
+	13250 4100 13850 4100
+$Comp
+L Device:C_Small C?
+U 1 1 5BCC9591
+P 1150 6000
+AR Path="/5BB122CA/5BCC9591" Ref="C?"  Part="1"
+AR Path="/5BB12371/5BCC9591" Ref="C?"  Part="1"
+F 0 "C?" H 1058 5954 50  0000 R CNN
+F 1 "1uF" H 1058 6045 50  0000 R CNN
+F 2 "Capacitor_SMD:C_0603_1608Metric_Pad1.05x0.95mm_HandSolder" H 1150 6000 50  0001 C CNN
+F 3 "~" H 1150 6000 50  0001 C CNN
+F 4 "EMK107B7104KAHT" H 1150 6000 50  0001 C CNN "Manufacturer Part Number"
+	1    1150 6000
+	-1   0    0    1
+$EndComp
 $EndSCHEMATC

Commit message: Agregada memoria FLASH a PCB_C
Parts:
- removed C? (x2): 100nF, symbol Device:C_Small
- removed U?: NTB0104BQ,115, NTB0104BQ115, symbol SamacSys_Parts:NTB0104BQ,115
- added C?: 1uF, Capacitor_SMD:C_0603_1608Metric_Pad1.05x0.95mm_HandSolder, symbol Device:C_Small
- added IC?: IS25LP080D-JULE-TR, SON50P200X300X60-8N, symbol SamacSys_Parts:IS25LP080D-JULE-TR
Connections:
- net labels added: FLASH_CS, FLASH_MISO, FLASH_MOSI, FLASH_SCK, IO_EN
- net labels removed: EXT_IO4, EXT_IO5, EXT_IO6, IO4, IO5, IO6, IO_B_EN
- wire segments 338 -> 330
Other:
- note removed: "Buffer IO_B"

Commit message: Footprints para PCB_C
Parts:
- removed C?: 4.3pF, symbol Device:C_Small
- removed C? (x2): 1uF, Capacitor_SMD:C_0603_1608Metric_Pad1.05x0.95mm_HandSolder, symbol Device:C_Small
- removed C?: 20pF, symbol Device:C_Small
- removed C? (x14): 100nF, symbol Device:C_Small
- added C? (x2): 1uF, Capacitor_SMD:C_0603_1608Metric_Pad1.05x0.95mm_HandSolder, symbol Device:C_Small
- added C? (x14): 100nF, Capacitor_SMD:C_0603_1608Metric_Pad1.05x0.95mm_HandSolder, symbol Device:C_Small
- added C?: 20pF, Capacitor_SMD:C_0603_1608Metric_Pad1.05x0.95mm_HandSolder, symbol Device:C_Small
- added C?: 4.3pF, Capacitor_SMD:C_0603_1608Metric_Pad1.05x0.95mm_HandSolder, symbol Device:C_Small
- C?: footprint (none) -> Capacitor_SMD:C_0603_1608Metric_Pad1.05x0.95mm_HandSolder; Manufacturer Part Number (none) -> 885012006001
- C?: footprint (none) -> Capacitor_SMD:C_0603_1608Metric_Pad1.05x0.95mm_HandSolder; Manufacturer Part Number (none) -> GCM1885C2A200JA16D
- C?: footprint (none) -> Capacitor_SMD:C_0805_2012Metric_Pad1.15x1.40mm_HandSolder; Dielectric (none) -> X7R; Manufacturer Part Number (none) -> GRM21BR71A475KE51K
- J?: footprint (none) -> Connector_USB:USB_Micro-B_Molex-105017-0001; Manufacturer Part Number (none) -> 105017-0001
- J?: footprint (none) -> Connector_PinHeader_2.54mm:PinHeader_1x06_P2.54mm_Vertical
- R? (x6): footprint (none) -> Resistor_SMD:R_0603_1608Metric_Pad1.05x0.95mm_HandSolder

Commit message: Corrección de conector de expansión en PCB_C
Connections:
- wire segments 330 -> 332
Changed lines of the file:
@@
 L power:+BATT #PWR?
 U 1 1 5BCB9E27
-P 13250 4100
-F 0 "#PWR?" H 13250 3950 50  0001 C CNN
-F 1 "+BATT" H 13264 4275 50  0000 C CNN
-F 2 "" H 13250 4100 50  0001 C CNN
-F 3 "" H 13250 4100 50  0001 C CNN
-	1    13250 4100
+P 13650 3500
+F 0 "#PWR?" H 13650 3350 50  0001 C CNN
+F 1 "+BATT" H 13664 3675 50  0000 C CNN
+F 2 "" H 13650 3500 50  0001 C CNN
+F 3 "" H 13650 3500 50  0001 C CNN
+	1    13650 3500
 	1    0    0    -1
 $EndComp
@@
 L power:+3V3 #PWR?
 U 1 1 5BCB9E2D
-P 13000 4100
-F 0 "#PWR?" H 13000 3950 50  0001 C CNN
-F 1 "+3V3" H 13014 4275 50  0000 C CNN
-F 2 "" H 13000 4100 50  0001 C CNN
-F 3 "" H 13000 4100 50  0001 C CNN
-	1    13000 4100
+P 13350 3500
+F 0 "#PWR?" H 13350 3350 50  0001 C CNN
+F 1 "+3V3" H 13364 3675 50  0000 C CNN
+F 2 "" H 13350 3500 50  0001 C CNN
+F 3 "" H 13350 3500 50  0001 C CNN
+	1    13350 3500
 	1    0    0    -1
 $EndComp
@@
 L power:+5V #PWR?
 U 1 1 5BCB9E33
-P 12800 4100
-F 0 "#PWR?" H 12800 3950 50  0001 C CNN
-F 1 "+5V" H 12814 4275 50  0000 C CNN
-F 2 "" H 12800 4100 50  0001 C CNN
-F 3 "" H 12800 4100 50  0001 C CNN
-	1    12800 4100
-	1    0    0    -1
-$EndComp
-$Comp
-L power:GND #PWR?
-U 1 1 5BCB9E39
-P 13750 4850
-F 0 "#PWR?" H 13750 4600 50  0001 C CNN
-F 1 "GND" H 13754 4676 50  0000 C CNN
-F 2 "" H 13750 4850 50  0001 C CNN
-F 3 "" H 13750 4850 50  0001 C CNN
-	1    13750 4850
-	1    0    0    -1
-$EndComp
-Wire Wire Line
-	13750 4850 13750 4750
-Wire Wire Line
-	13750 4550 13850 4550
-Wire Wire Line
-	13850 4650 13750 4650
-Connection ~ 13750 4650
-Wire Wire Line
-	13750 4650 13750 4550
-Wire Wire Line
-	13850 4750 13750 4750
-Connection ~ 13750 4750
-Wire Wire Line
-	13750 4750 13750 4650
-Text Notes 13250 3000 0    118  ~ 0
+P 13100 3500
+F 0 "#PWR?" H 13100 3350 50  0001 C CNN
+F 1 "+5V" H 13114 3675 50  0000 C CNN
+F 2 "" H 13100 3500 50  0001 C CNN
+F 3 "" H 13100 3500 50  0001 C CNN
+	1    13100 3500
+	1    0    0    -1
+$EndComp
+Text Notes 13250 3100 0    118  ~ 0
 Conector de expansión\n
 Wire Notes Line
-	16000 2800 12550 2800
+	16000 2900 12500 2900
 Wire Notes Line
-	12550 2800 12550 5400
+	12500 2900 12500 5500
 Wire Notes Line
-	12550 5400 16000 5400
+	12500 5500 16000 5500
 Wire Notes Line
-	16000 2800 16000 5400
-Text Label 15200 3400 0    50   ~ 0
+	16000 2900 16000 5500
+Text Label 15200 3600 0    50   ~ 0
 EXT_IO0
-Text Label 15200 3500 0    50   ~ 0
+Text Label 15200 3700 0    50   ~ 0
 EXT_IO1
-Text Label 15200 3600 0    50   ~ 0
+Text Label 15200 3800 0    50   ~ 0
 EXT_IO2
-Text Label 15200 3700 0    50   ~ 0
+Text Label 15200 3900 0    50   ~ 0
 EXT_IO3
 Wire Wire Line
-	15150 3400 15600 3400
-Wire Wire Line
-	15150 3500 15600 3500
-Wire Wire Line
 	15150 3600 15600 3600
 Wire Wire Line
 	15150 3700 15600 3700
+Wire Wire Line
+	15150 3800 15600 3800
+Wire Wire Line
+	15150 3900 15600 3900
 $Comp
 L AXTEC_IC:Conector_Expansion_CanSat J?
 U 1 1 5BCB9E14
-P 14500 3950
-F 0 "J?" H 14550 4800 50  0000 C CNN
-F 1 "Conector_Expansion_CanSat" H 14500 4700 50  0000 C CNN
-F 2 "AXTEC:Conector_Expansion_CanSat" H 14500 4450 50  0001 C CNN
-F 3 "" H 14500 4450 50  0001 C CNN
-	1    14500 3950
-	1    0    0    -1
-$EndComp
-Wire Wire Line
-	13400 3400 13850 3400
-Wire Wire Line
-	13850 3500 13400 3500
-Wire Wire Line
-	13850 3600 13400 3600
-Wire Wire Line
-	13400 3700 13850 3700
-Wire Wire Line
-	13400 3800 13850 3800
-Wire Wire Line
-	13400 3900 13850 3900
-Text Label 13450 3400 0    50   ~ 0
+P 14500 4150
+F 0 "J?" H 14550 5000 50  0000 C CNN
+F 1 "Conector_Expansion_CanSat" H 14500 4900 50  0000 C CNN
+F 2 "AXTEC:Conector_Expansion_CanSat" H 14500 4650 50  0001 C CNN
+F 3 "" H 14500 4650 50  0001 C CNN
+	1    14500 4150
+	1    0    0    -1
+$EndComp
+Wire Wire Line
+	13400 4500 13850 4500
+Wire Wire Line
+	13850 4600 13400 4600
+Wire Wire Line
+	13850 4700 13400 4700
+Wire Wire Line
+	13400 4800 13850 4800
+Wire Wire Line
+	13400 4900 13850 4900
+Wire Wire Line
+	13400 5000 13850 5000
+Text Label 13450 4500 0    50   ~ 0
 EXT_SDO
-Text Label 13450 3500 0    50   ~ 0
+Text Label 13450 4600 0    50   ~ 0
 EXT_SDI
-Text Label 13450 3600 0    50   ~ 0
+Text Label 13450 4700 0    50   ~ 0
 EXT_SCLK
-Text Label 13450 3700 0    50   ~ 0
+Text Label 13450 4800 0    50   ~ 0
 EXT_CS
-Text Label 13450 3800 0    50   ~ 0
+Text Label 13450 4900 0    50   ~ 0
 SCL_EXT
-Text Label 13450 3900 0    50   ~ 0
+Text Label 13450 5000 0    50   ~ 0
 SDA_EXT
-Wire Wire Line
-	12800 4300 13850 4300
-Wire Wire Line
-	12800 4300 12800 4100
-Wire Wire Line
-	13000 4100 13000 4200
-Wire Wire Line
-	13000 4200 13850 4200
-Wire Wire Line
-	13250 4100 13850 4100
 $Comp
 L SamacSys_Parts:IS25LP080D-JULE-TR IC?
@@
 	0    1    -1   0
 $EndComp
+Wire Wire Line
+	13850 3650 13650 3650
+Wire Wire Line
+	13650 3650 13650 3500
+Wire Wire Line
+	13350 3500 13350 3750
+Wire Wire Line
+	13350 3750 13850 3750
+Wire Wire Line
+	13100 3500 13100 3850
+Wire Wire Line
+	13100 3850 13850 3850
+$Comp
+L power:GND #PWR?
+U 1 1 5BE79E5A
+P 13100 5050
+F 0 "#PWR?" H 13100 4800 50  0001 C CNN
+F 1 "GND" H 13104 4876 50  0000 C CNN
+F 2 "" H 13100 5050 50  0001 C CNN
+F 3 "" H 13100 5050 50  0001 C CNN
+	1    13100 5050
+	1    0    0    -1
+$EndComp
+Wire Wire Line
+	13850 4100 13750 4100
+Wire Wire Line
+	13100 4100 13100 5050
+Wire Wire Line
+	13850 4200 13750 4200
+Wire Wire Line
+	13750 4200 13750 4100
+Connection ~ 13750 4100
+Wire Wire Line
+	13750 4100 13100 4100
+Wire Wire Line
+	13850 4300 13750 4300
+Wire Wire Line
+	13750 4300 13750 4200
+Connection ~ 13750 4200
 $EndSCHEMATC
