File: Hardware/Satelite/PCB_C/PCB_C.sch (KiCad schematic (older format))
At the start: 43 parts

Commit message: Switch analógico para cambiar entre los niveles de tensión de los buffers en PCB_C
Parts:
- removed Q? (x2): SSM3J338R,LF, SamacSys_Parts:SSM3J332RLFT, symbol SamacSys_Parts:SSM3J338R,LF
- removed R?: 10K, Resistor_SMD:R_0603_1608Metric_Pad1.05x0.95mm_HandSolder, symbol Device:R
- added Q?: BC817, Package_TO_SOT_SMD:SOT-23, symbol Transistor_BJT:BC817
- added R?: 100k, Resistor_SMD:R_0603_1608Metric_Pad1.05x0.95mm_HandSolder, symbol Device:R
- added R?: 1k, Resistor_SMD:R_0603_1608Metric_Pad1.05x0.95mm_HandSolder, symbol Device:R
- added U?: SN74LVC1G3157DCKR, SOT65P210X110-6N, symbol SamacSys_Parts:SN74LVC1G3157DCKR
- R?: value 10K -> 10k
Connections:
- net labels added: SWITCH_IO_V
- net labels removed: ENABLE_3V3_IO, ENABLE_5V_IO
- wire segments 325 -> 326
Other:
- note added: "Por defecto en +3V3"
Changed lines of the file:
@@
 $EndComp
-$Comp
-L SamacSys_Parts:SSM3J338R,LF Q?
-U 1 1 5C2117E2
-P 13850 7050
-F 0 "Q?" V 14418 7150 50  0000 C CNN
-F 1 "SSM3J338R,LF" V 14326 7150 50  0000 C CNN
-F 2 "SamacSys_Parts:SSM3J332RLFT" H 14300 7000 50  0001 L CNN
-F 3 "http://toshiba.semicon-storage.com/info/docget.jsp?did=30384&prodName=SSM3J338R" H 14300 6900 50  0001 L CNN
-F 4 "MOSFET Small-signal MOSFET Vdss= -12V, ID= -6A" H 14300 6800 50  0001 L CNN "Description"
-F 5 "Toshiba" H 14300 6600 50  0001 L CNN "Manufacturer_Name"
-F 6 "SSM3J338R,LF" H 14300 6500 50  0001 L CNN "Manufacturer Part Number"
-F 7 "SSM3J338R,LF" H 14300 6200 50  0001 L CNN "Arrow Part Number"
-F 8 "https://www.arrow.com/en/products/ssm3j338rlf/toshiba" H 14300 6100 50  0001 L CNN "Arrow Price/Stock"
-	1    13850 7050
-	0    -1   -1   0
-$EndComp
-$Comp
-L SamacSys_Parts:SSM3J338R,LF Q?
-U 1 1 5C2117EE
-P 13850 7700
-F 0 "Q?" V 14418 7800 50  0000 C CNN
-F 1 "SSM3J338R,LF" V 14326 7800 50  0000 C CNN
-F 2 "SamacSys_Parts:SSM3J332RLFT" H 14300 7650 50  0001 L CNN
-F 3 "http://toshiba.semicon-storage.com/info/docget.jsp?did=30384&prodName=SSM3J338R" H 14300 7550 50  0001 L CNN
-F 4 "MOSFET Small-signal MOSFET Vdss= -12V, ID= -6A" H 14300 7450 50  0001 L CNN "Description"
-F 5 "Toshiba" H 14300 7250 50  0001 L CNN "Manufacturer_Name"
-F 6 "SSM3J338R,LF" H 14300 7150 50  0001 L CNN "Manufacturer Part Number"
-F 7 "SSM3J338R,LF" H 14300 6850 50  0001 L CNN "Arrow Part Number"
-F 8 "https://www.arrow.com/en/products/ssm3j338rlf/toshiba" H 14300 6750 50  0001 L CNN "Arrow Price/Stock"
-	1    13850 7700
-	0    -1   -1   0
-$EndComp
-Wire Wire Line
-	13850 7700 13850 7750
-Wire Wire Line
-	13850 7750 14050 7750
-Wire Wire Line
-	13850 7050 13850 7100
-Wire Wire Line
-	13850 7100 14050 7100
-$Comp
-L Device:R R?
-U 1 1 5C2117F9
-P 14050 6900
-F 0 "R?" H 14120 6946 50  0000 L CNN
-F 1 "10K" H 14120 6854 50  0000 L CNN
-F 2 "Resistor_SMD:R_0603_1608Metric_Pad1.05x0.95mm_HandSolder" V 13980 6900 50  0001 C CNN
-F 3 "~" H 14050 6900 50  0001 C CNN
-	1    14050 6900
-	1    0    0    -1
-$EndComp
-Wire Wire Line
-	14050 7050 14050 7100
-Connection ~ 14050 7100
 $Comp
 L Device:R R?
 U 1 1 5C211802
-P 14050 7550
-F 0 "R?" H 14120 7596 50  0000 L CNN
-F 1 "10K" H 14120 7504 50  0000 L CNN
-F 2 "Resistor_SMD:R_0603_1608Metric_Pad1.05x0.95mm_HandSolder" V 13980 7550 50  0001 C CNN
-F 3 "~" H 14050 7550 50  0001 C CNN
-	1    14050 7550
-	1    0    0    -1
-$EndComp
-Wire Wire Line
-	14050 7700 14050 7750
-Connection ~ 14050 7750
+P 14500 6750
+F 0 "R?" H 14570 6796 50  0000 L CNN
+F 1 "10k" H 14570 6704 50  0000 L CNN
+F 2 "Resistor_SMD:R_0603_1608Metric_Pad1.05x0.95mm_HandSolder" V 14430 6750 50  0001 C CNN
+F 3 "~" H 14500 6750 50  0001 C CNN
+	1    14500 6750
+	1    0    0    -1
+$EndComp
 Wire Wire Line
 	11000 9650 11000 9700
@@
 $EndComp
 $Comp
-L power:VDD #PWR?
-U 1 1 5C294E4A
-P 13300 6600
-F 0 "#PWR?" H 13300 6450 50  0001 C CNN
-F 1 "VDD" H 13317 6775 50  0000 C CNN
-F 2 "" H 13300 6600 50  0001 C CNN
-F 3 "" H 13300 6600 50  0001 C CNN
-	1    13300 6600
-	1    0    0    -1
-$EndComp
-Wire Wire Line
-	13300 6600 13300 6750
-Wire Wire Line
-	13300 7400 13450 7400
-Wire Wire Line
-	13450 6750 13300 6750
-Connection ~ 13300 6750
-Wire Wire Line
-	13300 6750 13300 7400
-Wire Wire Line
-	14050 7100 14950 7100
-Wire Wire Line
-	14050 7750 15000 7750
-$Comp
 L power:+3V3 #PWR?
 U 1 1 5C2EE791
-P 14400 6700
-F 0 "#PWR?" H 14400 6550 50  0001 C CNN
-F 1 "+3V3" H 14415 6873 50  0000 C CNN
-F 2 "" H 14400 6700 50  0001 C CNN
-F 3 "" H 14400 6700 50  0001 C CNN
-	1    14400 6700
-	1    0    0    -1
-$EndComp
-Wire Wire Line
-	14400 6700 14400 6750
-Wire Wire Line
-	14400 6750 14050 6750
-Connection ~ 14050 6750
+P 12700 6550
+F 0 "#PWR?" H 12700 6400 50  0001 C CNN
+F 1 "+3V3" H 12715 6723 50  0000 C CNN
+F 2 "" H 12700 6550 50  0001 C CNN
+F 3 "" H 12700 6550 50  0001 C CNN
+	1    12700 6550
+	1    0    0    -1
+$EndComp
 $Comp
 L power:+5V #PWR?
 U 1 1 5C30537D
-P 14400 7350
-F 0 "#PWR?" H 14400 7200 50  0001 C CNN
-F 1 "+5V" H 14415 7523 50  0000 C CNN
-F 2 "" H 14400 7350 50  0001 C CNN
-F 3 "" H 14400 7350 50  0001 C CNN
-	1    14400 7350
-	1    0    0    -1
-$EndComp
-Wire Wire Line
-	14400 7350 14400 7400
-Wire Wire Line
-	14400 7400 14050 7400
-Connection ~ 14050 7400
-Text Label 14350 7100 0    50   ~ 0
-ENABLE_5V_IO
-Text Label 14350 7750 0    50   ~ 0
-ENABLE_3V3_IO
+P 12950 6550
+F 0 "#PWR?" H 12950 6400 50  0001 C CNN
+F 1 "+5V" H 12965 6723 50  0000 C CNN
+F 2 "" H 12950 6550 50  0001 C CNN
+F 3 "" H 12950 6550 50  0001 C CNN
+	1    12950 6550
+	1    0    0    -1
+$EndComp
 Wire Notes Line
 	12500 5800 12500 8050
@@
 Text Notes 13200 6050 0    118  ~ 0
 Selección de tensión IO
-Text Label 8350 3000 0    50   ~ 0
-ENABLE_5V_IO
 Text Label 8350 3900 0    50   ~ 0
-ENABLE_3V3_IO
+SWITCH_IO_V
 Wire Wire Line
 	11000 10900 11000 10800
@@
 Wire Wire Line
 	9800 10800 9150 10800
-Wire Wire Line
-	8250 3000 8900 3000
 Wire Wire Line
 	8250 3900 8900 3900
@@
 Text Label 6300 5400 0    50   ~ 0
 FLASH_CS
+$Comp
+L SamacSys_Parts:SN74LVC1G3157DCKR U?
+U 1 1 5C393362
+P 13600 6850
+F 0 "U?" H 13600 7216 50  0000 C CNN
+F 1 "SN74LVC1G3157DCKR" H 13600 7124 50  0000 C CNN
+F 2 "SOT65P210X110-6N" H 13950 7050 50  0001 L CNN
+F 3 "http://www.ti.com/lit/ds/symlink/sn74lvc1g3157.pdf" H 13950 6950 50  0001 L CNN
+F 4 "SN74LVC1G3157DCKR, Analogue Switch Single SPDT, 3, 5V, 6-Pin, SC-70" H 13950 6850 50  0001 L CNN "Description"
+F 5 "1.1" H 13950 6750 50  0001 L CNN "Height"
+F 6 "Texas Instruments" H 13950 6650 50  0001 L CNN "Manufacturer_Name"
+F 7 "SN74LVC1G3157DCKR" H 13950 6550 50  0001 L CNN "Manufacturer Part Number"
+F 8 "6282769P" H 13950 6450 50  0001 L CNN "RS Part Number"
+F 9 "http://uk.rs-online.com/web/p/products/6282769P" H 13950 6350 50  0001 L CNN "RS Price/Stock"
+F 10 "SN74LVC1G3157DCKR" H 13950 6250 50  0001 L CNN "Arrow Part Number"
+F 11 "https://www.arrow.com/en/products/sn74lvc1g3157dckr/texas-instruments" H 13950 6150 50  0001 L CNN "Arrow Price/Stock"
+	1    13600 6850
+	1    0    0    -1
+$EndComp
+Text Label 15300 7350 0    50   ~ 0
+SWITCH_IO_V
+Wire Wire Line
+	12700 6550 12700 6850
+Wire Wire Line
+	12700 6850 13100 6850
+Wire Wire Line
+	12950 6550 12950 6750
+Wire Wire Line
+	12950 6750 13100 6750
+$Comp
+L power:GND #PWR?
+U 1 1 5C435B93
+P 12700 7100
+F 0 "#PWR?" H 12700 6850 50  0001 C CNN
+F 1 "GND" H 12704 6926 50  0000 C CNN
+F 2 "" H 12700 7100 50  0001 C CNN
+F 3 "" H 12700 7100 50  0001 C CNN
+	1    12700 7100
+	1    0    0    -1
+$EndComp
+Wire Wire Line
+	12700 7100 12700 6950
+Wire Wire Line
+	12700 6950 13100 6950
+$Comp
+L Transistor_BJT:BC817 Q?
+U 1 1 5C450AE0
+P 14600 7350
+F 0 "Q?" H 14791 7396 50  0000 L CNN
+F 1 "BC817" H 14791 7304 50  0000 L CNN
+F 2 "Package_TO_SOT_SMD:SOT-23" H 14800 7275 50  0001 L CIN
+F 3 "http://www.fairchildsemi.com/ds/BC/BC817.pdf" H 14600 7350 50  0001 L CNN
+F 4 "BC817-40W,135" H 14600 7350 50  0001 C CNN "Manufacturer Part Number"
+	1    14600 7350
+	-1   0    0    -1
+$EndComp
+$Comp
+L power:+5V #PWR?
+U 1 1 5C46BB9A
+P 14100 6550
+F 0 "#PWR?" H 14100 6400 50  0001 C CNN
+F 1 "+5V" H 14115 6723 50  0000 C CNN
+F 2 "" H 14100 6550 50  0001 C CNN
+F 3 "" H 14100 6550 50  0001 C CNN
+	1    14100 6550
+	1    0    0    -1
+$EndComp
+Wire Wire Line
+	14100 6550 14100 6750
+$Comp
+L power:VDD #PWR?
+U 1 1 5C487256
+P 14300 6550
+F 0 "#PWR?" H 14300 6400 50  0001 C CNN
+F 1 "VDD" H 14317 6725 50  0000 C CNN
+F 2 "" H 14300 6550 50  0001 C CNN
+F 3 "" H 14300 6550 50  0001 C CNN
+	1    14300 6550
+	1    0    0    -1
+$EndComp
+Wire Wire Line
+	14300 6550 14300 6850
+Wire Wire Line
+	14300 6850 14100 6850
+$Comp
+L power:+5V #PWR?
+U 1 1 5C4F508E
+P 14500 6550
+F 0 "#PWR?" H 14500 6400 50  0001 C CNN
+F 1 "+5V" H 14515 6723 50  0000 C CNN
+F 2 "" H 14500 6550 50  0001 C CNN
+F 3 "" H 14500 6550 50  0001 C CNN
+	1    14500 6550
+	1    0    0    -1
+$EndComp
+Wire Wire Line
+	14500 6550 14500 6600
+Wire Wire Line
+	14500 6900 14500 6950
+$Comp
+L power:GND #PWR?
+U 1 1 5C52C216
+P 14500 7650
+F 0 "#PWR?" H 14500 7400 50  0001 C CNN
+F 1 "GND" H 14504 7476 50  0000 C CNN
+F 2 "" H 14500 7650 50  0001 C CNN
+F 3 "" H 14500 7650 50  0001 C CNN
+	1    14500 7650
+	1    0    0    -1
+$EndComp
+Wire Wire Line
+	14500 7550 14500 7650
+Connection ~ 14500 6950
+Wire Wire Line
+	14500 6950 14500 7150
+$Comp
+L Device:R R?
+U 1 1 5C59B777
+P 14900 6750
+F 0 "R?" H 14970 6796 50  0000 L CNN
+F 1 "100k" H 14970 6704 50  0000 L CNN
+F 2 "Resistor_SMD:R_0603_1608Metric_Pad1.05x0.95mm_HandSolder" V 14830 6750 50  0001 C CNN
+F 3 "~" H 14900 6750 50  0001 C CNN
+	1    14900 6750
+	1    0    0    -1
+$EndComp
+Wire Wire Line
+	14900 6600 14500 6600
+Connection ~ 14500 6600
+Wire Wire Line
+	14900 6900 14900 7350
+Wire Wire Line
+	14900 7350 14800 7350
+$Comp
+L Device:R R?
+U 1 1 5C5D409B
+P 15050 7350
+F 0 "R?" H 15120 7396 50  0000 L CNN
+F 1 "1k" H 15120 7304 50  0000 L CNN
+F 2 "Resistor_SMD:R_0603_1608Metric_Pad1.05x0.95mm_HandSolder" V 14980 7350 50  0001 C CNN
+F 3 "~" H 15050 7350 50  0001 C CNN
+	1    15050 7350
+	0    1    1    0
+$EndComp
+Connection ~ 14900 7350
+Wire Wire Line
+	14100 6950 14500 6950
+Wire Wire Line
+	15200 7350 15800 7350
+Text Notes 13200 7250 0    50   ~ 0
+Por defecto en +3V3
 $EndSCHEMATC

Commit message: Modificaciones en conectores, netlist para PCB C
Parts:
- IC1: renamed from IC?; footprint SOT95P270X145-6N -> SamacSys_Parts:SOT95P270X145-6N
- IC2: renamed from IC?; footprint SON50P200X300X60-8N -> SamacSys_Parts:SON50P200X300X60-8N
- IC3: renamed from IC?; footprint RSE(R-PUQFN-N10) -> SamacSys_Parts:RSE(R-PUQFN-N10)
- J2: renamed from J?; footprint (none) -> Connector_PinHeader_2.54mm:PinHeader_1x03_P2.54mm_Vertical
- J3: renamed from J?; footprint (none) -> AXTEC:Conector_PCB_B-C
- U1, U4: renamed from U?; footprint NTB0104BQ115 -> SamacSys_Parts:NTB0104BQ115
- U2: renamed from U?; footprint SOP65P490X110-8N -> SamacSys_Parts:SOP65P490X110-8N
- U5: renamed from U?; footprint SOT65P210X110-6N -> SamacSys_Parts:SOT65P210X110-6N
- Y1: renamed from Y?; footprint LFXTAL016178_1 -> SamacSys_Parts:LFXTAL016178_1
- Y2: renamed from Y?; footprint (none) -> Crystal:Crystal_SMD_0603-2Pin_6.0x3.5mm_HandSoldering
- gave numbers to parts that had none: 33

Commit message: Agregados agujeros de montaje para PCB C
Parts:
- added MH1: MH_CanSat, AXTEC:MH_CanSat, symbol AXTEC_IC:MH_CanSat
Connections:
- wire segments 326 -> 329
Other:
- note added: "AGUJEROS DE MONTAJE"
Changed lines of the file:
@@
 Text Notes 13200 7250 0    50   ~ 0
 Por defecto en +3V3
+$Comp
+L AXTEC_IC:MH_CanSat MH1
+U 1 1 5BCAAD71
+P 1900 7400
+F 0 "MH1" H 2178 7515 50  0000 L CNN
+F 1 "MH_CanSat" H 2178 7424 50  0000 L CNN
+F 2 "AXTEC:MH_CanSat" H 1900 7400 50  0001 C CNN
+F 3 "" H 1900 7400 50  0001 C CNN
+	1    1900 7400
+	1    0    0    -1
+$EndComp
+$Comp
+L power:GND #PWR081
+U 1 1 5BCAAE9A
+P 1900 7600
+F 0 "#PWR081" H 1900 7350 50  0001 C CNN
+F 1 "GND" H 1905 7427 50  0000 C CNN
+F 2 "" H 1900 7600 50  0001 C CNN
+F 3 "" H 1900 7600 50  0001 C CNN
+	1    1900 7600
+	-1   0    0    -1
+$EndComp
+Wire Wire Line
+	1750 7500 1900 7500
+Connection ~ 1900 7500
+Wire Wire Line
+	1900 7500 2050 7500
+Wire Wire Line
+	1900 7600 1900 7500
+Wire Notes Line
+	550  6550 3550 6550
+Wire Notes Line
+	3550 6550 3550 8200
+Wire Notes Line
+	3550 8200 550  8200
+Wire Notes Line
+	550  8200 550  6550
+Text Notes 900  6800 0    118  ~ 0
+AGUJEROS DE MONTAJE
 $EndSCHEMATC

Commit message: Capacitores 0402 para PCB_C
Parts:
- C1: footprint Capacitor_SMD:C_0603_1608Metric_Pad1.05x0.95mm_HandSolder -> Capacitor_SMD:C_0402_1005Metric; Manufacturer Part Number LMK107B7105MA-T -> GRM155R61E105KA12D
- C10, C11, C12, C14, C15, C16, C17, C18, C19, C2, C21, C5, C6, C9: footprint Capacitor_SMD:C_0603_1608Metric_Pad1.05x0.95mm_HandSolder -> Capacitor_SMD:C_0402_1005Metric; Manufacturer Part Number EMK107B7104KAHT -> GCM155R71C104KA55D
- C3, C4: footprint Capacitor_SMD:C_0603_1608Metric_Pad1.05x0.95mm_HandSolder -> Capacitor_SMD:C_0402_1005Metric; Manufacturer Part Number 885012006001 -> GRM1555C1H4R3WA01D
- C7, C8: footprint Capacitor_SMD:C_0603_1608Metric_Pad1.05x0.95mm_HandSolder -> Capacitor_SMD:C_0402_1005Metric; Manufacturer Part Number GCM1885C2A200JA16D -> GCM1555C1H200JA16D
- Y2: footprint Crystal:Crystal_SMD_0603-2Pin_6.0x3.5mm_HandSoldering -> Crystal:Crystal_HC49-4H_Vertical
Changed lines of the file:
@@
 F 0 "C3" H 5108 5304 50  0000 R CNN
 F 1 "4.3pF" H 5108 5395 50  0000 R CNN
-F 2 "Capacitor_SMD:C_0603_1608Metric_Pad1.05x0.95mm_HandSolder" H 5200 5350 50  0001 C CNN
+F 2 "Capacitor_SMD:C_0402_1005Metric" H 5200 5350 50  0001 C CNN
 F 3 "~" H 5200 5350 50  0001 C CNN
-F 4 "885012006001" H 5200 5350 50  0001 C CNN "Manufacturer Part Number"
+F 4 "GRM1555C1H4R3WA01D" H 5200 5350 50  0001 C CNN "Manufacturer Part Number"
 	1    5200 5350
 	0    1    1    0
@@
 F 0 "Y2" V 6058 3781 50  0000 L CNN
 F 1 "Crystal" V 6150 3781 50  0000 L CNN
-F 2 "Crystal:Crystal_SMD_0603-2Pin_6.0x3.5mm_HandSoldering" H 6150 3650 50  0001 C CNN
+F 2 "Crystal:Crystal_HC49-4H_Vertical" H 6150 3650 50  0001 C CNN
 F 3 "~" H 6150 3650 50  0001 C CNN
 F 4 "8 MHz" V 6242 3781 50  0000 L CNN "Frequency"
@@
 F 0 "C7" H 5708 3404 50  0000 R CNN
 F 1 "20pF" H 5708 3495 50  0000 R CNN
-F 2 "Capacitor_SMD:C_0603_1608Metric_Pad1.05x0.95mm_HandSolder" H 5800 3450 50  0001 C CNN
+F 2 "Capacitor_SMD:C_0402_1005Metric" H 5800 3450 50  0001 C CNN
 F 3 "~" H 5800 3450 50  0001 C CNN
-F 4 "GCM1885C2A200JA16D" H 5800 3450 50  0001 C CNN "Manufacturer Part Number"
+F 4 "GCM1555C1H200JA16D" H 5800 3450 50  0001 C CNN "Manufacturer Part Number"
 	1    5800 3450
 	0    1    1    0
@@
 F 0 "C1" H 1058 5954 50  0000 R CNN
 F 1 "1uF" H 1058 6045 50  0000 R CNN
-F 2 "Capacitor_SMD:C_0603_1608Metric_Pad1.05x0.95mm_HandSolder" H 1150 6000 50  0001 C CNN
+F 2 "Capacitor_SMD:C_0402_1005Metric" H 1150 6000 50  0001 C CNN
 F 3 "~" H 1150 6000 50  0001 C CNN
-F 4 "LMK107B7105MA-T" H 1150 6000 50  0001 C CNN "Manufacturer Part Number"
+F 4 "GRM155R61E105KA12D" H 1150 6000 50  0001 C CNN "Manufacturer Part Number"
 	1    1150 6000
 	-1   0    0    1
@@
 F 0 "C6" H 5842 2596 50  0000 L CNN
 F 1 "100nF" H 5842 2505 50  0000 L CNN
-F 2 "Capacitor_SMD:C_0603_1608Metric_Pad1.05x0.95mm_HandSolder" H 5750 2550 50  0001 C CNN
+F 2 "Capacitor_SMD:C_0402_1005Metric" H 5750 2550 50  0001 C CNN
 F 3 "~" H 5750 2550 50  0001 C CNN
-F 4 "EMK107B7104KAHT" H 5750 2550 50  0001 C CNN "Manufacturer Part Number"
+F 4 "GCM155R71C104KA55D" H 5750 2550 50  0001 C CNN "Manufacturer Part Number"
 	1    5750 2550
 	-1   0    0    -1
@@
 F 0 "C17" H 9192 5396 50  0000 L CNN
 F 1 "100nF" H 9192 5305 50  0000 L CNN
-F 2 "Capacitor_SMD:C_0603_1608Metric_Pad1.05x0.95mm_HandSolder" H 9100 5350 50  0001 C CNN
+F 2 "Capacitor_SMD:C_0402_1005Metric" H 9100 5350 50  0001 C CNN
 F 3 "~" H 9100 5350 50  0001 C CNN
-F 4 "EMK107B7104KAHT" H 9100 5350 50  0001 C CNN "Manufacturer Part Number"
+F 4 "GCM155R71C104KA55D" H 9100 5350 50  0001 C CNN "Manufacturer Part Number"
 	1    9100 5350
 	1    0    0    -1
@@
 F 0 "C16" H 9192 4296 50  0000 L CNN
 F 1 "100nF" H 9192 4205 50  0000 L CNN
-F 2 "Capacitor_SMD:C_0603_1608Metric_Pad1.05x0.95mm_HandSolder" H 9100 4250 50  0001 C CNN
+F 2 "Capacitor_SMD:C_0402_1005Metric" H 9100 4250 50  0001 C CNN
 F 3 "~" H 9100 4250 50  0001 C CNN
-F 4 "EMK107B7104KAHT" H 9100 4250 50  0001 C CNN "Manufacturer Part Number"
+F 4 "GCM155R71C104KA55D" H 9100 4250 50  0001 C CNN "Manufacturer Part Number"
 	1    9100 4250
 	1    0    0    -1
@@
 F 0 "C15" H 9192 2696 50  0000 L CNN
 F 1 "100nF" H 9192 2605 50  0000 L CNN
-F 2 "Capacitor_SMD:C_0603_1608Metric_Pad1.05x0.95mm_HandSolder" H 9100 2650 50  0001 C CNN
+F 2 "Capacitor_SMD:C_0402_1005Metric" H 9100 2650 50  0001 C CNN
 F 3 "~" H 9100 2650 50  0001 C CNN
-F 4 "EMK107B7104KAHT" H 9100 2650 50  0001 C CNN "Manufacturer Part Number"
+F 4 "GCM155R71C104KA55D" H 9100 2650 50  0001 C CNN "Manufacturer Part Number"
 	1    9100 2650
 	1    0    0    -1
@@
 F 0 "C10" H 8192 1596 50  0000 L CNN
 F 1 "100nF" H 8192 1505 50  0000 L CNN
-F 2 "Capacitor_SMD:C_0603_1608Metric_Pad1.05x0.95mm_HandSolder" H 8100 1550 50  0001 C CNN
+F 2 "Capacitor_SMD:C_0402_1005Metric" H 8100 1550 50  0001 C CNN
 F 3 "~" H 8100 1550 50  0001 C CNN
-F 4 "EMK107B7104KAHT" H 8100 1550 50  0001 C CNN "Manufacturer Part Number"
+F 4 "GCM155R71C104KA55D" H 8100 1550 50  0001 C CNN "Manufacturer Part Number"
 	1    8100 1550
 	-1   0    0    -1
@@
 F 0 "C12" H 8592 1596 50  0000 L CNN
 F 1 "100nF" H 8592 1505 50  0000 L CNN
-F 2 "Capacitor_SMD:C_0603_1608Metric_Pad1.05x0.95mm_HandSolder" H 8500 1550 50  0001 C CNN
+F 2 "Capacitor_SMD:C_0402_1005Metric" H 8500 1550 50  0001 C CNN
 F 3 "~" H 8500 1550 50  0001 C CNN
-F 4 "EMK107B7104KAHT" H 8500 1550 50  0001 C CNN "Manufacturer Part Number"
+F 4 "GCM155R71C104KA55D" H 8500 1550 50  0001 C CNN "Manufacturer Part Number"
 	1    8500 1550
 	-1   0    0    -1
@@
 F 0 "C14" H 8992 1596 50  0000 L CNN
 F 1 "100nF" H 8992 1505 50  0000 L CNN
-F 2 "Capacitor_SMD:C_0603_1608Metric_Pad1.05x0.95mm_HandSolder" H 8900 1550 50  0001 C CNN
+F 2 "Capacitor_SMD:C_0402_1005Metric" H 8900 1550 50  0001 C CNN
 F 3 "~" H 8900 1550 50  0001 C CNN
-F 4 "EMK107B7104KAHT" H 8900 1550 50  0001 C CNN "Manufacturer Part Number"
+F 4 "GCM155R71C104KA55D" H 8900 1550 50  0001 C CNN "Manufacturer Part Number"
 	1    8900 1550
 	-1   0    0    -1
@@
 F 0 "C18" H 9392 1596 50  0000 L CNN
 F 1 "100nF" H 9392 1505 50  0000 L CNN
-F 2 "Capacitor_SMD:C_0603_1608Metric_Pad1.05x0.95mm_HandSolder" H 9300 1550 50  0001 C CNN
+F 2 "Capacitor_SMD:C_0402_1005Metric" H 9300 1550 50  0001 C CNN
 F 3 "~" H 9300 1550 50  0001 C CNN
-F 4 "EMK107B7104KAHT" H 9300 1550 50  0001 C CNN "Manufacturer Part Number"
+F 4 "GCM155R71C104KA55D" H 9300 1550 50  0001 C CNN "Manufacturer Part Number"
 	1    9300 1550
 	-1   0    0    -1
@@
 F 0 "C21" H 11242 9846 50  0000 L CNN
 F 1 "100nF" H 11242 9755 50  0000 L CNN
-F 2 "Capacitor_SMD:C_0603_1608Metric_Pad1.05x0.95mm_HandSolder" H 11150 9800 50  0001 C CNN
+F 2 "Capacitor_SMD:C_0402_1005Metric" H 11150 9800 50  0001 C CNN
 F 3 "~" H 11150 9800 50  0001 C CNN
-F 4 "EMK107B7104KAHT" H 11150 9800 50  0001 C CNN "Manufacturer Part Number"
+F 4 "GCM155R71C104KA55D" H 11150 9800 50  0001 C CNN "Manufacturer Part Number"
 	1    11150 9800
 	1    0    0    -1
@@
 F 0 "C19" H 9592 9846 50  0000 L CNN
 F 1 "100nF" H 9592 9755 50  0000 L CNN
-F 2 "Capacitor_SMD:C_0603_1608Metric_Pad1.05x0.95mm_HandSolder" H 9500 9800 50  0001 C CNN
+F 2 "Capacitor_SMD:C_0402_1005Metric" H 9500 9800 50  0001 C CNN
 F 3 "~" H 9500 9800 50  0001 C CNN
-F 4 "EMK107B7104KAHT" H 9500 9800 50  0001 C CNN "Manufacturer Part Number"
+F 4 "GCM155R71C104KA55D" H 9500 9800 50  0001 C CNN "Manufacturer Part Number"
 	1    9500 9800
 	-1   0    0    -1
@@
 F 0 "C9" H 6692 10046 50  0000 L CNN
 F 1 "100nF" H 6692 9955 50  0000 L CNN
-F 2 "Capacitor_SMD:C_0603_1608Metric_Pad1.05x0.95mm_HandSolder" H 6600 10000 50  0001 C CNN
+F 2 "Capacitor_SMD:C_0402_1005Metric" H 6600 10000 50  0001 C CNN
 F 3 "~" H 6600 10000 50  0001 C CNN
-F 4 "EMK107B7104KAHT" H 6600 10000 50  0001 C CNN "Manufacturer Part Number"
+F 4 "GCM155R71C104KA55D" H 6600 10000 50  0001 C CNN "Manufacturer Part Number"
 	1    6600 10000
 	-1   0    0    -1
@@
 F 0 "C11" H 8442 10046 50  0000 L CNN
 F 1 "100nF" H 8442 9955 50  0000 L CNN
-F 2 "Capacitor_SMD:C_0603_1608Metric_Pad1.05x0.95mm_HandSolder" H 8350 10000 50  0001 C CNN
+F 2 "Capacitor_SMD:C_0402_1005Metric" H 8350 10000 50  0001 C CNN
 F 3 "~" H 8350 10000 50  0001 C CNN
-F 4 "EMK107B7104KAHT" H 8350 10000 50  0001 C CNN "Manufacturer Part Number"
+F 4 "GCM155R71C104KA55D" H 8350 10000 50  0001 C CNN "Manufacturer Part Number"
 	1    8350 10000
 	1    0    0    -1
@@
 F 0 "C5" H 5692 9846 50  0000 L CNN
 F 1 "100nF" H 5692 9755 50  0000 L CNN
-F 2 "Capacitor_SMD:C_0603_1608Metric_Pad1.05x0.95mm_HandSolder" H 5600 9800 50  0001 C CNN
+F 2 "Capacitor_SMD:C_0402_1005Metric" H 5600 9800 50  0001 C CNN
 F 3 "~" H 5600 9800 50  0001 C CNN
-F 4 "EMK107B7104KAHT" H 5600 9800 50  0001 C CNN "Manufacturer Part Number"
+F 4 "GCM155R71C104KA55D" H 5600 9800 50  0001 C CNN "Manufacturer Part Number"
 	1    5600 9800
 	1    0    0    -1
@@
 F 0 "C2" H 4042 9846 50  0000 L CNN
 F 1 "100nF" H 4042 9755 50  0000 L CNN
-F 2 "Capacitor_SMD:C_0603_1608Metric_Pad1.05x0.95mm_HandSolder" H 3950 9800 50  0001 C CNN
+F 2 "Capacitor_SMD:C_0402_1005Metric" H 3950 9800 50  0001 C CNN
 F 3 "~" H 3950 9800 50  0001 C CNN
-F 4 "EMK107B7104KAHT" H 3950 9800 50  0001 C CNN "Manufacturer Part Number"
+F 4 "GCM155R71C104KA55D" H 3950 9800 50  0001 C CNN "Manufacturer Part Number"
 	1    3950 9800
 	-1   0    0    -1
@@
 F 0 "C8" H 5708 3804 50  0000 R CNN
 F 1 "20pF" H 5708 3895 50  0000 R CNN
-F 2 "Capacitor_SMD:C_0603_1608Metric_Pad1.05x0.95mm_HandSolder" H 5800 3850 50  0001 C CNN
+F 2 "Capacitor_SMD:C_0402_1005Metric" H 5800 3850 50  0001 C CNN
 F 3 "~" H 5800 3850 50  0001 C CNN
-F 4 "GCM1885C2A200JA16D" H 5800 3850 50  0001 C CNN "Manufacturer Part Number"
+F 4 "GCM1555C1H200JA16D" H 5800 3850 50  0001 C CNN "Manufacturer Part Number"
 	1    5800 3850
 	0    1    -1   0
@@
 F 0 "C4" H 5108 5704 50  0000 R CNN
 F 1 "4.3pF" H 5108 5795 50  0000 R CNN
-F 2 "Capacitor_SMD:C_0603_1608Metric_Pad1.05x0.95mm_HandSolder" H 5200 5750 50  0001 C CNN
+F 2 "Capacitor_SMD:C_0402_1005Metric" H 5200 5750 50  0001 C CNN
 F 3 "~" H 5200 5750 50  0001 C CNN
-F 4 "885012006001" H 5200 5750 50  0001 C CNN "Manufacturer Part Number"
+F 4 "GRM1555C1H4R3WA01D" H 5200 5750 50  0001 C CNN "Manufacturer Part Number"
 	1    5200 5750
 	0    1    -1   0

Commit message: Diseño inicial de PCB C (WIP)
Parts:
- C13: footprint Capacitor_SMD:C_0603_1608Metric_Pad1.05x0.95mm_HandSolder -> Capacitor_SMD:C_0402_1005Metric; Manufacturer Part Number LMK107B7105MA-T -> GRM155R61E105KA12D
Changed lines of the file:
@@
 F 0 "C13" H 8708 7354 50  0000 R CNN
 F 1 "1uF" H 8708 7445 50  0000 R CNN
-F 2 "Capacitor_SMD:C_0603_1608Metric_Pad1.05x0.95mm_HandSolder" H 8800 7400 50  0001 C CNN
+F 2 "Capacitor_SMD:C_0402_1005Metric" H 8800 7400 50  0001 C CNN
 F 3 "~" H 8800 7400 50  0001 C CNN
-F 4 "LMK107B7105MA-T" H 8800 7400 50  0001 C CNN "Manufacturer Part Number"
+F 4 "GRM155R61E105KA12D" H 8800 7400 50  0001 C CNN "Manufacturer Part Number"
 	1    8800 7400
 	-1   0    0    1

Commit message: Nuevo conector B-C
Connections:
- wire segments 329 -> 346
