File: Hardware/Satelite/PCB_C/PCB_C.sch (KiCad schematic (older format))
At the start: 45 parts, among them IC1 MCP1501T-33E_CHY, IC2 IS25LP080D-JULE-TR, IC3 BQ24392RSER, J1 Conn_01x06, J2 JUMPER, J3 Conector_PCB_B-C, J4 Conector_Expansion_CanSat, J5 USB_B_Micro, Q1 BC817, U1 NTB0104BQ,115, U2 TCA9802DGKR, U3 STM32F303RETx, U4 NTB0104BQ,115, U5 SN74LVC1G3157DCKR, Y1 LFXTAL016178, Y2 Crystal

Commit message: La parte del conector B-C que va en el PCB_B fue movido a bottom mientras que la parte que va en el PCB_C permanece en top
Parts:
- J3: footprint AXTEC:Conector_PCB_B-C -> AXTEC:Conector_PCB_B-C_Lado_C
Changed lines of the file:
@@
 F 0 "J3" H 14250 2317 50  0000 C CNN
 F 1 "Conector_PCB_B-C" H 14250 2225 50  0000 C CNN
-F 2 "AXTEC:Conector_PCB_B-C" H 14150 2350 50  0001 C CNN
+F 2 "AXTEC:Conector_PCB_B-C_Lado_C" H 14150 2350 50  0001 C CNN
 F 3 "" H 14150 2350 50  0001 C CNN
 	1    14250 1600

Commit message: PCB C (WIP)
Parts:
- J3: Notes (none) -> Hecho con dos 10132797-025100LF y sus dos opuestos 10132798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
Changed lines of the file:
@@
 Text Label 6300 4900 0    50   ~ 0
 IO_A_EN
-Text Label 8350 3100 0    50   ~ 0
+Text Label 8350 4100 0    50   ~ 0
 I_SENSE_BATT
-Wire Wire Line
-	8250 3100 8900 3100
 Wire Wire Line
 	8250 3200 9850 3200
@@
 Text Label 8350 2500 0    50   ~ 0
 V_SENSE_3V3
-Text Label 8350 4100 0    50   ~ 0
+Text Label 8350 3100 0    50   ~ 0
 I_SENSE_5V
 Wire Wire Line
@@
 $EndComp
 Wire Wire Line
-	8250 4100 9100 4100
-Wire Wire Line
-	9100 4100 9100 4150
+	8250 4100 8900 4100
 $Comp
 L power:GND #PWR035
 U 1 1 5E677B4C
-P 9100 4350
-F 0 "#PWR035" H 9100 4100 50  0001 C CNN
-F 1 "GND" H 9104 4176 50  0000 C CNN
-F 2 "" H 9100 4350 50  0001 C CNN
-F 3 "" H 9100 4350 50  0001 C CNN
-	1    9100 4350
+P 9100 3700
+F 0 "#PWR035" H 9100 3450 50  0001 C CNN
+F 1 "GND" H 9104 3526 50  0000 C CNN
+F 2 "" H 9100 3700 50  0001 C CNN
+F 3 "" H 9100 3700 50  0001 C CNN
+	1    9100 3700
 	1    0    0    -1
 $EndComp
@@
 L Device:C_Small C?
 U 1 1 5BCFE120
-P 9100 4250
+P 9100 3600
 AR Path="/5BB122CA/5BCFE120" Ref="C?"  Part="1"
 AR Path="/5BB123AC/5BCFE120" Ref="C?"  Part="1"
 AR Path="/5BCFE120" Ref="C16"  Part="1"
-F 0 "C16" H 9192 4296 50  0000 L CNN
-F 1 "100nF" H 9192 4205 50  0000 L CNN
-F 2 "Capacitor_SMD:C_0402_1005Metric" H 9100 4250 50  0001 C CNN
-F 3 "~" H 9100 4250 50  0001 C CNN
-F 4 "GCM155R71C104KA55D" H 9100 4250 50  0001 C CNN "Manufacturer Part Number"
-	1    9100 4250
+F 0 "C16" H 9192 3646 50  0000 L CNN
+F 1 "100nF" H 9192 3555 50  0000 L CNN
+F 2 "Capacitor_SMD:C_0402_1005Metric" H 9100 3600 50  0001 C CNN
+F 3 "~" H 9100 3600 50  0001 C CNN
+F 4 "GCM155R71C104KA55D" H 9100 3600 50  0001 C CNN "Manufacturer Part Number"
+	1    9100 3600
 	1    0    0    -1
 $EndComp
@@
 F 2 "AXTEC:Conector_PCB_B-C_Lado_C" H 14150 2350 50  0001 C CNN
 F 3 "" H 14150 2350 50  0001 C CNN
+F 4 "Hecho con dos 10132797-025100LF y sus dos opuestos 10132798-022100LF" H 0   0   50  0001 C CNN "Notes"
 	1    14250 1600
 	1    0    0    -1
@@
 AGUJEROS DE MONTAJE
 $Comp
-L power:GND #PWR?
+L power:GND #PWR0101
 U 1 1 5BF7325F
 P 13200 2900
-F 0 "#PWR?" H 13200 2650 50  0001 C CNN
+F 0 "#PWR0101" H 13200 2650 50  0001 C CNN
 F 1 "GND" H 13204 2726 50  0000 C CNN
 F 2 "" H 13200 2900 50  0001 C CNN
@@
 	14950 3350 14950 3250
 $Comp
-L power:GND #PWR?
+L power:GND #PWR0102
 U 1 1 5BFE9BDC
 P 15200 3100
-F 0 "#PWR?" H 15200 2850 50  0001 C CNN
+F 0 "#PWR0102" H 15200 2850 50  0001 C CNN
 F 1 "GND" H 15204 2926 50  0000 C CNN
 F 2 "" H 15200 3100 50  0001 C CNN
@@
 Wire Wire Line
 	15000 2000 15600 2000
+Wire Wire Line
+	9100 3100 9100 3500
+Wire Wire Line
+	8250 3100 9100 3100
 $EndSCHEMATC
