File: Hardware/Satelite/PCB_C/_autosave-PCB_C.kicad_pcb (KiCad board)
At the start: 2 copper layers, 54 x 54 mm, 53 parts, among them IC1 MCP1501T-33E_CHY, IC2 IS25LP080D-JULE-TR, IC3 BQ24392RSER, IC4 MS563702BA03-50, IC5 BMX055, J1 Conn_01x06, J2 JUMPER, J3 Conector_PCB_B-C, J4 Conector_Expansion_CanSat, J5 USB_B_Micro, Q1 BC817, U1 NTB0104BQ,115, U2 TCA9802DGKR, U3 STM32F303RETx, U4 NTB0104BQ,115, U5 SN74LVC1G3157DCKR, U6 Si7006-A20-IM1, Y1 LFXTAL016178, Y2 Crystal

Commit message: PCB C (WIP)
Routing:
- net +5V: track 0.00 -> 37.4 mm
- net /V_SENSE_5V: track 0.00 -> 17.5 mm
- net /V_SENSE_3V3: track 7.15 -> 23.7 mm, vias 1 -> 2
- net GND: track 70.2 -> 72.1 mm
Changed lines of the file:
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@@
     (thickness 1.6)
     (drawings 0)
-    (tracks 185)
+    (tracks 214)
     (zones 0)
     (modules 53)
@@
   (via (at 0.8636 16.002) (size 0.6) (drill 0.3) (layers F.Cu B.Cu) (net 1))
   (segment (start 1.801 16.002) (end 0.8636 16.002) (width 0.4) (layer F.Cu) (net 1))
-  (segment (start -1.75 -20.75) (end 0.0508 -20.75) (width 0.3) (layer F.Cu) (net 1))
-  (segment (start 0.0508 -20.75) (end 1.85 -20.75) (width 0.3) (layer F.Cu) (net 1))
-  (via (at 0.0508 -20.75) (size 0.6) (drill 0.3) (layers F.Cu B.Cu) (net 1))
+  (segment (start 1.85 -20.75) (end 3.3764 -20.75) (width 0.3) (layer F.Cu) (net 1))
+  (segment (start 3.6068 -20.9804) (end 3.6068 -21.8948) (width 0.3) (layer F.Cu) (net 1))
+  (segment (start 3.3764 -20.75) (end 3.6068 -20.9804) (width 0.3) (layer F.Cu) (net 1))
+  (via (at -4.318 -20.32) (size 0.6) (drill 0.3) (layers F.Cu B.Cu) (net 1))
+  (segment (start -1.75 -20.75) (end -3.888 -20.75) (width 0.3) (layer F.Cu) (net 1))
+  (segment (start -3.888 -20.75) (end -4.318 -20.32) (width 0.3) (layer F.Cu) (net 1))
   (segment (start 5.1124 -24.25) (end 1.85 -24.25) (width 0.3) (layer F.Cu) (net 2))
   (segment (start 5.9666 -9.6012) (end 5.9666 -23.3958) (width 0.3) (layer F.Cu) (net 2))
@@
   (segment (start -0.557602 -3.1992) (end -1.27 -3.911598) (width 0.25) (layer F.Cu) (net 11))
   (segment (start 2.4996 -3.1992) (end -0.557602 -3.1992) (width 0.25) (layer F.Cu) (net 11))
+  (via (at -0.9144 -7.112) (size 0.6) (drill 0.3) (layers F.Cu B.Cu) (net 11))
+  (segment (start -1.27 -3.911598) (end -0.9144 -4.267198) (width 0.25) (layer B.Cu) (net 11))
+  (segment (start -0.9144 -4.267198) (end -0.9144 -7.112) (width 0.25) (layer B.Cu) (net 11))
+  (segment (start -0.9144 -7.112) (end -0.9144 -8.5344) (width 0.25) (layer F.Cu) (net 11))
+  (segment (start -1.75 -19.35) (end -1.75 -19.75) (width 0.25) (layer F.Cu) (net 11))
+  (segment (start -1.97401 -19.12599) (end -1.75 -19.35) (width 0.25) (layer F.Cu) (net 11))
+  (segment (start -1.97401 -9.59401) (end -1.97401 -19.12599) (width 0.25) (layer F.Cu) (net 11))
+  (segment (start -0.9144 -8.5344) (end -1.97401 -9.59401) (width 0.25) (layer F.Cu) (net 11))
   (via (at -2.4384 -4.1656) (size 0.6) (drill 0.3) (layers F.Cu B.Cu) (net 12))
   (segment (start -2.794 -3.025) (end -2.794 -3.81) (width 0.3) (layer B.Cu) (net 12))
@@
   (segment (start 4.318 8.4836) (end 3.81 8.9916) (width 0.25) (layer F.Cu) (net 15))
   (segment (start 3.81 8.9916) (end -0.1524 8.9916) (width 0.25) (layer F.Cu) (net 15))
+  (segment (start 1.85 -21.25) (end -1.75 -21.25) (width 0.3) (layer F.Cu) (net 45))
+  (segment (start -15.6972 -2.4028) (end -18.1 0) (width 0.3) (layer F.Cu) (net 45))
+  (segment (start -15.6972 -8.6868) (end -15.6972 -2.4028) (width 0.3) (layer F.Cu) (net 45))
+  (segment (start -7.5028 -21.25) (end -8.636 -20.1168) (width 0.3) (layer F.Cu) (net 45))
+  (segment (start -1.75 -21.25) (end -7.5028 -21.25) (width 0.3) (layer F.Cu) (net 45))
+  (segment (start -8.636 -20.1168) (end -8.636 -11.684) (width 0.3) (layer F.Cu) (net 45))
+  (segment (start -8.636 -11.684) (end -10.8204 -9.4996) (width 0.3) (layer F.Cu) (net 45))
+  (segment (start -10.8204 -9.4996) (end -14.8844 -9.4996) (width 0.3) (layer F.Cu) (net 45))
+  (segment (start -14.8844 -9.4996) (end -15.6972 -8.6868) (width 0.3) (layer F.Cu) (net 45))
+  (segment (start 0.5496 -7.7308) (end 0.5496 -5.6492) (width 0.25) (layer F.Cu) (net 49))
+  (segment (start -1.524 -9.8044) (end 0.5496 -7.7308) (width 0.25) (layer F.Cu) (net 49))
+  (segment (start -1.524 -18.6944) (end -1.524 -9.8044) (width 0.25) (layer F.Cu) (net 49))
+  (segment (start -0.5904 -20.25) (end -0.3556 -20.0152) (width 0.25) (layer F.Cu) (net 49))
+  (segment (start -1.75 -20.25) (end -0.5904 -20.25) (width 0.25) (layer F.Cu) (net 49))
+  (segment (start -0.3556 -20.0152) (end -0.3556 -19.304) (width 0.25) (layer F.Cu) (net 49))
+  (segment (start -0.6604 -18.9992) (end -1.2192 -18.9992) (width 0.25) (layer F.Cu) (net 49))
+  (segment (start -0.3556 -19.304) (end -0.6604 -18.9992) (width 0.25) (layer F.Cu) (net 49))
+  (segment (start -1.2192 -18.9992) (end -1.524 -18.6944) (width 0.25) (layer F.Cu) (net 49))
   (zone (net 1) (net_name GND) (layer F.Cu) (hatch edge 0.508)
     (connect_pads (clearance 0.25))
