File: Hardware/Satelite/PCB_C/IMU.sch (KiCad schematic (older format))
At the start: 3 parts

Commit message: Cambio en el simbolo de SW1 en PCB_A
Parts:
- removed C? (x2): 100nF, symbol Device:C_Small
- added C? (x2): 100nF, Capacitor_SMD:C_0603_1608Metric_Pad1.05x0.95mm_HandSolder, symbol Device:C_Small
Changed lines of the file:
@@
 L power:GND #PWR?
 U 1 1 5BB72101
-P 4350 3550
-F 0 "#PWR?" H 4350 3300 50  0001 C CNN
-F 1 "GND" H 4355 3377 50  0000 C CNN
-F 2 "" H 4350 3550 50  0001 C CNN
-F 3 "" H 4350 3550 50  0001 C CNN
-	1    4350 3550
+P 4300 3550
+F 0 "#PWR?" H 4300 3300 50  0001 C CNN
+F 1 "GND" H 4305 3377 50  0000 C CNN
+F 2 "" H 4300 3550 50  0001 C CNN
+F 3 "" H 4300 3550 50  0001 C CNN
+	1    4300 3550
 	1    0    0    -1
 $EndComp
@@
 L power:+3V3 #PWR?
 U 1 1 5BB72133
-P 4350 3050
-F 0 "#PWR?" H 4350 2900 50  0001 C CNN
-F 1 "+3V3" H 4365 3223 50  0000 C CNN
-F 2 "" H 4350 3050 50  0001 C CNN
-F 3 "" H 4350 3050 50  0001 C CNN
-	1    4350 3050
+P 4300 3050
+F 0 "#PWR?" H 4300 2900 50  0001 C CNN
+F 1 "+3V3" H 4315 3223 50  0000 C CNN
+F 2 "" H 4300 3050 50  0001 C CNN
+F 3 "" H 4300 3050 50  0001 C CNN
+	1    4300 3050
 	1    0    0    -1
 $EndComp
@@
 	5050 3050 5250 3050
 Wire Wire Line
-	5250 3250 4350 3250
-$Comp
-L Device:C_Small C?
-U 1 1 5BB721B3
-P 4350 3400
-AR Path="/5BB122CA/5BB721B3" Ref="C?"  Part="1"
-AR Path="/5BB12371/5BB721B3" Ref="C?"  Part="1"
-AR Path="/5BB123AC/5BB721B3" Ref="C?"  Part="1"
-F 0 "C?" H 4258 3354 50  0000 R CNN
-F 1 "100nF" H 4258 3445 50  0000 R CNN
-F 2 "" H 4350 3400 50  0001 C CNN
-F 3 "~" H 4350 3400 50  0001 C CNN
-	1    4350 3400
-	-1   0    0    1
-$EndComp
+	4300 3050 4300 3250
+Connection ~ 4300 3250
 Wire Wire Line
-	4350 3050 4350 3250
-Connection ~ 4350 3250
+	4300 3250 4300 3300
 Wire Wire Line
-	4350 3250 4350 3300
-Wire Wire Line
-	4350 3500 4350 3550
+	4300 3500 4300 3550
 Wire Wire Line
 	5250 3350 5200 3350
@@
 L power:GND #PWR?
 U 1 1 5BB7256E
-P 7300 4050
-F 0 "#PWR?" H 7300 3800 50  0001 C CNN
-F 1 "GND" H 7305 3877 50  0000 C CNN
-F 2 "" H 7300 4050 50  0001 C CNN
-F 3 "" H 7300 4050 50  0001 C CNN
-	1    7300 4050
+P 7400 4050
+F 0 "#PWR?" H 7400 3800 50  0001 C CNN
+F 1 "GND" H 7405 3877 50  0000 C CNN
+F 2 "" H 7400 4050 50  0001 C CNN
+F 3 "" H 7400 4050 50  0001 C CNN
+	1    7400 4050
 	1    0    0    -1
 $EndComp
 Wire Wire Line
-	7300 4050 7300 3150
-$Comp
-L Device:C_Small C?
-U 1 1 5BB7266C
-P 7050 3350
-AR Path="/5BB122CA/5BB7266C" Ref="C?"  Part="1"
-AR Path="/5BB12371/5BB7266C" Ref="C?"  Part="1"
-AR Path="/5BB123AC/5BB7266C" Ref="C?"  Part="1"
-F 0 "C?" H 6958 3304 50  0000 R CNN
-F 1 "100nF" H 6958 3395 50  0000 R CNN
-F 2 "" H 7050 3350 50  0001 C CNN
-F 3 "~" H 7050 3350 50  0001 C CNN
-	1    7050 3350
-	-1   0    0    1
-$EndComp
+	7400 4050 7400 3150
 $Comp
 L power:+3V3 #PWR?
@@
 Wire Wire Line
 	7050 3050 7050 3250
-Connection ~ 7050 3250
 $Comp
 L power:GND #PWR?
@@
 Wire Wire Line
 	6450 3050 6600 3050
-Wire Wire Line
-	6450 3150 7300 3150
 Wire Wire Line
 	6450 3250 7050 3250
@@
 	1    0    0    -1
 $EndComp
+Wire Wire Line
+	4300 3250 5250 3250
+$Comp
+L Device:C_Small C?
+U 1 1 5BCC83DC
+P 4300 3400
+AR Path="/5BB122CA/5BCC83DC" Ref="C?"  Part="1"
+AR Path="/5BB123AC/5BCC83DC" Ref="C?"  Part="1"
+F 0 "C?" H 4392 3446 50  0000 L CNN
+F 1 "100nF" H 4392 3355 50  0000 L CNN
+F 2 "Capacitor_SMD:C_0603_1608Metric_Pad1.05x0.95mm_HandSolder" H 4300 3400 50  0001 C CNN
+F 3 "~" H 4300 3400 50  0001 C CNN
+F 4 "EMK107B7104KAHT" H 4300 3400 50  0001 C CNN "Manufacturer Part Number"
+	1    4300 3400
+	1    0    0    -1
+$EndComp
+$Comp
+L Device:C_Small C?
+U 1 1 5BCC861B
+P 7050 3350
+AR Path="/5BB122CA/5BCC861B" Ref="C?"  Part="1"
+AR Path="/5BB123AC/5BCC861B" Ref="C?"  Part="1"
+F 0 "C?" H 7142 3396 50  0000 L CNN
+F 1 "100nF" H 7142 3305 50  0000 L CNN
+F 2 "Capacitor_SMD:C_0603_1608Metric_Pad1.05x0.95mm_HandSolder" H 7050 3350 50  0001 C CNN
+F 3 "~" H 7050 3350 50  0001 C CNN
+F 4 "EMK107B7104KAHT" H 7050 3350 50  0001 C CNN "Manufacturer Part Number"
+	1    7050 3350
+	1    0    0    -1
+$EndComp
+Wire Wire Line
+	6450 3150 7400 3150
+Connection ~ 7050 3250
 $EndSCHEMATC

Commit message: Modificaciones en conectores, netlist para PCB C
Parts:
- IC5: renamed from IC?; footprint LGA_PACKAGE_20_PINS -> SamacSys_Parts:LGA_PACKAGE_20_PINS
- gave numbers to parts that had none: 2
Changed lines of the file:
@@
 $EndDescr
 $Comp
-L SamacSys_Parts:BMX055 IC?
+L SamacSys_Parts:BMX055 IC5
 U 1 1 5BB71FEC
 P 5250 3050
-F 0 "IC?" H 5850 3315 50  0000 C CNN
+F 0 "IC5" H 5850 3315 50  0000 C CNN
 F 1 "BMX055" H 5850 3224 50  0000 C CNN
-F 2 "LGA_PACKAGE_20_PINS" H 6300 3150 50  0001 L CNN
+F 2 "SamacSys_Parts:LGA_PACKAGE_20_PINS" H 6300 3150 50  0001 L CNN
 F 3 "http://www.mouser.com/ds/2/621/BST-BMX055-DS000-02-586421.pdf" H 6300 3050 50  0001 L CNN
 F 4 "Small versatile 9-axis sensor module" H 6300 2950 50  0001 L CNN "Description"
@@
 GYRO_INT
 $Comp
-L power:GND #PWR?
+L power:GND #PWR073
 U 1 1 5BB72101
 P 4300 3550
-F 0 "#PWR?" H 4300 3300 50  0001 C CNN
+F 0 "#PWR073" H 4300 3300 50  0001 C CNN
 F 1 "GND" H 4305 3377 50  0000 C CNN
 F 2 "" H 4300 3550 50  0001 C CNN
@@
 $EndComp
 $Comp
-L power:+3V3 #PWR?
+L power:+3V3 #PWR072
 U 1 1 5BB72133
 P 4300 3050
-F 0 "#PWR?" H 4300 2900 50  0001 C CNN
+F 0 "#PWR072" H 4300 2900 50  0001 C CNN
 F 1 "+3V3" H 4315 3223 50  0000 C CNN
 F 2 "" H 4300 3050 50  0001 C CNN
@@
 	4650 3350 4650 3550
 $Comp
-L power:GND #PWR?
+L power:GND #PWR074
 U 1 1 5BB7221A
 P 4650 3550
-F 0 "#PWR?" H 4650 3300 50  0001 C CNN
+F 0 "#PWR074" H 4650 3300 50  0001 C CNN
 F 1 "GND" H 4655 3377 50  0000 C CNN
 F 2 "" H 4650 3550 50  0001 C CNN
@@
 	5200 3350 4650 3350
 $Comp
-L power:+3V3 #PWR?
+L power:+3V3 #PWR075
 U 1 1 5BB72267
 P 5000 3600
-F 0 "#PWR?" H 5000 3450 50  0001 C CNN
+F 0 "#PWR075" H 5000 3450 50  0001 C CNN
 F 1 "+3V3" H 5015 3773 50  0000 C CNN
 F 2 "" H 5000 3600 50  0001 C CNN
@@
 	5050 3950 5250 3950
 $Comp
-L power:GND #PWR?
+L power:GND #PWR080
 U 1 1 5BB7256E
 P 7400 4050
-F 0 "#PWR?" H 7400 3800 50  0001 C CNN
+F 0 "#PWR080" H 7400 3800 50  0001 C CNN
 F 1 "GND" H 7405 3877 50  0000 C CNN
 F 2 "" H 7400 4050 50  0001 C CNN
@@
 	7400 4050 7400 3150
 $Comp
-L power:+3V3 #PWR?
+L power:+3V3 #PWR078
 U 1 1 5BB726DE
 P 7050 3050
-F 0 "#PWR?" H 7050 2900 50  0001 C CNN
+F 0 "#PWR078" H 7050 2900 50  0001 C CNN
 F 1 "+3V3" H 7065 3223 50  0000 C CNN
 F 2 "" H 7050 3050 50  0001 C CNN
@@
 	7050 3050 7050 3250
 $Comp
-L power:GND #PWR?
+L power:GND #PWR079
 U 1 1 5BB72CBF
 P 7050 4050
-F 0 "#PWR?" H 7050 3800 50  0001 C CNN
+F 0 "#PWR079" H 7050 3800 50  0001 C CNN
 F 1 "GND" H 7055 3877 50  0000 C CNN
 F 2 "" H 7050 4050 50  0001 C CNN
@@
 	6500 3350 6450 3350
 $Comp
-L power:GND #PWR?
+L power:GND #PWR077
 U 1 1 5BB7368C
 P 6850 4050
-F 0 "#PWR?" H 6850 3800 50  0001 C CNN
+F 0 "#PWR077" H 6850 3800 50  0001 C CNN
 F 1 "GND" H 6855 3877 50  0000 C CNN
 F 2 "" H 6850 4050 50  0001 C CNN
@@
 	6650 3950 6650 4050
 $Comp
-L power:GND #PWR?
+L power:GND #PWR076
 U 1 1 5BB741F0
 P 6650 4050
-F 0 "#PWR?" H 6650 3800 50  0001 C CNN
+F 0 "#PWR076" H 6650 3800 50  0001 C CNN
 F 1 "GND" H 6655 3877 50  0000 C CNN
 F 2 "" H 6650 4050 50  0001 C CNN
@@
 P 4300 3400
 AR Path="/5BB122CA/5BCC83DC" Ref="C?"  Part="1"
-AR Path="/5BB123AC/5BCC83DC" Ref="C?"  Part="1"
-F 0 "C?" H 4392 3446 50  0000 L CNN
+AR Path="/5BB123AC/5BCC83DC" Ref="C24"  Part="1"
+F 0 "C24" H 4392 3446 50  0000 L CNN
 F 1 "100nF" H 4392 3355 50  0000 L CNN
 F 2 "Capacitor_SMD:C_0603_1608Metric_Pad1.05x0.95mm_HandSolder" H 4300 3400 50  0001 C CNN
@@
 P 7050 3350
 AR Path="/5BB122CA/5BCC861B" Ref="C?"  Part="1"
-AR Path="/5BB123AC/5BCC861B" Ref="C?"  Part="1"
-F 0 "C?" H 7142 3396 50  0000 L CNN
+AR Path="/5BB123AC/5BCC861B" Ref="C25"  Part="1"
+F 0 "C25" H 7142 3396 50  0000 L CNN
 F 1 "100nF" H 7142 3305 50  0000 L CNN
 F 2 "Capacitor_SMD:C_0603_1608Metric_Pad1.05x0.95mm_HandSolder" H 7050 3350 50  0001 C CNN

Commit message: Capacitores 0402 para PCB_C
Parts:
- C24, C25: footprint Capacitor_SMD:C_0603_1608Metric_Pad1.05x0.95mm_HandSolder -> Capacitor_SMD:C_0402_1005Metric; Manufacturer Part Number EMK107B7104KAHT -> GCM155R71C104KA55D
Changed lines of the file:
@@
 F 0 "C24" H 4392 3446 50  0000 L CNN
 F 1 "100nF" H 4392 3355 50  0000 L CNN
-F 2 "Capacitor_SMD:C_0603_1608Metric_Pad1.05x0.95mm_HandSolder" H 4300 3400 50  0001 C CNN
+F 2 "Capacitor_SMD:C_0402_1005Metric" H 4300 3400 50  0001 C CNN
 F 3 "~" H 4300 3400 50  0001 C CNN
-F 4 "EMK107B7104KAHT" H 4300 3400 50  0001 C CNN "Manufacturer Part Number"
+F 4 "GCM155R71C104KA55D" H 4300 3400 50  0001 C CNN "Manufacturer Part Number"
 	1    4300 3400
 	1    0    0    -1
@@
 F 0 "C25" H 7142 3396 50  0000 L CNN
 F 1 "100nF" H 7142 3305 50  0000 L CNN
-F 2 "Capacitor_SMD:C_0603_1608Metric_Pad1.05x0.95mm_HandSolder" H 7050 3350 50  0001 C CNN
+F 2 "Capacitor_SMD:C_0402_1005Metric" H 7050 3350 50  0001 C CNN
 F 3 "~" H 7050 3350 50  0001 C CNN
-F 4 "EMK107B7104KAHT" H 7050 3350 50  0001 C CNN "Manufacturer Part Number"
+F 4 "GCM155R71C104KA55D" H 7050 3350 50  0001 C CNN "Manufacturer Part Number"
 	1    7050 3350
 	1    0    0    -1

Commit message: Agregados part number faltantes en PCB_C
Parts:
- IC5: Manufacturer Part Number (none) -> BMX055; Manufacturer_Part_Number BMX055 -> (none)
Changed lines of the file:
@@
 F 3 "http://www.mouser.com/ds/2/621/BST-BMX055-DS000-02-586421.pdf" H 6300 3050 50  0001 L CNN
 F 4 "Small versatile 9-axis sensor module" H 6300 2950 50  0001 L CNN "Description"
-F 5 "" H 6300 2850 50  0001 L CNN "Height"
-F 6 "Bosch Sensortec" H 6300 2750 50  0001 L CNN "Manufacturer_Name"
-F 7 "BMX055" H 6300 2650 50  0001 L CNN "Manufacturer_Part_Number"
-F 8 "" H 6300 2550 50  0001 L CNN "RS Part Number"
-F 9 "" H 6300 2450 50  0001 L CNN "RS Price/Stock"
-F 10 "BMX055" H 6300 2350 50  0001 L CNN "Arrow Part Number"
-F 11 "" H 6300 2250 50  0001 L CNN "Arrow Price/Stock"
+F 5 "Bosch Sensortec" H 6300 2750 50  0001 L CNN "Manufacturer_Name"
+F 6 "BMX055" H 6300 2650 50  0001 L CNN "Manufacturer Part Number"
+F 7 "BMX055" H 6300 2350 50  0001 L CNN "Arrow Part Number"
 	1    5250 3050
 	1    0    0    -1

Commit message: Uso de 3.3V internos para todos los sensores en PCB_C y agregado de divisor resistivo para la señal de 5V proveniente del BQ24392.
Connections:
- net labels added: +3V3_Internal
- net labels removed: +3V3
Changed lines of the file:
@@
-	1    0    0    -1
-$EndComp
-$Comp
-L power:+3V3 #PWR072
-U 1 1 5BB72133
-P 4300 3050
-F 0 "#PWR072" H 4300 2900 50  0001 C CNN
-F 1 "+3V3" H 4315 3223 50  0000 C CNN
-F 2 "" H 4300 3050 50  0001 C CNN
-F 3 "" H 4300 3050 50  0001 C CNN
-	1    4300 3050
 	1    0    0    -1
 $EndComp
@@
 Wire Wire Line
 	5200 3350 4650 3350
-$Comp
-L power:+3V3 #PWR075
-U 1 1 5BB72267
-P 5000 3600
-F 0 "#PWR075" H 5000 3450 50  0001 C CNN
-F 1 "+3V3" H 5015 3773 50  0000 C CNN
-F 2 "" H 5000 3600 50  0001 C CNN
-F 3 "" H 5000 3600 50  0001 C CNN
-	1    5000 3600
-	1    0    0    -1
-$EndComp
 Wire Wire Line
-	5250 3650 5000 3650
+	5250 3650 4950 3650
 Wire Wire Line
-	5000 3650 5000 3600
+	4950 3650 4950 3600
 Wire Wire Line
 	5250 3850 5050 3850
@@
 Wire Wire Line
 	7400 4050 7400 3150
-$Comp
-L power:+3V3 #PWR078
-U 1 1 5BB726DE
-P 7050 3050
-F 0 "#PWR078" H 7050 2900 50  0001 C CNN
-F 1 "+3V3" H 7065 3223 50  0000 C CNN
-F 2 "" H 7050 3050 50  0001 C CNN
-F 3 "" H 7050 3050 50  0001 C CNN
-	1    7050 3050
-	1    0    0    -1
-$EndComp
 Wire Wire Line
 	7050 3050 7050 3250
@@
 	6450 3150 7400 3150
 Connection ~ 7050 3250
+$Comp
+L AXTEC_IC:+3V3_Internal #PWR?
+U 1 1 5C5DF040
+P 4300 3050
+AR Path="/5C5DF040" Ref="#PWR?"  Part="1"
+AR Path="/5BB123AC/5C5DF040" Ref="#PWR20"  Part="1"
+F 0 "#PWR20" H 4300 3450 50  0001 C CNN
+F 1 "+3V3_Internal" H 4285 3223 50  0000 C CNN
+F 2 "" H 4300 3050 50  0001 C CNN
+F 3 "" H 4300 3050 50  0001 C CNN
+	1    4300 3050
+	1    0    0    -1
+$EndComp
+$Comp
+L AXTEC_IC:+3V3_Internal #PWR?
+U 1 1 5C5DF52E
+P 7050 3050
+AR Path="/5C5DF52E" Ref="#PWR?"  Part="1"
+AR Path="/5BB123AC/5C5DF52E" Ref="#PWR23"  Part="1"
+F 0 "#PWR23" H 7050 3450 50  0001 C CNN
+F 1 "+3V3_Internal" H 7035 3223 50  0000 C CNN
+F 2 "" H 7050 3050 50  0001 C CNN
+F 3 "" H 7050 3050 50  0001 C CNN
+	1    7050 3050
+	1    0    0    -1
+$EndComp
+$Comp
+L AXTEC_IC:+3V3_Internal #PWR?
+U 1 1 5C5E21C8
+P 4950 3600
+AR Path="/5C5E21C8" Ref="#PWR?"  Part="1"
+AR Path="/5BB123AC/5C5E21C8" Ref="#PWR25"  Part="1"
+F 0 "#PWR25" H 4950 4000 50  0001 C CNN
+F 1 "+3V3_Internal" H 4935 3773 50  0000 C CNN
+F 2 "" H 4950 3600 50  0001 C CNN
+F 3 "" H 4950 3600 50  0001 C CNN
+	1    4950 3600
+	1    0    0    -1
+$EndComp
 $EndSCHEMATC
