File: Hardware/Satelite/PCB_C/Sensor presión.sch (KiCad schematic (older format))
At the start: 2 parts

Commit message: Cambio en el simbolo de SW1 en PCB_A
Parts:
- C?: footprint (none) -> Capacitor_SMD:C_0603_1608Metric_Pad1.05x0.95mm_HandSolder; Manufacturer Part Number (none) -> EMK107B7104KAHT
Changed lines of the file:
@@
 F 0 "C?" H 4708 3654 50  0000 R CNN
 F 1 "1uF" H 4708 3745 50  0000 R CNN
-F 2 "" H 4800 3700 50  0001 C CNN
+F 2 "Capacitor_SMD:C_0603_1608Metric_Pad1.05x0.95mm_HandSolder" H 4800 3700 50  0001 C CNN
 F 3 "~" H 4800 3700 50  0001 C CNN
+F 4 "EMK107B7104KAHT" H 4800 3700 50  0001 C CNN "Manufacturer Part Number"
 	1    4800 3700
 	-1   0    0    1

Commit message: Footprints para PCB_C
Parts:
- C?: Manufacturer Part Number EMK107B7104KAHT -> LMK107B7105MA-T
Changed lines of the file:
@@
 F 2 "Capacitor_SMD:C_0603_1608Metric_Pad1.05x0.95mm_HandSolder" H 4800 3700 50  0001 C CNN
 F 3 "~" H 4800 3700 50  0001 C CNN
-F 4 "EMK107B7104KAHT" H 4800 3700 50  0001 C CNN "Manufacturer Part Number"
+F 4 "LMK107B7105MA-T" H 4800 3700 50  0001 C CNN "Manufacturer Part Number"
 	1    4800 3700
 	-1   0    0    1

Commit message: Modificaciones en conectores, netlist para PCB C
Parts:
- IC4: renamed from IC?; footprint MS5637_1 -> SamacSys_Parts:MS5637_1
- gave numbers to parts that had none: 1
Changed lines of the file:
@@
 $EndDescr
 $Comp
-L SamacSys_Parts:MS563702BA03-50 IC?
+L SamacSys_Parts:MS563702BA03-50 IC4
 U 1 1 5BB71B9C
 P 5250 3350
-F 0 "IC?" H 5750 3615 50  0000 C CNN
+F 0 "IC4" H 5750 3615 50  0000 C CNN
 F 1 "MS563702BA03-50" H 5750 3524 50  0000 C CNN
-F 2 "MS5637_1" H 6100 3450 50  0001 L CNN
+F 2 "SamacSys_Parts:MS5637_1" H 6100 3450 50  0001 L CNN
 F 3 "http://docs-europe.electrocomponents.com/webdocs/142c/0900766b8142cddb.pdf" H 6100 3350 50  0001 L CNN
 F 4 "Sensor Pressure 2bar Barometric SMD MS563702BA03-50, Barometric Pressure Sensor, 1200mbar 0 ??? 3.6 V Output, 4-Pin QFN" H 6100 3250 50  0001 L CNN "Description"
@@
 $EndComp
 $Comp
-L power:+3V3 #PWR?
+L power:+3V3 #PWR069
 U 1 1 5BB71C29
 P 4800 3250
-F 0 "#PWR?" H 4800 3100 50  0001 C CNN
+F 0 "#PWR069" H 4800 3100 50  0001 C CNN
 F 1 "+3V3" H 4815 3423 50  0000 C CNN
 F 2 "" H 4800 3250 50  0001 C CNN
@@
 $EndComp
 $Comp
-L power:GND #PWR?
+L power:GND #PWR070
 U 1 1 5BB71C54
 P 4800 3800
-F 0 "#PWR?" H 4800 3550 50  0001 C CNN
+F 0 "#PWR070" H 4800 3550 50  0001 C CNN
 F 1 "GND" H 4805 3627 50  0000 C CNN
 F 2 "" H 4800 3800 50  0001 C CNN
@@
 P 4800 3700
 AR Path="/5BB122CA/5BB71D0F" Ref="C?"  Part="1"
-AR Path="/5BB12371/5BB71D0F" Ref="C?"  Part="1"
-F 0 "C?" H 4708 3654 50  0000 R CNN
+AR Path="/5BB12371/5BB71D0F" Ref="C23"  Part="1"
+F 0 "C23" H 4708 3654 50  0000 R CNN
 F 1 "1uF" H 4708 3745 50  0000 R CNN
 F 2 "Capacitor_SMD:C_0603_1608Metric_Pad1.05x0.95mm_HandSolder" H 4800 3700 50  0001 C CNN
@@
 Connection ~ 4800 3350
 $Comp
-L power:GND #PWR?
+L power:GND #PWR071
 U 1 1 5BB71DBB
 P 6350 3800
-F 0 "#PWR?" H 6350 3550 50  0001 C CNN
+F 0 "#PWR071" H 6350 3550 50  0001 C CNN
 F 1 "GND" H 6355 3627 50  0000 C CNN
 F 2 "" H 6350 3800 50  0001 C CNN

Commit message: Capacitores 0402 para PCB_C
Parts:
- C23: footprint Capacitor_SMD:C_0603_1608Metric_Pad1.05x0.95mm_HandSolder -> Capacitor_SMD:C_0402_1005Metric; Manufacturer Part Number LMK107B7105MA-T -> GRM155R61E105KA12D
Changed lines of the file:
@@
 F 0 "C23" H 4708 3654 50  0000 R CNN
 F 1 "1uF" H 4708 3745 50  0000 R CNN
-F 2 "Capacitor_SMD:C_0603_1608Metric_Pad1.05x0.95mm_HandSolder" H 4800 3700 50  0001 C CNN
+F 2 "Capacitor_SMD:C_0402_1005Metric" H 4800 3700 50  0001 C CNN
 F 3 "~" H 4800 3700 50  0001 C CNN
-F 4 "LMK107B7105MA-T" H 4800 3700 50  0001 C CNN "Manufacturer Part Number"
+F 4 "GRM155R61E105KA12D" H 4800 3700 50  0001 C CNN "Manufacturer Part Number"
 	1    4800 3700
 	-1   0    0    1

Commit message: Agregados part number faltantes en PCB_C
Parts:
- IC4: Manufacturer Part Number (none) -> MS563702BA03-50; Manufacturer_Part_Number MS563702BA03-50 -> (none)
Changed lines of the file:
@@
 F 3 "http://docs-europe.electrocomponents.com/webdocs/142c/0900766b8142cddb.pdf" H 6100 3350 50  0001 L CNN
 F 4 "Sensor Pressure 2bar Barometric SMD MS563702BA03-50, Barometric Pressure Sensor, 1200mbar 0 ??? 3.6 V Output, 4-Pin QFN" H 6100 3250 50  0001 L CNN "Description"
-F 5 "" H 6100 3150 50  0001 L CNN "Height"
-F 6 "TE Connectivity" H 6100 3050 50  0001 L CNN "Manufacturer_Name"
-F 7 "MS563702BA03-50" H 6100 2950 50  0001 L CNN "Manufacturer_Part_Number"
-F 8 "1704370" H 6100 2850 50  0001 L CNN "RS Part Number"
-F 9 "http://uk.rs-online.com/web/p/products/1704370" H 6100 2750 50  0001 L CNN "RS Price/Stock"
-F 10 "MS563702BA03-50" H 6100 2650 50  0001 L CNN "Arrow Part Number"
-F 11 "https://www.arrow.com/en/products/ms563702ba03-50/te-connectivity" H 6100 2550 50  0001 L CNN "Arrow Price/Stock"
+F 5 "TE Connectivity" H 6100 3050 50  0001 L CNN "Manufacturer_Name"
+F 6 "MS563702BA03-50" H 6100 2950 50  0001 L CNN "Manufacturer Part Number"
+F 7 "1704370" H 6100 2850 50  0001 L CNN "RS Part Number"
+F 8 "http://uk.rs-online.com/web/p/products/1704370" H 6100 2750 50  0001 L CNN "RS Price/Stock"
+F 9 "MS563702BA03-50" H 6100 2650 50  0001 L CNN "Arrow Part Number"
+F 10 "https://www.arrow.com/en/products/ms563702ba03-50/te-connectivity" H 6100 2550 50  0001 L CNN "Arrow Price/Stock"
 	1    5250 3350
 	1    0    0    -1

Commit message: Uso de 3.3V internos para todos los sensores en PCB_C y agregado de divisor resistivo para la señal de 5V proveniente del BQ24392.
Connections:
- net labels added: +3V3_Internal
- net labels removed: +3V3
Changed lines of the file:
@@
-$EndComp
-$Comp
-L power:+3V3 #PWR069
-U 1 1 5BB71C29
-P 4800 3250
-F 0 "#PWR069" H 4800 3100 50  0001 C CNN
-F 1 "+3V3" H 4815 3423 50  0000 C CNN
-F 2 "" H 4800 3250 50  0001 C CNN
-F 3 "" H 4800 3250 50  0001 C CNN
-	1    4800 3250
-	1    0    0    -1
 $EndComp
 $Comp
@@
 Wire Wire Line
 	5050 3450 5250 3450
+$Comp
+L AXTEC_IC:+3V3_Internal #PWR?
+U 1 1 5C5DEA8F
+P 4800 3250
+AR Path="/5C5DEA8F" Ref="#PWR?"  Part="1"
+AR Path="/5BB12371/5C5DEA8F" Ref="#PWR19"  Part="1"
+F 0 "#PWR19" H 4800 3650 50  0001 C CNN
+F 1 "+3V3_Internal" H 4785 3423 50  0000 C CNN
+F 2 "" H 4800 3250 50  0001 C CNN
+F 3 "" H 4800 3250 50  0001 C CNN
+	1    4800 3250
+	1    0    0    -1
+$EndComp
 $EndSCHEMATC
